File: KiCad/nixieAccurateClock/nixieAccurateClock.kicad_sch (KiCad schematic)
At the start: 7 parts, among them J1 Conn_01x02_Pin, J2 Conn_01x02_Pin, J3 Conn_01x02_Pin, SW1 SW_DIP_x02

Commit message: WIP final feature push
Parts:
- removed R1, R2: 100k, Resistor_SMD:R_0603_1608Metric, symbol Device:R
- removed SW1: SW_DIP_x02, Button_Switch_THT:SW_DIP_SPSTx02_Slide_6.7x6.64mm_W7.62mm_P2.54mm_LowProfile, symbol Switch:SW_DIP_x02
- added H1, H2, H3, H4: MountingHole_Pad, MountingHole:MountingHole_2.7mm_M2.5_Pad_Via, symbol Mechanical:MountingHole_Pad
- added RN1: 100k, Resistor_THT:R_Array_SIP9, symbol Device:R_Network08
- added RV1: 100k, Potentiometer_THT:Potentiometer_Bourns_3299Z_Horizontal, symbol Device:R_Potentiometer
- added SW1: SW_DIP_x08, symbol Switch:SW_DIP_x08
Connections:
- net +3.3V: now also RN1.1 (common), RV1.1
- net DST_check: now also RN1.2 (R1), SW1.1; no longer U1.9 (ICE_28)
- net DST_force: now also RN1.3 (R2), SW1.2; no longer U1.11 (ICE_32)
- net GND: now also H1.1, H2.1, H3.1, H4.1, RV1.3, SW1.10, SW1.11, SW1.12, SW1.13, SW1.14, SW1.15, SW1.16, SW1.9
- net brightness_control: now reaches U1.59 (ADC2|PB)
- net brightness_control: now also RV1.2
- new net 24h_mode: RN1.7 (R6), SW1.6
- new net RESERVED_1: RN1.8 (R7), SW1.7
- new net RESERVED_2: RN1.9 (R8), SW1.8
- new net anti-poison_force: RN1.6 (R5), SW1.5
- new net anti-poison_routine: RN1.5 (R4), SW1.4
- new net manual_brightness: RN1.4 (R3), SW1.3

Commit message: clean up placement and pin assignment
Parts:
- RV1: footprint Potentiometer_THT:Potentiometer_Bourns_3299Z_Horizontal -> Potentiometer_THT:Potentiometer_Bourns_3266Y_Vertical
- SW1: footprint (none) -> Button_Switch_THT:SW_DIP_SPSTx08_Slide_6.7x21.88mm_W7.62mm_P2.54mm_LowProfile
Connections:
- net +3.3V: now also U1.55 (+3.3V), U1.6 (+3.3V), U1.73 (+3.3V), U1.74 (+3.3V), U1.75 (+3.3V)
- net 24h_mode: now also U1.11 (ICE_32)
- net DST_check: now also U1.16 (ICE_43)
- net DST_force: now also U1.15 (ICE_42)
- net GPS_1PPS: now also U1.29 (ICE_46); no longer U1.52 (ICE_20_G3)
- net GPS_1PPS2: now also U1.31 (ICE_48); no longer U1.48 (ICE_18)
- net GPS_RSTN: now also U1.70 (PICO_PMOD_B4); no longer U1.69 (PICO_PMOD_A4)
- net HV_CLOCK: now also U1.32 (ICE_2); no longer U1.14 (ICE_38)
- net HV_DATA: now also U1.34 (ICE_4); no longer U1.16 (ICE_43)
- net HV_POLARITY: now also U1.22 (ICE_9); no longer U1.15 (ICE_42)
- net PPS_TRIMMED: now also U1.20 (ICE_6); no longer U1.13 (ICE_36)
- net RESERVED_1: now also U1.10 (ICE_31)
- net RESERVED_2: now also U1.9 (ICE_28)
- net anti-poison_force: now also U1.12 (ICE_34)
- net anti-poison_routine: now also U1.13 (ICE_36)
- net manual_brightness: now also U1.14 (ICE_38)
Other:
- moved on the sheet: H3, H4

Commit message: reroute daughter board
Swapped standoffs and pin header orientation on IN-14 daughter board so that standoffs face outward.  This allows using the daughter board mounting for the mother board mounting.
Parts:
- removed H1, H2, H3: MountingHole_Pad, MountingHole:MountingHole_2.7mm_M2.5_Pad_Via, symbol Mechanical:MountingHole_Pad
- RV1: footprint Potentiometer_THT:Potentiometer_Bourns_3266Y_Vertical -> Potentiometer_THT:Potentiometer_Bourns_3266Z_Horizontal
- renumbered H4 to H1
Changed lines of the file:
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@@
-    (stroke (width 0) (type default))
-  )
-  (wire (pts (xy 241.3 135.89) (xy 241.3 133.35))
     (stroke (width 0) (type default))
   )
@@
     (stroke (width 0) (type default))
   )
-  (wire (pts (xy 248.92 143.51) (xy 248.92 140.97))
-    (stroke (width 0) (type default))
-  )
   (wire (pts (xy 72.39 78.74) (xy 74.93 78.74))
     (stroke (width 0) (type default))
@@
   )
   (wire (pts (xy 72.39 83.82) (xy 74.93 83.82))
-    (stroke (width 0) (type default))
-  )
-  (wire (pts (xy 234.95 128.27) (xy 234.95 125.73))
     (stroke (width 0) (type default))
   )
@@
       (effects (font (size 1.27 1.27)) (justify right))
     )
-    (property "Footprint" "Potentiometer_THT:Potentiometer_Bourns_3266Y_Vertical" (at 46.99 93.98 0)
+    (property "Footprint" "Potentiometer_THT:Potentiometer_Bourns_3266Z_Horizontal" (at 46.99 93.98 0)
       (effects (font (size 1.27 1.27)) hide)
     )
@@
         (path "/55aab698-7558-4fe2-95ad-faa6da60ef89"
           (reference "RV1") (unit 1)
-        )
-      )
-    )
-  )
-  (symbol (lib_id "power:GND") (at 234.95 128.27 0) (unit 1)
-    (in_bom yes) (on_board yes) (dnp no) (fields_autoplaced)
-    (property "Reference" "#PWR07" (at 234.95 134.62 0)
-      (effects (font (size 1.27 1.27)) hide)
-    )
-    (property "Value" "GND" (at 234.95 133.35 0)
-      (effects (font (size 1.27 1.27)))
-    )
-    (property "Footprint" "" (at 234.95 128.27 0)
-      (effects (font (size 1.27 1.27)) hide)
-    )
-    (property "Datasheet" "" (at 234.95 128.27 0)
-      (effects (font (size 1.27 1.27)) hide)
-    )
-    (pin "1")
-    (instances
-      (project "nixieAccurateClock"
-        (path "/55aab698-7558-4fe2-95ad-faa6da60ef89"
-          (reference "#PWR07") (unit 1)
         )
       )
@@
         (path "/55aab698-7558-4fe2-95ad-faa6da60ef89"
           (reference "#PWR010") (unit 1)
-        )
-      )
-    )
-  )
-  (symbol (lib_id "power:GND") (at 241.3 135.89 0) (unit 1)
-    (in_bom yes) (on_board yes) (dnp no) (fields_autoplaced)
-    (property "Reference" "#PWR08" (at 241.3 142.24 0)
-      (effects (font (size 1.27 1.27)) hide)
-    )
-    (property "Value" "GND" (at 241.3 140.97 0)
-      (effects (font (size 1.27 1.27)))
-    )
-    (property "Footprint" "" (at 241.3 135.89 0)
-      (effects (font (size 1.27 1.27)) hide)
-    )
-    (property "Datasheet" "" (at 241.3 135.89 0)
-      (effects (font (size 1.27 1.27)) hide)
-    )
-    (pin "1")
-    (instances
-      (project "nixieAccurateClock"
-        (path "/55aab698-7558-4fe2-95ad-faa6da60ef89"
-          (reference "#PWR08") (unit 1)
         )
       )
@@
     )
   )
-  (symbol (lib_id "Mechanical:MountingHole_Pad") (at 248.92 138.43 0) (unit 1)
-    (in_bom yes) (on_board yes) (dnp no) (fields_autoplaced)
-    (property "Reference" "H3" (at 251.46 135.89 0)
-      (effects (font (size 1.27 1.27)) (justify left))
-    )
-    (property "Value" "MountingHole_Pad" (at 251.46 138.43 0)
-      (effects (font (size 1.27 1.27)) (justify left))
-    )
-    (property "Footprint" "MountingHole:MountingHole_2.7mm_M2.5_Pad_Via" (at 248.92 138.43 0)
-      (effects (font (size 1.27 1.27)) hide)
-    )
-    (property "Datasheet" "~" (at 248.92 138.43 0)
-      (effects (font (size 1.27 1.27)) hide)
-    )
-    (pin "1")
-    (instances
-      (project "nixieAccurateClock"
-        (path "/55aab698-7558-4fe2-95ad-faa6da60ef89"
-          (reference "H3") (unit 1)
-        )
-      )
-    )
-  )
   (symbol (lib_id "power:GND") (at 264.16 52.07 0) (unit 1)
     (in_bom yes) (on_board yes) (dnp no)
@@
     )
   )
-  (symbol (lib_id "power:GND") (at 248.92 143.51 0) (unit 1)
-    (in_bom yes) (on_board yes) (dnp no) (fields_autoplaced)
-    (property "Reference" "#PWR09" (at 248.92 149.86 0)
-      (effects (font (size 1.27 1.27)) hide)
-    )
-    (property "Value" "GND" (at 248.92 148.59 0)
-      (effects (font (size 1.27 1.27)))
-    )
-    (property "Footprint" "" (at 248.92 143.51 0)
-      (effects (font (size 1.27 1.27)) hide)
-    )
-    (property "Datasheet" "" (at 248.92 143.51 0)
-      (effects (font (size 1.27 1.27)) hide)
-    )
-    (pin "1")
-    (instances
-      (project "nixieAccurateClock"
-        (path "/55aab698-7558-4fe2-95ad-faa6da60ef89"
-          (reference "#PWR09") (unit 1)
-        )
-      )
-    )
-  )
   (symbol (lib_id "power:+5V") (at 90.17 119.38 180) (unit 1)
     (in_bom yes) (on_board yes) (dnp no) (fields_autoplaced)
@@
     )
   )
-  (symbol (lib_id "Mechanical:MountingHole_Pad") (at 234.95 123.19 0) (unit 1)
-    (in_bom yes) (on_board yes) (dnp no) (fields_autoplaced)
-    (property "Reference" "H1" (at 237.49 120.65 0)
-      (effects (font (size 1.27 1.27)) (justify left))
-    )
-    (property "Value" "MountingHole_Pad" (at 237.49 123.19 0)
-      (effects (font (size 1.27 1.27)) (justify left))
-    )
-    (property "Footprint" "MountingHole:MountingHole_2.7mm_M2.5_Pad_Via" (at 234.95 123.19 0)
-      (effects (font (size 1.27 1.27)) hide)
-    )
-    (property "Datasheet" "~" (at 234.95 123.19 0)
-      (effects (font (size 1.27 1.27)) hide)
-    )
-    (pin "1")
-    (instances
-      (project "nixieAccurateClock"
-        (path "/55aab698-7558-4fe2-95ad-faa6da60ef89"
-          (reference "H1") (unit 1)
-        )
-      )
-    )
-  )
   (symbol (lib_id "Mechanical:MountingHole_Pad") (at 255.27 146.05 0) (unit 1)
     (in_bom yes) (on_board yes) (dnp no) (fields_autoplaced)
-    (property "Reference" "H4" (at 257.81 143.51 0)
+    (property "Reference" "H1" (at 257.81 143.51 0)
       (effects (font (size 1.27 1.27)) (justify left))
     )
@@
       (project "nixieAccurateClock"
         (path "/55aab698-7558-4fe2-95ad-faa6da60ef89"
-          (reference "H4") (unit 1)
+          (reference "H1") (unit 1)
         )
       )
@@
         )
       )
-    )
-  )
-  (symbol (lib_id "Mechanical:MountingHole_Pad") (at 241.3 130.81 0) (unit 1)
-    (in_bom yes) (on_board yes) (dnp no) (fields_autoplaced)
-    (property "Reference" "H2" (at 243.84 128.27 0)
-      (effects (font (size 1.27 1.27)) (justify left))
-    )
-    (property "Value" "MountingHole_Pad" (at 243.84 130.81 0)
-      (effects (font (size 1.27 1.27)) (justify left))
-    )
-    (property "Footprint" "MountingHole:MountingHole_2.7mm_M2.5_Pad_Via" (at 241.3 130.81 0)
-      (effects (font (size 1.27 1.27)) hide)
-    )
-    (property "Datasheet" "~" (at 241.3 130.81 0)
-      (effects (font (size 1.27 1.27)) hide)
-    )
-    (pin "1")
-    (instances
-      (project "nixieAccurateClock"
-        (path "/55aab698-7558-4fe2-95ad-faa6da60ef89"
-          (reference "H2") (unit 1)
-        )
-      )

Commit message: simplify nixie daughter board
Remove cathode pins that would not be usable for current sensing anyway.
Pivot to using anode pin as shunt measurement with a R2R flash ADC (not yet implemented).
Connections:
- net HV_POLARITY: no longer names the net of U1.22 (ICE_9)
Changed lines of the file:
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@@
-    (stroke (width 0) (type default))
-  )
-  (wire (pts (xy 71.12 38.1) (xy 74.93 38.1))
     (stroke (width 0) (type default))
   )
@@
       (effects (font (size 1.27 1.27)) (justify right) hide)
     )
-  )
-  (global_label "HV_POLARITY" (shape output) (at 71.12 38.1 180) (fields_autoplaced)
-    (effects (font (size 1.27 1.27)) (justify right))
-    (property "Intersheetrefs" "${INTERSHEET_REFS}" (at 56.0999 38.1 0)
-      (effects (font (size 1.27 1.27)) (justify right) hide)
-    )

Commit message: Signal condition shunt signal
Textbook reference and LTSpice simulation for receipts.

I attempted a differential amplifier based solution but I failed to get it to work.  If it did work it would require more components and likely give little additional benefit.

ADC implementation WIP.
Connections:
- net GPS_1PPS renamed GPS_{1PPS}
- net GPS_1PPS2 renamed GPS_{1PPS2}
- net GPS_BOOT_SEL renamed GPS_{BOOT_SEL}
- net GPS_RSTN renamed GPS_{RSTN}
- net GPS_RXD renamed GPS_{RXD}
- net GPS_TXD renamed GPS_{TXD}
- net HV_CLOCK renamed CLOCK_{HV}
- net HV_DATA renamed DATA_{HV}
- net HV_GATE renamed HV_{GATE}
- net HV_SENSE renamed HV_{SENSE}
- net PPS_TRIMMED renamed PPS_{TRIMMED}
Other:
- added sheet LSD_ADC (LSD_ADC.kicad_sch)

Commit message: give pico iCE better mounting
Connections:
- net LSD_{ADC_D0}: now also U1.52 (ICE_20_G3)
- net LSD_{ADC_D1}: now also U1.50 (ICE_26)
- net LSD_{ADC_D2}: now also U1.48 (ICE_18)
- net LSD_{ADC_D3}: now also U1.46 (ICE_23)
- net LSD_{ADC_MODE}: now also U1.47 (ICE_19)
- net LSD_{ADC_~{INT}}: now also U1.51 (ICE_21)
- net LSD_{ADC_~{RD}}: now also U1.49 (ICE_27)
- net LSD_{ADC_~{WR}/RDY}: now also U1.45 (ICE_25)
