File: KiCad/nixieAccurateClock/nixieAccurateClock.kicad_sch (KiCad schematic)
At the start: 8 parts, among them J1 Conn_01x02_Pin, J2 Conn_01x02_Pin, J3 Conn_01x02_Pin, SW1 SW_DIP_x08

Commit message: ERC and DRC pass
Connections:
- net LSD_{ADC_D4}: now also U1.28 (ICE_45)
- net LSD_{ADC_D5}: now also U1.27 (ICE_44_G6)
- net LSD_{ADC_D6}: now also U1.22 (ICE_9)
- net LSD_{ADC_D7}: now also U1.21 (ICE_10|PB)
- net LSD_{ADC_~{CS}}: now also U1.30 (ICE_47)
- net LSD_{ADC_~{OFL}}: now also U1.19 (ICE_11)
Changed lines of the file:
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@@
+    (stroke (width 0) (type default))
+  )
+  (wire (pts (xy 134.62 53.34) (xy 138.43 53.34))
     (stroke (width 0) (type default))
   )
@@
     (stroke (width 0) (type default))
   )
+  (wire (pts (xy 134.62 58.42) (xy 138.43 58.42))
+    (stroke (width 0) (type default))
+  )
   (wire (pts (xy 71.12 35.56) (xy 74.93 35.56))
     (stroke (width 0) (type default))
@@
     (stroke (width 0) (type default))
   )
+  (wire (pts (xy 71.12 40.64) (xy 74.93 40.64))
+    (stroke (width 0) (type default))
+  )
   (wire (pts (xy 93.98 21.59) (xy 93.98 22.86))
     (stroke (width 0) (type default))
   )
+  (wire (pts (xy 134.62 50.8) (xy 138.43 50.8))
+    (stroke (width 0) (type default))
+  )
   (wire (pts (xy 46.99 99.06) (xy 46.99 97.79))
     (stroke (width 0) (type default))
@@
     (stroke (width 0) (type default))
   )
+  (wire (pts (xy 71.12 43.18) (xy 74.93 43.18))
+    (stroke (width 0) (type default))
+  )
   (wire (pts (xy 242.57 83.82) (xy 246.38 83.82))
     (stroke (width 0) (type default))
@@
   )
   (wire (pts (xy 134.62 43.18) (xy 138.43 43.18))
+    (stroke (width 0) (type default))
+  )
+  (wire (pts (xy 71.12 38.1) (xy 74.93 38.1))
     (stroke (width 0) (type default))
   )
@@
     )
   )
-  (global_label "LSD_{ADC_D4}" (shape input) (at 40.64 44.45 180) (fields_autoplaced)
-    (effects (font (size 1.27 1.27)) (justify right))
-    (property "Intersheetrefs" "${INTERSHEET_REFS}" (at 28.4358 44.45 0)
-      (effects (font (size 1.27 1.27)) (justify right) hide)
+  (global_label "LSD_{ADC_D4}" (shape input) (at 138.43 53.34 0) (fields_autoplaced)
+    (effects (font (size 1.27 1.27)) (justify left))
+    (property "Intersheetrefs" "${INTERSHEET_REFS}" (at 150.6342 53.34 0)
+      (effects (font (size 1.27 1.27)) (justify left) hide)
     )
   )
@@
     )
   )
-  (global_label "LSD_{ADC_D7}" (shape input) (at 40.64 52.07 180) (fields_autoplaced)
-    (effects (font (size 1.27 1.27)) (justify right))
-    (property "Intersheetrefs" "${INTERSHEET_REFS}" (at 28.4358 52.07 0)
-      (effects (font (size 1.27 1.27)) (justify right) hide)
-    )
-  )
-  (global_label "LSD_{ADC_D6}" (shape input) (at 40.64 49.53 180) (fields_autoplaced)
-    (effects (font (size 1.27 1.27)) (justify right))
-    (property "Intersheetrefs" "${INTERSHEET_REFS}" (at 28.4358 49.53 0)
+  (global_label "LSD_{ADC_D7}" (shape input) (at 71.12 40.64 180) (fields_autoplaced)
+    (effects (font (size 1.27 1.27)) (justify right))
+    (property "Intersheetrefs" "${INTERSHEET_REFS}" (at 58.9158 40.64 0)
+      (effects (font (size 1.27 1.27)) (justify right) hide)
+    )
+  )
+  (global_label "LSD_{ADC_D6}" (shape input) (at 71.12 38.1 180) (fields_autoplaced)
+    (effects (font (size 1.27 1.27)) (justify right))
+    (property "Intersheetrefs" "${INTERSHEET_REFS}" (at 58.9158 38.1 0)
       (effects (font (size 1.27 1.27)) (justify right) hide)
     )
@@
     )
   )
-  (global_label "LSD_{ADC_~{OFL}}" (shape input) (at 43.18 66.04 180) (fields_autoplaced)
-    (effects (font (size 1.27 1.27)) (justify right))
-    (property "Intersheetrefs" "${INTERSHEET_REFS}" (at 30.2016 66.04 0)
-      (effects (font (size 1.27 1.27)) (justify right) hide)
-    )
-  )
-  (global_label "LSD_{ADC_~{CS}}" (shape output) (at 40.64 59.69 180) (fields_autoplaced)
-    (effects (font (size 1.27 1.27)) (justify right))
-    (property "Intersheetrefs" "${INTERSHEET_REFS}" (at 28.4358 59.69 0)
-      (effects (font (size 1.27 1.27)) (justify right) hide)
+  (global_label "LSD_{ADC_~{OFL}}" (shape input) (at 71.12 43.18 180) (fields_autoplaced)
+    (effects (font (size 1.27 1.27)) (justify right))
+    (property "Intersheetrefs" "${INTERSHEET_REFS}" (at 58.1416 43.18 0)
+      (effects (font (size 1.27 1.27)) (justify right) hide)
+    )
+  )
+  (global_label "LSD_{ADC_~{CS}}" (shape output) (at 138.43 58.42 0) (fields_autoplaced)
+    (effects (font (size 1.27 1.27)) (justify left))
+    (property "Intersheetrefs" "${INTERSHEET_REFS}" (at 150.6342 58.42 0)
+      (effects (font (size 1.27 1.27)) (justify left) hide)
     )
   )
@@
     )
   )
-  (global_label "LSD_{ADC_D5}" (shape input) (at 40.64 46.99 180) (fields_autoplaced)
-    (effects (font (size 1.27 1.27)) (justify right))
-    (property "Intersheetrefs" "${INTERSHEET_REFS}" (at 28.4358 46.99 0)
-      (effects (font (size 1.27 1.27)) (justify right) hide)
-    )
-  )
+  (global_label "LSD_{ADC_D5}" (shape input) (at 138.43 50.8 0) (fields_autoplaced)
+    (effects (font (size 1.27 1.27)) (justify left))
+    (property "Intersheetrefs" "${INTERSHEET_REFS}" (at 150.6342 50.8 0)
+      (effects (font (size 1.27 1.27)) (justify left) hide)
+    )
+  )

Commit message: Add decoupling caps
Parts:
- removed RN1: 100k, Resistor_THT:R_Array_SIP9, symbol Device:R_Network08

Commit message: WIP two stage HV supply
Other:
- added sheet 20V_supply (20V_supply.kicad_sch)
- company: (none) -> Paul Willis
Changed lines of the file:
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@@
   (title_block
     (title "Nixie Accurate Clock")
+    (rev "A")
+    (company "Paul Willis")
   )
   (junction (at 264.16 36.83) (diameter 0) (color 0 0 0 0)
@@
   (symbol (lib_id "power:+3.3V") (at 105.41 119.38 180) (unit 1)
     (in_bom yes) (on_board yes) (dnp no) (fields_autoplaced)
-    (property "Reference" "#PWR09" (at 105.41 115.57 0)
+    (property "Reference" "#PWR05" (at 105.41 115.57 0)
       (effects (font (size 1.27 1.27)) hide)
     )
@@
       (project "nixieAccurateClock"
         (path "/55aab698-7558-4fe2-95ad-faa6da60ef89"
-          (reference "#PWR09") (unit 1)
+          (reference "#PWR05") (unit 1)
         )
       )
@@
   (symbol (lib_id "power:GND") (at 147.32 81.28 180) (unit 1)
     (in_bom yes) (on_board yes) (dnp no) (fields_autoplaced)
-    (property "Reference" "#PWR04" (at 147.32 74.93 0)
+    (property "Reference" "#PWR07" (at 147.32 74.93 0)
       (effects (font (size 1.27 1.27)) hide)
     )
@@
       (project "nixieAccurateClock"
         (path "/55aab698-7558-4fe2-95ad-faa6da60ef89"
-          (reference "#PWR04") (unit 1)
+          (reference "#PWR07") (unit 1)
         )
       )
@@
   (symbol (lib_id "power:GND") (at 147.32 71.12 180) (unit 1)
     (in_bom yes) (on_board yes) (dnp no) (fields_autoplaced)
-    (property "Reference" "#PWR03" (at 147.32 64.77 0)
+    (property "Reference" "#PWR06" (at 147.32 64.77 0)
       (effects (font (size 1.27 1.27)) hide)
     )
@@
       (project "nixieAccurateClock"
         (path "/55aab698-7558-4fe2-95ad-faa6da60ef89"
-          (reference "#PWR03") (unit 1)
+          (reference "#PWR06") (unit 1)
         )
       )
@@
         )
         (path "/55aab698-7558-4fe2-95ad-faa6da60ef89"
+          (reference "#PWR04") (unit 1)
+        )
+      )
+    )
+  )
+  (symbol (lib_id "power:GND") (at 255.27 151.13 0) (unit 1)
+    (in_bom yes) (on_board yes) (dnp no) (fields_autoplaced)
+    (property "Reference" "#PWR09" (at 255.27 157.48 0)
+      (effects (font (size 1.27 1.27)) hide)
+    )
+    (property "Value" "GND" (at 255.27 156.21 0)
+      (effects (font (size 1.27 1.27)))
+    )
+    (property "Footprint" "" (at 255.27 151.13 0)
+      (effects (font (size 1.27 1.27)) hide)
+    )
+    (property "Datasheet" "" (at 255.27 151.13 0)
+      (effects (font (size 1.27 1.27)) hide)
+    )
+    (pin "1")
+    (instances
+      (project "nixieAccurateClock"
+        (path "/55aab698-7558-4fe2-95ad-faa6da60ef89"
+          (reference "#PWR09") (unit 1)
+        )
+      )
+    )
+  )
+  (symbol (lib_id "power:+3.3V") (at 46.99 88.9 0) (unit 1)
+    (in_bom yes) (on_board yes) (dnp no) (fields_autoplaced)
+    (property "Reference" "#PWR01" (at 46.99 92.71 0)
+      (effects (font (size 1.27 1.27)) hide)
+    )
+    (property "Value" "+3.3V" (at 46.99 83.82 0)
+      (effects (font (size 1.27 1.27)))
+    )
+    (property "Footprint" "" (at 46.99 88.9 0)
+      (effects (font (size 1.27 1.27)) hide)
+    )
+    (property "Datasheet" "" (at 46.99 88.9 0)
+      (effects (font (size 1.27 1.27)) hide)
+    )
+    (pin "1")
+    (instances
+      (project "nixieAccurateClock"
+        (path "/55aab698-7558-4fe2-95ad-faa6da60ef89"
           (reference "#PWR01") (unit 1)
         )
@@
     )
   )
-  (symbol (lib_id "power:GND") (at 255.27 151.13 0) (unit 1)
-    (in_bom yes) (on_board yes) (dnp no) (fields_autoplaced)
-    (property "Reference" "#PWR010" (at 255.27 157.48 0)
-      (effects (font (size 1.27 1.27)) hide)
-    )
-    (property "Value" "GND" (at 255.27 156.21 0)
-      (effects (font (size 1.27 1.27)))
-    )
-    (property "Footprint" "" (at 255.27 151.13 0)
-      (effects (font (size 1.27 1.27)) hide)
-    )
-    (property "Datasheet" "" (at 255.27 151.13 0)
-      (effects (font (size 1.27 1.27)) hide)
-    )
-    (pin "1")
-    (instances
-      (project "nixieAccurateClock"
-        (path "/55aab698-7558-4fe2-95ad-faa6da60ef89"
-          (reference "#PWR010") (unit 1)
-        )
-      )
-    )
-  )
-  (symbol (lib_id "power:+3.3V") (at 46.99 88.9 0) (unit 1)
-    (in_bom yes) (on_board yes) (dnp no) (fields_autoplaced)
-    (property "Reference" "#PWR05" (at 46.99 92.71 0)
-      (effects (font (size 1.27 1.27)) hide)
-    )
-    (property "Value" "+3.3V" (at 46.99 83.82 0)
-      (effects (font (size 1.27 1.27)))
-    )
-    (property "Footprint" "" (at 46.99 88.9 0)
-      (effects (font (size 1.27 1.27)) hide)
-    )
-    (property "Datasheet" "" (at 46.99 88.9 0)
-      (effects (font (size 1.27 1.27)) hide)
-    )
-    (pin "1")
-    (instances
-      (project "nixieAccurateClock"
-        (path "/55aab698-7558-4fe2-95ad-faa6da60ef89"
-          (reference "#PWR05") (unit 1)
-        )
-      )
-    )
-  )
   (symbol (lib_id "power:GND") (at 147.32 91.44 180) (unit 1)
     (in_bom yes) (on_board yes) (dnp no) (fields_autoplaced)
-    (property "Reference" "#PWR06" (at 147.32 85.09 0)
+    (property "Reference" "#PWR08" (at 147.32 85.09 0)
       (effects (font (size 1.27 1.27)) hide)
     )
@@
       (project "nixieAccurateClock"
         (path "/55aab698-7558-4fe2-95ad-faa6da60ef89"
-          (reference "#PWR06") (unit 1)
+          (reference "#PWR08") (unit 1)
         )
       )
@@
   (symbol (lib_id "power:GND") (at 46.99 99.06 0) (unit 1)
     (in_bom yes) (on_board yes) (dnp no) (fields_autoplaced)
-    (property "Reference" "#PWR07" (at 46.99 105.41 0)
+    (property "Reference" "#PWR02" (at 46.99 105.41 0)
       (effects (font (size 1.27 1.27)) hide)
     )
@@
       (project "nixieAccurateClock"
         (path "/55aab698-7558-4fe2-95ad-faa6da60ef89"
-          (reference "#PWR07") (unit 1)
+          (reference "#PWR02") (unit 1)
         )
       )
@@
         )
         (path "/55aab698-7558-4fe2-95ad-faa6da60ef89"
-          (reference "#PWR02") (unit 1)
+          (reference "#PWR010") (unit 1)
         )
       )
@@
   (symbol (lib_id "power:+5V") (at 90.17 119.38 180) (unit 1)
     (in_bom yes) (on_board yes) (dnp no) (fields_autoplaced)
-    (property "Reference" "#PWR08" (at 90.17 115.57 0)
+    (property "Reference" "#PWR03" (at 90.17 115.57 0)
       (effects (font (size 1.27 1.27)) hide)
     )
@@
       (project "nixieAccurateClock"
         (path "/55aab698-7558-4fe2-95ad-faa6da60ef89"
-          (reference "#PWR08") (unit 1)
+          (reference "#PWR03") (unit 1)
         )
       )
@@
     (instances
       (project "nixieAccurateClock"
-        (path "/55aab698-7558-4fe2-95ad-faa6da60ef89" (page "4"))
+        (path "/55aab698-7558-4fe2-95ad-faa6da60ef89" (page "5"))
+      )
+    )
+  )
+  (sheet (at 222.25 109.22) (size 12.7 3.81) (fields_autoplaced)
+    (stroke (width 0.1524) (type solid))
+    (fill (color 0 0 0 0.0000))
+    (property "Sheetname" "20V_supply" (at 222.25 108.5084 0)
+      (effects (font (size 1.27 1.27)) (justify left bottom))
+    )
+    (property "Sheetfile" "20V_supply.kicad_sch" (at 222.25 113.6146 0)
+      (effects (font (size 1.27 1.27)) (justify left top))
+    )
+    (instances
+      (project "nixieAccurateClock"
+        (path "/55aab698-7558-4fe2-95ad-faa6da60ef89" (page "3"))
       )
     )
@@
     (instances
       (project "nixieAccurateClock"
-        (path "/55aab698-7558-4fe2-95ad-faa6da60ef89" (page "5"))
+        (path "/55aab698-7558-4fe2-95ad-faa6da60ef89" (page "6"))
       )
     )
@@
     (instances
       (project "nixieAccurateClock"
-        (path "/55aab698-7558-4fe2-95ad-faa6da60ef89" (page "3"))
+        (path "/55aab698-7558-4fe2-95ad-faa6da60ef89" (page "2"))
       )
     )
@@
     (instances
       (project "nixieAccurateClock"
-        (path "/55aab698-7558-4fe2-95ad-faa6da60ef89" (page "2"))
-      )
-    )
+        (path "/55aab698-7558-4fe2-95ad-faa6da60ef89" (page "4"))
+      )
+    )

Commit message: HV bleed circuit
Connections:
- net HV_{GATE}: no longer names the net of U1.64 (PICO_PMOD_B1)
Other:
- added sheet HV_bleed (HV_bleed.kicad_sch)
Changed lines of the file:
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@@
-    (stroke (width 0) (type default))
-  )
-  (wire (pts (xy 72.39 78.74) (xy 74.93 78.74))
     (stroke (width 0) (type default))
   )
@@
     (property "Intersheetrefs" "${INTERSHEET_REFS}" (at 150.6342 50.8 0)
       (effects (font (size 1.27 1.27)) (justify left) hide)
-    )
-  )
-  (global_label "HV_{GATE}" (shape output) (at 72.39 78.74 180) (fields_autoplaced)
-    (effects (font (size 1.27 1.27)) (justify right))
-    (property "Intersheetrefs" "${INTERSHEET_REFS}" (at 63.3547 78.74 0)
-      (effects (font (size 1.27 1.27)) (justify right) hide)
     )
   )
@@
     (instances
       (project "nixieAccurateClock"
+        (path "/55aab698-7558-4fe2-95ad-faa6da60ef89" (page "6"))
+      )
+    )
+  )
+  (sheet (at 198.12 130.81) (size 12.7 3.81) (fields_autoplaced)
+    (stroke (width 0.1524) (type solid))
+    (fill (color 0 0 0 0.0000))
+    (property "Sheetname" "HV_bleed" (at 198.12 130.0984 0)
+      (effects (font (size 1.27 1.27)) (justify left bottom))
+    )
+    (property "Sheetfile" "HV_bleed.kicad_sch" (at 198.12 135.2046 0)
+      (effects (font (size 1.27 1.27)) (justify left top))
+    )
+    (instances
+      (project "nixieAccurateClock"
         (path "/55aab698-7558-4fe2-95ad-faa6da60ef89" (page "5"))
       )
@@
     (instances
       (project "nixieAccurateClock"
-        (path "/55aab698-7558-4fe2-95ad-faa6da60ef89" (page "6"))
-      )
-    )
+        (path "/55aab698-7558-4fe2-95ad-faa6da60ef89" (page "7"))
+      )
+    )

Commit message: Add HV control
Stop tracking SPICE simulations
Changed lines of the file:
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@@
+    )
+  )
+  (global_label "HV_{CONTROL}" (shape output) (at 71.12 30.48 180) (fields_autoplaced)
+    (effects (font (size 1.27 1.27)) (justify right))
+    (property "Intersheetrefs" "${INTERSHEET_REFS}" (at 58.8431 30.48 0)
+      (effects (font (size 1.27 1.27)) (justify right) hide)
     )
   )

Commit message: finish schematic features
Parts:
- added J4, J5: Conn_01x02_Pin, Connector_PinHeader_2.54mm:PinHeader_1x02_P2.54mm_Vertical, symbol Connector:Conn_01x02_Pin
Connections:
- net +3.3V: now also J5.2 (Pin_2); no longer U1.5 (+3.3V), U1.55 (+3.3V), U1.56 (+3.3V), U1.6 (+3.3V), U1.73 (+3.3V), U1.74 (+3.3V), U1.75 (+3.3V)
- net +5V: now also J4.2 (Pin_2); no longer U1.79 (+5V)
- net HV_{SENSE} renamed HV_{MEASURE}
- new net 3.3V_{SENSE}: J5.1 (Pin_1), U1.5 (+3.3V), U1.55 (+3.3V), U1.56 (+3.3V), U1.6 (+3.3V), U1.73 (+3.3V), U1.74 (+3.3V), U1.75 (+3.3V)
- new net 5V_{SENSE}: J4.1 (Pin_1), U1.79 (+5V)
Other:
- sheet 20V_supply renamed 20V supply
- sheet HV_bleed renamed HV bleed
- sheet LSD_ADC renamed LSD ADC
