File: KiCad/nixieAccurateClock/nixieAccurateClock.kicad_pcb (KiCad board)
At the start: 2 copper layers, 221 x 109.2 mm, 19 parts, among them J1 Conn_02x20_Odd_Even, J2 Conn_02x20_Odd_Even, J3 Conn_Coaxial, Q1 PZTA42, SW1 SW_DIP_x02, U1 PX1125T

Commit message: proper ERC and DRC pass
Parts:
- removed H1, H2, H3, H4: MountingHole_Pad, MountingHole:MountingHole_2.5mm_Pad_Via
- removed the R1 at (202.6, 103.4)
- removed the R2 at (228.6, 102.4)
- added J4: Conn_Coaxial, 00_lib:SMA_Amphenol_132289_EdgeMount, F.Cu at (28.2, 98.2)
- added R4: 10M, Resistor_SMD:R_0603_1608Metric, F.Cu at (228.6, 102.4)
- added R5: 100k, Resistor_SMD:R_0603_1608Metric, F.Cu at (231.1, 102.4)
- added U2: PX1125T, 00_lib:PX1125T, F.Cu at (50.8, 92.3)
- J1, J2: value Conn_02x20_Odd_Even -> Conn_01x02_Pin; footprint Connector_PinSocket_2.54mm:PinSocket_2x20_P2.54mm_Vertical -> Connector_PinHeader_2.54mm:PinHeader_1x02_P2.54mm_Vertical
- J3: value Conn_Coaxial -> Conn_01x02_Pin; footprint 00_lib:SMA_Amphenol_132289_EdgeMount -> Connector_PinHeader_2.54mm:PinHeader_1x02_P2.54mm_Vertical
- R3: value 100k -> 2k
- U1: value PX1125T -> ~; footprint 00_lib:PX1125T -> 00_lib:pico iCE
- moved J3 126.6 mm to (152.4, 73.7), turned to 90 degrees
- moved J2 92.5 mm to (144.8, 119.4), turned to 90 degrees
- moved J1 90.4 mm to (160.0, 119.4), turned to 90 degrees
- moved U1 58.7 mm to (109.2, 86.4), turned to 0 degrees
- moved BT1 30.5 mm to (142.2, 109.2), turned to 90 degrees
- moved R1 30.5 mm to (127.0, 67.8)
- moved R2 30.5 mm to (127.0, 83.0)
- moved SW1 30.5 mm to (127.0, 73.7)
- moved R3 28.6 mm to (202.6, 103.3)
- renumbered R5 to R1, R4 to R2
Connections:
- BT1 pad 1: /+3V3_STDBY -> +3V3_STDBY
- J1 pad 1: /ICE_FLASH_IO2 -> /~{RESET}
- J1 pad 2: /~{ICE_RST} -> GND
- J2 pad 1: /ICE_SSN -> /~{USB_BOOT}
- J2 pad 2: /ICE_SO -> GND
- J3 pad 1: Net-(J3-In) -> /~{ICE_RST}
- R1 pad 1: +3V3 -> +3.3V
- R1 pad 2: /ICE_28 -> /DST_check
- R2 pad 1: /ICE_32 -> /DST_force
- R2 pad 2: +3V3 -> +3.3V
- R3 pad 1: /ADC3 -> HV_GATE
- R3 pad 2: GND -> Net-(Q1-B)
- SW1 pad 1: /ICE_28 -> /DST_check
- SW1 pad 2: /ICE_32 -> /DST_force
- U1 pad 1: /PICO_PMOD_A1 -> unconnected-(U1-ICE_FLASH_IO2-Pad1)
- U1 pad 10: GND -> unconnected-(U1-ICE_31-Pad10)
- U1 pad 11: Net-(J3-In) -> /DST_force
- U1 pad 12: GND -> unconnected-(U1-ICE_34-Pad12)
- U1 pad 13: GND -> unconnected-(U1-ICE_36-Pad13)
- U1 pad 2: unconnected-(U1-SPI_MISO-Pad2) -> /~{ICE_RST}
- U1 pad 20: /PICO_PMOD_B3 -> unconnected-(U1-ICE_6-Pad20)
- U1 pad 21: /PICO_PMOD_B2 -> unconnected-(U1-ICE_10|PB-Pad21)
- U1 pad 22: /+3V3_STDBY -> unconnected-(U1-ICE_9-Pad22)
- U1 pad 23: +3V3 -> unconnected-(U1-VIO_BANK_2-Pad23)
- U1 pad 24: GND -> unconnected-(U1-VIO_BANK_2-Pad24)
- U1 pad 3: /PICO_PMOD_A2 -> unconnected-(U1-ICE_FLASH_IO3-Pad3)
- U1 pad 4: /PICO_PMOD_A3 -> GND
- U1 pad 5: unconnected-(U1-NC-Pad5) -> +3.3V
- U1 pad 7: unconnected-(U1-NC-Pad7) -> GND
- U1 pad 8: /PICO_PMOD_A4 -> GND
- U1 pad 9: unconnected-(U1-SPI_CSN-Pad9) -> /DST_check
Routing:
- net /ADC3: track 230.4 -> 0.00 mm, vias 1 -> 0
- net /PICO_PMOD_B1: track 220.5 -> 0.00 mm, vias 1 -> 0
- net HV_SENSE: track 0.00 -> 202.9 mm, vias 0 -> 1
- net HV_GATE: track 0.00 -> 190.0 mm, vias 0 -> 1
- net +3V3_STDBY: track 0.00 -> 146.2 mm
- net GPS_BOOT_SEL: track 0.00 -> 138.8 mm, vias 0 -> 1
- net /+3V3_STDBY: track 117.6 -> 0.00 mm
- net /PICO_PMOD_A1: track 110.8 -> 0.00 mm, vias 1 -> 0
- net GPS_RSTN: track 0.00 -> 106.7 mm, vias 0 -> 1
- net /PICO_PMOD_A2: track 100.8 -> 0.00 mm, vias 1 -> 0
- net /PICO_PMOD_A3: track 90.7 -> 0.00 mm, vias 1 -> 0
- net GPS_1PPS2: track 0.00 -> 81.5 mm
- net /PICO_PMOD_A4: track 76.2 -> 0.00 mm, vias 1 -> 0
- net GPS_1PPS: track 0.00 -> 73.8 mm
- net +3.3V: track 0.00 -> 72.4 mm
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- added copper zone on B.Cu, net GND
- removed copper zone on B.Cu, net +5V
Other:
- board text added: "~{ICE RESET}"
- board text added: "~{RESET}"
- board text added: "~{USB BOOT}"

Commit message: WIP nixies
Parts:
- added N1: IN-14, 00_lib:nixies-us-IN-14, F.Cu at (40.6, 38.1)
- added N2: IN-14, 00_lib:nixies-us-IN-14, F.Cu at (63.5, 38.1)
- added N3: IN-14, 00_lib:nixies-us-IN-14, F.Cu at (91.4, 38.1)
- added N4: IN-14, 00_lib:nixies-us-IN-14, F.Cu at (119.4, 38.1)
- added N5: IN-14, 00_lib:nixies-us-IN-14, F.Cu at (147.3, 38.1)
- added N6: IN-14, 00_lib:nixies-us-IN-14, F.Cu at (175.3, 38.1)
- added R10: 33k, Resistor_SMD:R_1206_3216Metric, F.Cu at (159.6, 38.0)
- added R11: 33k, Resistor_SMD:R_1206_3216Metric, F.Cu at (187.6, 38.0)
- added R6: 33k, Resistor_SMD:R_1206_3216Metric, F.Cu at (48.3, 48.3)
- added R7: 33k, Resistor_SMD:R_1206_3216Metric, F.Cu at (75.8, 38.0)
- added R8: 33k, Resistor_SMD:R_1206_3216Metric, F.Cu at (103.7, 38.0)
- added R9: 33k, Resistor_SMD:R_1206_3216Metric, F.Cu at (131.7, 38.0)
- added U3: HV509K6-G, 00_lib:QFN32_5X5MC_MCH, F.Cu at (40.7, 53.1)
- added U4: HV509K6-G, 00_lib:QFN32_5X5MC_MCH, F.Cu at (76.7, 32.5)
- added U5: HV509K6-G, 00_lib:QFN32_5X5MC_MCH, F.Cu at (104.6, 32.5)
- added U6: HV509K6-G, 00_lib:QFN32_5X5MC_MCH, F.Cu at (132.6, 32.5)
- added U7: HV509K6-G, 00_lib:QFN32_5X5MC_MCH, F.Cu at (160.5, 32.5)
- added U8: HV509K6-G, 00_lib:QFN32_5X5MC_MCH, F.Cu at (188.4, 32.5)
- moved J1 116.9 mm to (43.2, 121.9)
- moved J2 111.8 mm to (33.0, 121.9)
- moved J3 110.2 mm to (53.3, 121.9)
- moved C1 97.7 mm to (139.7, 68.6)
- moved D1 97.7 mm to (127.0, 68.6)
- moved Q1 97.7 mm to (116.8, 68.6)
- moved R4 97.7 mm to (139.7, 61.8)
- moved R3 97.7 mm to (113.7, 62.7)
- moved R5 97.7 mm to (142.2, 61.8)
- moved L1 95.4 mm to (101.6, 68.6)
- moved BT1 73.6 mm to (80.8, 68.6), turned to 180 degrees
- moved R2 72.3 mm to (63.5, 117.7)
- moved R1 71.2 mm to (76.2, 117.7), turned to 90 degrees
- moved SW1 70.6 mm to (71.1, 116.8), turned to -90 degrees
- moved U1 52.4 mm to (58.4, 99.1), turned to -90 degrees
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Connections:
- net Net-(D1-K) renamed VPP
- U1 pad 13: unconnected-(U1-ICE_36-Pad13) -> PPS_TRIMMED
- U1 pad 14: unconnected-(U1-ICE_38-Pad14) -> HV_CLOCK
- U1 pad 15: unconnected-(U1-ICE_42-Pad15) -> HV_POLARITY
- U1 pad 16: unconnected-(U1-ICE_43-Pad16) -> HV_DATA
Routing:
- net HV_GATE: track 190.0 -> 4.26 mm, vias 1 -> 0
- net HV_SENSE: track 202.9 -> 30.0 mm, vias 1 -> 0
- net +3V3_STDBY: track 146.2 -> 0.00 mm
- net GPS_BOOT_SEL: track 138.8 -> 0.00 mm, vias 1 -> 0
- net GPS_RSTN: track 106.7 -> 0.00 mm, vias 1 -> 0
- net +5V: track 104.8 -> 0.00 mm, vias 1 -> 0
- net GPS_1PPS2: track 81.5 -> 0.00 mm
- net GPS_1PPS: track 73.8 -> 0.00 mm
- net /~{RESET}: track 67.3 -> 0.00 mm
- net /~{ICE_RST}: track 65.2 -> 0.00 mm
- net +3.3V: track 72.4 -> 12.7 mm
- net GPS_TXD: track 45.1 -> 0.00 mm
- net GPS_RXD: track 44.5 -> 0.00 mm
- net /~{USB_BOOT}: track 37.7 -> 0.00 mm
- net /Nixies/Nixie1/N_1: track 0.00 -> 27.0 mm
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Other:
- board size 221 x 109.2 mm -> 170.2 x 101.6 mm
- board text removed: "ON: Check for DST"
- board text removed: "ON: Force DST on"
- board text removed: "USB-C"

Commit message: IN-14 daughter board
Parts:
- removed N1, N2, N3, N4, N5, N6: IN-14, 00_lib:nixies-us-IN-14
- removed R10, R11, R6, R7, R8, R9: 33k, Resistor_SMD:R_1206_3216Metric
- U3, U4, U5, U6, U7, U8: value HV509K6-G -> ~; footprint 00_lib:QFN32_5X5MC_MCH -> 00_lib:IN-14 daughter board
- moved U8 144.4 mm to (44.0, 32.5), turned to -90 degrees
- moved U3 132.9 mm to (172.0, 32.5)
- moved U7 92.5 mm to (68.0, 32.5), turned to -90 degrees
- moved U4 71.3 mm to (148.0, 32.5), turned to -90 degrees
- moved U6 36.6 mm to (96.0, 32.5), turned to -90 degrees
- moved U5 15.4 mm to (120.0, 32.5), turned to -90 degrees
- moved BT1 4.51 mm to (81.8, 73.0)
Connections:
- U3 pad 1: /Nixies/Nixie1/N_RHDP -> VPP
- U3 pad 10: /Nixies/Nixie1/N_3 -> unconnected-(U3-N_1-Pad10)
- U3 pad 11: /Nixies/Nixie1/N_2 -> unconnected-(U3-N_6-Pad11)
- U3 pad 12: /Nixies/Nixie1/N_1 -> PPS_TRIMMED
- U3 pad 14: VPP -> Net-(U3-DOUT)
- U3 pad 15: GND -> unconnected-(U3-N_8-Pad15)
- U3 pad 17: HV_DATA -> unconnected-(U3-N_9-Pad17)
- U3 pad 19: HV_CLOCK -> unconnected-(U3-N_0-Pad19)
- U3 pad 2: /Nixies/Nixie1/N_LHDP -> HV_DATA
- U3 pad 20: +3.3V -> unconnected-(U3-N_RHDP-Pad20)
- U3 pad 21: HV_POLARITY -> unconnected-(U3-HVGND-Pad21)
- U3 pad 22: PPS_TRIMMED -> +5V
- U3 pad 23: unconnected-(U3-NC-Pad23) -> GND
- U3 pad 3: /Nixies/Nixie1/N_0 -> unconnected-(U3-N_2-Pad3)
- U3 pad 4: /Nixies/Nixie1/N_9 -> HV_CLOCK
- U3 pad 5: /Nixies/Nixie1/N_8 -> unconnected-(U3-N_3-Pad5)
- U3 pad 6: /Nixies/Nixie1/N_7 -> +3.3V
- U3 pad 7: /Nixies/Nixie1/N_6 -> unconnected-(U3-N_4-Pad7)
- U3 pad 8: /Nixies/Nixie1/N_5 -> HV_POLARITY
- U3 pad 9: /Nixies/Nixie1/N_4 -> unconnected-(U3-N_5-Pad9)
- U4 pad 1: /Nixies/Nixie2/N_RHDP -> VPP
- U4 pad 10: /Nixies/Nixie2/N_3 -> unconnected-(U4-N_1-Pad10)
- U4 pad 11: /Nixies/Nixie2/N_2 -> unconnected-(U4-N_6-Pad11)
- U4 pad 12: /Nixies/Nixie2/N_1 -> PPS_TRIMMED
- U4 pad 14: VPP -> Net-(U4-DOUT)
- U4 pad 15: GND -> unconnected-(U4-N_8-Pad15)
- U4 pad 17: /Nixies/Nixie1/DOUT -> unconnected-(U4-N_9-Pad17)
- U4 pad 19: HV_CLOCK -> unconnected-(U4-N_0-Pad19)
- U4 pad 2: /Nixies/Nixie2/N_LHDP -> Net-(U3-DOUT)
- U4 pad 20: +3.3V -> unconnected-(U4-N_RHDP-Pad20)
- U4 pad 21: HV_POLARITY -> unconnected-(U4-HVGND-Pad21)
- U4 pad 22: PPS_TRIMMED -> +5V
- U4 pad 23: unconnected-(U4-NC-Pad23) -> GND
- U4 pad 3: /Nixies/Nixie2/N_0 -> unconnected-(U4-N_2-Pad3)
- U4 pad 4: /Nixies/Nixie2/N_9 -> HV_CLOCK
- U4 pad 5: /Nixies/Nixie2/N_8 -> unconnected-(U4-N_3-Pad5)
- U4 pad 6: /Nixies/Nixie2/N_7 -> +3.3V
- U4 pad 7: /Nixies/Nixie2/N_6 -> unconnected-(U4-N_4-Pad7)
- U4 pad 8: /Nixies/Nixie2/N_5 -> HV_POLARITY
- U4 pad 9: /Nixies/Nixie2/N_4 -> unconnected-(U4-N_5-Pad9)
- U5 pad 1: /Nixies/Nixie3/N_RHDP -> VPP
- U5 pad 10: /Nixies/Nixie3/N_3 -> unconnected-(U5-N_1-Pad10)
- U5 pad 11: /Nixies/Nixie3/N_2 -> unconnected-(U5-N_6-Pad11)
- U5 pad 12: /Nixies/Nixie3/N_1 -> PPS_TRIMMED
- U5 pad 14: VPP -> Net-(U5-DOUT)
- U5 pad 15: GND -> unconnected-(U5-N_8-Pad15)
- U5 pad 17: /Nixies/Nixie2/DOUT -> unconnected-(U5-N_9-Pad17)
- U5 pad 19: HV_CLOCK -> unconnected-(U5-N_0-Pad19)
- U5 pad 2: /Nixies/Nixie3/N_LHDP -> Net-(U4-DOUT)
- U5 pad 20: +3.3V -> unconnected-(U5-N_RHDP-Pad20)
- U5 pad 21: HV_POLARITY -> unconnected-(U5-HVGND-Pad21)
- U5 pad 22: PPS_TRIMMED -> +5V
- U5 pad 23: unconnected-(U5-NC-Pad23) -> GND
- U5 pad 3: /Nixies/Nixie3/N_0 -> unconnected-(U5-N_2-Pad3)
- U5 pad 4: /Nixies/Nixie3/N_9 -> HV_CLOCK
- U5 pad 5: /Nixies/Nixie3/N_8 -> unconnected-(U5-N_3-Pad5)
- U5 pad 6: /Nixies/Nixie3/N_7 -> +3.3V
- U5 pad 7: /Nixies/Nixie3/N_6 -> unconnected-(U5-N_4-Pad7)
- U5 pad 8: /Nixies/Nixie3/N_5 -> HV_POLARITY
- U5 pad 9: /Nixies/Nixie3/N_4 -> unconnected-(U5-N_5-Pad9)
- U6 pad 1: /Nixies/Nixie4/N_RHDP -> VPP
- U6 pad 10: /Nixies/Nixie4/N_3 -> unconnected-(U6-N_1-Pad10)
- U6 pad 11: /Nixies/Nixie4/N_2 -> unconnected-(U6-N_6-Pad11)
- U6 pad 12: /Nixies/Nixie4/N_1 -> PPS_TRIMMED
- U6 pad 14: VPP -> Net-(U6-DOUT)
- U6 pad 15: GND -> unconnected-(U6-N_8-Pad15)
- U6 pad 17: /Nixies/Nixie3/DOUT -> unconnected-(U6-N_9-Pad17)
- U6 pad 19: HV_CLOCK -> unconnected-(U6-N_0-Pad19)
- U6 pad 2: /Nixies/Nixie4/N_LHDP -> Net-(U5-DOUT)
- U6 pad 20: +3.3V -> unconnected-(U6-N_RHDP-Pad20)
- U6 pad 21: HV_POLARITY -> unconnected-(U6-HVGND-Pad21)
- U6 pad 22: PPS_TRIMMED -> +5V
- U6 pad 23: unconnected-(U6-NC-Pad23) -> GND
- U6 pad 3: /Nixies/Nixie4/N_0 -> unconnected-(U6-N_2-Pad3)
- U6 pad 4: /Nixies/Nixie4/N_9 -> HV_CLOCK
- U6 pad 5: /Nixies/Nixie4/N_8 -> unconnected-(U6-N_3-Pad5)
- U6 pad 6: /Nixies/Nixie4/N_7 -> +3.3V
- U6 pad 7: /Nixies/Nixie4/N_6 -> unconnected-(U6-N_4-Pad7)
- U6 pad 8: /Nixies/Nixie4/N_5 -> HV_POLARITY
- U6 pad 9: /Nixies/Nixie4/N_4 -> unconnected-(U6-N_5-Pad9)
- U7 pad 1: /Nixies/Nixie5/N_RHDP -> VPP
- U7 pad 10: /Nixies/Nixie5/N_3 -> unconnected-(U7-N_1-Pad10)
- U7 pad 11: /Nixies/Nixie5/N_2 -> unconnected-(U7-N_6-Pad11)
- U7 pad 12: /Nixies/Nixie5/N_1 -> PPS_TRIMMED
- U7 pad 14: VPP -> Net-(U7-DOUT)
- U7 pad 15: GND -> unconnected-(U7-N_8-Pad15)
- U7 pad 17: /Nixies/Nixie4/DOUT -> unconnected-(U7-N_9-Pad17)
- U7 pad 19: HV_CLOCK -> unconnected-(U7-N_0-Pad19)
- U7 pad 2: /Nixies/Nixie5/N_LHDP -> Net-(U6-DOUT)
- U7 pad 20: +3.3V -> unconnected-(U7-N_RHDP-Pad20)
- U7 pad 21: HV_POLARITY -> unconnected-(U7-HVGND-Pad21)
- U7 pad 22: PPS_TRIMMED -> +5V
- U7 pad 23: unconnected-(U7-NC-Pad23) -> GND
- U7 pad 3: /Nixies/Nixie5/N_0 -> unconnected-(U7-N_2-Pad3)
- U7 pad 4: /Nixies/Nixie5/N_9 -> HV_CLOCK
- U7 pad 5: /Nixies/Nixie5/N_8 -> unconnected-(U7-N_3-Pad5)
- U7 pad 6: /Nixies/Nixie5/N_7 -> +3.3V
- U7 pad 7: /Nixies/Nixie5/N_6 -> unconnected-(U7-N_4-Pad7)
- U7 pad 8: /Nixies/Nixie5/N_5 -> HV_POLARITY
- U7 pad 9: /Nixies/Nixie5/N_4 -> unconnected-(U7-N_5-Pad9)
- U8 pad 1: /Nixies/Nixie6/N_RHDP -> VPP
- U8 pad 10: /Nixies/Nixie6/N_3 -> unconnected-(U8-N_1-Pad10)
- U8 pad 11: /Nixies/Nixie6/N_2 -> unconnected-(U8-N_6-Pad11)
- U8 pad 12: /Nixies/Nixie6/N_1 -> PPS_TRIMMED
- U8 pad 14: VPP -> unconnected-(U8-DOUT-Pad14)
- U8 pad 15: GND -> unconnected-(U8-N_8-Pad15)
- U8 pad 17: /Nixies/Nixie5/DOUT -> unconnected-(U8-N_9-Pad17)
- U8 pad 19: HV_CLOCK -> unconnected-(U8-N_0-Pad19)
- U8 pad 2: /Nixies/Nixie6/N_LHDP -> Net-(U7-DOUT)
- U8 pad 20: +3.3V -> unconnected-(U8-N_RHDP-Pad20)
- U8 pad 21: HV_POLARITY -> unconnected-(U8-HVGND-Pad21)
- U8 pad 22: PPS_TRIMMED -> +5V
- U8 pad 23: unconnected-(U8-NC-Pad23) -> GND
- U8 pad 3: /Nixies/Nixie6/N_0 -> unconnected-(U8-N_2-Pad3)
- U8 pad 4: /Nixies/Nixie6/N_9 -> HV_CLOCK
- U8 pad 5: /Nixies/Nixie6/N_8 -> unconnected-(U8-N_3-Pad5)
- U8 pad 6: /Nixies/Nixie6/N_7 -> +3.3V
- U8 pad 7: /Nixies/Nixie6/N_6 -> unconnected-(U8-N_4-Pad7)
- U8 pad 8: /Nixies/Nixie6/N_5 -> HV_POLARITY
- U8 pad 9: /Nixies/Nixie6/N_4 -> unconnected-(U8-N_5-Pad9)
Routing:
- net /Nixies/Nixie1/N_1: track 27.0 -> 0.00 mm
- net /Nixies/Nixie1/N_2: track 19.9 -> 0.00 mm
- net /Nixies/Nixie1/N_3: track 13.3 -> 0.00 mm
- net /Nixies/Nixie1/N_8: track 12.9 -> 0.00 mm
- net /Nixies/Nixie1/N_7: track 9.88 -> 0.00 mm
- net /Nixies/Nixie1/N_4: track 9.30 -> 0.00 mm
- net /Nixies/Nixie1/N_6: track 7.63 -> 0.00 mm
- net HV_SENSE: track 30.0 -> 22.9 mm
- net /Nixies/Nixie1/N_5: track 6.61 -> 0.00 mm
Other:
- board size 170.2 x 101.6 mm -> 153 x 101.5 mm

Commit message: WIP final feature push
Parts:
- removed R1, R2: 100k, Resistor_SMD:R_0603_1608Metric
- removed SW1: SW_DIP_x02, Button_Switch_THT:SW_DIP_SPSTx02_Slide_6.7x6.64mm_W7.62mm_P2.54mm_LowProfile
- added H1: MountingHole_Pad, MountingHole:MountingHole_2.7mm_M2.5_Pad_Via, F.Cu at (4.00, 4.00)
- added H2: MountingHole_Pad, MountingHole:MountingHole_2.7mm_M2.5_Pad_Via, F.Cu at (146.0, 4.00)
- added H3: MountingHole_Pad, MountingHole:MountingHole_2.7mm_M2.5_Pad_Via, F.Cu at (4.00, 81.0)
- added H4: MountingHole_Pad, MountingHole:MountingHole_2.7mm_M2.5_Pad_Via, F.Cu at (146.0, 81.0)
- moved J2 76.0 mm to (76.0, 59.2)
- moved J1 64.4 mm to (76.1, 66.5)
- moved BT1 51.5 mm to (130.0, 55.0), turned to -90 degrees
- moved J3 51.3 mm to (75.7, 75.8)
- moved J4 43.0 mm to (2.54, 40.0)
- moved U1 42.8 mm to (32.5, 65.0)
- moved U3 40.4 mm to (141.5, 6.00)
- moved U4 40.4 mm to (117.5, 6.00)
- moved U5 37.5 mm to (93.5, 6.00)
- moved U6 37.5 mm to (69.5, 6.00)
- moved U2 37.0 mm to (18.0, 40.0), turned to 90 degrees
- moved U7 34.8 mm to (45.5, 6.00)
- moved U8 34.8 mm to (21.5, 6.00)
- moved R5 30.9 mm to (129.3, 33.7)
- moved C1 30.9 mm to (126.8, 40.5)
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Connections:
- net Net-(D1-A) renamed /High voltage supply/HV_BOOST
- U8 pad 10: unconnected-(U8-N_1-Pad10) -> /Nixies/N_1
- U8 pad 11: unconnected-(U8-N_6-Pad11) -> /Nixies/N_6
- U8 pad 13: unconnected-(U8-N_7-Pad13) -> /Nixies/N_7
- U8 pad 15: unconnected-(U8-N_8-Pad15) -> /Nixies/N_8
- U8 pad 17: unconnected-(U8-N_9-Pad17) -> /Nixies/N_9
- U8 pad 19: unconnected-(U8-N_0-Pad19) -> /Nixies/N_0
- U8 pad 3: unconnected-(U8-N_2-Pad3) -> /Nixies/N_2
- U8 pad 5: unconnected-(U8-N_3-Pad5) -> /Nixies/N_3
- U8 pad 7: unconnected-(U8-N_4-Pad7) -> /Nixies/N_4
- U8 pad 9: unconnected-(U8-N_5-Pad9) -> /Nixies/N_5
Routing:
- net +3.3V: track 12.7 -> 0.00 mm
- net Net-(J4-In): track 7.34 -> 0.00 mm
- net /DST_check: track 5.08 -> 0.00 mm
- net /DST_force: track 5.08 -> 0.00 mm
- net GND: vias 1 -> 0
- added copper zone on In1.Cu, net GND
- added copper zone on In2.Cu, net GND
Other:
- board size 153 x 101.5 mm -> 150 x 85 mm
- copper layers 2 -> 4

Commit message: clean up placement and pin assignment
Parts:
- added RN1: 100k, Resistor_THT:R_Array_SIP9, F.Cu at (81.1, 48.9)
- added RV1: 100k, Potentiometer_THT:Potentiometer_Bourns_3266Y_Vertical, F.Cu at (72.8, 59.7)
- added SW1: SW_DIP_x08, Button_Switch_THT:SW_DIP_SPSTx08_Slide_6.7x21.88mm_W7.62mm_P2.54mm_LowProfile, F.Cu at (85.1, 51.4)
- moved J3 24.1 mm to (68.6, 52.7)
- moved J2 23.0 mm to (68.6, 37.5)
- moved J1 22.7 mm to (68.6, 45.1)
- moved BT1 15.1 mm to (144.2, 60.0), turned to 180 degrees
- moved D1 14.2 mm to (128.3, 40.5)
- moved C1 14.2 mm to (141.0, 40.5)
- moved L1 14.2 mm to (102.9, 40.5)
- moved Q1 14.2 mm to (118.1, 40.5)
- moved R1 14.2 mm to (115.0, 34.6)
- moved R2 14.2 mm to (141.0, 33.7)
- moved R3 14.2 mm to (143.5, 33.7)
- moved H3 11.0 mm to (3.00, 70.0)
- moved H4 11.0 mm to (146.0, 70.0)
- moved U1 3.90 mm to (32.2, 61.1)
- moved J4 1.00 mm to (2.54, 39.0)
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- renumbered R3 to R1, R4 to R2, R5 to R3
Connections:
- net Net-(J4-In) renamed /GPS/RF_IN
- U1 pad 10: unconnected-(U1-ICE_31-Pad10) -> /RESERVED_1
- U1 pad 11: /DST_force -> /24h_mode
- U1 pad 12: unconnected-(U1-ICE_34-Pad12) -> /anti-poison_force
- U1 pad 13: PPS_TRIMMED -> /anti-poison_routine
- U1 pad 14: HV_CLOCK -> /manual_brightness
- U1 pad 15: HV_POLARITY -> /DST_force
- U1 pad 16: HV_DATA -> /DST_check
- U1 pad 20: unconnected-(U1-ICE_6-Pad20) -> PPS_TRIMMED
- U1 pad 22: unconnected-(U1-ICE_9-Pad22) -> HV_POLARITY
- U1 pad 29: unconnected-(U1-ICE_46-Pad29) -> GPS_1PPS
- U1 pad 31: unconnected-(U1-ICE_48-Pad31) -> GPS_1PPS2
- U1 pad 32: unconnected-(U1-ICE_2-Pad32) -> HV_CLOCK
- U1 pad 34: unconnected-(U1-ICE_4-Pad34) -> HV_DATA
- U1 pad 48: GPS_1PPS2 -> unconnected-(U1-ICE_18-Pad48)
- U1 pad 52: GPS_1PPS -> unconnected-(U1-ICE_20_G3-Pad52)
- U1 pad 55: unconnected-(U1-+3.3V-Pad55) -> +3.3V
- U1 pad 59: unconnected-(U1-ADC2|PB-Pad59) -> /brightness_control
- U1 pad 6: unconnected-(U1-+3.3V-Pad6) -> +3.3V
- U1 pad 69: GPS_RSTN -> unconnected-(U1-PICO_PMOD_A4-Pad69)
- U1 pad 70: unconnected-(U1-PICO_PMOD_B4-Pad70) -> GPS_RSTN
- U1 pad 73: unconnected-(U1-+3.3V-Pad73) -> +3.3V
- U1 pad 74: unconnected-(U1-+3.3V-Pad74) -> +3.3V
- U1 pad 75: unconnected-(U1-+3.3V-Pad75) -> +3.3V
- U1 pad 9: /DST_check -> /RESERVED_2
Routing:
- added copper zone on F.Cu, net +3.3V
- added copper zone on B.Cu, net +5V
- removed copper zone on B.Cu, net GND
- removed copper zone on F.Cu, net GND
Other:
- board size 150 x 85 mm -> 150 x 74 mm
- board text added: "24 hour mode"
- board text added: "DST check"
- board text added: "DST force"
- board text added: "OFF"
- board text added: "ON"
- board text added: "RESERVED 1"
- board text added: "RESERVED 2"
- board text added: "anti-poison force"
- board text added: "anti-poison routine"
- board text added: "manual brightness"

Commit message: reroute daughter board
Swapped standoffs and pin header orientation on IN-14 daughter board so that standoffs face outward.  This allows using the daughter board mounting for the mother board mounting.
Parts:
- removed the H1 at (4.00, 4.00)
- removed H2, H3: MountingHole_Pad, MountingHole:MountingHole_2.7mm_M2.5_Pad_Via
- RV1: footprint Potentiometer_THT:Potentiometer_Bourns_3266Y_Vertical -> Potentiometer_THT:Potentiometer_Bourns_3266Z_Horizontal
- moved RV1 67.8 mm to (6.04, 48.0)
- moved R3 46.7 mm to (98.0, 44.2), turned to 90 degrees
- moved R2 41.8 mm to (100.5, 44.2), turned to -90 degrees
- moved J1 36.2 mm to (32.5, 42.6)
- moved J2 36.2 mm to (32.5, 35.0)
- moved U3 35.4 mm to (112.6, 26.5), turned to 90 degrees
- moved U4 33.0 mm to (91.6, 26.5), turned to 90 degrees
- moved U5 32.2 mm to (68.6, 26.5), turned to 90 degrees
- moved C1 31.3 mm to (110.0, 36.2)
- moved U6 30.7 mm to (46.6, 26.5), turned to 90 degrees
- moved U7 29.3 mm to (24.6, 26.5), turned to 90 degrees
- moved D1 28.8 mm to (100.5, 33.0)
- moved U8 27.2 mm to (3.62, 26.5), turned to 90 degrees
- moved J3 25.6 mm to (45.0, 42.6)
- moved L1 23.3 mm to (79.7, 38.8)
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- renumbered H4 to H1
Routing:
- net HV_SENSE: track 22.9 -> 2.54 mm
- net HV_GATE: track 4.26 -> 0.00 mm
- net +5V: track 0.00 -> 3.26 mm, vias 0 -> 1
- net VPP: track 16.3 -> 18.4 mm
- net /High voltage supply/HV_BOOST: track 17.1 -> 18.2 mm
Other:
- board size 150 x 74 mm -> 129 x 77 mm

Commit message: simplify nixie daughter board
Remove cathode pins that would not be usable for current sensing anyway.
Pivot to using anode pin as shunt measurement with a R2R flash ADC (not yet implemented).
Parts:
- moved H1 4.00 mm to (125.0, 76.0)
- moved U1 4.00 mm to (33.2, 67.1)
- moved RN1 3.00 mm to (68.6, 55.2)
- moved SW1 3.00 mm to (72.6, 57.7)
- moved J1 2.00 mm to (32.5, 44.6)
- moved J2 2.00 mm to (32.5, 37.0)
- moved J3 2.00 mm to (45.0, 44.6)
- moved RV1 2.00 mm to (6.04, 50.0)
- moved R1 1.54 mm to (92.1, 34.3)
- moved C1 1.54 mm to (110.3, 37.8)
- moved D1 1.54 mm to (100.8, 34.5)
- moved L1 1.54 mm to (80.0, 40.2)
- moved Q1 1.54 mm to (95.3, 40.2)
- moved R2 1.54 mm to (100.9, 45.8)
- moved R3 1.54 mm to (98.3, 45.8)
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Connections:
- U1 pad 22: HV_POLARITY -> unconnected-(U1-ICE_9-Pad22)
- U3 pad 1: VPP -> /Nixies/HV_daisy_1
- U3 pad 10: unconnected-(U3-N_1-Pad10) -> GND
- U3 pad 2: HV_DATA -> +5V
- U3 pad 23: GND -> (no net)
- U3 pad 3: unconnected-(U3-N_2-Pad3) -> PPS_TRIMMED
- U3 pad 4: HV_CLOCK -> HV_DATA
- U3 pad 5: unconnected-(U3-N_3-Pad5) -> GND
- U3 pad 8: HV_POLARITY -> HV_CLOCK
- U3 pad 9: unconnected-(U3-N_5-Pad9) -> VPP
- U4 pad 1: VPP -> unconnected-(U4-DOUT-Pad1)
- U4 pad 10: unconnected-(U4-N_1-Pad10) -> GND
- U4 pad 2: Net-(U3-DOUT) -> +5V
- U4 pad 23: GND -> (no net)
- U4 pad 3: unconnected-(U4-N_2-Pad3) -> PPS_TRIMMED
- U4 pad 4: HV_CLOCK -> /Nixies/HV_daisy_5
- U4 pad 5: unconnected-(U4-N_3-Pad5) -> GND
- U4 pad 8: HV_POLARITY -> HV_CLOCK
- U4 pad 9: unconnected-(U4-N_5-Pad9) -> VPP
- U5 pad 1: VPP -> /Nixies/HV_daisy_2
- U5 pad 10: unconnected-(U5-N_1-Pad10) -> GND
- U5 pad 2: Net-(U4-DOUT) -> +5V
- U5 pad 23: GND -> (no net)
- U5 pad 3: unconnected-(U5-N_2-Pad3) -> PPS_TRIMMED
- U5 pad 4: HV_CLOCK -> /Nixies/HV_daisy_1
- U5 pad 5: unconnected-(U5-N_3-Pad5) -> GND
- U5 pad 8: HV_POLARITY -> HV_CLOCK
- U5 pad 9: unconnected-(U5-N_5-Pad9) -> VPP
- U6 pad 1: VPP -> /Nixies/HV_daisy_3
- U6 pad 10: unconnected-(U6-N_1-Pad10) -> GND
- U6 pad 2: Net-(U5-DOUT) -> +5V
- U6 pad 23: GND -> (no net)
- U6 pad 3: unconnected-(U6-N_2-Pad3) -> PPS_TRIMMED
- U6 pad 4: HV_CLOCK -> /Nixies/HV_daisy_2
- U6 pad 5: unconnected-(U6-N_3-Pad5) -> GND
- U6 pad 8: HV_POLARITY -> HV_CLOCK
- U6 pad 9: unconnected-(U6-N_5-Pad9) -> VPP
- U7 pad 1: VPP -> /Nixies/HV_daisy_4
- U7 pad 10: unconnected-(U7-N_1-Pad10) -> GND
- U7 pad 2: Net-(U6-DOUT) -> +5V
- U7 pad 23: GND -> (no net)
- U7 pad 3: unconnected-(U7-N_2-Pad3) -> PPS_TRIMMED
- U7 pad 4: HV_CLOCK -> /Nixies/HV_daisy_3
- U7 pad 5: unconnected-(U7-N_3-Pad5) -> GND
- U7 pad 8: HV_POLARITY -> HV_CLOCK
- U7 pad 9: unconnected-(U7-N_5-Pad9) -> VPP
- U8 pad 1: VPP -> /Nixies/HV_daisy_5
- U8 pad 10: /Nixies/N_1 -> GND
- U8 pad 2: Net-(U7-DOUT) -> +5V
- U8 pad 23: GND -> (no net)
- U8 pad 3: /Nixies/N_2 -> PPS_TRIMMED
- U8 pad 4: HV_CLOCK -> /Nixies/HV_daisy_4
- U8 pad 5: /Nixies/N_3 -> GND
- U8 pad 7: /Nixies/N_4 -> unconnected-(U8-ANODE-Pad7)
- U8 pad 8: HV_POLARITY -> HV_CLOCK
- U8 pad 9: /Nixies/N_5 -> VPP
Routing:
- net /GPS/RF_IN: track 0.00 -> 13.5 mm
- net /manual_brightness: track 0.00 -> 4.02 mm
- net /anti-poison_routine: track 0.00 -> 4.02 mm
- net /anti-poison_force: track 0.00 -> 4.02 mm
- net /RESERVED_2: track 0.00 -> 4.02 mm
- net /RESERVED_1: track 0.00 -> 4.02 mm
- net /DST_force: track 0.00 -> 4.02 mm
- net /DST_check: track 0.00 -> 4.02 mm
- net /24h_mode: track 0.00 -> 4.02 mm
- net VPP: track 18.4 -> 19.5 mm
Other:
- board size 129 x 77 mm -> 129 x 80 mm
