File: KiCad/nixieAccurateClock/nixieAccurateClock.kicad_pcb (KiCad board)
At the start: 4 copper layers, 129 x 80 mm, 24 parts, among them J1 Conn_01x02_Pin, J2 Conn_01x02_Pin, J3 Conn_01x02_Pin, J4 Conn_Coaxial, Q1 PZTA42, SW1 SW_DIP_x08, U2 PX1125T

Commit message: Signal condition shunt signal
Textbook reference and LTSpice simulation for receipts.

I attempted a differential amplifier based solution but I failed to get it to work.  If it did work it would require more components and likely give little additional benefit.

ADC implementation WIP.
Connections:
- U4 pad 7: unconnected-(U4-ANODE-Pad7) -> LSD_SHUNT
