File: KiCad/nixieAccurateClock/nixieAccurateClock.kicad_pcb (KiCad board)
At the start: 4 copper layers, 129 x 80 mm, 42 parts, among them J1 Conn_01x02_Pin, J2 Conn_01x02_Pin, J3 Conn_01x02_Pin, J4 Conn_Coaxial, Q1 PZTA42, Q2 PZTA42, SW1 SW_DIP_x08, U10 TXB0108PWR, U11 TXB0108PWR, U2 PX1125T

Commit message: tie level shift OE to ground
OE on the TX0108 is internally tied high and should be softly pulled low for power-on sequencing.
Connections:
- R6 pad 1: +3.3V -> GND
- R7 pad 1: +3.3V -> GND
Routing:
- net GND: track 58.3 -> 62.6 mm, vias 14 -> 16

Commit message: simulate HV supply concept
LM5156 simulation is infeasible

LTSpice model demonstrating that a two stage buck from 5 to 210 is possible.  Both stages run away, but the LM5156 should provide feedback to keep it on target.
Parts:
- removed the C1 at (110.3, 38.4)
- removed the R1 at (100.9, 46.4)
- removed the R2 at (92.2, 35.6)
- added C10: 1n, Capacitor_SMD:C_0603_1608Metric, F.Cu at (-48.4, -2.30)
- added C11: 1u, Capacitor_SMD:C_0603_1608Metric, F.Cu at (-48.4, 0.21)
- added C2: 1u, Capacitor_SMD:C_0603_1608Metric, F.Cu at (-34.3, -4.81)
- added C3: 10u, Capacitor_THT:CP_Radial_D10.0mm_P5.00mm, F.Cu at (-28.8, -2.80)
- added C4: 0.1u, Capacitor_SMD:C_0603_1608Metric, F.Cu at (-34.3, -7.32)
- added C5: 1u, Capacitor_SMD:C_0603_1608Metric, F.Cu at (-34.3, -2.30)
- added C6: 1u, Capacitor_SMD:C_0603_1608Metric, F.Cu at (-34.3, 0.21)
- added C7: 1u, Capacitor_SMD:C_0603_1608Metric, F.Cu at (-48.4, -4.81)
- added C8: 10u, Capacitor_THT:CP_Radial_D10.0mm_P5.00mm, F.Cu at (-64.3, 14.3)
- added C9: 1u, Capacitor_SMD:C_0603_1608Metric, F.Cu at (-48.4, -7.32)
- added D2: SM4004, Diode_SMD:D_MELF, F.Cu at (-46.4, 6.14)
- added L2: 820u, 00_lib:IND_MSS1583_COC, F.Cu at (-59.1, 0.00)
- added Q3: MMBT3904, Package_TO_SOT_SMD:SOT-23, F.Cu at (14.0, 18.2)
- added R1: 62k, Resistor_SMD:R_0603_1608Metric, F.Cu at (-32.8, 22.0)
- added R1: 160k, Resistor_SMD:R_0201_0603Metric, F.Cu at (-31.1, 12.1)
- added R10: 10M, Resistor_SMD:R_0603_1608Metric, F.Cu at (-40.4, -4.81)
- added R11: 4.7k, Resistor_SMD:R_0603_1608Metric, F.Cu at (-44.4, -7.32)
- added R12: 1k, Resistor_SMD:R_0201_0603Metric, F.Cu at (-44.9, 11.2)
- added R13: 1k, Resistor_SMD:R_0201_0603Metric, F.Cu at (-44.9, 12.9)
- added R14: 100k, Resistor_SMD:R_0603_1608Metric, F.Cu at (-40.4, -2.30)
- added R15: 40m, Resistor_SMD:R_0201_0603Metric, F.Cu at (-44.9, 14.7)
- added R16: 100k, Resistor_SMD:R_0603_1608Metric, F.Cu at (-48.4, 2.72)
- added R17: 220k, Resistor_SMD:R_0603_1608Metric, F.Cu at (-44.4, -4.81)
- added R18: 100k, Resistor_SMD:R_0603_1608Metric, F.Cu at (-44.4, 0.21)
- added R19: 10k, Resistor_SMD:R_0603_1608Metric, F.Cu at (-44.4, -2.30)
- added R2: 27k, Resistor_SMD:R_0603_1608Metric, F.Cu at (-32.8, 24.5)
- added R2: 62k, Resistor_SMD:R_0201_0603Metric, F.Cu at (-31.1, 13.8)
- added R20: 470, Resistor_SMD:R_0603_1608Metric, F.Cu at (-44.4, 2.72)
- added R21: 10M, Resistor_SMD:R_0603_1608Metric, F.Cu at (-40.4, -7.32)
- added R6: 100k, Resistor_SMD:R_0603_1608Metric, F.Cu at (-34.3, 10.2)
- added R7: 470, Resistor_SMD:R_0603_1608Metric, F.Cu at (-34.3, 7.74)
- added R8: 4.7k, Resistor_SMD:R_0603_1608Metric, F.Cu at (-34.3, 12.8)
- added R9: 62k, Resistor_SMD:R_0201_0603Metric, F.Cu at (-44.9, 9.45)
- added TP1: TestPoint, TestPoint:TestPoint_Loop_D2.54mm_Drill1.5mm_Beaded, F.Cu at (-27.4, 13.7)
- added TP2: TestPoint, TestPoint:TestPoint_Loop_D2.54mm_Drill1.5mm_Beaded, F.Cu at (-41.2, 11.1)
- added U3: LM51561HPWPR, 00_lib:PWP0014H-IPC_A, F.Cu at (-17.3, 13.6)
- added U4: LM51561HPWPR, 00_lib:PWP0014H-IPC_A, F.Cu at (-50.8, 19.9)
- L1: value l=820u -> 15u; footprint 00_lib:IND_MSS1583_COC -> 00_lib:IND_VLS6045EX-150M
- Q1, Q2: value PZTA42 -> BSP88
- R3: value 100k -> 40m; footprint Resistor_SMD:R_0603_1608Metric -> Resistor_SMD:R_0201_0603Metric
- moved R4 138.5 mm to (-34.3, 2.72), turned to 0 degrees
- moved R5 137.8 mm to (-34.3, 5.23), turned to 0 degrees
- moved R3 133.1 mm to (-31.1, 15.6), turned to 0 degrees
- moved Q1 127.3 mm to (-27.4, 7.10)
- moved D1 124.5 mm to (-16.6, -6.41), turned to 0 degrees
- moved L1 104.4 mm to (-18.7, 6.75)
- moved Q2 62.9 mm to (-51.1, 12.7), turned to 0 degrees
- moved R22 42.2 mm to (61.5, 10.6), turned to 0 degrees
- moved R26 39.1 mm to (18.4, 18.2), turned to 180 degrees
- moved U12 35.1 mm to (59.4, 15.2), turned to 180 degrees
- moved C13 33.8 mm to (60.8, 20.3), turned to 90 degrees
- moved U11 28.2 mm to (48.5, 15.2), turned to 180 degrees
- moved C14 26.0 mm to (58.0, 20.3), turned to 90 degrees
- moved C16 21.5 mm to (38.7, 10.0), turned to -90 degrees
- moved C12 19.7 mm to (40.6, 21.0)
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- renumbered C2 to C1, C3 to C12, C4 to C13, C5 to C14, C6 to C15, C7 to C16, R6 to R22, R7 to R23, R8 to R24, R9 to R25, R10 to R26, R11 to R27, U8 to U10, U9 to U11, U10 to U12, U11 to U13, U3 to U5, U4 to U6, U5 to U7, U6 to U8, U7 to U9
Connections:
- D1 pad 1: VPP -> +20V
- D1 pad 2: /High voltage supply/HV_{BOOST} -> Net-(D1-A)
- L1 pad 2: /High voltage supply/HV_{BOOST} -> Net-(D1-A)
- Q1 pad 1: /High voltage supply/HV_{BASE} -> Net-(Q1-G)
- Q1 pad 2: /High voltage supply/HV_{BOOST} -> Net-(D1-A)
- Q1 pad 3: GND -> Net-(Q1-S)
- Q2 pad 1: /LSD_ADC/LSD_{SHUNT_div} -> Net-(Q2-G)
- Q2 pad 2: /LSD_ADC/V_{SHUNT} -> /High voltage supply/HV_{BOOST}
- Q2 pad 3: /LSD_ADC/LSD_{SHUNT_SC_Emitter} -> Net-(Q2-S)
- R3 pad 1: HV_{SENSE} -> Net-(Q1-S)
- R4 pad 1: VPP -> Net-(U3-PGOOD)
- R4 pad 2: /High voltage supply/HV_{BLEED-1} -> +5V
- R5 pad 1: /High voltage supply/HV_{BLEED-1} -> GND
- R5 pad 2: GND -> Net-(U3-RT)
Routing:
- net HV_{SENSE}: track 107.4 -> 5.60 mm, vias 5 -> 0
- net /LSD_ADC/V_{SHUNT}: track 73.9 -> 4.55 mm, vias 4 -> 0
- net DATA_{HV}: track 140.0 -> 77.8 mm
- net VPP: track 187.2 -> 131.2 mm
- net HV_{GATE}: track 84.2 -> 33.3 mm, vias 3 -> 1
- net LSD_{ADC_~{INT}}: track 34.1 -> 0.00 mm
- net LSD_{ADC_~{RD}}: track 30.0 -> 0.00 mm
- net LSD_{ADC_D0}: track 25.9 -> 0.00 mm
- net LSD_{ADC_MODE}: track 25.9 -> 0.00 mm
- net LSD_{ADC_D1}: track 22.2 -> 0.00 mm
- net LSD_{ADC_D6}: track 71.5 -> 49.3 mm
- net LSD_{ADC_~{WR}/RDY}: track 21.5 -> 0.00 mm
- net /LSD_ADC/LSD_{ADC_5V_~{CS}}: track 25.8 -> 4.46 mm
- net LSD_{ADC_D7}: track 76.6 -> 55.5 mm
- net /LSD_ADC/LSD_{ADC_5V_D4}: track 24.2 -> 3.91 mm
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
Commit message: HV bleed circuit
Parts:
- added C12: 1u, Capacitor_SMD:C_0603_1608Metric, F.Cu at (-51.1, 43.1)
- added D3: SM4004, Diode_SMD:D_MELF, F.Cu at (-45.1, 44.0)
- added Q3: BSP88, Package_TO_SOT_SMD:SOT-223-3_TabPin2, F.Cu at (-58.0, 46.0)
- added Q4: BSP88, Package_TO_SOT_SMD:SOT-223-3_TabPin2, F.Cu at (-58.0, 54.2)
- added Q5: BSP88, Package_TO_SOT_SMD:SOT-223-3_TabPin2, F.Cu at (-58.0, 64.5)
- added R22: 4.7k, Resistor_SMD:R_0603_1608Metric, F.Cu at (-51.1, 45.6)
- added R23: 1M, Resistor_SMD:R_0603_1608Metric, F.Cu at (-51.1, 48.1)
- added R24: 10k, Resistor_THT:R_Axial_DIN0617_L17.0mm_D6.0mm_P20.32mm_Horizontal, F.Cu at (-61.0, 38.1)
- added R25: 100k, Resistor_SMD:R_0603_1608Metric, F.Cu at (-51.1, 50.7)
- R28: renamed from R26; value 100k -> 10k
- R29: renamed from R27; value 470 -> 10k
- renumbered C11 to C10, C8 to C11, C12 to C13, C13 to C14, C14 to C15, C15 to C16, C16 to C17, C4 to C2, C5 to C3, C2 to C4, C6 to C5, C3 to C6, C9 to C7, C7 to C8, C10 to C9, R4 to R1, R11 to R10, R17 to R11, R9 to R12, R12 to R13, R13 to R14, R19 to R15, R15 to R16, R18 to R17, R20 to R18, R21 to R19, R10 to R20, R14 to R21, R24 to R26, R25 to R27, R5 to R3, R22 to R30, R23 to R31, R1 to R4, R7 to R5, R3 to R6, R6 to R7, R16 to R9, U8 to U6, U6 to U7, U9 to U8, U7 to U9
Connections:
- C4 pad 1: Net-(U3-VCC) -> /20V_supply/VCC_{LM5156_20V}
- R1 pad 2: +5V -> /20V_supply/VCC_{LM5156_20V}
- R10 pad 1: Net-(U4-BIAS) -> Net-(U4-EN_UVLO_SYNC)
- R12 pad 1: +20V -> Net-(U4-EN_UVLO_SYNC)
- R12 pad 2: Net-(U4-BIAS) -> +20V
- R2 pad 2: Net-(U3-BIAS) -> Net-(U3-EN_UVLO_SYNC)
- R4 pad 1: +5V -> Net-(U3-EN_UVLO_SYNC)
- R4 pad 2: Net-(U3-BIAS) -> +5V
- U1 pad 64: HV_{GATE} -> unconnected-(U1-PICO_PMOD_B1-Pad64)
- U3 pad 1: Net-(U3-BIAS) -> +5V
- U3 pad 14: Net-(U3-BIAS) -> Net-(U3-EN_UVLO_SYNC)
- U3 pad 3: Net-(U3-VCC) -> /20V_supply/VCC_{LM5156_20V}
- U4 pad 1: Net-(U4-BIAS) -> +20V
- U4 pad 14: Net-(U4-BIAS) -> Net-(U4-EN_UVLO_SYNC)
Routing:
- net unconnected-(U1-PICO_PMOD_B1-Pad64): track 0.00 -> 33.3 mm, vias 0 -> 1
- net HV_{GATE}: track 33.3 -> 0.00 mm, vias 1 -> 0

Commit message: Add HV control
Stop tracking SPICE simulations
Parts:
- removed the R1 at (-31.1, 12.1)
- removed the R1 at (-34.3, 2.72)
- removed the R2 at (-32.8, 24.5)
- removed the R2 at (-31.1, 13.8)
- added C18: 0.1u, Capacitor_SMD:C_0603_1608Metric, F.Cu at (-79.9, 5.26)
- added R1: 100k, Resistor_SMD:R_0603_1608Metric, F.Cu at (-65.9, 5.26)
- added R2: 27k, Resistor_SMD:R_0603_1608Metric, F.Cu at (-65.9, 7.77)
- R18: value 470 -> 15k
- R19: value 10M -> 2.7M
- moved D1 50.5 mm to (-63.9, 11.2)
- moved Q5 49.0 mm to (-94.4, 31.6)
- moved R4 37.8 mm to (-61.9, -2.27)
- moved U3 37.5 mm to (-54.7, 16.8)
- moved R19 31.9 mm to (-71.9, -2.27)
- moved R20 31.9 mm to (-71.9, 0.24)
- moved R21 31.9 mm to (-71.9, 2.75)
- moved C4 31.9 mm to (-65.9, 0.24)
- moved R10 31.9 mm to (-75.9, -2.27)
- moved R11 31.9 mm to (-75.9, 0.24)
- moved R15 31.9 mm to (-75.9, 2.75)
- moved R17 31.9 mm to (-75.9, 5.26)
- moved C10 31.6 mm to (-79.9, 2.75)
- moved C2 31.6 mm to (-65.9, -4.78)
- moved C5 31.6 mm to (-65.9, 2.75)
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Connections:
- net /20V_supply/VCC_{LM5156_20V} renamed /20V_supply/20V_{VCC}
- net Net-(C10-Pad1) renamed /High voltage supply/HV_{COMP-1}
- net Net-(C5-Pad1) renamed /20V_supply/20V_{COMP-1}
- net Net-(D1-A) renamed /20V_supply/20V_{BOOST}
- net Net-(Q1-G) renamed /20V_supply/20V_{GATE}
- net Net-(Q1-S) renamed /20V_supply/20V_{CS}
- net Net-(Q2-G) renamed /High voltage supply/HV_{GATE}
- net Net-(Q2-S) renamed /High voltage supply/HV_{SOURCE}
- net Net-(R13-Pad2) renamed /High voltage supply/HV_{CS-1}
- net Net-(U3-COMP) renamed /20V_supply/20V_{COMP}
- net Net-(U3-EN_UVLO_SYNC) renamed /20V_supply/20V_{UVLO}
- net Net-(U3-FB) renamed /20V_supply/20V_{FB}
- net Net-(U3-PGOOD) renamed /20V_supply/20V_{PGOOD}
- net Net-(U3-RT) renamed /20V_supply/20V_{RT}
- net Net-(U3-SS) renamed /20V_supply/20V_{SS}
- net Net-(U4-COMP) renamed /High voltage supply/HV_{COMP}
- net Net-(U4-CS) renamed /High voltage supply/HV_{CS}
- net Net-(U4-EN_UVLO_SYNC) renamed /High voltage supply/HV_{UVLO}
- net Net-(U4-PGOOD) renamed /High voltage supply/HV_{PGOOD}
- net Net-(U4-RT) renamed /High voltage supply/HV_{RT}
- net Net-(U4-SS) renamed /High voltage supply/HV_{SS}
- net Net-(U4-VCC) renamed /High voltage supply/HV_{VCC}
- R17 pad 1: Net-(U4-FB) -> /High voltage supply/HV_{FB}
- R17 pad 2: VPP -> HV_{CONTROL}
- R18 pad 2: Net-(U4-FB) -> /High voltage supply/HV_{FB}
- R19 pad 1: VPP -> /High voltage supply/HV_{FB}
- R19 pad 2: GND -> VPP
- U4 pad 10: Net-(U4-FB) -> /High voltage supply/HV_{FB}

Commit message: finish schematic features
Parts:
- removed the C18 at (-79.9, 5.26)
- added C13: 1u, Capacitor_SMD:C_0603_1608Metric, F.Cu at (-38.3, 10.4)
- added J10: Conn_02x05_Odd_Even, Connector_PinSocket_2.54mm:PinSocket_2x05_P2.54mm_Horizontal, F.Cu at (-41.6, 33.6)
- added J4: Conn_01x02_Pin, Connector_PinHeader_2.54mm:PinHeader_1x02_P2.54mm_Vertical, F.Cu at (-35.9, 50.4)
- added J5: Conn_01x02_Pin, Connector_PinHeader_2.54mm:PinHeader_1x02_P2.54mm_Vertical, F.Cu at (-31.3, 50.4)
- added J7: Conn_01x02_Pin, Connector_PinHeader_2.54mm:PinHeader_1x02_P2.54mm_Vertical, F.Cu at (-35.9, 59.6)
- added J8: Conn_01x02_Pin, Connector_PinHeader_2.54mm:PinHeader_1x02_P2.54mm_Vertical, F.Cu at (-86.8, 61.6)
- added J9: Conn_01x02_Pin, Connector_PinHeader_2.54mm:PinHeader_1x02_P2.54mm_Vertical, F.Cu at (-65.2, 31.2)
- added TP10: TestPoint, TestPoint:TestPoint_Loop_D2.54mm_Drill1.5mm_Beaded, F.Cu at (-69.8, 21.3)
- added TP11: TestPoint, TestPoint:TestPoint_Loop_D2.54mm_Drill1.5mm_Beaded, F.Cu at (-69.8, 26.3)
- added TP12: TestPoint, TestPoint:TestPoint_Loop_D2.54mm_Drill1.5mm_Beaded, F.Cu at (-64.7, 21.3)
- added TP13: TestPoint, TestPoint:TestPoint_Loop_D2.54mm_Drill1.5mm_Beaded, F.Cu at (-64.7, 26.3)
- added TP14: TestPoint, TestPoint:TestPoint_Loop_D2.54mm_Drill1.5mm_Beaded, F.Cu at (-59.7, 21.3)
- added TP15: TestPoint, TestPoint:TestPoint_Loop_D2.54mm_Drill1.5mm_Beaded, F.Cu at (-59.7, 26.3)
- added TP16: TestPoint, TestPoint:TestPoint_Loop_D2.54mm_Drill1.5mm_Beaded, F.Cu at (-52.6, 11.7)
- added TP17: TestPoint, TestPoint:TestPoint_Loop_D2.54mm_Drill1.5mm_Beaded, F.Cu at (-52.6, 16.7)
- added TP18: TestPoint, TestPoint:TestPoint_Loop_D2.54mm_Drill1.5mm_Beaded, F.Cu at (-52.6, 21.8)
- added TP19: TestPoint, TestPoint:TestPoint_Loop_D2.54mm_Drill1.5mm_Beaded, F.Cu at (-52.6, 26.8)
- added TP20: TestPoint, TestPoint:TestPoint_Loop_D2.54mm_Drill1.5mm_Beaded, F.Cu at (-52.6, 50.6)
- added TP21: TestPoint, TestPoint:TestPoint_Loop_D2.54mm_Drill1.5mm_Beaded, F.Cu at (-52.6, 55.7)
- added TP22: TestPoint, TestPoint:TestPoint_Loop_D2.54mm_Drill1.5mm_Beaded, F.Cu at (-52.6, 60.7)
- added TP23: TestPoint, TestPoint:TestPoint_Loop_D2.54mm_Drill1.5mm_Beaded, F.Cu at (-52.6, 65.8)
- added TP3: TestPoint, TestPoint:TestPoint_Loop_D2.54mm_Drill1.5mm_Beaded, F.Cu at (-86.6, 51.7)
- added TP4: TestPoint, TestPoint:TestPoint_Loop_D2.54mm_Drill1.5mm_Beaded, F.Cu at (-86.6, 56.8)
- added TP5: TestPoint, TestPoint:TestPoint_Loop_D2.54mm_Drill1.5mm_Beaded, F.Cu at (-81.6, 41.6)
- added TP6: TestPoint, TestPoint:TestPoint_Loop_D2.54mm_Drill1.5mm_Beaded, F.Cu at (-81.6, 46.7)
- added TP7: TestPoint, TestPoint:TestPoint_Loop_D2.54mm_Drill1.5mm_Beaded, F.Cu at (-81.6, 51.7)
- added TP8: TestPoint, TestPoint:TestPoint_Loop_D2.54mm_Drill1.5mm_Beaded, F.Cu at (-74.8, 21.3)
- added TP9: TestPoint, TestPoint:TestPoint_Loop_D2.54mm_Drill1.5mm_Beaded, F.Cu at (-74.8, 26.3)
- C10: value 1u -> 1n
- C11, C6: value 10u -> 1u; footprint Capacitor_THT:CP_Radial_D10.0mm_P5.00mm -> Capacitor_SMD:C_0603_1608Metric
- C12, C4: value 1u -> 0.1u
- C2: value 0.1u -> 1u
- C3, C8: value 1u -> 10u; footprint Capacitor_SMD:C_0603_1608Metric -> Capacitor_THT:CP_Radial_D10.0mm_P5.00mm
- C9: value 1n -> 1u
- R1: value 100k -> 62k
- R10: value 4.7k -> 10M
- R11: value 220k -> 4.7k
- R12: value 62k -> 1k
- R14: value 1k -> 100k; footprint Resistor_SMD:R_0201_0603Metric -> Resistor_SMD:R_0603_1608Metric
- R15: value 10k -> 40m; footprint Resistor_SMD:R_0603_1608Metric -> Resistor_SMD:R_0201_0603Metric
- R16, R6: value 40m -> 100k; footprint Resistor_SMD:R_0201_0603Metric -> Resistor_SMD:R_0603_1608Metric
- R17: value 100k -> 220k
- R18: value 15k -> 2.7M
- R19: value 2.7M -> 10k
- R20: value 10M -> 100k
- R21: value 100k -> 15k
- R22: value 4.7k -> 1M
- R23: value 1M -> 10k; footprint Resistor_SMD:R_0603_1608Metric -> Resistor_THT:R_Axial_DIN0617_L17.0mm_D6.0mm_P20.32mm_Horizontal
- R24: value 10k -> 4.7k; footprint Resistor_THT:R_Axial_DIN0617_L17.0mm_D6.0mm_P20.32mm_Horizontal -> Resistor_SMD:R_0603_1608Metric
- R3: value 100k -> 40m; footprint Resistor_SMD:R_0603_1608Metric -> Resistor_SMD:R_0201_0603Metric
- R4: value 62k -> 100k
- R5: value 470 -> 100k
- R7: value 100k -> 470
- R9: value 100k -> 62k; footprint Resistor_SMD:R_0603_1608Metric -> Resistor_SMD:R_0201_0603Metric
- moved R3 68.4 mm to (-83.3, 60.2)
- moved C3 62.9 mm to (-75.5, 59.9)
- moved L1 55.7 mm to (-63.4, 62.3)
- moved Q5 53.3 mm to (-45.2, 52.2)
- moved C6 52.4 mm to (-77.1, 47.9)
- moved TP1 47.0 mm to (-86.6, 41.6)
- moved C2 46.5 mm to (-77.1, 40.3)
- moved R1 46.5 mm to (-77.1, 50.4)
- moved R7 46.5 mm to (-73.1, 47.9)
- moved R8 46.5 mm to (-73.1, 50.4)
- moved R2 46.5 mm to (-77.1, 52.9)
- moved D1 45.1 mm to (-63.3, 56.3)
- moved C4 44.1 mm to (-77.1, 42.8)
- moved C5 44.1 mm to (-77.1, 45.4)
- moved R4 44.1 mm to (-73.1, 40.3)
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- renumbered C13 to C14, C14 to C15, C15 to C16, C16 to C17, C17 to C18, J4 to J6, R30 to R26, R31 to R27, R26 to R28, R27 to R29, R28 to R30, R29 to R31, U7 to U6, U9 to U7, U6 to U8, U8 to U9
Connections:
- net /20V_supply/20V_{GATE} renamed /20V supply/20V_{GATE}
- net /LSD_ADC/LSD_{ADC_5V_D0} renamed /LSD ADC/LSD_{ADC_5V_D0}
- net /LSD_ADC/LSD_{ADC_5V_D1} renamed /LSD ADC/LSD_{ADC_5V_D1}
- net /LSD_ADC/LSD_{ADC_5V_D2} renamed /LSD ADC/LSD_{ADC_5V_D2}
- net /LSD_ADC/LSD_{ADC_5V_D3} renamed /LSD ADC/LSD_{ADC_5V_D3}
- net /LSD_ADC/LSD_{ADC_5V_D4} renamed /LSD ADC/LSD_{ADC_5V_D4}
- net /LSD_ADC/LSD_{ADC_5V_D5} renamed /LSD ADC/LSD_{ADC_5V_D5}
- net /LSD_ADC/LSD_{ADC_5V_D6} renamed /LSD ADC/LSD_{ADC_5V_D6}
- net /LSD_ADC/LSD_{ADC_5V_D7} renamed /LSD ADC/LSD_{ADC_5V_D7}
- net /LSD_ADC/LSD_{ADC_5V_MODE} renamed /LSD ADC/LSD_{ADC_5V_MODE}
- net /LSD_ADC/LSD_{ADC_5V_~{CS}} renamed /LSD ADC/LSD_{ADC_5V_~{CS}}
- net /LSD_ADC/LSD_{ADC_5V_~{INT}} renamed /LSD ADC/LSD_{ADC_5V_~{INT}}
- net /LSD_ADC/LSD_{ADC_5V_~{OFL}} renamed /LSD ADC/LSD_{ADC_5V_~{OFL}}
- net /LSD_ADC/LSD_{ADC_5V_~{RD}} renamed /LSD ADC/LSD_{ADC_5V_~{RD}}
- net /LSD_ADC/LSD_{ADC_5V_~{WR}/RDY} renamed /LSD ADC/LSD_{ADC_5V_~{WR}/RDY}
- net /LSD_ADC/OE_{lvl-shift-1} renamed /LSD ADC/OE_{lvl-shift-1}
- net /LSD_ADC/OE_{lvl-shift-2} renamed /LSD ADC/OE_{lvl-shift-2}
- net /LSD_ADC/VCC_{ADC} renamed /LSD ADC/VCC_{ADC}
- net /LSD_ADC/VCC_{lvl-shift-A-1} renamed /LSD ADC/VCC_{lvl-shift-A-1}
- net /LSD_ADC/VCC_{lvl-shift-A-2} renamed /LSD ADC/VCC_{lvl-shift-A-2}
- net /LSD_ADC/VCC_{lvl-shift-B-1} renamed /LSD ADC/VCC_{lvl-shift-B-1}
- net /LSD_ADC/VCC_{lvl-shift-B-2} renamed /LSD ADC/VCC_{lvl-shift-B-2}
- BT1 pad 1: +3V3_STDBY -> /GPS/3.3V_STDBY_{SENSE}
- C10 pad 1: /High voltage supply/HV_{COMP-1} -> /High voltage supply/HV_{COMP}
- C11 pad 1: VPP -> /High voltage supply/HV_{COMP-1}
- C12 pad 1: /HV_bleed/HV_Bleed_{source} -> /High voltage supply/HV_{FB}
- C2 pad 1: /20V_supply/20V_{SS} -> /20V supply/20V_{VCC}
- C3 pad 1: /20V_supply/20V_{COMP} -> /20V supply/20V_{SENSE}
- C4 pad 1: /20V_supply/20V_{VCC} -> /20V supply/20V_{SS}
- C5 pad 1: /20V_supply/20V_{COMP-1} -> /20V supply/20V_{COMP}
- C6 pad 1: +20V -> /20V supply/20V_{COMP-1}
- C7 pad 1: GND -> /High voltage supply/HV_{VCC}
- C7 pad 2: /High voltage supply/HV_{SS} -> GND
- C8 pad 1: /High voltage supply/HV_{VCC} -> /High voltage supply/HV_{SENSE}
- C9 pad 1: /High voltage supply/HV_{COMP} -> GND
- C9 pad 2: GND -> /High voltage supply/HV_{SS}
- D1 pad 1: +20V -> /20V supply/20V_{SENSE}
- D1 pad 2: /20V_supply/20V_{BOOST} -> /20V supply/20V_{BOOST}
- D2 pad 1: VPP -> /High voltage supply/HV_{SENSE}
- D3 pad 1: /HV_bleed/HV_Bleed_{gate} -> /HV bleed/HV_bleed_{gate}
- D3 pad 2: /HV_bleed/HV_Bleed_{pulldown} -> /HV bleed/HV_bleed_{pulldown}
- L1 pad 2: /20V_supply/20V_{BOOST} -> /20V supply/20V_{BOOST}
- Q1 pad 2: /20V_supply/20V_{BOOST} -> /20V supply/20V_{BOOST}
- Q1 pad 3: /20V_supply/20V_{CS} -> /20V supply/20V_{CS}
- Q3 pad 1: +5V -> /HV bleed/HV_bleed_{gate}
- Q3 pad 2: /HV_bleed/HV_Bleed_{gate} -> /HV bleed/HV_bleed_{drain}
- Q3 pad 3: GND -> /HV bleed/HV_bleed_{source}
- Q4 pad 1: /HV_bleed/HV_Bleed_{gate} -> +5V
- Q4 pad 2: /HV_bleed/HV_Bleed_{drain} -> /HV bleed/HV_bleed_{gate}
- Q4 pad 3: /HV_bleed/HV_Bleed_{source} -> GND
- Q5 pad 1: /LSD_ADC/LSD_{SHUNT_div} -> /LSD ADC/LSD_{SHUNT_div}
- Q5 pad 2: /LSD_ADC/V_{SHUNT} -> /LSD ADC/V_{SHUNT}
- Q5 pad 3: /LSD_ADC/LSD_{SHUNT_SC_Emitter} -> /LSD ADC/LSD_{SHUNT_SC_Emitter}
- R1 pad 1: /20V_supply/20V_{PGOOD} -> /20V supply/20V_{UVLO}
- R1 pad 2: /20V_supply/VCC_{LM5156_20V} -> +5V
- R10 pad 1: /High voltage supply/HV_{UVLO} -> VPP
- R10 pad 2: GND -> HV_{MEASURE}
- R11 pad 1: GND -> /High voltage supply/HV_{UVLO}
- R11 pad 2: /High voltage supply/HV_{RT} -> GND
- R12 pad 1: /High voltage supply/HV_{UVLO} -> /High voltage supply/HV_{CS}
- R12 pad 2: +20V -> /High voltage supply/HV_{CS-1}
- R13 pad 1: /High voltage supply/HV_{CS} -> /High voltage supply/HV_{CS-1}
- R13 pad 2: /High voltage supply/HV_{CS-1} -> /High voltage supply/HV_{SOURCE}
- R14 pad 1: /High voltage supply/HV_{CS-1} -> HV_{MEASURE}
- R14 pad 2: /High voltage supply/HV_{SOURCE} -> GND
- R15 pad 1: /High voltage supply/HV_{COMP} -> /High voltage supply/HV_{SOURCE}
- R15 pad 2: /High voltage supply/HV_{COMP-1} -> GND
- R16 pad 1: /High voltage supply/HV_{SOURCE} -> /High voltage supply/HV_{PGOOD}
- R16 pad 2: GND -> /High voltage supply/HV_{VCC}
- R17 pad 1: /High voltage supply/HV_{FB} -> GND
- R17 pad 2: HV_{CONTROL} -> /High voltage supply/HV_{RT}
- R18 pad 1: GND -> /High voltage supply/HV_{FB}
- R18 pad 2: /High voltage supply/HV_{FB} -> /High voltage supply/HV_{SENSE}
- R19 pad 1: /High voltage supply/HV_{FB} -> /High voltage supply/HV_{COMP}
- R19 pad 2: VPP -> /High voltage supply/HV_{COMP-1}
- R2 pad 2: /20V_supply/20V_{UVLO} -> /20V supply/20V_{UVLO}
- R20 pad 1: VPP -> /High voltage supply/HV_{FB}
- R20 pad 2: HV_{SENSE} -> HV_{CONTROL}
- R21 pad 1: HV_{SENSE} -> GND
- R21 pad 2: GND -> /High voltage supply/HV_{FB}
- R22 pad 1: GND -> /HV bleed/HV_bleed_{pulldown}
- R22 pad 2: +5V -> VPP
- R23 pad 1: /HV_bleed/HV_Bleed_{pulldown} -> VPP
- R23 pad 2: VPP -> /HV bleed/HV_bleed_{drain}
- R24 pad 1: VPP -> GND
- R24 pad 2: /HV_bleed/HV_Bleed_{drain} -> +5V
- R25 pad 1: /HV_bleed/HV_Bleed_{source} -> /HV bleed/HV_bleed_{source}
- R28 pad 2: /LSD_ADC/LSD_{SHUNT_div} -> /LSD ADC/LSD_{SHUNT_div}
- R29 pad 1: /LSD_ADC/LSD_{SHUNT_div} -> /LSD ADC/LSD_{SHUNT_div}
- R3 pad 1: GND -> /20V supply/20V_{CS}
- R3 pad 2: /20V_supply/20V_{RT} -> GND
- R30 pad 2: /LSD_ADC/V_{SHUNT} -> /LSD ADC/V_{SHUNT}
- R31 pad 1: /LSD_ADC/LSD_{SHUNT_SC_Emitter} -> /LSD ADC/LSD_{SHUNT_SC_Emitter}
- R4 pad 1: /20V_supply/20V_{UVLO} -> /20V supply/20V_{PGOOD}
- R4 pad 2: +5V -> /20V supply/20V_{VCC}
- R5 pad 1: /20V_supply/20V_{COMP} -> GND
- R5 pad 2: /20V_supply/20V_{COMP-1} -> /20V supply/20V_{RT}
- R6 pad 1: /20V_supply/20V_{CS} -> /20V supply/20V_{FB}
- R6 pad 2: GND -> /20V supply/20V_{SENSE}
- R7 pad 1: /20V_supply/20V_{FB} -> /20V supply/20V_{COMP}
- R7 pad 2: +20V -> /20V supply/20V_{COMP-1}
- R8 pad 2: /20V_supply/20V_{FB} -> /20V supply/20V_{FB}
- R9 pad 1: /High voltage supply/HV_{PGOOD} -> /High voltage supply/HV_{UVLO}
- R9 pad 2: +5V -> +20V
- TP1 pad 1: /20V_supply/20V_{PGOOD} -> /20V supply/20V_{BOOST}
- TP2 pad 1: /High voltage supply/HV_{PGOOD} -> /20V supply/20V_{UVLO}
- U1 pad 5: +3.3V -> /3.3V_{SENSE}
- U1 pad 55: +3.3V -> /3.3V_{SENSE}
- U1 pad 56: +3.3V -> /3.3V_{SENSE}
- U1 pad 6: +3.3V -> /3.3V_{SENSE}
- U1 pad 61: HV_{SENSE} -> HV_{MEASURE}
- U1 pad 73: +3.3V -> /3.3V_{SENSE}
- U1 pad 74: +3.3V -> /3.3V_{SENSE}
- U1 pad 75: +3.3V -> /3.3V_{SENSE}
- U1 pad 79: +5V -> /5V_{SENSE}
- U10 pad 1: unconnected-(U10-DOUT-Pad1) -> /Nixies/D_{IN-PRECISE}
- U11 pad 1: /LSD_ADC/V_{SHUNT} -> /LSD ADC/V_{SHUNT}
- U3 pad 10: /20V_supply/20V_{FB} -> /20V supply/20V_{FB}
- U3 pad 11: /20V_supply/20V_{SS} -> /20V supply/20V_{SS}
- U3 pad 12: /20V_supply/20V_{RT} -> /20V supply/20V_{RT}
- U3 pad 13: /20V_supply/20V_{PGOOD} -> /20V supply/20V_{PGOOD}
- U3 pad 14: /20V_supply/20V_{UVLO} -> /20V supply/20V_{UVLO}
- U3 pad 3: /20V_supply/20V_{VCC} -> /20V supply/20V_{VCC}
- U3 pad 7: /20V_supply/20V_{CS} -> /20V supply/20V_{CS}
- U3 pad 8: /20V_supply/20V_{COMP} -> /20V supply/20V_{COMP}
Routing:
- net /3.3V_{SENSE}: track 0.00 -> 57.2 mm, vias 0 -> 3
- net +3.3V: track 73.9 -> 16.6 mm, vias 11 -> 8
- net +5V: track 41.7 -> 32.2 mm, vias 14 -> 12
- net /5V_{SENSE}: track 0.00 -> 9.54 mm, vias 0 -> 2
- net HV_{SENSE}: track 5.60 -> 0.00 mm
- net HV_{MEASURE}: track 0.00 -> 5.60 mm

Commit message: ERC pass
layout WIP
All components arranged except power supplies.
Most nets routed (all except power supplies and ADC lines).
Parts:
- removed the Q3 at (14.0, 18.2)
- moved J7 153.5 mm to (117.4, 67.3), turned to 90 degrees
- moved J6 149.9 mm to (150.3, 64.5), turned to 0 degrees
- moved RV1 139.2 mm to (144.8, 73.7), turned to 180 degrees
- moved J4 131.9 mm to (88.8, 93.3), turned to -90 degrees
- moved J5 125.9 mm to (88.8, 88.2), turned to -90 degrees
- moved H1 122.9 mm to (4.00, 97.6)
- moved U2 120.0 mm to (135.6, 62.5), turned to 0 degrees
- moved J2 110.8 mm to (142.7, 48.3)
- moved TP23 107.6 mm to (50.8, 36.1)
- moved C1 103.7 mm to (126.0, 68.4), turned to 180 degrees
- moved TP22 100.4 mm to (44.7, 36.1)
- moved J1 95.6 mm to (128.0, 48.3)
- moved REF** 91.0 mm to (47.8, 96.5)
- moved U1 89.1 mm to (119.7, 88.7), turned to 90 degrees
- moved TP21 85.4 mm to (30.5, 36.1)
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Connections:
- U1 pad 10: /RESERVED_1 -> HV_{CONTROL}
- U1 pad 11: /24h_mode -> LSD_{ADC_D3}
- U1 pad 12: /anti-poison_force -> LSD_{ADC_~{OFL}}
- U1 pad 13: /anti-poison_routine -> LSD_{ADC_D2}
- U1 pad 14: /manual_brightness -> LSD_{ADC_D7}
- U1 pad 15: /DST_force -> LSD_{ADC_D1}
- U1 pad 16: /DST_check -> LSD_{ADC_D6}
- U1 pad 18: unconnected-(U1-ICE_35_G0-Pad18) -> LSD_{ADC_D5}
- U1 pad 19: LSD_{ADC_~{OFL}} -> LSD_{ADC_D0}
- U1 pad 20: PPS_{TRIMMED} -> LSD_{ADC_D4}
- U1 pad 21: LSD_{ADC_D7} -> PPS_{TRIMMED}
- U1 pad 22: LSD_{ADC_D6} -> LSD_{ADC_MODE}
- U1 pad 27: LSD_{ADC_D5} -> LSD_{ADC_~{WR}/RDY}
- U1 pad 28: LSD_{ADC_D4} -> LSD_{ADC_~{RD}}
- U1 pad 29: GPS_{1PPS} -> GPS_{1PPS2}
- U1 pad 30: LSD_{ADC_~{CS}} -> LSD_{ADC_~{INT}}
- U1 pad 31: GPS_{1PPS2} -> GPS_{1PPS}
- U1 pad 32: CLOCK_{HV} -> LSD_{ADC_~{CS}}
- U1 pad 33: unconnected-(U1-ICE_3-Pad33) -> DATA_{HV}
- U1 pad 34: DATA_{HV} -> CLOCK_{HV}
- U1 pad 45: LSD_{ADC_~{WR}/RDY} -> /DST_force
- U1 pad 46: LSD_{ADC_D3} -> /DST_check
- U1 pad 47: LSD_{ADC_MODE} -> /anti-poison_routine
- U1 pad 48: LSD_{ADC_D2} -> /manual_brightness
- U1 pad 49: LSD_{ADC_~{RD}} -> /24h_mode
- U1 pad 50: LSD_{ADC_D1} -> /anti-poison_force
- U1 pad 51: LSD_{ADC_~{INT}} -> /RESERVED_2
- U1 pad 52: LSD_{ADC_D0} -> /RESERVED_1
- U1 pad 59: /brightness_control -> HV_{MEASURE}
- U1 pad 61: HV_{MEASURE} -> /brightness_control
- U1 pad 63: GPS_{BOOT_SEL} -> GPS_{RXD}
- U1 pad 65: unconnected-(U1-PICO_PMOD_A2-Pad65) -> GPS_{TXD}
- U1 pad 66: GPS_{RXD} -> unconnected-(U1-PICO_PMOD_B2-Pad66)
- U1 pad 67: unconnected-(U1-PICO_PMOD_A3-Pad67) -> GPS_{RSTN}
- U1 pad 68: GPS_{TXD} -> unconnected-(U1-PICO_PMOD_B3-Pad68)
- U1 pad 69: unconnected-(U1-PICO_PMOD_A4-Pad69) -> GPS_{BOOT_SEL}
- U1 pad 70: GPS_{RSTN} -> unconnected-(U1-PICO_PMOD_B4-Pad70)
- U1 pad 9: /RESERVED_2 -> SENSE_{PRECISE}
Routing:
- net /LSD ADC/V_{SHUNT}: track 0.00 -> 102.4 mm
- net +3V3_STDBY: track 137.6 -> 54.3 mm, vias 1 -> 0
- net LSD_{ADC_D5}: track 83.0 -> 3.93 mm, vias 3 -> 1
- net LSD_{ADC_~{CS}}: track 77.5 -> 4.45 mm, vias 3 -> 1
- net LSD_{ADC_D4}: track 76.8 -> 4.19 mm, vias 3 -> 1
- net GPS_{1PPS}: track 73.3 -> 15.2 mm, vias 1 -> 0
- net LSD_{ADC_D7}: track 55.5 -> 4.08 mm, vias 2 -> 1
- net CLOCK_{HV}: track 184.9 -> 231.3 mm, vias 2 -> 1
- net LSD_{ADC_D6}: track 49.3 -> 3.83 mm, vias 2 -> 1
- net LSD_{ADC_~{OFL}}: track 49.6 -> 4.33 mm, vias 3 -> 1
- net /LSD ADC/LSD_{SHUNT_SC_Emitter}: track 0.00 -> 43.8 mm, vias 0 -> 2
- net /3.3V_{SENSE}: track 57.2 -> 16.4 mm, vias 3 -> 4
- net GPS_{1PPS2}: track 51.9 -> 17.4 mm, vias 1 -> 0
- net unconnected-(U1-PICO_PMOD_B1-Pad64): track 33.3 -> 0.00 mm, vias 1 -> 0
- net VPP: track 131.2 -> 161.2 mm, vias 0 -> 1
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- added copper zone on F.Cu, net /3.3V_{SENSE}
- added copper zone on B.Cu, net /5V_{SENSE}
- removed copper zone on B.Cu, net GND
Other:
- board size 129 x 80 mm -> 152.4 x 101.6 mm
- board text added: "+3.3V"
- board text added: "+3.3V standby"
- board text added: "+5V"
- board text added: "Nixie Accurate Clock, Rev A https://github.com/willis936/nixie-clock-ice"
- board text removed: "Nixie Accurate Clock Rev A https://github.com/willis936/nixie-clock-ice"

Commit message: tear it apart again
I didn't fix the pico iCE pinout after flipping it over.

I still haven't, but routing is now a fresh start.
Parts:
- moved C14 122.2 mm to (205.9, 55.7)
- moved C17 122.2 mm to (194.9, 60.2)
- moved C18 122.2 mm to (194.9, 57.6)
- moved R27 122.2 mm to (205.1, 60.9)
- moved U11 122.2 mm to (200.2, 47.9)
- moved U12 122.2 mm to (200.2, 36.9)
- moved U13 122.2 mm to (200.2, 58.9)
- moved C15 122.2 mm to (205.2, 35.6)
- moved C16 122.2 mm to (205.2, 38.4)
- moved R30 122.2 mm to (192.2, 48.1)
- moved R26 122.2 mm to (195.5, 34.9)
- moved J4 61.0 mm to (82.4, 153.9)
- moved SW1 61.0 mm to (73.9, 158.7)
- moved J5 61.0 mm to (82.4, 148.8)
- moved J6 51.8 mm to (111.8, 99.1), turned to -90 degrees
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Routing:
- net CLOCK_{HV}: track 231.3 -> 166.5 mm
- net DATA_{HV}: track 64.7 -> 4.24 mm
- net +3V3_STDBY: track 54.3 -> 0.00 mm
- net PPS_{TRIMMED}: track 228.0 -> 173.9 mm
- net /~{ICE_RST}: track 49.9 -> 0.00 mm, vias 1 -> 0
- net /brightness_control: track 44.4 -> 0.00 mm, vias 1 -> 0
- net GPS_{RSTN}: track 43.4 -> 0.00 mm
- net /~{RESET}: track 38.9 -> 0.00 mm
- net /RESERVED_1: track 37.1 -> 0.00 mm
- net /RESERVED_2: track 37.0 -> 0.00 mm
- net GPS_{BOOT_SEL}: track 36.7 -> 0.00 mm
- net GPS_{TXD}: track 34.9 -> 0.00 mm
- net GPS_{RXD}: track 34.8 -> 0.00 mm
- net /anti-poison_force: track 34.6 -> 0.00 mm
- net /~{USB_BOOT}: track 33.8 -> 0.00 mm
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- removed copper zone on F.Cu, net /3.3V_{SENSE}
- removed copper zone on B.Cu, net /5V_{SENSE}
Other:
- board text removed: "+3.3V standby"
