File: KiCad/nixieAccurateClock/nixieAccurateClock.kicad_pcb (KiCad board)
At the start: 4 copper layers, 152.4 x 101.6 mm, 111 parts, among them J1 Conn_01x02_Pin, J2 Conn_01x02_Pin, J3 Conn_01x02_Pin, J4 Conn_01x02_Pin, J5 Conn_Coaxial, J6 Conn_01x02_Pin, J7 Conn_01x02_Pin, J8 Conn_01x02_Pin, J9 Conn_02x05_Odd_Even, Q1 BSP88, Q2 BSP88, Q3 BSP88, Q4 BSP88, Q5 BSP88, SW1 SW_DIP_x08, U1 MCP23008-xSO, U13 ADC0820BCWMX, U14 TXB0108PWR, U15 TXB0108PWR, U2 pico iCE, U3 LTR-329ALS-01, U4 PX1125T, U5 LM51561HPWPR, U6 LM51561HPWPR

Commit message: swap bleed resistor for SMD
Parts:
- added REF**: Symbol_HighVoltage_Type2_CopperTop_VerySmall, Symbol:Symbol_HighVoltage_Type2_CopperTop_VerySmall, F.Cu at (61.0, 69.2)
- R25: footprint Resistor_THT:R_Axial_DIN0617_L17.0mm_D6.0mm_P20.32mm_Horizontal -> Resistor_SMD:R_2512_6332Metric
- moved R25 14.5 mm to (26.0, 44.5)
Routing:
- net HV_{SENSE}: track 40.2 -> 52.0 mm, vias 1 -> 2
- net /HV bleed/HV_bleed_{drain}: track 19.8 -> 22.6 mm

Commit message: Switch to SMT test points
Parts:
- TP1, TP10, TP11, TP12, TP13, TP14, TP15, TP16, TP17, TP18, TP19, TP2, TP20, TP3, TP4, TP5, TP6, TP7, TP8, TP9: footprint TestPoint:TestPoint_Loop_D2.54mm_Drill1.5mm_Beaded -> 00_lib:TestPoint_Keystone_5019_Minature

Commit message: Add fiducials
Parts:
- added FID1: Fiducial, Fiducial:Fiducial_1mm_Mask3mm, F.Cu at (9.12, 92.5)
- added FID2: Fiducial, Fiducial:Fiducial_1mm_Mask3mm, F.Cu at (143.3, 92.5)
- added FID3: Fiducial, Fiducial:Fiducial_1mm_Mask3mm, F.Cu at (143.3, 9.12)
- moved BT1 24.3 mm to (147.5, 74.0), turned to 180 degrees
- moved SW1 7.62 mm to (126.6, 39.4)
- moved U1 7.62 mm to (117.8, 48.3)
- moved C1 7.62 mm to (122.4, 40.6)
Routing:
- net /GPS/3.3V_STDBY_{SENSE}: track 20.0 -> 28.0 mm
- net /INT_{IO-expander}: track 37.0 -> 44.6 mm
- net /~{RESET}_{IO-expander}: track 41.6 -> 49.2 mm
- net /brightness_control: track 62.5 -> 57.8 mm
- net I2C_{DATA}: track 161.9 -> 165.1 mm
- net I2C_{CLOCK}: track 156.3 -> 159.5 mm
Other:
- board text removed: "Migrate this stuff up a little."

Commit message: switch to 27k R_anode
Add voltage rail jumpers for different 5V and 3.3V standby applications
Parts:
- added J5: Conn_01x02_Pin, Connector_PinHeader_2.54mm:PinHeader_1x02_P2.54mm_Vertical, F.Cu at (156.8, 122.3)
- added J8: Conn_01x02_Pin, Connector_PinHeader_2.54mm:PinHeader_1x02_P2.54mm_Vertical, F.Cu at (31.5, 89.0)
- moved C12 44.9 mm to (71.2, 94.5)
- moved J4 44.9 mm to (131.3, 70.4)
- moved C11 44.9 mm to (67.0, 88.8)
- moved C13 44.9 mm to (74.0, 95.5)
- moved C14 44.9 mm to (76.2, 89.0)
- moved J1 44.9 mm to (100.8, 128.3)
- moved R14 44.9 mm to (69.2, 102.5)
- moved R15 44.9 mm to (71.0, 102.5)
- moved R17 44.9 mm to (70.7, 98.5)
- moved R20 44.9 mm to (76.2, 91.0)
- moved R21 44.9 mm to (73.7, 93.8)
- moved R22 44.9 mm to (76.2, 84.5)
- moved R23 44.9 mm to (76.2, 86.8)
- moved R27 44.9 mm to (130.0, 43.8)
- moved R30 44.9 mm to (54.7, 50.7)
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- renumbered J8 to J10, J9 to J11, J5 to J6, J6 to J7, J7 to J9
Connections:
- BT1 pad 1: /GPS/3.3V_STDBY_{SENSE} -> +3V3_STDBY
- J7 pad 1: /GPS/3.3V_STDBY_{SENSE} -> +3V3_STDBY
- J7 pad 2: +3V3_STDBY -> /GPS/3.3V_STDBY_GPS_{SENSE}
- R3 pad 2: +5V -> /20V supply/5V_20V_{SENSE}
- U2 pad 77: +3V3_STDBY -> /3.3V_STDBY_SRAM_{SENSE}
- U4 pad 22: +3V3_STDBY -> /GPS/3.3V_STDBY_GPS_{SENSE}
- U5 pad 1: +5V -> /20V supply/5V_20V_{SENSE}
Routing:
- net +3V3_STDBY: track 53.3 -> 0.00 mm
- net /3.3V_STDBY_SRAM_{SENSE}: track 0.00 -> 30.7 mm
- net /GPS/3.3V_STDBY_{SENSE}: track 28.0 -> 0.00 mm
- net /GPS/3.3V_STDBY_GPS_{SENSE}: track 0.00 -> 21.1 mm
- net /20V supply/5V_20V_{SENSE}: track 0.00 -> 4.66 mm
- net +5V: track 29.0 -> 24.6 mm, vias 14 -> 13
- net DATA_{HV}: vias 1 -> 0
- added copper zone on F.Cu, net +3V3_STDBY
Other:
- board text added: "210V"

Commit message: clean up pico iCE traces
Parts:
- C10, C5: footprint Capacitor_THT:CP_Radial_D10.0mm_P5.00mm -> Capacitor_SMD:CP_Elec_8x10
- R1, R2: value 4.7k -> 1k
- SW1: footprint Button_Switch_THT:SW_DIP_SPSTx08_Slide_6.7x21.88mm_W7.62mm_P2.54mm_LowProfile -> Button_Switch_SMD:SW_DIP_SPSTx08_Slide_6.7x21.88mm_W8.61mm_P2.54mm_LowProfile
- moved R31 44.2 mm to (73.9, 41.4), turned to 90 degrees
- moved SW1 9.76 mm to (162.4, 80.0)
- moved TP20 8.70 mm to (83.6, 76.5)
- moved C5 2.57 mm to (57.1, 120.2)
Routing:
- net +3.3V: track 43.7 -> 0.00 mm, vias 11 -> 0
- net +5V: track 24.6 -> 12.0 mm, vias 13 -> 9
- net HV_{SENSE}: track 52.0 -> 56.8 mm
- net /INT_{IO-expander}: track 44.6 -> 48.6 mm
- net /~{RESET}_{IO-expander}: track 49.2 -> 53.2 mm
- net SENSE_{PRECISE}: track 136.1 -> 132.7 mm
- net /LSD ADC/V_{SHUNT}: track 119.8 -> 116.6 mm
- net HV_{MEASURE}: track 140.5 -> 137.6 mm, vias 5 -> 3
- net CLOCK_{HV}: track 239.4 -> 242.3 mm, vias 3 -> 2
- net LSD_{ADC_~{WR}/RDY}: track 91.0 -> 93.8 mm
- net GND: track 110.0 -> 112.2 mm, vias 29 -> 27
- net LSD_{ADC_~{INT}}: track 83.0 -> 85.2 mm
- net LSD_{ADC_~{RD}}: track 82.9 -> 84.7 mm
- net VPP: track 196.1 -> 194.5 mm
- net LSD_{ADC_MODE}: track 77.9 -> 79.3 mm
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Other:
- board text added: "GPS"
- board text added: "SRAM"
