File: KiCad/nixieAccurateClock/gps.kicad_sch (KiCad schematic)
At the start: 4 parts

Commit message: WIP two stage HV supply
Other:
- title: GPS -> Nixie Accurate Clock
Changed lines of the file:
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@@
   (paper "A4")
   (title_block
-    (title "GPS")
+    (title "Nixie Accurate Clock")
+    (rev "A")
   )
   (junction (at 72.39 110.49) (diameter 0) (color 0 0 0 0)
@@
         )
         (path "/55aab698-7558-4fe2-95ad-faa6da60ef89/9610945c-9df3-4d66-a574-d19433fdc707"
-          (reference "C2") (unit 1)
+          (reference "C1") (unit 1)
         )
       )
@@
         )
         (path "/55aab698-7558-4fe2-95ad-faa6da60ef89/9610945c-9df3-4d66-a574-d19433fdc707"
-          (reference "#PWR020") (unit 1)
+          (reference "#PWR016") (unit 1)
         )
       )
@@
         )
         (path "/55aab698-7558-4fe2-95ad-faa6da60ef89/9610945c-9df3-4d66-a574-d19433fdc707"
-          (reference "#PWR023") (unit 1)
+          (reference "#PWR011") (unit 1)
         )
       )
@@
         )
         (path "/55aab698-7558-4fe2-95ad-faa6da60ef89/9610945c-9df3-4d66-a574-d19433fdc707"
-          (reference "#PWR021") (unit 1)
+          (reference "#PWR017") (unit 1)
         )
       )
@@
         )
         (path "/55aab698-7558-4fe2-95ad-faa6da60ef89/9610945c-9df3-4d66-a574-d19433fdc707"
-          (reference "#PWR018") (unit 1)
+          (reference "#PWR013") (unit 1)
         )
       )
@@
         )
         (path "/55aab698-7558-4fe2-95ad-faa6da60ef89/9610945c-9df3-4d66-a574-d19433fdc707"
-          (reference "#PWR024") (unit 1)
+          (reference "#PWR012") (unit 1)
         )
       )
@@
         )
         (path "/55aab698-7558-4fe2-95ad-faa6da60ef89/9610945c-9df3-4d66-a574-d19433fdc707"
-          (reference "#PWR019") (unit 1)
+          (reference "#PWR015") (unit 1)
         )
       )
@@
         )
         (path "/55aab698-7558-4fe2-95ad-faa6da60ef89/9610945c-9df3-4d66-a574-d19433fdc707"
-          (reference "#PWR022") (unit 1)
-        )
-      )
+          (reference "#PWR014") (unit 1)
+        )
+      )

Commit message: simulate HV supply concept
LM5156 simulation is infeasible

LTSpice model demonstrating that a two stage buck from 5 to 210 is possible.  Both stages run away, but the LM5156 should provide feedback to keep it on target.
Parts:
- gave numbers to parts that had none: 4
Changed lines of the file:
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@@
   (symbol (lib_id "Device:C_Small") (at 96.52 119.38 0) (mirror y) (unit 1)
     (in_bom yes) (on_board yes) (dnp no)
-    (property "Reference" "C?" (at 99.06 118.1163 0)
+    (property "Reference" "C1" (at 99.06 118.1163 0)
       (effects (font (size 1.27 1.27)) (justify right))
     )
@@
       (effects (font (size 1.27 1.27)) hide)
     )
+    (property "Sim.Enable" "0" (at 96.52 119.38 0)
+      (effects (font (size 1.27 1.27)) hide)
+    )
     (pin "2")
     (pin "1")
     (instances
       (project "nixieAccurateClock"
-        (path "/55aab698-7558-4fe2-95ad-faa6da60ef89/919829db-9d44-4db4-a8a4-73523a1d66d3"
-          (reference "C?") (unit 1)
-        )
         (path "/55aab698-7558-4fe2-95ad-faa6da60ef89/9610945c-9df3-4d66-a574-d19433fdc707"
           (reference "C1") (unit 1)
@@
   (symbol (lib_id "power:GND") (at 160.02 92.71 90) (mirror x) (unit 1)
     (in_bom yes) (on_board yes) (dnp no)
-    (property "Reference" "#PWR?" (at 166.37 92.71 0)
+    (property "Reference" "#PWR016" (at 166.37 92.71 0)
       (effects (font (size 1.27 1.27)) hide)
     )
@@
     (instances
       (project "nixieAccurateClock"
-        (path "/55aab698-7558-4fe2-95ad-faa6da60ef89"
-          (reference "#PWR?") (unit 1)
-        )
         (path "/55aab698-7558-4fe2-95ad-faa6da60ef89/9610945c-9df3-4d66-a574-d19433fdc707"
           (reference "#PWR016") (unit 1)
@@
   (symbol (lib_id "power:GND") (at 72.39 125.73 0) (mirror y) (unit 1)
     (in_bom yes) (on_board yes) (dnp no)
-    (property "Reference" "#PWR?" (at 72.39 132.08 0)
+    (property "Reference" "#PWR011" (at 72.39 132.08 0)
       (effects (font (size 1.27 1.27)) hide)
     )
@@
     (instances
       (project "nixieAccurateClock"
-        (path "/55aab698-7558-4fe2-95ad-faa6da60ef89"
-          (reference "#PWR?") (unit 1)
-        )
         (path "/55aab698-7558-4fe2-95ad-faa6da60ef89/9610945c-9df3-4d66-a574-d19433fdc707"
           (reference "#PWR011") (unit 1)
@@
   (symbol (lib_id "power:GND") (at 184.15 99.06 0) (mirror y) (unit 1)
     (in_bom yes) (on_board yes) (dnp no)
-    (property "Reference" "#PWR?" (at 184.15 105.41 0)
+    (property "Reference" "#PWR017" (at 184.15 105.41 0)
       (effects (font (size 1.27 1.27)) hide)
     )
@@
     (instances
       (project "nixieAccurateClock"
-        (path "/55aab698-7558-4fe2-95ad-faa6da60ef89"
-          (reference "#PWR?") (unit 1)
-        )
         (path "/55aab698-7558-4fe2-95ad-faa6da60ef89/9610945c-9df3-4d66-a574-d19433fdc707"
           (reference "#PWR017") (unit 1)
@@
   (symbol (lib_id "power:GND") (at 106.68 82.55 180) (unit 1)
     (in_bom yes) (on_board yes) (dnp no)
-    (property "Reference" "#PWR?" (at 106.68 76.2 0)
+    (property "Reference" "#PWR013" (at 106.68 76.2 0)
       (effects (font (size 1.27 1.27)) hide)
     )
@@
     (instances
       (project "nixieAccurateClock"
-        (path "/55aab698-7558-4fe2-95ad-faa6da60ef89"
-          (reference "#PWR?") (unit 1)
-        )
         (path "/55aab698-7558-4fe2-95ad-faa6da60ef89/9610945c-9df3-4d66-a574-d19433fdc707"
           (reference "#PWR013") (unit 1)
@@
   (symbol (lib_id "power:+3.3V") (at 96.52 128.27 180) (unit 1)
     (in_bom yes) (on_board yes) (dnp no) (fields_autoplaced)
-    (property "Reference" "#PWR?" (at 96.52 124.46 0)
+    (property "Reference" "#PWR012" (at 96.52 124.46 0)
       (effects (font (size 1.27 1.27)) hide)
     )
@@
     (instances
       (project "nixieAccurateClock"
-        (path "/55aab698-7558-4fe2-95ad-faa6da60ef89"
-          (reference "#PWR?") (unit 1)
-        )
         (path "/55aab698-7558-4fe2-95ad-faa6da60ef89/9610945c-9df3-4d66-a574-d19433fdc707"
           (reference "#PWR012") (unit 1)
@@
   (symbol (lib_id "Device:Battery_Cell") (at 72.39 118.11 0) (unit 1)
     (in_bom yes) (on_board yes) (dnp no) (fields_autoplaced)
-    (property "Reference" "BT?" (at 76.2 114.9985 0)
+    (property "Reference" "BT1" (at 76.2 114.9985 0)
       (effects (font (size 1.27 1.27)) (justify left))
     )
@@
       (effects (font (size 1.27 1.27)) hide)
     )
+    (property "Sim.Enable" "0" (at 72.39 118.11 0)
+      (effects (font (size 1.27 1.27)) hide)
+    )
     (pin "1")
     (pin "2")
     (instances
       (project "nixieAccurateClock"
-        (path "/55aab698-7558-4fe2-95ad-faa6da60ef89"
-          (reference "BT?") (unit 1)
-        )
         (path "/55aab698-7558-4fe2-95ad-faa6da60ef89/9610945c-9df3-4d66-a574-d19433fdc707"
           (reference "BT1") (unit 1)
@@
   (symbol (lib_id "power:GND") (at 156.21 82.55 0) (mirror x) (unit 1)
     (in_bom yes) (on_board yes) (dnp no)
-    (property "Reference" "#PWR?" (at 156.21 76.2 0)
+    (property "Reference" "#PWR015" (at 156.21 76.2 0)
       (effects (font (size 1.27 1.27)) hide)
     )
@@
     (instances
       (project "nixieAccurateClock"
-        (path "/55aab698-7558-4fe2-95ad-faa6da60ef89"
-          (reference "#PWR?") (unit 1)
-        )
         (path "/55aab698-7558-4fe2-95ad-faa6da60ef89/9610945c-9df3-4d66-a574-d19433fdc707"
           (reference "#PWR015") (unit 1)
@@
   (symbol (lib_id "00_lib:PX1125T") (at 109.22 87.63 0) (unit 1)
     (in_bom yes) (on_board yes) (dnp no) (fields_autoplaced)
-    (property "Reference" "U?" (at 132.08 80.01 0)
+    (property "Reference" "U2" (at 132.08 80.01 0)
       (effects (font (size 1.27 1.27)))
     )
@@
     (instances
       (project "nixieAccurateClock"
-        (path "/55aab698-7558-4fe2-95ad-faa6da60ef89"
-          (reference "U?") (unit 1)
-        )
         (path "/55aab698-7558-4fe2-95ad-faa6da60ef89/9610945c-9df3-4d66-a574-d19433fdc707"
           (reference "U2") (unit 1)
@@
   (symbol (lib_id "power:GND") (at 106.68 120.65 0) (mirror y) (unit 1)
     (in_bom yes) (on_board yes) (dnp no)
-    (property "Reference" "#PWR?" (at 106.68 127 0)
+    (property "Reference" "#PWR014" (at 106.68 127 0)
       (effects (font (size 1.27 1.27)) hide)
     )
@@
     (instances
       (project "nixieAccurateClock"
-        (path "/55aab698-7558-4fe2-95ad-faa6da60ef89"
-          (reference "#PWR?") (unit 1)
-        )
         (path "/55aab698-7558-4fe2-95ad-faa6da60ef89/9610945c-9df3-4d66-a574-d19433fdc707"
           (reference "#PWR014") (unit 1)
@@
   (symbol (lib_id "Connector:Conn_Coaxial") (at 184.15 90.17 0) (unit 1)
     (in_bom yes) (on_board yes) (dnp no) (fields_autoplaced)
-    (property "Reference" "J?" (at 187.96 89.1932 0)
+    (property "Reference" "J4" (at 187.96 89.1932 0)
       (effects (font (size 1.27 1.27)) (justify left))
     )
@@
       (effects (font (size 1.27 1.27)) hide)
     )
+    (property "Sim.Enable" "0" (at 184.15 90.17 0)
+      (effects (font (size 1.27 1.27)) hide)
+    )
     (pin "1")
     (pin "2")
     (instances
       (project "nixieAccurateClock"
-        (path "/55aab698-7558-4fe2-95ad-faa6da60ef89"
-          (reference "J?") (unit 1)
-        )
         (path "/55aab698-7558-4fe2-95ad-faa6da60ef89/9610945c-9df3-4d66-a574-d19433fdc707"
           (reference "J4") (unit 1)

Commit message: finish schematic features
Parts:
- added J7: Conn_01x02_Pin, Connector_PinHeader_2.54mm:PinHeader_1x02_P2.54mm_Vertical, symbol Connector:Conn_01x02_Pin
- renumbered J4 to J6
Connections:
- net +3V3_STDBY: now also J7.2 (Pin_2); no longer BT1.1 (+)
- new net 3.3V_STDBY_{SENSE}: BT1.1 (+), J7.1 (Pin_1)
Other:
- company: (none) -> Paul Willis
- moved on the sheet: BT1

Commit message: ERC pass
Close look at pico iCE pinout
Add light sensor
Rough layout for non-HV
Parts:
- renumbered C1 to C3, U2 to U4
Changed lines of the file:
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@@
   (symbol (lib_id "Device:C_Small") (at 96.52 119.38 0) (mirror y) (unit 1)
     (in_bom yes) (on_board yes) (dnp no)
-    (property "Reference" "C1" (at 99.06 118.1163 0)
+    (property "Reference" "C3" (at 99.06 118.1163 0)
       (effects (font (size 1.27 1.27)) (justify right))
     )
@@
       (project "nixieAccurateClock"
         (path "/55aab698-7558-4fe2-95ad-faa6da60ef89/9610945c-9df3-4d66-a574-d19433fdc707"
-          (reference "C1") (unit 1)
+          (reference "C3") (unit 1)
         )
       )
@@
   (symbol (lib_id "power:GND") (at 160.02 92.71 90) (mirror x) (unit 1)
     (in_bom yes) (on_board yes) (dnp no)
-    (property "Reference" "#PWR013" (at 166.37 92.71 0)
+    (property "Reference" "#PWR021" (at 166.37 92.71 0)
       (effects (font (size 1.27 1.27)) hide)
     )
@@
       (project "nixieAccurateClock"
         (path "/55aab698-7558-4fe2-95ad-faa6da60ef89/9610945c-9df3-4d66-a574-d19433fdc707"
-          (reference "#PWR013") (unit 1)
+          (reference "#PWR021") (unit 1)
         )
       )
@@
   (symbol (lib_id "power:GND") (at 72.39 135.89 0) (mirror y) (unit 1)
     (in_bom yes) (on_board yes) (dnp no)
-    (property "Reference" "#PWR017" (at 72.39 142.24 0)
+    (property "Reference" "#PWR025" (at 72.39 142.24 0)
       (effects (font (size 1.27 1.27)) hide)
     )
@@
       (project "nixieAccurateClock"
         (path "/55aab698-7558-4fe2-95ad-faa6da60ef89/9610945c-9df3-4d66-a574-d19433fdc707"
-          (reference "#PWR017") (unit 1)
+          (reference "#PWR025") (unit 1)
         )
       )
@@
   (symbol (lib_id "power:GND") (at 184.15 99.06 0) (mirror y) (unit 1)
     (in_bom yes) (on_board yes) (dnp no)
-    (property "Reference" "#PWR014" (at 184.15 105.41 0)
+    (property "Reference" "#PWR022" (at 184.15 105.41 0)
       (effects (font (size 1.27 1.27)) hide)
     )
@@
       (project "nixieAccurateClock"
         (path "/55aab698-7558-4fe2-95ad-faa6da60ef89/9610945c-9df3-4d66-a574-d19433fdc707"
-          (reference "#PWR014") (unit 1)
+          (reference "#PWR022") (unit 1)
         )
       )
@@
   (symbol (lib_id "power:GND") (at 106.68 82.55 180) (unit 1)
     (in_bom yes) (on_board yes) (dnp no)
-    (property "Reference" "#PWR011" (at 106.68 76.2 0)
+    (property "Reference" "#PWR019" (at 106.68 76.2 0)
       (effects (font (size 1.27 1.27)) hide)
     )
@@
       (project "nixieAccurateClock"
         (path "/55aab698-7558-4fe2-95ad-faa6da60ef89/9610945c-9df3-4d66-a574-d19433fdc707"
-          (reference "#PWR011") (unit 1)
+          (reference "#PWR019") (unit 1)
         )
       )
@@
   (symbol (lib_id "power:+3.3V") (at 96.52 128.27 180) (unit 1)
     (in_bom yes) (on_board yes) (dnp no) (fields_autoplaced)
-    (property "Reference" "#PWR016" (at 96.52 124.46 0)
+    (property "Reference" "#PWR024" (at 96.52 124.46 0)
       (effects (font (size 1.27 1.27)) hide)
     )
@@
       (project "nixieAccurateClock"
         (path "/55aab698-7558-4fe2-95ad-faa6da60ef89/9610945c-9df3-4d66-a574-d19433fdc707"
-          (reference "#PWR016") (unit 1)
+          (reference "#PWR024") (unit 1)
         )
       )
@@
   (symbol (lib_id "power:GND") (at 156.21 82.55 0) (mirror x) (unit 1)
     (in_bom yes) (on_board yes) (dnp no)
-    (property "Reference" "#PWR012" (at 156.21 76.2 0)
+    (property "Reference" "#PWR020" (at 156.21 76.2 0)
       (effects (font (size 1.27 1.27)) hide)
     )
@@
       (project "nixieAccurateClock"
         (path "/55aab698-7558-4fe2-95ad-faa6da60ef89/9610945c-9df3-4d66-a574-d19433fdc707"
-          (reference "#PWR012") (unit 1)
+          (reference "#PWR020") (unit 1)
         )
       )
@@
   (symbol (lib_id "00_lib:PX1125T") (at 109.22 87.63 0) (unit 1)
     (in_bom yes) (on_board yes) (dnp no) (fields_autoplaced)
-    (property "Reference" "U2" (at 132.08 80.01 0)
+    (property "Reference" "U4" (at 132.08 80.01 0)
       (effects (font (size 1.27 1.27)))
     )
@@
       (project "nixieAccurateClock"
         (path "/55aab698-7558-4fe2-95ad-faa6da60ef89/9610945c-9df3-4d66-a574-d19433fdc707"
-          (reference "U2") (unit 1)
+          (reference "U4") (unit 1)
         )
       )
@@
   (symbol (lib_id "power:GND") (at 106.68 120.65 0) (mirror y) (unit 1)
     (in_bom yes) (on_board yes) (dnp no)
-    (property "Reference" "#PWR015" (at 106.68 127 0)
+    (property "Reference" "#PWR023" (at 106.68 127 0)
       (effects (font (size 1.27 1.27)) hide)
     )
@@
       (project "nixieAccurateClock"
         (path "/55aab698-7558-4fe2-95ad-faa6da60ef89/9610945c-9df3-4d66-a574-d19433fdc707"
-          (reference "#PWR015") (unit 1)
-        )
-      )
+          (reference "#PWR023") (unit 1)
+        )
+      )
