File: KiCad/nixieAccurateClock/gps.kicad_sch (KiCad schematic)
At the start: 5 parts, among them J6 Conn_Coaxial, J7 Conn_01x02_Pin, U4 PX1125T

Commit message: Fill out BOM
Parts:
- BT1: Model (none) -> 103; Price (none) -> 1.50
- C3: Model (none) -> CL10B104KB8NNWC; Price (none) -> 0.10
- J5: renamed from J6; Model (none) -> 132289; Price (none) -> 7.55
- J6: renamed from J7; Model (none) -> PH1-02-UA; Price (none) -> 0.10
- U4: Height 2.6 -> (none); Manufacturer_Name SkyTraq -> (none); Manufacturer_Part_Number PX1125T -> (none); Price (none) -> 27.80
Changed lines of the file:
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@@
       (effects (font (size 1.27 1.27)) hide)
     )
-    (property "Datasheet" "~" (at 96.52 119.38 0)
-      (effects (font (size 1.27 1.27)) hide)
-    )
-    (property "Sim.Enable" "0" (at 96.52 119.38 0)
+    (property "Datasheet" "https://mm.digikey.com/Volume0/opasdata/d220001/medias/docus/658/CL10B104KB8NNWC_Spec.pdf" (at 96.52 119.38 0)
+      (effects (font (size 1.27 1.27)) hide)
+    )
+    (property "Sim.Enable" "" (at 96.52 119.38 0)
+      (effects (font (size 1.27 1.27)) hide)
+    )
+    (property "Model" "CL10B104KB8NNWC" (at 96.52 119.38 0)
+      (effects (font (size 1.27 1.27)) hide)
+    )
+    (property "Price" "0.10" (at 96.52 119.38 0)
       (effects (font (size 1.27 1.27)) hide)
     )
@@
   (symbol (lib_id "power:GND") (at 160.02 92.71 90) (mirror x) (unit 1)
     (in_bom yes) (on_board yes) (dnp no)
-    (property "Reference" "#PWR021" (at 166.37 92.71 0)
+    (property "Reference" "#PWR020" (at 166.37 92.71 0)
       (effects (font (size 1.27 1.27)) hide)
     )
@@
       (project "nixieAccurateClock"
         (path "/55aab698-7558-4fe2-95ad-faa6da60ef89/9610945c-9df3-4d66-a574-d19433fdc707"
-          (reference "#PWR021") (unit 1)
+          (reference "#PWR020") (unit 1)
         )
       )
@@
   (symbol (lib_id "Connector:Conn_01x02_Pin") (at 62.23 116.84 0) (mirror x) (unit 1)
     (in_bom yes) (on_board yes) (dnp no)
-    (property "Reference" "J7" (at 64.77 118.11 0)
+    (property "Reference" "J6" (at 64.77 118.11 0)
       (effects (font (size 1.27 1.27)) (justify right))
     )
@@
       (effects (font (size 1.27 1.27)) hide)
     )
-    (property "Datasheet" "~" (at 62.23 116.84 0)
+    (property "Datasheet" "https://app.adam-tech.com/products/download/data_sheet/201605/ph1-xx-ua-data-sheet.pdf" (at 62.23 116.84 0)
       (effects (font (size 1.27 1.27)) hide)
     )
@@
       (effects (font (size 1.27 1.27)) hide)
     )
-    (pin "1")
-    (pin "2")
-    (instances
-      (project "nixieAccurateClock"
-        (path "/55aab698-7558-4fe2-95ad-faa6da60ef89/9610945c-9df3-4d66-a574-d19433fdc707"
-          (reference "J7") (unit 1)
+    (property "Model" "PH1-02-UA" (at 62.23 116.84 0)
+      (effects (font (size 1.27 1.27)) hide)
+    )
+    (property "Price" "0.10" (at 62.23 116.84 0)
+      (effects (font (size 1.27 1.27)) hide)
+    )
+    (pin "1")
+    (pin "2")
+    (instances
+      (project "nixieAccurateClock"
+        (path "/55aab698-7558-4fe2-95ad-faa6da60ef89/9610945c-9df3-4d66-a574-d19433fdc707"
+          (reference "J6") (unit 1)
         )
       )
@@
   (symbol (lib_id "power:GND") (at 72.39 135.89 0) (mirror y) (unit 1)
     (in_bom yes) (on_board yes) (dnp no)
-    (property "Reference" "#PWR025" (at 72.39 142.24 0)
+    (property "Reference" "#PWR024" (at 72.39 142.24 0)
       (effects (font (size 1.27 1.27)) hide)
     )
@@
       (project "nixieAccurateClock"
         (path "/55aab698-7558-4fe2-95ad-faa6da60ef89/9610945c-9df3-4d66-a574-d19433fdc707"
-          (reference "#PWR025") (unit 1)
+          (reference "#PWR024") (unit 1)
         )
       )
@@
   (symbol (lib_id "power:GND") (at 184.15 99.06 0) (mirror y) (unit 1)
     (in_bom yes) (on_board yes) (dnp no)
-    (property "Reference" "#PWR022" (at 184.15 105.41 0)
+    (property "Reference" "#PWR021" (at 184.15 105.41 0)
       (effects (font (size 1.27 1.27)) hide)
     )
@@
       (project "nixieAccurateClock"
         (path "/55aab698-7558-4fe2-95ad-faa6da60ef89/9610945c-9df3-4d66-a574-d19433fdc707"
-          (reference "#PWR022") (unit 1)
+          (reference "#PWR021") (unit 1)
         )
       )
@@
   (symbol (lib_id "power:GND") (at 106.68 82.55 180) (unit 1)
     (in_bom yes) (on_board yes) (dnp no)
-    (property "Reference" "#PWR019" (at 106.68 76.2 0)
+    (property "Reference" "#PWR018" (at 106.68 76.2 0)
       (effects (font (size 1.27 1.27)) hide)
     )
@@
       (project "nixieAccurateClock"
         (path "/55aab698-7558-4fe2-95ad-faa6da60ef89/9610945c-9df3-4d66-a574-d19433fdc707"
-          (reference "#PWR019") (unit 1)
+          (reference "#PWR018") (unit 1)
         )
       )
@@
   (symbol (lib_id "power:+3.3V") (at 96.52 128.27 180) (unit 1)
     (in_bom yes) (on_board yes) (dnp no) (fields_autoplaced)
-    (property "Reference" "#PWR024" (at 96.52 124.46 0)
+    (property "Reference" "#PWR023" (at 96.52 124.46 0)
       (effects (font (size 1.27 1.27)) hide)
     )
@@
       (project "nixieAccurateClock"
         (path "/55aab698-7558-4fe2-95ad-faa6da60ef89/9610945c-9df3-4d66-a574-d19433fdc707"
-          (reference "#PWR024") (unit 1)
+          (reference "#PWR023") (unit 1)
         )
       )
@@
       (effects (font (size 1.27 1.27)) hide)
     )
-    (property "Datasheet" "~" (at 72.39 126.746 90)
+    (property "Datasheet" "https://www.keyelco.com/userAssets/file/M65p3.pdf" (at 72.39 126.746 90)
       (effects (font (size 1.27 1.27)) hide)
     )
@@
       (effects (font (size 1.27 1.27)) hide)
     )
+    (property "Model" "103" (at 72.39 128.27 0)
+      (effects (font (size 1.27 1.27)) hide)
+    )
+    (property "Price" "1.50" (at 72.39 128.27 0)
+      (effects (font (size 1.27 1.27)) hide)
+    )
     (pin "1")
     (pin "2")
@@
   (symbol (lib_id "power:GND") (at 156.21 82.55 0) (mirror x) (unit 1)
     (in_bom yes) (on_board yes) (dnp no)
-    (property "Reference" "#PWR020" (at 156.21 76.2 0)
+    (property "Reference" "#PWR019" (at 156.21 76.2 0)
       (effects (font (size 1.27 1.27)) hide)
     )
@@
       (project "nixieAccurateClock"
         (path "/55aab698-7558-4fe2-95ad-faa6da60ef89/9610945c-9df3-4d66-a574-d19433fdc707"
-          (reference "#PWR020") (unit 1)
+          (reference "#PWR019") (unit 1)
         )
       )
@@
       (effects (font (size 1.27 1.27)) (justify left top) hide)
     )
-    (property "Height" "2.6" (at 151.13 482.55 0)
-      (effects (font (size 1.27 1.27)) (justify left top) hide)
-    )
-    (property "Mouser Part Number" "" (at 151.13 582.55 0)
-      (effects (font (size 1.27 1.27)) (justify left top) hide)
-    )
-    (property "Mouser Price/Stock" "" (at 151.13 682.55 0)
-      (effects (font (size 1.27 1.27)) (justify left top) hide)
-    )
-    (property "Manufacturer_Name" "SkyTraq" (at 151.13 782.55 0)
-      (effects (font (size 1.27 1.27)) (justify left top) hide)
-    )
-    (property "Manufacturer_Part_Number" "PX1125T" (at 151.13 882.55 0)
-      (effects (font (size 1.27 1.27)) (justify left top) hide)
-    )
     (property "Sim.Enable" "0" (at 109.22 87.63 0)
+      (effects (font (size 1.27 1.27)) hide)
+    )
+    (property "Price" "27.80" (at 109.22 87.63 0)
       (effects (font (size 1.27 1.27)) hide)
     )
@@
   (symbol (lib_id "power:GND") (at 106.68 120.65 0) (mirror y) (unit 1)
     (in_bom yes) (on_board yes) (dnp no)
-    (property "Reference" "#PWR023" (at 106.68 127 0)
+    (property "Reference" "#PWR022" (at 106.68 127 0)
       (effects (font (size 1.27 1.27)) hide)
     )
@@
       (project "nixieAccurateClock"
         (path "/55aab698-7558-4fe2-95ad-faa6da60ef89/9610945c-9df3-4d66-a574-d19433fdc707"
-          (reference "#PWR023") (unit 1)
+          (reference "#PWR022") (unit 1)
         )
       )
@@
   (symbol (lib_id "Connector:Conn_Coaxial") (at 184.15 90.17 0) (unit 1)
     (in_bom yes) (on_board yes) (dnp no) (fields_autoplaced)
-    (property "Reference" "J6" (at 187.96 89.1932 0)
+    (property "Reference" "J5" (at 187.96 89.1932 0)
       (effects (font (size 1.27 1.27)) (justify left))
     )
@@
       (effects (font (size 1.27 1.27)) hide)
     )
-    (property "Datasheet" " ~" (at 184.15 90.17 0)
+    (property "Datasheet" "https://www.mouser.com/datasheet/2/18/1/amphs06501_1-2259276.pdf" (at 184.15 90.17 0)
       (effects (font (size 1.27 1.27)) hide)
     )
@@
       (effects (font (size 1.27 1.27)) hide)
     )
-    (pin "1")
-    (pin "2")
-    (instances
-      (project "nixieAccurateClock"
-        (path "/55aab698-7558-4fe2-95ad-faa6da60ef89/9610945c-9df3-4d66-a574-d19433fdc707"
-          (reference "J6") (unit 1)
-        )
-      )
+    (property "Model" "132289" (at 184.15 90.17 0)
+      (effects (font (size 1.27 1.27)) hide)
+    )
+    (property "Price" "7.55" (at 184.15 90.17 0)
+      (effects (font (size 1.27 1.27)) hide)
+    )
+    (pin "1")
+    (pin "2")
+    (instances
+      (project "nixieAccurateClock"
+        (path "/55aab698-7558-4fe2-95ad-faa6da60ef89/9610945c-9df3-4d66-a574-d19433fdc707"
+          (reference "J5") (unit 1)
+        )
+      )

Commit message: Add retailer links
Parts:
- BT1: Digikey link (none) -> https://www.digikey.com/en/products/detail/103/36-103-ND/33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; Mouser link (none) -> https://www.mouser.com/ProductDetail/Keystone-Electronics/1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
- C3: Digikey link (none) -> https://www.digikey.com/en/products/detail/samsung-electro-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; Mouser link (none) -> https://www.mouser.com/ProductDetail/Samsung-Electro-Mechan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
- J5: Digikey link (none) -> https://www.digikey.com/en/products/detail/amphenol-rf/1322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; Mouser link (none) -> https://www.mouser.com/ProductDetail/Amphenol-RF/132289?qs=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
- J6: Digikey link (none) -> https://www.digikey.com/en/products/detail/adam-tech/PH1-02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; Mouser link (none) -> https://www.mouser.com/ProductDetail/Samtec/TSW-102-07-G-S?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
- U4: Digikey link (none) -> N/A; Mouser link (none) -> N/A
Changed lines of the file:
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@@
+      (effects (font (size 1.27 1.27)) hide)
+    )
+    (property "Digikey link" "https://www.digikey.com/en/products/detail/samsung-electro-mechanics/CL10A105KA8NNNC/3886760" (at 96.52 119.38 0)
+      (effects (font (size 1.27 1.27)) hide)
+    )
+    (property "Mouser link" "https://www.mouser.com/ProductDetail/Samsung-Electro-Mechanics/CL10A105KA8NNNC?qs=hqM3L16%252BxldY%252BnK4KzDJVg%3D%3D" (at 96.52 119.38 0)
       (effects (font (size 1.27 1.27)) hide)
     )
@@
     )
     (property "Price" "0.10" (at 62.23 116.84 0)
+      (effects (font (size 1.27 1.27)) hide)
+    )
+    (property "Digikey link" "https://www.digikey.com/en/products/detail/adam-tech/PH1-02-UA/9830266" (at 62.23 116.84 0)
+      (effects (font (size 1.27 1.27)) hide)
+    )
+    (property "Mouser link" "https://www.mouser.com/ProductDetail/Samtec/TSW-102-07-G-S?qs=iT52DjcXudsNPhlNCDp8vw%3D%3D" (at 62.23 116.84 0)
       (effects (font (size 1.27 1.27)) hide)
     )
@@
       (effects (font (size 1.27 1.27)) hide)
     )
+    (property "Digikey link" "https://www.digikey.com/en/products/detail/103/36-103-ND/331620" (at 72.39 128.27 0)
+      (effects (font (size 1.27 1.27)) hide)
+    )
+    (property "Mouser link" "https://www.mouser.com/ProductDetail/Keystone-Electronics/103?qs=Q3RoVmURDolsdXuDGYj49g%3D%3D" (at 72.39 128.27 0)
+      (effects (font (size 1.27 1.27)) hide)
+    )
     (pin "1")
     (pin "2")
@@
     )
     (property "Price" "27.80" (at 109.22 87.63 0)
+      (effects (font (size 1.27 1.27)) hide)
+    )
+    (property "Digikey link" "N/A" (at 109.22 87.63 0)
+      (effects (font (size 1.27 1.27)) hide)
+    )
+    (property "Mouser link" "N/A" (at 109.22 87.63 0)
       (effects (font (size 1.27 1.27)) hide)
     )
@@
       (effects (font (size 1.27 1.27)) hide)
     )
+    (property "Digikey link" "https://www.digikey.com/en/products/detail/amphenol-rf/132289/1989875" (at 184.15 90.17 0)
+      (effects (font (size 1.27 1.27)) hide)
+    )
+    (property "Mouser link" "https://www.mouser.com/ProductDetail/Amphenol-RF/132289?qs=nhkRCwpTkeb9ti20UXE5Cg%3D%3D" (at 184.15 90.17 0)
+      (effects (font (size 1.27 1.27)) hide)
+    )
