File: KiCad/nixieAccurateClock/hv_supply.kicad_sch (KiCad schematic)
At the start: 7 parts, among them Q1 PZTA42

Commit message: proper ERC and DRC pass
Parts:
- renumbered C1 to C?, D1 to D?, L1 to L?, Q1 to Q?, R2 to R?, R3 to R?, R1 to R?
Connections:
- net ADC3 renamed HV_SENSE
- net PICO_PMOD_B1 renamed HV_GATE
Other:
- title: (none) -> High voltage supply

Commit message: WIP nixies
Connections:
- net VPP: now reaches C?.1, D?.1 (K), R?.1
Changed lines of the file:
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@@
   (junction (at 175.26 93.98) (diameter 0) (color 0 0 0 0)
+  )
+  (junction (at 175.26 81.28) (diameter 0) (color 0 0 0 0)
+  )
+  (wire (pts (xy 175.26 78.74) (xy 175.26 81.28))
+    (stroke (width 0) (type default))
   )
   (wire (pts (xy 137.16 81.28) (xy 137.16 83.82))
@@
   (symbol (lib_id "power:GND") (at 175.26 105.41 0) (unit 1)
     (in_bom yes) (on_board yes) (dnp no) (fields_autoplaced)
-    (property "Reference" "#PWR013" (at 175.26 111.76 0)
+    (property "Reference" "#PWR014" (at 175.26 111.76 0)
       (effects (font (size 1.27 1.27)) hide)
     )
@@
       (project "nixieAccurateClock"
         (path "/55aab698-7558-4fe2-95ad-faa6da60ef89/f2852417-d6c8-4bbe-bd15-a29bc4083bd0"
-          (reference "#PWR013") (unit 1)
+          (reference "#PWR014") (unit 1)
         )
       )
@@
         )
       )
+    )
+  )
+  (symbol (lib_id "power:VPP") (at 175.26 78.74 0) (unit 1)
+    (in_bom yes) (on_board yes) (dnp no) (fields_autoplaced)
+    (property "Reference" "#PWR013" (at 175.26 82.55 0)
+      (effects (font (size 1.27 1.27)) hide)
+    )
+    (property "Value" "VPP" (at 175.26 73.66 0)
+      (effects (font (size 1.27 1.27)))
+    )
+    (property "Footprint" "" (at 175.26 78.74 0)
+      (effects (font (size 1.27 1.27)) hide)
+    )
+    (property "Datasheet" "" (at 175.26 78.74 0)
+      (effects (font (size 1.27 1.27)) hide)
+    )
+    (pin "1")
+    (instances
+      (project "nixieAccurateClock"
+        (path "/55aab698-7558-4fe2-95ad-faa6da60ef89/f2852417-d6c8-4bbe-bd15-a29bc4083bd0"
+          (reference "#PWR013") (unit 1)
+        )
+      )

Commit message: WIP final feature push
Connections:
- net HV_BOOST: now reaches D?.2 (A), L?.2, Q?.2 (C)
Changed lines of the file:
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@@
     (effects (font (size 1.27 1.27)) (justify left top))
+  )
+  (label "HV_BOOST" (at 133.35 81.28 0) (fields_autoplaced)
+    (effects (font (size 1.27 1.27)) (justify left bottom))
   )
   (global_label "HV_GATE" (shape input) (at 99.06 88.9 180) (fields_autoplaced)
@@
   (symbol (lib_id "power:GND") (at 137.16 97.79 0) (unit 1)
     (in_bom yes) (on_board yes) (dnp no)
-    (property "Reference" "#PWR011" (at 137.16 104.14 0)
+    (property "Reference" "#PWR014" (at 137.16 104.14 0)
       (effects (font (size 1.27 1.27)) hide)
     )
@@
       (project "nixieAccurateClock"
         (path "/55aab698-7558-4fe2-95ad-faa6da60ef89/f2852417-d6c8-4bbe-bd15-a29bc4083bd0"
-          (reference "#PWR011") (unit 1)
+          (reference "#PWR014") (unit 1)
         )
       )
@@
   (symbol (lib_id "power:GND") (at 175.26 105.41 0) (unit 1)
     (in_bom yes) (on_board yes) (dnp no) (fields_autoplaced)
-    (property "Reference" "#PWR014" (at 175.26 111.76 0)
+    (property "Reference" "#PWR017" (at 175.26 111.76 0)
       (effects (font (size 1.27 1.27)) hide)
     )
@@
       (project "nixieAccurateClock"
         (path "/55aab698-7558-4fe2-95ad-faa6da60ef89/f2852417-d6c8-4bbe-bd15-a29bc4083bd0"
-          (reference "#PWR014") (unit 1)
+          (reference "#PWR017") (unit 1)
         )
       )
@@
   (symbol (lib_id "power:GND") (at 156.21 99.06 0) (unit 1)
     (in_bom yes) (on_board yes) (dnp no)
-    (property "Reference" "#PWR012" (at 156.21 105.41 0)
+    (property "Reference" "#PWR015" (at 156.21 105.41 0)
       (effects (font (size 1.27 1.27)) hide)
     )
@@
       (project "nixieAccurateClock"
         (path "/55aab698-7558-4fe2-95ad-faa6da60ef89/f2852417-d6c8-4bbe-bd15-a29bc4083bd0"
-          (reference "#PWR012") (unit 1)
+          (reference "#PWR015") (unit 1)
         )
       )
@@
         )
         (path "/55aab698-7558-4fe2-95ad-faa6da60ef89/f2852417-d6c8-4bbe-bd15-a29bc4083bd0"
-          (reference "#PWR010") (unit 1)
+          (reference "#PWR013") (unit 1)
         )
       )
@@
         )
         (path "/55aab698-7558-4fe2-95ad-faa6da60ef89/f2852417-d6c8-4bbe-bd15-a29bc4083bd0"
-          (reference "R4") (unit 1)
+          (reference "R2") (unit 1)
         )
       )
@@
         )
         (path "/55aab698-7558-4fe2-95ad-faa6da60ef89/f2852417-d6c8-4bbe-bd15-a29bc4083bd0"
-          (reference "R5") (unit 1)
+          (reference "R3") (unit 1)
         )
       )
@@
         )
         (path "/55aab698-7558-4fe2-95ad-faa6da60ef89/f2852417-d6c8-4bbe-bd15-a29bc4083bd0"
-          (reference "R3") (unit 1)
+          (reference "R1") (unit 1)
         )
       )
@@
   (symbol (lib_id "power:VPP") (at 175.26 78.74 0) (unit 1)
     (in_bom yes) (on_board yes) (dnp no) (fields_autoplaced)
-    (property "Reference" "#PWR013" (at 175.26 82.55 0)
+    (property "Reference" "#PWR016" (at 175.26 82.55 0)
       (effects (font (size 1.27 1.27)) hide)
     )
@@
       (project "nixieAccurateClock"
         (path "/55aab698-7558-4fe2-95ad-faa6da60ef89/f2852417-d6c8-4bbe-bd15-a29bc4083bd0"
-          (reference "#PWR013") (unit 1)
-        )
-      )
+          (reference "#PWR016") (unit 1)
+        )
+      )

Commit message: Signal condition shunt signal
Textbook reference and LTSpice simulation for receipts.

I attempted a differential amplifier based solution but I failed to get it to work.  If it did work it would require more components and likely give little additional benefit.

ADC implementation WIP.
Parts:
- R?: value 2k -> 2.2k
Connections:
- net HV_BOOST renamed HV_{BOOST}
- net HV_GATE renamed HV_{GATE}
- net HV_SENSE renamed HV_{SENSE}
Other:
- moved on the sheet: L?, R?

Commit message: DRC pass except ADC
Parts:
- added R? (x2): 100k, Resistor_SMD:R_0603_1608Metric, symbol Device:R
Connections:
- net GND: now also R?.2
- net VPP: now also R?.1
- net HV_{BASE}: now reaches Q?.1 (B), R?.2
- new net HV_{BLEED-1}: R?.1, R?.2

Commit message: WIP HV supply simulation
Parts:
- L?: value 680u -> ${SIM.PARAMS}; Model (none) -> MSS1583-824
Changed lines of the file:
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@@
       (effects (font (size 1.27 1.27)) (justify left) hide)
+    )
+    (property "Sim.Library" "lib.pretty\\MPSA42.LIB" (at 134.62 88.9 0)
+      (effects (font (size 1.27 1.27)) hide)
+    )
+    (property "Sim.Name" "MPSA42" (at 134.62 88.9 0)
+      (effects (font (size 1.27 1.27)) hide)
+    )
+    (property "Sim.Device" "NPN" (at 134.62 88.9 0)
+      (effects (font (size 1.27 1.27)) hide)
+    )
+    (property "Sim.Type" "GUMMELPOON" (at 134.62 88.9 0)
+      (effects (font (size 1.27 1.27)) hide)
+    )
+    (property "Sim.Pins" "1=B 2=C 3=E" (at 134.62 88.9 0)
+      (effects (font (size 1.27 1.27)) hide)
     )
     (pin "3")
@@
       (effects (font (size 1.27 1.27)))
     )
-    (property "Value" "680u" (at 123.19 78.74 90)
+    (property "Value" "${SIM.PARAMS}" (at 123.19 78.74 90)
       (effects (font (size 1.27 1.27)))
     )
@@
       (effects (font (size 1.27 1.27)) hide)
     )
-    (property "Datasheet" "~" (at 123.19 81.28 0)
+    (property "Datasheet" "https://www.coilcraft.com/getmedia/fbfe8ea7-f5d8-4484-859e-2285f427326d/mss1583.pdf" (at 123.19 81.28 0)
+      (effects (font (size 1.27 1.27)) hide)
+    )
+    (property "Model" "MSS1583-824" (at 123.19 81.28 90)
+      (effects (font (size 1.27 1.27)) hide)
+    )
+    (property "Sim.Device" "L" (at 123.19 81.28 0)
+      (effects (font (size 1.27 1.27)) hide)
+    )
+    (property "Sim.Params" "l=820u" (at 123.19 81.28 0)
+      (effects (font (size 1.27 1.27)) hide)
+    )
+    (property "Sim.Pins" "1=+ 2=-" (at 123.19 81.28 0)
       (effects (font (size 1.27 1.27)) hide)
     )
@@
       (effects (font (size 1.27 1.27)) hide)
     )
+    (property "Sim.Library" "lib.pretty\\1N4004RL.LIB" (at 147.32 81.28 0)
+      (effects (font (size 1.27 1.27)) hide)
+    )
+    (property "Sim.Name" "D1n4004rl" (at 147.32 81.28 0)
+      (effects (font (size 1.27 1.27)) hide)
+    )
