File: KiCad/nixieAccurateClock/hv_supply.kicad_sch (KiCad schematic)
At the start: 9 parts

Commit message: fix sims
SPICE asy files had improper netlist orders for their models
FIxing this reveals that the LSD ADC circuit needed resistor tweaks, but now behaves much better (~70% of FS range for a 145 V nixie).
The HV supply still does not sim properly.  Will investigate a dedicated driver IC.
Parts:
- R?: value 2.2k -> 470
Changed lines of the file:
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@@
       (effects (font (size 1.27 1.27)))
     )
-    (property "Value" "2.2k" (at 105.41 85.09 90)
+    (property "Value" "470" (at 105.41 85.09 90)
       (effects (font (size 1.27 1.27)))
     )

Commit message: tie level shift OE to ground
OE on the TX0108 is internally tied high and should be softly pulled low for power-on sequencing.
Other:
- moved on the sheet: R?
Changed lines of the file:
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@@
   (junction (at 175.26 81.28) (diameter 0) (color 0 0 0 0)
   )
-  (junction (at 105.41 158.75) (diameter 0) (color 0 0 0 0)
+  (junction (at 210.82 138.43) (diameter 0) (color 0 0 0 0)
   )
   (wire (pts (xy 175.26 78.74) (xy 175.26 81.28))
@@
     (stroke (width 0) (type default))
   )
-  (wire (pts (xy 105.41 171.45) (xy 105.41 168.91))
-    (stroke (width 0) (type default))
-  )
-  (wire (pts (xy 105.41 158.75) (xy 105.41 156.21))
+  (wire (pts (xy 210.82 151.13) (xy 210.82 148.59))
+    (stroke (width 0) (type default))
+  )
+  (wire (pts (xy 210.82 138.43) (xy 210.82 135.89))
     (stroke (width 0) (type default))
   )
@@
     (stroke (width 0) (type default))
   )
-  (wire (pts (xy 105.41 161.29) (xy 105.41 158.75))
-    (stroke (width 0) (type default))
-  )
-  (wire (pts (xy 105.41 158.75) (xy 106.68 158.75))
+  (wire (pts (xy 210.82 140.97) (xy 210.82 138.43))
+    (stroke (width 0) (type default))
+  )
+  (wire (pts (xy 210.82 138.43) (xy 212.09 138.43))
     (stroke (width 0) (type default))
   )
@@
     (stroke (width 0) (type default))
   )
-  (wire (pts (xy 105.41 146.05) (xy 105.41 148.59))
+  (wire (pts (xy 210.82 125.73) (xy 210.82 128.27))
     (stroke (width 0) (type default))
   )
@@
   )
   (text_box "10 second bleed resistors that use > 220 mW total (> 1 mA)."
-    (at 118.11 156.21 0) (size 29.21 7.62)
+    (at 223.52 135.89 0) (size 29.21 7.62)
     (stroke (width 0) (type default))
     (fill (type none))
@@
     (effects (font (size 1.27 1.27)) (justify left top))
   )
-  (label "HV_{BLEED-1}" (at 106.68 158.75 0) (fields_autoplaced)
+  (label "HV_{BLEED-1}" (at 212.09 138.43 0) (fields_autoplaced)
     (effects (font (size 1.27 1.27)) (justify left bottom))
   )
@@
     )
   )
-  (symbol (lib_id "Device:R") (at 105.41 165.1 0) (unit 1)
-    (in_bom yes) (on_board yes) (dnp no) (fields_autoplaced)
-    (property "Reference" "R?" (at 107.95 163.83 0)
-      (effects (font (size 1.27 1.27)) (justify left))
-    )
-    (property "Value" "100k" (at 107.95 166.37 0)
-      (effects (font (size 1.27 1.27)) (justify left))
-    )
-    (property "Footprint" "Resistor_SMD:R_0603_1608Metric" (at 103.632 165.1 90)
-      (effects (font (size 1.27 1.27)) hide)
-    )
-    (property "Datasheet" "~" (at 105.41 165.1 0)
+  (symbol (lib_id "Device:R") (at 210.82 144.78 0) (unit 1)
+    (in_bom yes) (on_board yes) (dnp no) (fields_autoplaced)
+    (property "Reference" "R?" (at 213.36 143.51 0)
+      (effects (font (size 1.27 1.27)) (justify left))
+    )
+    (property "Value" "100k" (at 213.36 146.05 0)
+      (effects (font (size 1.27 1.27)) (justify left))
+    )
+    (property "Footprint" "Resistor_SMD:R_0603_1608Metric" (at 209.042 144.78 90)
+      (effects (font (size 1.27 1.27)) hide)
+    )
+    (property "Datasheet" "~" (at 210.82 144.78 0)
       (effects (font (size 1.27 1.27)) hide)
     )
@@
     )
   )
-  (symbol (lib_id "power:VPP") (at 105.41 146.05 0) (unit 1)
-    (in_bom yes) (on_board yes) (dnp no) (fields_autoplaced)
-    (property "Reference" "#PWR016" (at 105.41 149.86 0)
-      (effects (font (size 1.27 1.27)) hide)
-    )
-    (property "Value" "VPP" (at 105.41 140.97 0)
-      (effects (font (size 1.27 1.27)))
-    )
-    (property "Footprint" "" (at 105.41 146.05 0)
-      (effects (font (size 1.27 1.27)) hide)
-    )
-    (property "Datasheet" "" (at 105.41 146.05 0)
+  (symbol (lib_id "power:VPP") (at 210.82 125.73 0) (unit 1)
+    (in_bom yes) (on_board yes) (dnp no) (fields_autoplaced)
+    (property "Reference" "#PWR016" (at 210.82 129.54 0)
+      (effects (font (size 1.27 1.27)) hide)
+    )
+    (property "Value" "VPP" (at 210.82 120.65 0)
+      (effects (font (size 1.27 1.27)))
+    )
+    (property "Footprint" "" (at 210.82 125.73 0)
+      (effects (font (size 1.27 1.27)) hide)
+    )
+    (property "Datasheet" "" (at 210.82 125.73 0)
       (effects (font (size 1.27 1.27)) hide)
     )
@@
     )
   )
-  (symbol (lib_id "Device:R") (at 105.41 152.4 0) (unit 1)
-    (in_bom yes) (on_board yes) (dnp no) (fields_autoplaced)
-    (property "Reference" "R?" (at 107.95 151.13 0)
-      (effects (font (size 1.27 1.27)) (justify left))
-    )
-    (property "Value" "100k" (at 107.95 153.67 0)
-      (effects (font (size 1.27 1.27)) (justify left))
-    )
-    (property "Footprint" "Resistor_SMD:R_0603_1608Metric" (at 103.632 152.4 90)
-      (effects (font (size 1.27 1.27)) hide)
-    )
-    (property "Datasheet" "~" (at 105.41 152.4 0)
+  (symbol (lib_id "Device:R") (at 210.82 132.08 0) (unit 1)
+    (in_bom yes) (on_board yes) (dnp no) (fields_autoplaced)
+    (property "Reference" "R?" (at 213.36 130.81 0)
+      (effects (font (size 1.27 1.27)) (justify left))
+    )
+    (property "Value" "100k" (at 213.36 133.35 0)
+      (effects (font (size 1.27 1.27)) (justify left))
+    )
+    (property "Footprint" "Resistor_SMD:R_0603_1608Metric" (at 209.042 132.08 90)
+      (effects (font (size 1.27 1.27)) hide)
+    )
+    (property "Datasheet" "~" (at 210.82 132.08 0)
       (effects (font (size 1.27 1.27)) hide)
     )
@@
     )
   )
-  (symbol (lib_id "power:GND") (at 105.41 171.45 0) (unit 1)
-    (in_bom yes) (on_board yes) (dnp no) (fields_autoplaced)
-    (property "Reference" "#PWR017" (at 105.41 177.8 0)
-      (effects (font (size 1.27 1.27)) hide)
-    )
-    (property "Value" "GND" (at 105.41 176.53 0)
-      (effects (font (size 1.27 1.27)))
-    )
-    (property "Footprint" "" (at 105.41 171.45 0)
-      (effects (font (size 1.27 1.27)) hide)
-    )
-    (property "Datasheet" "" (at 105.41 171.45 0)
-      (effects (font (size 1.27 1.27)) hide)
-    )
+  (symbol (lib_id "power:GND") (at 210.82 151.13 0) (unit 1)
+    (in_bom yes) (on_board yes) (dnp no) (fields_autoplaced)
+    (property "Reference" "#PWR017" (at 210.82 157.48 0)
+      (effects (font (size 1.27 1.27)) hide)
+    )
+    (property "Value" "GND" (at 210.82 156.21 0)
+      (effects (font (size 1.27 1.27)))
+    )
+    (property "Footprint" "" (at 210.82 151.13 0)
+      (effects (font (size 1.27 1.27)) hide)
+    )
+    (property "Datasheet" "" (at 210.82 151.13 0)
+      (effects (font (size 1.27 1.27)) hide)
+    )

Commit message: WIP two stage HV supply
Parts:
- removed L?: ${SIM.PARAMS}, 00_lib:IND_MSS1583_COC, symbol Device:L
- removed R?: 100k, Resistor_SMD:R_0603_1608Metric, symbol Device:R
- removed R?: 470, Resistor_SMD:R_0603_1608Metric, symbol Device:R
- added L2: 820u, 00_lib:IND_BOURNS_SRR1210, symbol Device:L
- added R19: 62k, Resistor_SMD:R_0201_0603Metric, symbol Device:R
- added R9: 47k, Resistor_SMD:R_0201_0603Metric, symbol Device:R
- added R?: 4.7k, Resistor_SMD:R_0603_1608Metric, symbol Device:R
- C?: value 47u -> 10u; footprint Capacitor_THT:C_Radial_D12.5mm_H20.0mm_P5.00mm -> Capacitor_THT:CP_Radial_D10.0mm_P5.00mm; Model UCS2E470MHD1TO -> UVC2G100MPD1TD
- R?: value 100k -> 10M
Connections:
- net HV_{BLEED-1} is gone; now on net GND: R?.2
- net HV_{BOOST}: no longer D?.2 (A)
- net VPP: no longer C?.1, D?.1 (K)
Other:
- title: High voltage supply -> Nixie Accurate Clock
- moved on the sheet: C?, D?, Q?, R?

Commit message: simulate HV supply concept
LM5156 simulation is infeasible

LTSpice model demonstrating that a two stage buck from 5 to 210 is possible.  Both stages run away, but the LM5156 should provide feedback to keep it on target.
Parts:
- removed C?: 10u, Capacitor_THT:CP_Radial_D10.0mm_P5.00mm, symbol Device:C_Polarized
- removed D?: SM4004, Diode_SMD:D_MELF, symbol Diode:SM4004
- removed Q?: PZTA42, Package_TO_SOT_SMD:SOT-223-3_TabPin2, symbol Transistor_BJT:PZTA42
- removed R19: 62k, Resistor_SMD:R_0201_0603Metric, symbol Device:R
- added C10, C7, C8: 1u, Capacitor_SMD:C_0603_1608Metric, symbol Device:C
- added C11: 10u, Capacitor_THT:CP_Radial_D10.0mm_P5.00mm, symbol Device:C_Polarized
- added C9: 1n, Capacitor_SMD:C_0603_1608Metric, symbol Device:C
- added D2: SM4004, Diode_SMD:D_MELF, symbol Diode:SM4004
- added Q2: BSP88, Package_TO_SOT_SMD:SOT-223-3_TabPin2, symbol 00_lib:BSP88
- added R10, R17: 100k, Resistor_SMD:R_0603_1608Metric, symbol Device:R
- added R12: 220k, Resistor_SMD:R_0603_1608Metric, symbol Device:R
- added R13, R14: 1k, Resistor_SMD:R_0201_0603Metric, symbol Device:R
- added R15: 10k, Resistor_SMD:R_0603_1608Metric, symbol Device:R
- added R16: 40m, Resistor_SMD:R_0201_0603Metric, symbol Device:R
- added R18: 470, Resistor_SMD:R_0603_1608Metric, symbol Device:R
- added TP2: TestPoint, TestPoint:TestPoint_Loop_D2.54mm_Drill1.5mm_Beaded, symbol Connector:TestPoint
- added U4: LM51561HPWPR, 00_lib:PWP0014H-IPC_A, symbol 00_lib:LM51561HPWPR
- L2: footprint 00_lib:IND_BOURNS_SRR1210 -> 00_lib:IND_MSS1583_COC
- R9: value 47k -> 62k; Model RC0603FR-0747KL -> RMCF0603FT62K0
- gave numbers to parts that had none: 4
Connections:
- net GND: now also R11.2, C10.2, C11.2, C7.1, C8.2, C9.2, R12.1, R16.2, R18.1, U4.15 (EP), U4.5 (PGND), U4.6 (AGND), U4.9 (DITHOFF)
- net HV_{BOOST}: now also L2.2, D2.2 (A), Q2.2 (D)
- net VPP: now also C11.1, D2.1 (K), R17.2
- net at R9.1: now also R11.1, U4.14 (EN_UVLO_SYNC)
- net +20V: now reaches R9.2
- net +20V: now also L2.1, U4.1 (BIAS)
- new net: Q2.3 (S), R14.2, R16.1
- new net: C9.1, R15.1, U4.8 (COMP)
- new net: R12.2, U4.12 (RT)
- new net: R17.1, R18.2, U4.10 (FB)
- new net: C10.1, R15.2
- new net: R10.1, TP2.1, U4.13 (PGOOD)
- new net: C7.2, U4.11 (SS)
- new net: C8.1, U4.3 (VCC)
- new net: Q2.1 (G), U4.4 (GATE)
- new net: R13.1, U4.7 (CS)
- new net: R13.2, R14.1
- new net +5V: R10.2
Other:
- moved on the sheet: L2, R11, R20, R21

Commit message: HV bleed circuit
Parts:
- renumbered R11 to R10, R12 to R11, R9 to R12, R10 to R9

Commit message: Add HV control
Stop tracking SPICE simulations
Parts:
- added C18: 0.1u, Capacitor_SMD:C_0603_1608Metric, symbol Device:C_Small
- R18: value 470 -> 15k; Model (none) -> RC0603FR-071K5L
- R19: value 10M -> 2.7M; Model (none) -> RC0603JR-072M7L
Connections:
- net GND: now also C18.2; no longer R19.2
- net VPP: now also R19.2; no longer R17.2, R19.1
- net HV_{SOURCE}: now reaches Q2.3 (S), R14.2, R16.1
- net HV_{UVLO}: now reaches R10.1, R12.1, U4.14 (EN_UVLO_SYNC)
- net HV_{COMP}: now reaches C9.1, R15.1, U4.8 (COMP)
- net HV_{RT}: now reaches R11.2, U4.12 (RT)
- net HV_{FB}: now reaches R17.1, R18.2, U4.10 (FB)
- net HV_{FB}: now also R19.1, C18.1
- net HV_{COMP-1}: now reaches C10.1, R15.2
- net HV_{PGOOD}: now reaches R9.1, TP2.1, U4.13 (PGOOD)
- net HV_{SS}: now reaches C7.2, U4.11 (SS)
- net HV_{VCC}: now reaches C8.1, U4.3 (VCC)
- net HV_{GATE}: now reaches Q2.1 (G), U4.4 (GATE)
- net HV_{CS}: now reaches R13.1, U4.7 (CS)
- net HV_{CS-1}: now reaches R13.2, R14.1
- new net HV_{CONTROL}: R17.2
Other:
- moved on the sheet: C7, C8, R14

Commit message: finish schematic features
Parts:
- added J9: Conn_01x02_Pin, Connector_PinHeader_2.54mm:PinHeader_1x02_P2.54mm_Vertical, symbol Connector:Conn_01x02_Pin
- added TP10, TP11, TP13, TP14, TP15, TP8, TP9: TestPoint, TestPoint:TestPoint_Loop_D2.54mm_Drill1.5mm_Beaded, symbol Connector:TestPoint
- renumbered C9 to C10, C10 to C11, C18 to C12, C8 to C7, C11 to C8, C7 to C9, R20 to R10, R10 to R11, R13 to R12, R14 to R13, R21 to R14, R16 to R15, R9 to R16, R11 to R17, R19 to R18, R15 to R19, R17 to R20, R18 to R21, R12 to R9, TP2 to TP12
Connections:
- net +5V is gone; now on net HV_{VCC}: R16.2
- net GND: now also TP15.1
- net HV_{BOOST}: now also TP8.1
- net HV_{COMP}: now also TP14.1
- net HV_{FB}: now also TP13.1
- net HV_{GATE}: now also TP10.1
- net HV_{SENSE}: now also C8.1, D2.1 (K), R18.2, J9.1 (Pin_1); no longer R10.2, R14.1
- net HV_{UVLO}: now also TP9.1
- net VPP: now also J9.2 (Pin_2); no longer C8.1, D2.1 (K), R18.2
- new net HV_{MEASURE}: R10.2, R14.1, TP11.1
Other:
- company: (none) -> Paul Willis
- moved on the sheet: R10, R11, R14

Commit message: ERC pass
Close look at pico iCE pinout
Add light sensor
Rough layout for non-HV
Parts:
- U6: renamed from U4; footprint 00_lib:PWP0014H-IPC_A -> 00_lib:PWP0014H-IPC_C
- renumbered C8 to C10, C9 to C11, C10 to C12, C11 to C13, C12 to C14, C7 to C9, R9 to R11, R10 to R12, R11 to R13, R12 to R14, R13 to R15, R14 to R16, R15 to R17, R16 to R18, R17 to R19, R18 to R20, R19 to R21, R20 to R22, R21 to R23
