File: KiCad/nixieAccurateClock/hv_supply.kicad_sch (KiCad schematic)
At the start: 30 parts, among them J10 Conn_01x02_Pin, Q2 BSP88, U6 LM51561HPWPR

Commit message: clean up SMPS routing
Parts:
- removed TP11, TP9: TestPoint, 00_lib:TestPoint_Keystone_5019_Minature, symbol Connector:TestPoint
- renumbered TP13 to TP10, TP8 to TP7, TP10 to TP8, TP12 to TP9
Changed lines of the file:
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@@
   (junction (at 63.5 44.45) (diameter 0) (color 0 0 0 0)
   )
-  (junction (at 41.91 52.07) (diameter 0) (color 0 0 0 0)
-  )
   (junction (at 236.22 44.45) (diameter 0) (color 0 0 0 0)
   )
@@
   (junction (at 184.15 44.45) (diameter 0) (color 0 0 0 0)
   )
-  (junction (at 41.91 67.31) (diameter 0) (color 0 0 0 0)
-  )
   (junction (at 198.12 44.45) (diameter 0) (color 0 0 0 0)
   )
@@
     (stroke (width 0) (type default))
   )
-  (wire (pts (xy 34.29 52.07) (xy 41.91 52.07))
-    (stroke (width 0) (type default))
-  )
   (wire (pts (xy 198.12 99.06) (xy 198.12 101.6))
     (stroke (width 0) (type default))
@@
     (stroke (width 0) (type default))
   )
-  (wire (pts (xy 41.91 67.31) (xy 64.77 67.31))
+  (wire (pts (xy 38.1 67.31) (xy 64.77 67.31))
     (stroke (width 0) (type default))
   )
@@
     (stroke (width 0) (type default))
   )
-  (wire (pts (xy 41.91 52.07) (xy 63.5 52.07))
+  (wire (pts (xy 34.29 52.07) (xy 63.5 52.07))
     (stroke (width 0) (type default))
   )
@@
     (stroke (width 0) (type default))
   )
-  (wire (pts (xy 38.1 67.31) (xy 41.91 67.31))
-    (stroke (width 0) (type default))
-  )
   (wire (pts (xy 198.12 41.91) (xy 198.12 44.45))
     (stroke (width 0) (type default))
@@
     (stroke (width 0) (type default))
   )
-  (wire (pts (xy 41.91 64.77) (xy 41.91 67.31))
-    (stroke (width 0) (type default))
-  )
   (wire (pts (xy 138.43 59.69) (xy 160.02 59.69))
     (stroke (width 0) (type default))
@@
   )
   (wire (pts (xy 124.46 95.25) (xy 124.46 97.79))
-    (stroke (width 0) (type default))
-  )
-  (wire (pts (xy 41.91 50.8) (xy 41.91 52.07))
     (stroke (width 0) (type default))
   )
@@
   (symbol (lib_id "Connector:TestPoint") (at 124.46 66.04 0) (unit 1)
     (in_bom yes) (on_board yes) (dnp no) (fields_autoplaced)
-    (property "Reference" "TP12" (at 127 61.468 0)
+    (property "Reference" "TP9" (at 127 61.468 0)
       (effects (font (size 1.27 1.27)) (justify left))
     )
@@
       (project "nixieAccurateClock"
         (path "/55aab698-7558-4fe2-95ad-faa6da60ef89/f2852417-d6c8-4bbe-bd15-a29bc4083bd0"
-          (reference "TP12") (unit 1)
+          (reference "TP9") (unit 1)
         )
       )
@@
   (symbol (lib_id "Connector:TestPoint") (at 160.02 40.64 0) (unit 1)
     (in_bom yes) (on_board yes) (dnp no) (fields_autoplaced)
-    (property "Reference" "TP8" (at 162.56 36.068 0)
+    (property "Reference" "TP7" (at 162.56 36.068 0)
       (effects (font (size 1.27 1.27)) (justify left))
     )
@@
       (project "nixieAccurateClock"
         (path "/55aab698-7558-4fe2-95ad-faa6da60ef89/f2852417-d6c8-4bbe-bd15-a29bc4083bd0"
-          (reference "TP8") (unit 1)
+          (reference "TP7") (unit 1)
         )
       )
@@
     )
   )
-  (symbol (lib_id "Connector:TestPoint") (at 41.91 64.77 0) (unit 1)
-    (in_bom yes) (on_board yes) (dnp no) (fields_autoplaced)
-    (property "Reference" "TP11" (at 44.45 60.198 0)
-      (effects (font (size 1.27 1.27)) (justify left))
-    )
-    (property "Value" "TestPoint" (at 44.45 62.738 0)
-      (effects (font (size 1.27 1.27)) (justify left))
-    )
-    (property "Footprint" "00_lib:TestPoint_Keystone_5019_Minature" (at 46.99 64.77 0)
-      (effects (font (size 1.27 1.27)) hide)
-    )
-    (property "Datasheet" "https://www.mouser.com/datasheet/2/215/019-743690.pdf" (at 46.99 64.77 0)
-      (effects (font (size 1.27 1.27)) hide)
-    )
-    (property "Model" "5019" (at 41.91 64.77 0)
-      (effects (font (size 1.27 1.27)) hide)
-    )
-    (property "Sim.Enable" "0" (at 41.91 64.77 0)
-      (effects (font (size 1.27 1.27)) hide)
-    )
-    (property "Price" "0.33" (at 41.91 64.77 0)
-      (effects (font (size 1.27 1.27)) hide)
-    )
-    (property "Digikey link" "https://www.digikey.com/en/products/detail/keystone-electronics/5019/3907343" (at 41.91 64.77 0)
-      (effects (font (size 1.27 1.27)) hide)
-    )
-    (property "Mouser link" "https://www.mouser.com/ProductDetail/Keystone-Electronics/5019?qs=wOxb8XianXjjCAsb90Ilzw%3D%3D" (at 41.91 64.77 0)
-      (effects (font (size 1.27 1.27)) hide)
-    )
-    (pin "1")
-    (instances
-      (project "nixieAccurateClock"
-        (path "/55aab698-7558-4fe2-95ad-faa6da60ef89/f2852417-d6c8-4bbe-bd15-a29bc4083bd0"
-          (reference "TP11") (unit 1)
-        )
-      )
-    )
-  )
   (symbol (lib_id "Device:R") (at 236.22 50.8 0) (unit 1)
     (in_bom yes) (on_board yes) (dnp no) (fields_autoplaced)
@@
         (path "/55aab698-7558-4fe2-95ad-faa6da60ef89/f2852417-d6c8-4bbe-bd15-a29bc4083bd0"
           (reference "R12") (unit 1)
-        )
-      )
-    )
-  )
-  (symbol (lib_id "Connector:TestPoint") (at 41.91 50.8 0) (unit 1)
-    (in_bom yes) (on_board yes) (dnp no) (fields_autoplaced)
-    (property "Reference" "TP9" (at 44.45 46.228 0)
-      (effects (font (size 1.27 1.27)) (justify left))
-    )
-    (property "Value" "TestPoint" (at 44.45 48.768 0)
-      (effects (font (size 1.27 1.27)) (justify left))
-    )
-    (property "Footprint" "00_lib:TestPoint_Keystone_5019_Minature" (at 46.99 50.8 0)
-      (effects (font (size 1.27 1.27)) hide)
-    )
-    (property "Datasheet" "https://www.mouser.com/datasheet/2/215/019-743690.pdf" (at 46.99 50.8 0)
-      (effects (font (size 1.27 1.27)) hide)
-    )
-    (property "Model" "5019" (at 41.91 50.8 0)
-      (effects (font (size 1.27 1.27)) hide)
-    )
-    (property "Sim.Enable" "0" (at 41.91 50.8 0)
-      (effects (font (size 1.27 1.27)) hide)
-    )
-    (property "Price" "0.33" (at 41.91 50.8 0)
-      (effects (font (size 1.27 1.27)) hide)
-    )
-    (property "Digikey link" "https://www.digikey.com/en/products/detail/keystone-electronics/5019/3907343" (at 41.91 50.8 0)
-      (effects (font (size 1.27 1.27)) hide)
-    )
-    (property "Mouser link" "https://www.mouser.com/ProductDetail/Keystone-Electronics/5019?qs=wOxb8XianXjjCAsb90Ilzw%3D%3D" (at 41.91 50.8 0)
-      (effects (font (size 1.27 1.27)) hide)
-    )
-    (pin "1")
-    (instances
-      (project "nixieAccurateClock"
-        (path "/55aab698-7558-4fe2-95ad-faa6da60ef89/f2852417-d6c8-4bbe-bd15-a29bc4083bd0"
-          (reference "TP9") (unit 1)
         )
       )
@@
   (symbol (lib_id "Connector:TestPoint") (at 124.46 73.66 0) (unit 1)
     (in_bom yes) (on_board yes) (dnp no) (fields_autoplaced)
-    (property "Reference" "TP13" (at 127 69.088 0)
+    (property "Reference" "TP10" (at 127 69.088 0)
       (effects (font (size 1.27 1.27)) (justify left))
     )
@@
       (project "nixieAccurateClock"
         (path "/55aab698-7558-4fe2-95ad-faa6da60ef89/f2852417-d6c8-4bbe-bd15-a29bc4083bd0"
-          (reference "TP13") (unit 1)
+          (reference "TP10") (unit 1)
         )
       )
@@
   (symbol (lib_id "Connector:TestPoint") (at 124.46 50.8 0) (unit 1)
     (in_bom yes) (on_board yes) (dnp no) (fields_autoplaced)
-    (property "Reference" "TP10" (at 127 46.228 0)
+    (property "Reference" "TP8" (at 127 46.228 0)
       (effects (font (size 1.27 1.27)) (justify left))
     )
@@
       (project "nixieAccurateClock"
         (path "/55aab698-7558-4fe2-95ad-faa6da60ef89/f2852417-d6c8-4bbe-bd15-a29bc4083bd0"
-          (reference "TP10") (unit 1)
-        )
-      )
+          (reference "TP8") (unit 1)
+        )
+      )
