File: KiCad/nixieAccurateClock/nixies.kicad_sch (KiCad schematic)
At the start: 0 parts

Commit message: IN-14 daughter board
Parts:
- added U3, U4, U5, U6, U7, U8: ~, 00_lib:IN-14 daughter board, symbol 00_lib:IN-14_daughter_board
Connections:
- net HV_DATA: now also U3.2 (DIN)
- new net: U5.14 (DOUT), U6.2 (DIN)
- new net: U4.14 (DOUT), U5.2 (DIN)
- new net: U7.14 (DOUT), U8.2 (DIN)
- new net: U6.14 (DOUT), U7.2 (DIN)
- new net: U3.14 (DOUT), U4.2 (DIN)
- new net +3.3V: U3.6 (+3.3V), U4.6 (+3.3V), U5.6 (+3.3V), U6.6 (+3.3V), U7.6 (+3.3V), U8.6 (+3.3V)
- new net +5V: U3.22 (+5V), U4.22 (+5V), U5.22 (+5V), U6.22 (+5V), U7.22 (+5V), U8.22 (+5V)
- new net GND: U3.23 (GND), U4.23 (GND), U5.23 (GND), U6.23 (GND), U7.23 (GND), U8.23 (GND)
- new net HV_CLOCK: U3.4 (CLOCK), U4.4 (CLOCK), U5.4 (CLOCK), U6.4 (CLOCK), U7.4 (CLOCK), U8.4 (CLOCK)
- new net HV_POLARITY: U3.8 (~{POLARITY}), U4.8 (~{POLARITY}), U5.8 (~{POLARITY}), U6.8 (~{POLARITY}), U7.8 (~{POLARITY}), U8.8 (~{POLARITY})
- new net PPS_TRIMMED: U3.12 (~{LATCH}), U4.12 (~{LATCH}), U5.12 (~{LATCH}), U6.12 (~{LATCH}), U7.12 (~{LATCH}), U8.12 (~{LATCH})
- new net VPP: U3.1 (VPP), U4.1 (VPP), U5.1 (VPP), U6.1 (VPP), U7.1 (VPP), U8.1 (VPP)
Other:
- removed sheet Nixie1
- removed sheet Nixie2
- removed sheet Nixie3
- removed sheet Nixie4
- removed sheet Nixie5
- removed sheet Nixie6

Commit message: WIP final feature push
Parts:
- removed U3, U4, U5, U6, U7, U8: ~, 00_lib:IN-14 daughter board, symbol 00_lib:IN-14_daughter_board
- added U3, U4, U5, U6, U7, U8: ~, 00_lib:IN-14 daughter board, symbol 00_lib:nixie_daughter_board
Connections:
- net +3.3V: now also U3.6 (+3.3V), U4.6 (+3.3V), U5.6 (+3.3V), U6.6 (+3.3V), U7.6 (+3.3V), U8.6 (+3.3V)
- net +5V: now also U3.22 (+5V), U4.22 (+5V), U5.22 (+5V), U6.22 (+5V), U7.22 (+5V), U8.22 (+5V)
- net GND: now also U3.23 (GND), U4.23 (GND), U5.23 (GND), U6.23 (GND), U7.23 (GND), U8.23 (GND)
- net HV_CLOCK: now also U3.4 (CLOCK), U4.4 (CLOCK), U5.4 (CLOCK), U6.4 (CLOCK), U7.4 (CLOCK), U8.4 (CLOCK)
- net HV_DATA: now also U3.2 (DIN)
- net HV_POLARITY: now also U3.8 (~{POLARITY}), U4.8 (~{POLARITY}), U5.8 (~{POLARITY}), U6.8 (~{POLARITY}), U7.8 (~{POLARITY}), U8.8 (~{POLARITY})
- net PPS_TRIMMED: now also U3.12 (~{LATCH}), U4.12 (~{LATCH}), U5.12 (~{LATCH}), U6.12 (~{LATCH}), U7.12 (~{LATCH}), U8.12 (~{LATCH})
- net VPP: now also U3.1 (VPP), U4.1 (VPP), U5.1 (VPP), U6.1 (VPP), U7.1 (VPP), U8.1 (VPP)
- new net: U7.14 (DOUT), U8.2 (DIN)
- new net: U4.14 (DOUT), U5.2 (DIN)
- new net: U3.14 (DOUT), U4.2 (DIN)
- new net: U6.14 (DOUT), U7.2 (DIN)
- new net: U5.14 (DOUT), U6.2 (DIN)
- new net N_0: U8.19 (N_0)
- new net N_1: U8.10 (N_1)
- new net N_2: U8.3 (N_2)
- new net N_3: U8.5 (N_3)
- new net N_4: U8.7 (N_4)
- new net N_5: U8.9 (N_5)
- new net N_6: U8.11 (N_6)
- new net N_7: U8.13 (N_7)
- new net N_8: U8.15 (N_8)
- new net N_9: U8.17 (N_9)

Commit message: simplify nixie daughter board
Remove cathode pins that would not be usable for current sensing anyway.
Pivot to using anode pin as shunt measurement with a R2R flash ADC (not yet implemented).
Connections:
- net HV_POLARITY is gone; now on net HV_CLOCK: U3.8 (CLOCK), U4.8 (CLOCK), U5.8 (CLOCK), U6.8 (CLOCK), U7.8 (CLOCK), U8.8 (CLOCK)
- net N_1 is gone; now on net GND: U8.10 (GND)
- net N_2 is gone; now on net PPS_TRIMMED: U8.3 (~{LATCH})
- net N_3 is gone; now on net GND: U8.5 (GND)
- net N_5 is gone; now on net VPP: U8.9 (VPP)
- net +5V: now also U3.2 (+5V), U4.2 (+5V), U5.2 (+5V), U6.2 (+5V), U7.2 (+5V), U8.2 (+5V); no longer U3.22 (+5V), U4.22 (+5V), U5.22 (+5V), U6.22 (+5V), U7.22 (+5V), U8.22 (+5V)
- net GND: now also U3.10 (GND), U3.5 (GND), U4.10 (GND), U4.5 (GND), U5.10 (GND), U5.5 (GND), U6.10 (GND), U6.5 (GND), U7.10 (GND), U7.5 (GND); no longer U3.23 (GND), U4.23 (GND), U5.23 (GND), U6.23 (GND), U7.23 (GND), U8.23 (GND)
- net HV_CLOCK: no longer U3.4 (CLOCK), U4.4 (CLOCK), U5.4 (CLOCK), U6.4 (CLOCK), U7.4 (CLOCK), U8.4 (CLOCK)
- net HV_DATA: now also U3.4 (DIN); no longer U3.2 (DIN)
- net PPS_TRIMMED: now also U3.3 (~{LATCH}), U4.3 (~{LATCH}), U5.3 (~{LATCH}), U6.3 (~{LATCH}), U7.3 (~{LATCH}); no longer U3.12 (~{LATCH}), U4.12 (~{LATCH}), U5.12 (~{LATCH}), U6.12 (~{LATCH}), U7.12 (~{LATCH}), U8.12 (~{LATCH})
- net VPP: now also U3.9 (VPP), U4.9 (VPP), U5.9 (VPP), U6.9 (VPP), U7.9 (VPP); no longer U3.1 (VPP), U4.1 (VPP), U5.1 (VPP), U6.1 (VPP), U7.1 (VPP), U8.1 (VPP)
- removed net N_0: U8.19 (N_0)
- net N_4: no longer names the net of U8.7 (ANODE)
- removed net N_6: U8.11 (N_6)
- removed net N_7: U8.13 (N_7)
- removed net N_8: U8.15 (N_8)
- removed net N_9: U8.17 (N_9)
- new net HV_daisy_1: U3.1 (DOUT), U5.4 (DIN)
- new net HV_daisy_2: U5.1 (DOUT), U6.4 (DIN)
- new net HV_daisy_3: U6.1 (DOUT), U7.4 (DIN)
- new net HV_daisy_4: U7.1 (DOUT), U8.4 (DIN)
- new net HV_daisy_5: U4.4 (DIN), U8.1 (DOUT)

Commit message: Signal condition shunt signal
Textbook reference and LTSpice simulation for receipts.

I attempted a differential amplifier based solution but I failed to get it to work.  If it did work it would require more components and likely give little additional benefit.

ADC implementation WIP.
Parts:
- renumbered U7 to U4, U8 to U6, U6 to U7, U4 to U8
Connections:
- net HV_daisy_3: no longer U7.1 (DOUT)
- net LSD_{SHUNT}: now reaches U8.7 (ANODE)
- net HV_CLOCK renamed CLOCK_{HV}
- net HV_DATA renamed DATA_{HV}
- net HV_daisy_1 renamed DAISY_{HV-1}
- net HV_daisy_2 renamed DAISY_{HV-2}
- net HV_daisy_4 renamed DAISY_{HV-4}
- net HV_daisy_5 renamed DAISY_{HV-5}
- net PPS_TRIMMED renamed PPS_{TRIMMED}
- new net DAISY_{HV-3}: U7.1 (DOUT)

Commit message: DRC pass except ADC
Parts:
- renumbered U5 to U4, U7 to U5, U4 to U6, U6 to U7
Connections:
- net HV_daisy_3 is gone; now on net DAISY_{HV-3}: U6.4 (DIN)

Commit message: give pico iCE better mounting
Parts:
- renumbered U6 to U4, U4 to U5, U7 to U6, U5 to U7

Commit message: Add decoupling caps
Parts:
- renumbered U5 to U4, U7 to U5, U4 to U6, U6 to U7
Changed lines of the file:
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@@
   (symbol (lib_id "power:GND") (at 104.14 110.49 270) (unit 1)
     (in_bom yes) (on_board yes) (dnp no) (fields_autoplaced)
-    (property "Reference" "#PWR034" (at 97.79 110.49 0)
+    (property "Reference" "#PWR027" (at 97.79 110.49 0)
       (effects (font (size 1.27 1.27)) hide)
     )
@@
       (project "nixieAccurateClock"
         (path "/55aab698-7558-4fe2-95ad-faa6da60ef89/1d5016d9-fde4-4367-b1de-5d16dd08b171"
-          (reference "#PWR034") (unit 1)
+          (reference "#PWR027") (unit 1)
         )
       )
@@
   (symbol (lib_id "00_lib:nixie_daughter_board") (at 175.26 124.46 0) (unit 1)
     (in_bom yes) (on_board yes) (dnp no) (fields_autoplaced)
-    (property "Reference" "U7" (at 188.595 102.87 0)
+    (property "Reference" "U5" (at 188.595 102.87 0)
       (effects (font (size 1.27 1.27)))
     )
@@
       (project "nixieAccurateClock"
         (path "/55aab698-7558-4fe2-95ad-faa6da60ef89/1d5016d9-fde4-4367-b1de-5d16dd08b171"
-          (reference "U7") (unit 1)
+          (reference "U5") (unit 1)
         )
       )
@@
         )
         (path "/55aab698-7558-4fe2-95ad-faa6da60ef89/1d5016d9-fde4-4367-b1de-5d16dd08b171"
-          (reference "#PWR033") (unit 1)
+          (reference "#PWR046") (unit 1)
         )
       )
@@
         )
         (path "/55aab698-7558-4fe2-95ad-faa6da60ef89/1d5016d9-fde4-4367-b1de-5d16dd08b171"
-          (reference "#PWR044") (unit 1)
+          (reference "#PWR030") (unit 1)
         )
       )
@@
         )
         (path "/55aab698-7558-4fe2-95ad-faa6da60ef89/1d5016d9-fde4-4367-b1de-5d16dd08b171"
-          (reference "#PWR048") (unit 1)
+          (reference "#PWR045") (unit 1)
         )
       )
@@
   (symbol (lib_id "power:GND") (at 168.91 139.7 270) (unit 1)
     (in_bom yes) (on_board yes) (dnp no) (fields_autoplaced)
-    (property "Reference" "#PWR043" (at 162.56 139.7 0)
+    (property "Reference" "#PWR041" (at 162.56 139.7 0)
       (effects (font (size 1.27 1.27)) hide)
     )
@@
       (project "nixieAccurateClock"
         (path "/55aab698-7558-4fe2-95ad-faa6da60ef89/1d5016d9-fde4-4367-b1de-5d16dd08b171"
-          (reference "#PWR043") (unit 1)
+          (reference "#PWR041") (unit 1)
         )
       )
@@
   (symbol (lib_id "power:GND") (at 39.37 139.7 270) (unit 1)
     (in_bom yes) (on_board yes) (dnp no) (fields_autoplaced)
-    (property "Reference" "#PWR027" (at 33.02 139.7 0)
+    (property "Reference" "#PWR037" (at 33.02 139.7 0)
       (effects (font (size 1.27 1.27)) hide)
     )
@@
       (project "nixieAccurateClock"
         (path "/55aab698-7558-4fe2-95ad-faa6da60ef89/1d5016d9-fde4-4367-b1de-5d16dd08b171"
-          (reference "#PWR027") (unit 1)
+          (reference "#PWR037") (unit 1)
         )
       )
@@
         )
         (path "/55aab698-7558-4fe2-95ad-faa6da60ef89/1d5016d9-fde4-4367-b1de-5d16dd08b171"
-          (reference "#PWR049") (unit 1)
+          (reference "#PWR048") (unit 1)
         )
       )
@@
         )
         (path "/55aab698-7558-4fe2-95ad-faa6da60ef89/1d5016d9-fde4-4367-b1de-5d16dd08b171"
-          (reference "#PWR028") (unit 1)
+          (reference "#PWR026") (unit 1)
         )
       )
@@
   (symbol (lib_id "00_lib:nixie_daughter_board") (at 110.49 124.46 0) (unit 1)
     (in_bom yes) (on_board yes) (dnp no) (fields_autoplaced)
-    (property "Reference" "U5" (at 123.825 102.87 0)
+    (property "Reference" "U4" (at 123.825 102.87 0)
       (effects (font (size 1.27 1.27)))
     )
@@
       (project "nixieAccurateClock"
         (path "/55aab698-7558-4fe2-95ad-faa6da60ef89/1d5016d9-fde4-4367-b1de-5d16dd08b171"
-          (reference "U5") (unit 1)
+          (reference "U4") (unit 1)
         )
       )
@@
         )
         (path "/55aab698-7558-4fe2-95ad-faa6da60ef89/1d5016d9-fde4-4367-b1de-5d16dd08b171"
-          (reference "#PWR046") (unit 1)
+          (reference "#PWR036") (unit 1)
         )
       )
@@
         )
         (path "/55aab698-7558-4fe2-95ad-faa6da60ef89/1d5016d9-fde4-4367-b1de-5d16dd08b171"
-          (reference "#PWR041") (unit 1)
+          (reference "#PWR047") (unit 1)
         )
       )
@@
         )
         (path "/55aab698-7558-4fe2-95ad-faa6da60ef89/1d5016d9-fde4-4367-b1de-5d16dd08b171"
-          (reference "#PWR032") (unit 1)
+          (reference "#PWR043") (unit 1)
         )
       )
@@
         )
         (path "/55aab698-7558-4fe2-95ad-faa6da60ef89/1d5016d9-fde4-4367-b1de-5d16dd08b171"
-          (reference "#PWR047") (unit 1)
+          (reference "#PWR042") (unit 1)
         )
       )
@@
         )
         (path "/55aab698-7558-4fe2-95ad-faa6da60ef89/1d5016d9-fde4-4367-b1de-5d16dd08b171"
-          (reference "#PWR031") (unit 1)
+          (reference "#PWR038") (unit 1)
         )
       )
@@
         )
         (path "/55aab698-7558-4fe2-95ad-faa6da60ef89/1d5016d9-fde4-4367-b1de-5d16dd08b171"
-          (reference "#PWR039") (unit 1)
+          (reference "#PWR040") (unit 1)
         )
       )
@@
         )
         (path "/55aab698-7558-4fe2-95ad-faa6da60ef89/1d5016d9-fde4-4367-b1de-5d16dd08b171"
-          (reference "#PWR040") (unit 1)
+          (reference "#PWR044") (unit 1)
         )
       )
@@
   (symbol (lib_id "00_lib:nixie_daughter_board") (at 110.49 153.67 0) (unit 1)
     (in_bom yes) (on_board yes) (dnp no) (fields_autoplaced)
-    (property "Reference" "U6" (at 123.825 132.08 0)
+    (property "Reference" "U7" (at 123.825 132.08 0)
       (effects (font (size 1.27 1.27)))
     )
@@
       (project "nixieAccurateClock"
         (path "/55aab698-7558-4fe2-95ad-faa6da60ef89/1d5016d9-fde4-4367-b1de-5d16dd08b171"
-          (reference "U6") (unit 1)
+          (reference "U7") (unit 1)
         )
       )
@@
         )
         (path "/55aab698-7558-4fe2-95ad-faa6da60ef89/1d5016d9-fde4-4367-b1de-5d16dd08b171"
-          (reference "#PWR030") (unit 1)
+          (reference "#PWR034") (unit 1)
         )
       )
@@
   (symbol (lib_id "power:GND") (at 168.91 110.49 270) (unit 1)
     (in_bom yes) (on_board yes) (dnp no) (fields_autoplaced)
-    (property "Reference" "#PWR042" (at 162.56 110.49 0)
+    (property "Reference" "#PWR029" (at 162.56 110.49 0)
       (effects (font (size 1.27 1.27)) hide)
     )
@@
       (project "nixieAccurateClock"
         (path "/55aab698-7558-4fe2-95ad-faa6da60ef89/1d5016d9-fde4-4367-b1de-5d16dd08b171"
-          (reference "#PWR042") (unit 1)
+          (reference "#PWR029") (unit 1)
         )
       )
@@
         )
         (path "/55aab698-7558-4fe2-95ad-faa6da60ef89/1d5016d9-fde4-4367-b1de-5d16dd08b171"
-          (reference "#PWR038") (unit 1)
+          (reference "#PWR035") (unit 1)
         )
       )
@@
         )
         (path "/55aab698-7558-4fe2-95ad-faa6da60ef89/1d5016d9-fde4-4367-b1de-5d16dd08b171"
-          (reference "#PWR036") (unit 1)
+          (reference "#PWR028") (unit 1)
         )
       )
@@
   (symbol (lib_id "00_lib:nixie_daughter_board") (at 45.72 153.67 0) (unit 1)
     (in_bom yes) (on_board yes) (dnp no) (fields_autoplaced)
-    (property "Reference" "U4" (at 59.055 132.08 0)
+    (property "Reference" "U6" (at 59.055 132.08 0)
       (effects (font (size 1.27 1.27)))
     )
@@
       (project "nixieAccurateClock"
         (path "/55aab698-7558-4fe2-95ad-faa6da60ef89/1d5016d9-fde4-4367-b1de-5d16dd08b171"
-          (reference "U4") (unit 1)
+          (reference "U6") (unit 1)
         )
       )
@@
         )
         (path "/55aab698-7558-4fe2-95ad-faa6da60ef89/1d5016d9-fde4-4367-b1de-5d16dd08b171"
-          (reference "#PWR045") (unit 1)
+          (reference "#PWR033") (unit 1)
         )
       )
@@
   (symbol (lib_id "power:GND") (at 39.37 110.49 270) (unit 1)
     (in_bom yes) (on_board yes) (dnp no) (fields_autoplaced)
-    (property "Reference" "#PWR026" (at 33.02 110.49 0)
+    (property "Reference" "#PWR025" (at 33.02 110.49 0)
       (effects (font (size 1.27 1.27)) hide)
     )
@@
       (project "nixieAccurateClock"
         (path "/55aab698-7558-4fe2-95ad-faa6da60ef89/1d5016d9-fde4-4367-b1de-5d16dd08b171"
-          (reference "#PWR026") (unit 1)
+          (reference "#PWR025") (unit 1)
         )
       )
@@
   (symbol (lib_id "power:GND") (at 104.14 139.7 270) (unit 1)
     (in_bom yes) (on_board yes) (dnp no) (fields_autoplaced)
-    (property "Reference" "#PWR035" (at 97.79 139.7 0)
+    (property "Reference" "#PWR039" (at 97.79 139.7 0)
       (effects (font (size 1.27 1.27)) hide)
     )
@@
       (project "nixieAccurateClock"
         (path "/55aab698-7558-4fe2-95ad-faa6da60ef89/1d5016d9-fde4-4367-b1de-5d16dd08b171"
-          (reference "#PWR035") (unit 1)
+          (reference "#PWR039") (unit 1)
         )
       )
@@
         )
         (path "/55aab698-7558-4fe2-95ad-faa6da60ef89/1d5016d9-fde4-4367-b1de-5d16dd08b171"
-          (reference "#PWR029") (unit 1)
+          (reference "#PWR031") (unit 1)
         )
       )
@@
         )
         (path "/55aab698-7558-4fe2-95ad-faa6da60ef89/1d5016d9-fde4-4367-b1de-5d16dd08b171"
-          (reference "#PWR037") (unit 1)
-        )
-      )
+          (reference "#PWR032") (unit 1)
+        )
+      )
