File: KiCad/nixieAccurateClock/nixies.kicad_sch (KiCad schematic)
At the start: 6 parts

Commit message: Switch to <6 mil package for level shifting
Parts:
- renumbered U3 to U4, U4 to U5, U5 to U6, U6 to U7, U7 to U8, U8 to U9

Commit message: add delay resistor to level shifter OE
Resistor is shown on TX0108 data sheet.
Likely helps slow OE with capacitive input to help with power-on sequencing.
Parts:
- renumbered U4 to U3, U5 to U4, U6 to U5, U7 to U6, U8 to U7, U9 to U8

Commit message: WIP two stage HV supply
Parts:
- renumbered U3 to U4, U6 to U5, U4 to U6, U5 to U8, U8 to U9
Other:
- title: Nixies -> Nixie Accurate Clock

Commit message: simulate HV supply concept
LM5156 simulation is infeasible

LTSpice model demonstrating that a two stage buck from 5 to 210 is possible.  Both stages run away, but the LM5156 should provide feedback to keep it on target.
Parts:
- renumbered U9 to U10, U4 to U5, U5 to U6, U6 to U7, U7 to U8, U8 to U9

Commit message: finish schematic features
Parts:
- added J10: Conn_02x05_Odd_Even, Connector_PinSocket_2.54mm:PinSocket_2x05_P2.54mm_Horizontal, symbol Connector_Generic:Conn_02x05_Odd_Even
- renumbered U7 to U6, U9 to U7, U6 to U8, U8 to U9
Connections:
- net +3.3V: now also J10.6 (Pin_6)
- net +5V: now also J10.2 (Pin_2)
- net CLOCK_{HV}: now also J10.8 (Pin_8)
- net GND: now also J10.5 (Pin_5)
- net PPS_{TRIMMED}: now also J10.3 (Pin_3)
- net VPP: now also J10.9 (Pin_9)
- net D_{IN-PRECISE}: now reaches U10.1 (DOUT)
- net D_{IN-PRECISE}: now also J10.4 (Pin_4)
- new net SENSE_{PRECISE}: J10.10 (Pin_10)
Other:
- company: (none) -> Paul Willis

Commit message: ERC pass
Close look at pico iCE pinout
Add light sensor
Rough layout for non-HV
Parts:
- renumbered U8 to U10, U9 to U11, U10 to U12, U5 to U7, U6 to U8, U7 to U9
Connections:
- net I2C_{DATA}: now reaches J10.1 (Pin_1)
- net I2C_{CLOCK}: now reaches J10.7 (Pin_7)

Commit message: DRC pass
it's messy
Connections:
- net I2C_{CLOCK} renamed CLOCK_{PRECISE}
- net I2C_{DATA} renamed DATA_{PRECISE}
