File: KiCad/nixieAccurateClock/nixies.kicad_sch (KiCad schematic)
At the start: 7 parts, among them J10 Conn_02x05_Odd_Even

Commit message: Fill out BOM
Parts:
- J9: renamed from J10; Model (none) -> SFH11-PBPC-D05-RA-BK; Price (none) -> 0.81
- U10, U11, U12, U7, U8, U9: Price (none) -> 21.41

Commit message: Add retailer links
Parts:
- J9: Digikey link (none) -> https://www.digikey.com/en/products/detail/sullins-connecto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; Mouser link (none) -> N/A
- U10, U11, U12, U7, U8, U9: Digikey link (none) -> N/A; Mouser link (none) -> N/A
Other:
- moved on the sheet: J9, U10, U11, U12, U7, U8, U9

Commit message: switch to 27k R_anode
Add voltage rail jumpers for different 5V and 3.3V standby applications
Parts:
- renumbered J9 to J11
Changed lines of the file:
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@@
   (symbol (lib_id "Connector_Generic:Conn_02x05_Odd_Even") (at 45.72 135.89 0) (unit 1)
     (in_bom yes) (on_board yes) (dnp no) (fields_autoplaced)
-    (property "Reference" "J9" (at 46.99 124.46 0)
+    (property "Reference" "J11" (at 46.99 124.46 0)
       (effects (font (size 1.27 1.27)))
     )
@@
       (project "nixieAccurateClock"
         (path "/55aab698-7558-4fe2-95ad-faa6da60ef89/1d5016d9-fde4-4367-b1de-5d16dd08b171"
-          (reference "J9") (unit 1)
+          (reference "J11") (unit 1)
         )
       )
