File: KiCad/nixieAccurateClock/LSD_ADC.kicad_sch (KiCad schematic)
At the start: 6 parts

Commit message: fix clearance rules on daughter board
0.4 mm clearance is not possible to obey with an HV driver IC package that has 0.25 mm pad spacing, but all HV lines can be kept at least 0.25 mm away from everything else and inner layers can be preferentially used.

WIP ADC interface, logic level convertor has been chosen.
Parts:
- added U10, U11: TXB0108DQSR, Package_SON:USON-20_2x4mm_P0.4mm, symbol Logic_LevelTranslator:TXB0108DQSR
Connections:
- net +5V: now also U10.16 (VCCB), U11.16 (VCCB)
- net GND: now also U10.15 (GND), U11.15 (GND)
- net LSD_{SHUNT_div}: now reaches Q?.1 (B), R?.1, R?.2
- net LSD_{SHUNT_SC_Emitter}: now reaches Q?.3 (E), R?.1
- net LSD_{ADC_5V_~{CS}}: now reaches U?.13 (~{CS})
- net LSD_{ADC_5V_~{CS}}: now also U11.19 (B2)
- net LSD_{ADC_5V_D4}: now reaches U?.14 (DB4)
- net LSD_{ADC_5V_D4}: now also U11.18 (B3)
- net LSD_{ADC_5V_D5}: now reaches U?.15 (DB5)
- net LSD_{ADC_5V_D5}: now also U11.17 (B4)
- net LSD_{ADC_5V_D6}: now reaches U?.16 (DB6)
- net LSD_{ADC_5V_D6}: now also U11.14 (B5)
- net LSD_{ADC_5V_D7}: now reaches U?.17 (DB7)
- net LSD_{ADC_5V_D7}: now also U11.13 (B6)
- net LSD_{ADC_5V_~{OFL}}: now reaches U?.18 (~{OFL})
- net LSD_{ADC_5V_~{OFL}}: now also U11.12 (B7)
- net LSD_{ADC_5V_D0}: now reaches U?.2 (DB0)
- net LSD_{ADC_5V_D0}: now also U10.20 (B1)
- net LSD_{ADC_5V_D1}: now reaches U?.3 (DB1)
- net LSD_{ADC_5V_D1}: now also U10.19 (B2)
- net LSD_{ADC_5V_D2}: now reaches U?.4 (DB2)
- net LSD_{ADC_5V_D2}: now also U10.18 (B3)
- net LSD_{ADC_5V_D3}: now reaches U?.5 (DB3)
- net LSD_{ADC_5V_D3}: now also U10.17 (B4)
- net LSD_{ADC_5V_~{WR}/RDY}: now reaches U?.6 (~{WR}/RDY)
- net LSD_{ADC_5V_~{WR}/RDY}: now also U10.14 (B5)
- net LSD_{ADC_5V_MODE}: now reaches U?.7 (MODE)
- net LSD_{ADC_5V_MODE}: now also U10.13 (B6)
- net LSD_{ADC_5V_~{RD}}: now reaches U?.8 (~{RD})
- net LSD_{ADC_5V_~{RD}}: now also U10.12 (B7)
- net LSD_{ADC_5V_~{INT}}: now reaches U?.9 (~{INT})
- net LSD_{ADC_5V_~{INT}}: now also U10.11 (B8)
- new net +3.3V: U10.5 (VCCA), U10.6 (OE), U11.5 (VCCA), U11.6 (OE)
- new net LSD_{ADC_D0}: U10.1 (A1)
- new net LSD_{ADC_D1}: U10.2 (A2)
- new net LSD_{ADC_D2}: U10.3 (A3)
- new net LSD_{ADC_D3}: U10.4 (A4)
- new net LSD_{ADC_D4}: U11.3 (A3)
- new net LSD_{ADC_D5}: U11.4 (A4)
- new net LSD_{ADC_D6}: U11.7 (A5)
- new net LSD_{ADC_D7}: U11.8 (A6)
- new net LSD_{ADC_MODE}: U10.8 (A6)
- new net LSD_{ADC_~{CS}}: U11.2 (A2)
- new net LSD_{ADC_~{INT}}: U10.10 (A8)
- new net LSD_{ADC_~{OFL}}: U11.9 (A7)
- new net LSD_{ADC_~{RD}}: U10.9 (A7)
- new net LSD_{ADC_~{WR}/RDY}: U10.7 (A5)
Other:
- moved on the sheet: Q?, R?

Commit message: give pico iCE better mounting
Other:
- moved on the sheet: Q?, R?, U10, U11

Commit message: Add decoupling caps
Parts:
- added C3, C4, C5, C6, C7: 0.1u, Capacitor_SMD:C_0603_1608Metric, symbol Device:C_Small
Connections:
- net +3.3V: now also C4.1, C6.1; no longer U10.5 (VCCA), U10.6 (OE), U11.5 (VCCA), U11.6 (OE)
- net +5V: now also C3.1, C5.1, C7.1; no longer U10.16 (VCCB), U11.16 (VCCB), U?.20 (V_{CC})
- new net VCC_{ADC}: C3.2, U?.20 (V_{CC})
- new net VCC_{lvl-shift-A-1}: C4.2, U10.5 (VCCA), U10.6 (OE)
- new net VCC_{lvl-shift-A-2}: C6.2, U11.5 (VCCA), U11.6 (OE)
- new net VCC_{lvl-shift-B-1}: C5.2, U10.16 (VCCB)
- new net VCC_{lvl-shift-B-2}: C7.2, U11.16 (VCCB)
Other:
- moved on the sheet: U10, U11

Commit message: fix sims
SPICE asy files had improper netlist orders for their models
FIxing this reveals that the LSD ADC circuit needed resistor tweaks, but now behaves much better (~70% of FS range for a 145 V nixie).
The HV supply still does not sim properly.  Will investigate a dedicated driver IC.
Parts:
- R?: value 2.2k -> 470
Changed lines of the file:
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@@
       (effects (font (size 1.27 1.27)) (justify left))
     )
-    (property "Value" "2.2k" (at 138.43 157.48 0)
+    (property "Value" "470" (at 138.43 157.48 0)
       (effects (font (size 1.27 1.27)) (justify left))
     )

Commit message: Switch to <6 mil package for level shifting
Parts:
- removed U10, U11: TXB0108DQSR, Package_SON:USON-20_2x4mm_P0.4mm, symbol Logic_LevelTranslator:TXB0108DQSR
- added U11, U12: TXB0108PWR, Package_SO:TSSOP-20_4.4x6.5mm_P0.65mm, symbol 00_lib:TXB0108PWR
Connections:
- net +3.3V: now also U11.10 (OE), U12.10 (OE)
- net GND: now also U11.11 (GND), U12.11 (GND)
- net LSD_{ADC_5V_D0}: now also U11.20 (B1)
- net LSD_{ADC_5V_D1}: now also U11.18 (B2)
- net LSD_{ADC_5V_D2}: now also U11.17 (B3)
- net LSD_{ADC_5V_D3}: now also U11.16 (B4)
- net LSD_{ADC_5V_D4}: now also U12.17 (B3)
- net LSD_{ADC_5V_D5}: now also U12.16 (B4)
- net LSD_{ADC_5V_D6}: now also U12.15 (B5)
- net LSD_{ADC_5V_D7}: now also U12.14 (B6)
- net LSD_{ADC_5V_MODE}: now also U11.14 (B6)
- net LSD_{ADC_5V_~{CS}}: now also U12.18 (B2)
- net LSD_{ADC_5V_~{INT}}: now also U11.12 (B8)
- net LSD_{ADC_5V_~{OFL}}: now also U12.13 (B7)
- net LSD_{ADC_5V_~{RD}}: now also U11.13 (B7)
- net LSD_{ADC_5V_~{WR}/RDY}: now also U11.15 (B5)
- net LSD_{ADC_D0}: now also U11.5 (A4)
- net LSD_{ADC_D1}: now also U11.4 (A3)
- net LSD_{ADC_D2}: now also U11.3 (A2)
- net LSD_{ADC_D3}: now also U11.1 (A1)
- net LSD_{ADC_D4}: now also U12.4 (A3)
- net LSD_{ADC_D5}: now also U12.5 (A4)
- net LSD_{ADC_D6}: now also U12.6 (A5)
- net LSD_{ADC_D7}: now also U12.7 (A6)
- net LSD_{ADC_MODE}: now also U11.7 (A6)
- net LSD_{ADC_~{CS}}: now also U12.3 (A2)
- net LSD_{ADC_~{INT}}: now also U11.9 (A8)
- net LSD_{ADC_~{OFL}}: now also U12.8 (A7)
- net LSD_{ADC_~{RD}}: now also U11.8 (A7)
- net LSD_{ADC_~{WR}/RDY}: now also U11.6 (A5)
- net VCC_{lvl-shift-A-1}: now also U11.2 (VCCA)
- net VCC_{lvl-shift-A-2}: now also U12.2 (VCCA)
- net VCC_{lvl-shift-B-1}: now also U11.19 (VCCB)
- net VCC_{lvl-shift-B-2}: now also U12.19 (VCCB)
