File: KiCad/nixieAccurateClock/LSD_ADC.kicad_sch (KiCad schematic)
At the start: 13 parts, among them U11 TXB0108PWR, U12 TXB0108PWR

Commit message: add delay resistor to level shifter OE
Resistor is shown on TX0108 data sheet.
Likely helps slow OE with capacitive input to help with power-on sequencing.
Parts:
- added R? (x2): 100k, Resistor_SMD:R_0603_1608Metric, symbol Device:R
- renumbered U11 to U10, U12 to U11
Connections:
- net +3.3V: now also R?.1, R?.1; no longer U10.10 (OE), U11.10 (OE)
- new net OE_{lvl-shift-1}: R?.2, U10.10 (OE)
- new net OE_{lvl-shift-2}: R?.2, U11.10 (OE)
Other:
- moved on the sheet: C4, C5, C6, C7, Q?, R?, U10, U11

Commit message: tie level shift OE to ground
OE on the TX0108 is internally tied high and should be softly pulled low for power-on sequencing.
Connections:
- net +3.3V: no longer R?.1, R?.1
- net GND: now also R?.1, R?.1
Changed lines of the file:
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@@
   (junction (at 93.98 124.46) (diameter 0) (color 0 0 0 0)
   )
+  (wire (pts (xy 241.3 60.96) (xy 241.3 62.23))
+    (stroke (width 0) (type default))
+  )
+  (wire (pts (xy 229.87 74.93) (xy 233.68 74.93))
+    (stroke (width 0) (type default))
+  )
+  (wire (pts (xy 114.3 185.42) (xy 114.3 190.5))
+    (stroke (width 0) (type default))
+  )
   (wire (pts (xy 166.37 50.8) (xy 166.37 52.07))
-    (stroke (width 0) (type default))
-  )
-  (wire (pts (xy 241.3 60.96) (xy 241.3 62.23))
-    (stroke (width 0) (type default))
-  )
-  (wire (pts (xy 229.87 74.93) (xy 233.68 74.93))
-    (stroke (width 0) (type default))
-  )
-  (wire (pts (xy 114.3 185.42) (xy 114.3 190.5))
     (stroke (width 0) (type default))
   )
@@
     )
   )
+  (symbol (lib_id "power:GND") (at 133.35 69.85 270) (unit 1)
+    (in_bom yes) (on_board yes) (dnp no)
+    (property "Reference" "#PWR?" (at 127 69.85 0)
+      (effects (font (size 1.27 1.27)) hide)
+    )
+    (property "Value" "GND" (at 129.54 69.85 90)
+      (effects (font (size 1.27 1.27)) (justify right))
+    )
+    (property "Footprint" "" (at 133.35 69.85 0)
+      (effects (font (size 1.27 1.27)) hide)
+    )
+    (property "Datasheet" "" (at 133.35 69.85 0)
+      (effects (font (size 1.27 1.27)) hide)
+    )
+    (pin "1")
+    (instances
+      (project "nixieAccurateClock"
+        (path "/55aab698-7558-4fe2-95ad-faa6da60ef89"
+          (reference "#PWR?") (unit 1)
+        )
+        (path "/55aab698-7558-4fe2-95ad-faa6da60ef89/919829db-9d44-4db4-a8a4-73523a1d66d3"
+          (reference "#PWR056") (unit 1)
+        )
+      )
+    )
+  )
   (symbol (lib_id "power:+5V") (at 246.38 50.8 0) (unit 1)
     (in_bom yes) (on_board yes) (dnp no)
@@
     )
   )
-  (symbol (lib_id "power:+3.3V") (at 208.28 69.85 90) (unit 1)
-    (in_bom yes) (on_board yes) (dnp no)
-    (property "Reference" "#PWR?" (at 212.09 69.85 0)
-      (effects (font (size 1.27 1.27)) hide)
-    )
-    (property "Value" "+3.3V" (at 201.93 69.85 90)
-      (effects (font (size 1.27 1.27)))
-    )
-    (property "Footprint" "" (at 208.28 69.85 0)
-      (effects (font (size 1.27 1.27)) hide)
-    )
-    (property "Datasheet" "" (at 208.28 69.85 0)
-      (effects (font (size 1.27 1.27)) hide)
-    )
-    (pin "1")
-    (instances
-      (project "nixieAccurateClock"
-        (path "/55aab698-7558-4fe2-95ad-faa6da60ef89"
-          (reference "#PWR?") (unit 1)
-        )
-        (path "/55aab698-7558-4fe2-95ad-faa6da60ef89/919829db-9d44-4db4-a8a4-73523a1d66d3"
-          (reference "#PWR057") (unit 1)
-        )
-      )
-    )
-  )
   (symbol (lib_id "Device:R") (at 93.98 111.76 0) (unit 1)
     (in_bom yes) (on_board yes) (dnp no) (fields_autoplaced)
@@
         (path "/55aab698-7558-4fe2-95ad-faa6da60ef89/919829db-9d44-4db4-a8a4-73523a1d66d3"
           (reference "Q2") (unit 1)
-        )
-      )
-    )
-  )
-  (symbol (lib_id "power:+3.3V") (at 133.35 69.85 90) (unit 1)
-    (in_bom yes) (on_board yes) (dnp no)
-    (property "Reference" "#PWR?" (at 137.16 69.85 0)
-      (effects (font (size 1.27 1.27)) hide)
-    )
-    (property "Value" "+3.3V" (at 127 69.85 90)
-      (effects (font (size 1.27 1.27)))
-    )
-    (property "Footprint" "" (at 133.35 69.85 0)
-      (effects (font (size 1.27 1.27)) hide)
-    )
-    (property "Datasheet" "" (at 133.35 69.85 0)
-      (effects (font (size 1.27 1.27)) hide)
-    )
-    (pin "1")
-    (instances
-      (project "nixieAccurateClock"
-        (path "/55aab698-7558-4fe2-95ad-faa6da60ef89"
-          (reference "#PWR?") (unit 1)
-        )
-        (path "/55aab698-7558-4fe2-95ad-faa6da60ef89/919829db-9d44-4db4-a8a4-73523a1d66d3"
-          (reference "#PWR056") (unit 1)
         )
       )
@@
         )
       )
+    )
+  )
+  (symbol (lib_id "power:GND") (at 208.28 69.85 270) (unit 1)
+    (in_bom yes) (on_board yes) (dnp no)
+    (property "Reference" "#PWR?" (at 201.93 69.85 0)
+      (effects (font (size 1.27 1.27)) hide)
+    )
+    (property "Value" "GND" (at 204.47 69.85 90)
+      (effects (font (size 1.27 1.27)) (justify right))
+    )
+    (property "Footprint" "" (at 208.28 69.85 0)
+      (effects (font (size 1.27 1.27)) hide)
+    )
+    (property "Datasheet" "" (at 208.28 69.85 0)
+      (effects (font (size 1.27 1.27)) hide)
+    )
+    (pin "1")
+    (instances
+      (project "nixieAccurateClock"
+        (path "/55aab698-7558-4fe2-95ad-faa6da60ef89"
+          (reference "#PWR?") (unit 1)
+        )
+        (path "/55aab698-7558-4fe2-95ad-faa6da60ef89/919829db-9d44-4db4-a8a4-73523a1d66d3"
+          (reference "#PWR057") (unit 1)
+        )
+      )

Commit message: WIP two stage HV supply
Parts:
- renumbered C3 to C10, C4 to C11, C5 to C12, C6 to C13, C7 to C14, U10 to U11, U11 to U12
Other:
- title: LSD ADC -> Nixie Accurate Clock
Changed lines of the file:
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@@
   (paper "A4")
   (title_block
-    (title "LSD ADC")
+    (title "Nixie Accurate Clock")
+    (rev "A")
   )
   (junction (at 114.3 163.83) (diameter 0) (color 0 0 0 0)
@@
   (symbol (lib_name "C_Small_1") (lib_id "Device:C_Small") (at 83.82 29.21 0) (unit 1)
     (in_bom yes) (on_board yes) (dnp no)
-    (property "Reference" "C3" (at 81.28 27.9463 0)
+    (property "Reference" "C10" (at 81.28 27.9463 0)
       (effects (font (size 1.27 1.27)) (justify right))
     )
@@
       (project "nixieAccurateClock"
         (path "/55aab698-7558-4fe2-95ad-faa6da60ef89/919829db-9d44-4db4-a8a4-73523a1d66d3"
-          (reference "C3") (unit 1)
+          (reference "C10") (unit 1)
         )
       )
@@
         )
         (path "/55aab698-7558-4fe2-95ad-faa6da60ef89/919829db-9d44-4db4-a8a4-73523a1d66d3"
-          (reference "#PWR050") (unit 1)
+          (reference "#PWR063") (unit 1)
         )
       )
@@
         )
         (path "/55aab698-7558-4fe2-95ad-faa6da60ef89/919829db-9d44-4db4-a8a4-73523a1d66d3"
-          (reference "#PWR054") (unit 1)
+          (reference "#PWR071") (unit 1)
         )
       )
@@
   (symbol (lib_name "C_Small_3") (lib_id "Device:C_Small") (at 246.38 54.61 0) (mirror y) (unit 1)
     (in_bom yes) (on_board yes) (dnp no)
-    (property "Reference" "C7" (at 248.92 53.3463 0)
+    (property "Reference" "C14" (at 248.92 53.3463 0)
       (effects (font (size 1.27 1.27)) (justify right))
     )
@@
       (project "nixieAccurateClock"
         (path "/55aab698-7558-4fe2-95ad-faa6da60ef89/919829db-9d44-4db4-a8a4-73523a1d66d3"
-          (reference "C7") (unit 1)
+          (reference "C14") (unit 1)
         )
       )
@@
   (symbol (lib_id "00_lib:TXB0108PWR") (at 168.91 80.01 0) (unit 1)
     (in_bom yes) (on_board yes) (dnp no) (fields_autoplaced)
-    (property "Reference" "U10" (at 171.1041 97.79 0)
+    (property "Reference" "U11" (at 171.1041 97.79 0)
       (effects (font (size 1.27 1.27)) (justify left))
     )
@@
       (project "nixieAccurateClock"
         (path "/55aab698-7558-4fe2-95ad-faa6da60ef89/919829db-9d44-4db4-a8a4-73523a1d66d3"
-          (reference "U10") (unit 1)
+          (reference "U11") (unit 1)
         )
       )
@@
   (symbol (lib_name "C_Small_2") (lib_id "Device:C_Small") (at 241.3 54.61 0) (unit 1)
     (in_bom yes) (on_board yes) (dnp no)
-    (property "Reference" "C6" (at 238.76 53.3463 0)
+    (property "Reference" "C13" (at 238.76 53.3463 0)
       (effects (font (size 1.27 1.27)) (justify right))
     )
@@
       (project "nixieAccurateClock"
         (path "/55aab698-7558-4fe2-95ad-faa6da60ef89/919829db-9d44-4db4-a8a4-73523a1d66d3"
-          (reference "C6") (unit 1)
+          (reference "C13") (unit 1)
         )
       )
@@
         )
         (path "/55aab698-7558-4fe2-95ad-faa6da60ef89/919829db-9d44-4db4-a8a4-73523a1d66d3"
-          (reference "R6") (unit 1)
+          (reference "R17") (unit 1)
         )
       )
@@
         )
         (path "/55aab698-7558-4fe2-95ad-faa6da60ef89/919829db-9d44-4db4-a8a4-73523a1d66d3"
-          (reference "#PWR056") (unit 1)
+          (reference "#PWR066") (unit 1)
         )
       )
@@
         )
         (path "/55aab698-7558-4fe2-95ad-faa6da60ef89/919829db-9d44-4db4-a8a4-73523a1d66d3"
-          (reference "#PWR055") (unit 1)
+          (reference "#PWR073") (unit 1)
         )
       )
@@
         )
         (path "/55aab698-7558-4fe2-95ad-faa6da60ef89/919829db-9d44-4db4-a8a4-73523a1d66d3"
-          (reference "R7") (unit 1)
+          (reference "R18") (unit 1)
         )
       )
@@
         )
         (path "/55aab698-7558-4fe2-95ad-faa6da60ef89/919829db-9d44-4db4-a8a4-73523a1d66d3"
-          (reference "#PWR052") (unit 1)
+          (reference "#PWR067") (unit 1)
         )
       )
@@
   (symbol (lib_id "power:GND") (at 114.3 190.5 0) (unit 1)
     (in_bom yes) (on_board yes) (dnp no) (fields_autoplaced)
-    (property "Reference" "#PWR061" (at 114.3 196.85 0)
+    (property "Reference" "#PWR065" (at 114.3 196.85 0)
       (effects (font (size 1.27 1.27)) hide)
     )
@@
       (project "nixieAccurateClock"
         (path "/55aab698-7558-4fe2-95ad-faa6da60ef89/919829db-9d44-4db4-a8a4-73523a1d66d3"
-          (reference "#PWR061") (unit 1)
+          (reference "#PWR065") (unit 1)
         )
       )
@@
   (symbol (lib_id "power:GND") (at 168.91 101.6 0) (unit 1)
     (in_bom yes) (on_board yes) (dnp no) (fields_autoplaced)
-    (property "Reference" "#PWR058" (at 168.91 107.95 0)
+    (property "Reference" "#PWR068" (at 168.91 107.95 0)
       (effects (font (size 1.27 1.27)) hide)
     )
@@
       (project "nixieAccurateClock"
         (path "/55aab698-7558-4fe2-95ad-faa6da60ef89/919829db-9d44-4db4-a8a4-73523a1d66d3"
-          (reference "#PWR058") (unit 1)
+          (reference "#PWR068") (unit 1)
         )
       )
@@
         )
         (path "/55aab698-7558-4fe2-95ad-faa6da60ef89/919829db-9d44-4db4-a8a4-73523a1d66d3"
-          (reference "R8") (unit 1)
+          (reference "R13") (unit 1)
         )
       )
@@
         )
         (path "/55aab698-7558-4fe2-95ad-faa6da60ef89/919829db-9d44-4db4-a8a4-73523a1d66d3"
-          (reference "R11") (unit 1)
+          (reference "R16") (unit 1)
         )
       )
@@
   (symbol (lib_id "power:VPP") (at 93.98 144.78 180) (unit 1)
     (in_bom yes) (on_board yes) (dnp no) (fields_autoplaced)
-    (property "Reference" "#PWR060" (at 93.98 140.97 0)
+    (property "Reference" "#PWR064" (at 93.98 140.97 0)
       (effects (font (size 1.27 1.27)) hide)
     )
@@
       (project "nixieAccurateClock"
         (path "/55aab698-7558-4fe2-95ad-faa6da60ef89/919829db-9d44-4db4-a8a4-73523a1d66d3"
-          (reference "#PWR060") (unit 1)
+          (reference "#PWR064") (unit 1)
         )
       )
@@
         )
         (path "/55aab698-7558-4fe2-95ad-faa6da60ef89/919829db-9d44-4db4-a8a4-73523a1d66d3"
-          (reference "#PWR053") (unit 1)
+          (reference "#PWR069") (unit 1)
         )
       )
@@
   (symbol (lib_id "power:GND") (at 243.84 101.6 0) (unit 1)
     (in_bom yes) (on_board yes) (dnp no) (fields_autoplaced)
-    (property "Reference" "#PWR059" (at 243.84 107.95 0)
+    (property "Reference" "#PWR072" (at 243.84 107.95 0)
       (effects (font (size 1.27 1.27)) hide)
     )
@@
       (project "nixieAccurateClock"
         (path "/55aab698-7558-4fe2-95ad-faa6da60ef89/919829db-9d44-4db4-a8a4-73523a1d66d3"
-          (reference "#PWR059") (unit 1)
+          (reference "#PWR072") (unit 1)
         )
       )
@@
         )
         (path "/55aab698-7558-4fe2-95ad-faa6da60ef89/919829db-9d44-4db4-a8a4-73523a1d66d3"
-          (reference "#PWR051") (unit 1)
+          (reference "#PWR061") (unit 1)
         )
       )
@@
         )
         (path "/55aab698-7558-4fe2-95ad-faa6da60ef89/919829db-9d44-4db4-a8a4-73523a1d66d3"
-          (reference "#PWR049") (unit 1)
+          (reference "#PWR062") (unit 1)
         )
       )
@@
         )
         (path "/55aab698-7558-4fe2-95ad-faa6da60ef89/919829db-9d44-4db4-a8a4-73523a1d66d3"
-          (reference "Q2") (unit 1)
+          (reference "Q3") (unit 1)
         )
       )
@@
   (symbol (lib_id "Device:C_Small") (at 166.37 54.61 0) (unit 1)
     (in_bom yes) (on_board yes) (dnp no)
-    (property "Reference" "C4" (at 163.83 53.3463 0)
+    (property "Reference" "C11" (at 163.83 53.3463 0)
       (effects (font (size 1.27 1.27)) (justify right))
     )
@@
       (project "nixieAccurateClock"
         (path "/55aab698-7558-4fe2-95ad-faa6da60ef89/919829db-9d44-4db4-a8a4-73523a1d66d3"
-          (reference "C4") (unit 1)
+          (reference "C11") (unit 1)
         )
       )
@@
   (symbol (lib_name "C_Small_4") (lib_id "Device:C_Small") (at 171.45 54.61 0) (mirror y) (unit 1)
     (in_bom yes) (on_board yes) (dnp no)
-    (property "Reference" "C5" (at 173.99 53.3463 0)
+    (property "Reference" "C12" (at 173.99 53.3463 0)
       (effects (font (size 1.27 1.27)) (justify right))
     )
@@
       (project "nixieAccurateClock"
         (path "/55aab698-7558-4fe2-95ad-faa6da60ef89/919829db-9d44-4db4-a8a4-73523a1d66d3"
-          (reference "C5") (unit 1)
+          (reference "C12") (unit 1)
         )
       )
@@
   (symbol (lib_name "TXB0108PWR_1") (lib_id "00_lib:TXB0108PWR") (at 243.84 80.01 0) (unit 1)
     (in_bom yes) (on_board yes) (dnp no) (fields_autoplaced)
-    (property "Reference" "U11" (at 246.0341 97.79 0)
+    (property "Reference" "U12" (at 246.0341 97.79 0)
       (effects (font (size 1.27 1.27)) (justify left))
     )
@@
       (project "nixieAccurateClock"
         (path "/55aab698-7558-4fe2-95ad-faa6da60ef89/919829db-9d44-4db4-a8a4-73523a1d66d3"
-          (reference "U11") (unit 1)
+          (reference "U12") (unit 1)
         )
       )
@@
         )
         (path "/55aab698-7558-4fe2-95ad-faa6da60ef89/919829db-9d44-4db4-a8a4-73523a1d66d3"
-          (reference "R10") (unit 1)
+          (reference "R15") (unit 1)
         )
       )
@@
         )
         (path "/55aab698-7558-4fe2-95ad-faa6da60ef89/919829db-9d44-4db4-a8a4-73523a1d66d3"
-          (reference "R9") (unit 1)
+          (reference "R14") (unit 1)
         )
       )
@@
         )
         (path "/55aab698-7558-4fe2-95ad-faa6da60ef89/919829db-9d44-4db4-a8a4-73523a1d66d3"
-          (reference "U9") (unit 1)
+          (reference "U10") (unit 1)
         )
       )
@@
         )
         (path "/55aab698-7558-4fe2-95ad-faa6da60ef89/919829db-9d44-4db4-a8a4-73523a1d66d3"
-          (reference "#PWR057") (unit 1)
-        )
-      )
+          (reference "#PWR070") (unit 1)
+        )
+      )

Commit message: simulate HV supply concept
LM5156 simulation is infeasible

LTSpice model demonstrating that a two stage buck from 5 to 210 is possible.  Both stages run away, but the LM5156 should provide feedback to keep it on target.
Parts:
- removed Q?: PZTA42, Package_TO_SOT_SMD:SOT-223-3_TabPin2, symbol Transistor_BJT:PZTA42
- added Q3: BSP88, Package_TO_SOT_SMD:SOT-223-3_TabPin2, symbol 00_lib:BSP88
- R24: renamed from R?; value 100k -> 10k
- R25: renamed from R?; value 470 -> 10k
- gave numbers to parts that had none: 5
- renumbered C10 to C12, C11 to C13, C12 to C14, C13 to C15, C14 to C16, U11 to U12, U12 to U13
Connections:
- net LSD_{SHUNT_SC_Emitter}: now also Q3.3 (S)
- net LSD_{SHUNT_div}: now also Q3.1 (G)
- net V_{SHUNT}: now also Q3.2 (D)

Commit message: HV bleed circuit
Parts:
- renumbered C12 to C13, C13 to C14, C14 to C15, C15 to C16, C16 to C17, Q3 to Q5, R22 to R26, R23 to R27, R24 to R28, R25 to R29, R26 to R30, R27 to R31

Commit message: finish schematic features
Parts:
- added TP20, TP21, TP22, TP23: TestPoint, TestPoint:TestPoint_Loop_D2.54mm_Drill1.5mm_Beaded, symbol Connector:TestPoint
- renumbered C13 to C14, C14 to C15, C15 to C16, C16 to C17, C17 to C18, R30 to R26, R31 to R27, R26 to R28, R27 to R29, R28 to R30, R29 to R31
Connections:
- net GND: now also TP23.1
- net LSD_{SHUNT_SC_Emitter}: now also TP22.1
- net LSD_{SHUNT_div}: now also TP20.1
- net V_{SHUNT}: now also TP21.1
Other:
- company: (none) -> Paul Willis

Commit message: ERC pass
Close look at pico iCE pinout
Add light sensor
Rough layout for non-HV
Parts:
- renumbered C14 to C16, C15 to C17, C16 to C18, C17 to C19, C18 to C20, R26 to R28, R27 to R29, R28 to R30, R29 to R31, R30 to R32, R31 to R33, U11 to U13, U12 to U14, U13 to U15

Commit message: DRC pass
it's messy
Parts:
- renumbered R28 to R27, R29 to R28, R30 to R29, R31 to R30, R32 to R31, R33 to R32, TP20 to TP17, TP21 to TP18, TP22 to TP19, TP23 to TP20
Connections:
- net HV_{SENSE} renamed HV_{MEASURE}
