File: KiCad/nixieAccurateClock/LSD_ADC.kicad_sch (KiCad schematic)
At the start: 19 parts, among them Q5 BSP88, U14 TXB0108PWR, U15 TXB0108PWR

Commit message: Fill out BOM
Parts:
- C16, C17, C18, C19, C20: Model (none) -> CL10B104KB8NNWC; Price (none) -> 0.10
- Q5: Model (none) -> BSP88; Price (none) -> 0.60
- R27, R28, R30: Model (none) -> RC0603JR-07100KL; Price (none) -> 0.10
- R29: Model (none) -> RMCF0603FT10M0; Price (none) -> 0.10
- R31, R32: Model (none) -> RC0603FR-0710KL; Price (none) -> 0.10
- TP17, TP18, TP19, TP20: Price (none) -> 0.38
- U13: value ~ -> ADC0820BCWMX; Model (none) -> ADC0820BCWMX/NOPB; Price (none) -> 5.93
- U14, U15: Model (none) -> TXB0108PWR; Price (none) -> 1.65

Commit message: Add retailer links
Parts:
- C16, C17, C18, C19, C20: Digikey link (none) -> https://www.digikey.com/en/products/detail/samsung-electro-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; Mouser link (none) -> https://www.mouser.com/ProductDetail/Samsung-Electro-Mechan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
- Q5: Digikey link (none) -> https://www.digikey.com/en/products/detail/infineon-technol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; Mouser link (none) -> https://www.mouser.com/ProductDetail/Infineon-Technologies/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
- R27, R28, R30: Digikey link (none) -> https://www.digikey.com/en/products/detail/yageo/RC0603JR-0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; Mouser link (none) -> https://www.mouser.com/ProductDetail/YAGEO/RC0603JR-07100KL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
- R29: Digikey link (none) -> https://www.digikey.com/en/products/detail/stackpole-electr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; Mouser link (none) -> https://www.mouser.com/ProductDetail/SEI-Stackpole/RMCF0603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
- R31, R32: Digikey link (none) -> https://www.digikey.com/en/products/detail/yageo/RC0603FR-0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; Mouser link (none) -> https://www.mouser.com/ProductDetail/YAGEO/RC0603FR-0710KL?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
- TP17, TP18, TP19, TP20: Digikey link (none) -> https://www.digikey.com/en/products/detail/keystone-electro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; Mouser link (none) -> https://www.mouser.com/ProductDetail/Keystone-Electronics/5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
- U13: Digikey link (none) -> https://www.digikey.com/en/products/detail/texas-instrument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; Mouser link (none) -> https://www.mouser.com/ProductDetail/Texas-Instruments/ADC0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
- U14, U15: Digikey link (none) -> https://www.digikey.com/en/products/detail/texas-instrument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; Mouser link (none) -> https://www.mouser.com/ProductDetail/Texas-Instruments/TXB0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

Commit message: Switch to SMT test points
Parts:
- TP17, TP18, TP19, TP20: footprint TestPoint:TestPoint_Loop_D2.54mm_Drill1.5mm_Beaded -> 00_lib:TestPoint_Keystone_5019_Minature; Digikey link https://www.digikey.com/en/products/detail/keystone-electronics/5001/255327 -> https://www.digikey.com/en/products/detail/keystone-electronics/5019/3907343; Model 5001 -> 5019; Mouser link https://www.mouser.com/ProductDetail/Keystone-Electronics/5001?qs=q0tsjPZWdm%2FW0vdr%2FwowKg%3D%3D -> https://www.mouser.com/ProductDetail/Keystone-Electronics/5019?qs=wOxb8XianXjjCAsb90Ilzw%3D%3D; Price 0.38 -> 0.33
Changed lines of the file:
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@@
       (effects (font (size 1.27 1.27)))
     )
-    (property "Footprint" "TestPoint:TestPoint_Loop_D2.54mm_Drill1.5mm_Beaded" (at 88.9 119.38 0)
-      (effects (font (size 1.27 1.27)) hide)
-    )
-    (property "Datasheet" "https://www.keyelco.com/userAssets/file/M65p56.pdf" (at 88.9 119.38 0)
-      (effects (font (size 1.27 1.27)) hide)
-    )
-    (property "Model" "5001" (at 88.9 124.46 0)
+    (property "Footprint" "00_lib:TestPoint_Keystone_5019_Minature" (at 88.9 119.38 0)
+      (effects (font (size 1.27 1.27)) hide)
+    )
+    (property "Datasheet" "https://www.mouser.com/datasheet/2/215/019-743690.pdf" (at 88.9 119.38 0)
+      (effects (font (size 1.27 1.27)) hide)
+    )
+    (property "Model" "5019" (at 88.9 124.46 0)
       (effects (font (size 1.27 1.27)) hide)
     )
@@
       (effects (font (size 1.27 1.27)) hide)
     )
-    (property "Price" "0.38" (at 88.9 124.46 0)
-      (effects (font (size 1.27 1.27)) hide)
-    )
-    (property "Digikey link" "https://www.digikey.com/en/products/detail/keystone-electronics/5001/255327" (at 88.9 124.46 0)
-      (effects (font (size 1.27 1.27)) hide)
-    )
-    (property "Mouser link" "https://www.mouser.com/ProductDetail/Keystone-Electronics/5001?qs=q0tsjPZWdm%2FW0vdr%2FwowKg%3D%3D" (at 88.9 124.46 0)
+    (property "Price" "0.33" (at 88.9 124.46 0)
+      (effects (font (size 1.27 1.27)) hide)
+    )
+    (property "Digikey link" "https://www.digikey.com/en/products/detail/keystone-electronics/5019/3907343" (at 88.9 124.46 0)
+      (effects (font (size 1.27 1.27)) hide)
+    )
+    (property "Mouser link" "https://www.mouser.com/ProductDetail/Keystone-Electronics/5019?qs=wOxb8XianXjjCAsb90Ilzw%3D%3D" (at 88.9 124.46 0)
       (effects (font (size 1.27 1.27)) hide)
     )
@@
       (effects (font (size 1.27 1.27)) (justify left))
     )
-    (property "Footprint" "TestPoint:TestPoint_Loop_D2.54mm_Drill1.5mm_Beaded" (at 130.81 160.02 0)
-      (effects (font (size 1.27 1.27)) hide)
-    )
-    (property "Datasheet" "https://www.keyelco.com/userAssets/file/M65p56.pdf" (at 130.81 160.02 0)
-      (effects (font (size 1.27 1.27)) hide)
-    )
-    (property "Model" "5001" (at 125.73 160.02 0)
+    (property "Footprint" "00_lib:TestPoint_Keystone_5019_Minature" (at 130.81 160.02 0)
+      (effects (font (size 1.27 1.27)) hide)
+    )
+    (property "Datasheet" "https://www.mouser.com/datasheet/2/215/019-743690.pdf" (at 130.81 160.02 0)
+      (effects (font (size 1.27 1.27)) hide)
+    )
+    (property "Model" "5019" (at 125.73 160.02 0)
       (effects (font (size 1.27 1.27)) hide)
     )
@@
       (effects (font (size 1.27 1.27)) hide)
     )
-    (property "Price" "0.38" (at 125.73 160.02 0)
-      (effects (font (size 1.27 1.27)) hide)
-    )
-    (property "Digikey link" "https://www.digikey.com/en/products/detail/keystone-electronics/5001/255327" (at 125.73 160.02 0)
-      (effects (font (size 1.27 1.27)) hide)
-    )
-    (property "Mouser link" "https://www.mouser.com/ProductDetail/Keystone-Electronics/5001?qs=q0tsjPZWdm%2FW0vdr%2FwowKg%3D%3D" (at 125.73 160.02 0)
+    (property "Price" "0.33" (at 125.73 160.02 0)
+      (effects (font (size 1.27 1.27)) hide)
+    )
+    (property "Digikey link" "https://www.digikey.com/en/products/detail/keystone-electronics/5019/3907343" (at 125.73 160.02 0)
+      (effects (font (size 1.27 1.27)) hide)
+    )
+    (property "Mouser link" "https://www.mouser.com/ProductDetail/Keystone-Electronics/5019?qs=wOxb8XianXjjCAsb90Ilzw%3D%3D" (at 125.73 160.02 0)
       (effects (font (size 1.27 1.27)) hide)
     )
@@
       (effects (font (size 1.27 1.27)))
     )
-    (property "Footprint" "TestPoint:TestPoint_Loop_D2.54mm_Drill1.5mm_Beaded" (at 107.95 181.61 0)
-      (effects (font (size 1.27 1.27)) hide)
-    )
-    (property "Datasheet" "https://www.keyelco.com/userAssets/file/M65p56.pdf" (at 107.95 181.61 0)
-      (effects (font (size 1.27 1.27)) hide)
-    )
-    (property "Model" "5001" (at 107.95 176.53 0)
+    (property "Footprint" "00_lib:TestPoint_Keystone_5019_Minature" (at 107.95 181.61 0)
+      (effects (font (size 1.27 1.27)) hide)
+    )
+    (property "Datasheet" "https://www.mouser.com/datasheet/2/215/019-743690.pdf" (at 107.95 181.61 0)
+      (effects (font (size 1.27 1.27)) hide)
+    )
+    (property "Model" "5019" (at 107.95 176.53 0)
       (effects (font (size 1.27 1.27)) hide)
     )
@@
       (effects (font (size 1.27 1.27)) hide)
     )
-    (property "Price" "0.38" (at 107.95 176.53 0)
-      (effects (font (size 1.27 1.27)) hide)
-    )
-    (property "Digikey link" "https://www.digikey.com/en/products/detail/keystone-electronics/5001/255327" (at 107.95 176.53 0)
-      (effects (font (size 1.27 1.27)) hide)
-    )
-    (property "Mouser link" "https://www.mouser.com/ProductDetail/Keystone-Electronics/5001?qs=q0tsjPZWdm%2FW0vdr%2FwowKg%3D%3D" (at 107.95 176.53 0)
+    (property "Price" "0.33" (at 107.95 176.53 0)
+      (effects (font (size 1.27 1.27)) hide)
+    )
+    (property "Digikey link" "https://www.digikey.com/en/products/detail/keystone-electronics/5019/3907343" (at 107.95 176.53 0)
+      (effects (font (size 1.27 1.27)) hide)
+    )
+    (property "Mouser link" "https://www.mouser.com/ProductDetail/Keystone-Electronics/5019?qs=wOxb8XianXjjCAsb90Ilzw%3D%3D" (at 107.95 176.53 0)
       (effects (font (size 1.27 1.27)) hide)
     )
@@
       (effects (font (size 1.27 1.27)) (justify left))
     )
-    (property "Footprint" "TestPoint:TestPoint_Loop_D2.54mm_Drill1.5mm_Beaded" (at 140.97 187.96 0)
-      (effects (font (size 1.27 1.27)) hide)
-    )
-    (property "Datasheet" "https://www.keyelco.com/userAssets/file/M65p56.pdf" (at 140.97 187.96 0)
-      (effects (font (size 1.27 1.27)) hide)
-    )
-    (property "Model" "5001" (at 135.89 187.96 0)
+    (property "Footprint" "00_lib:TestPoint_Keystone_5019_Minature" (at 140.97 187.96 0)
+      (effects (font (size 1.27 1.27)) hide)
+    )
+    (property "Datasheet" "https://www.mouser.com/datasheet/2/215/019-743690.pdf" (at 140.97 187.96 0)
+      (effects (font (size 1.27 1.27)) hide)
+    )
+    (property "Model" "5019" (at 135.89 187.96 0)
       (effects (font (size 1.27 1.27)) hide)
     )
@@
       (effects (font (size 1.27 1.27)) hide)
     )
-    (property "Price" "0.38" (at 135.89 187.96 0)
-      (effects (font (size 1.27 1.27)) hide)
-    )
-    (property "Digikey link" "https://www.digikey.com/en/products/detail/keystone-electronics/5001/255327" (at 135.89 187.96 0)
-      (effects (font (size 1.27 1.27)) hide)
-    )
-    (property "Mouser link" "https://www.mouser.com/ProductDetail/Keystone-Electronics/5001?qs=q0tsjPZWdm%2FW0vdr%2FwowKg%3D%3D" (at 135.89 187.96 0)
-      (effects (font (size 1.27 1.27)) hide)
-    )
+    (property "Price" "0.33" (at 135.89 187.96 0)
+      (effects (font (size 1.27 1.27)) hide)
+    )
+    (property "Digikey link" "https://www.digikey.com/en/products/detail/keystone-electronics/5019/3907343" (at 135.89 187.96 0)
+      (effects (font (size 1.27 1.27)) hide)
+    )
+    (property "Mouser link" "https://www.mouser.com/ProductDetail/Keystone-Electronics/5019?qs=wOxb8XianXjjCAsb90Ilzw%3D%3D" (at 135.89 187.96 0)
+      (effects (font (size 1.27 1.27)) hide)
+    )

Commit message: clean up SMPS routing
Parts:
- renumbered TP17 to TP14, TP18 to TP15, TP19 to TP16, TP20 to TP17
Changed lines of the file:
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@@
   (symbol (lib_id "Connector:TestPoint") (at 88.9 124.46 90) (unit 1)
     (in_bom yes) (on_board yes) (dnp no) (fields_autoplaced)
-    (property "Reference" "TP17" (at 85.598 119.38 90)
+    (property "Reference" "TP14" (at 85.598 119.38 90)
       (effects (font (size 1.27 1.27)))
     )
@@
       (project "nixieAccurateClock"
         (path "/55aab698-7558-4fe2-95ad-faa6da60ef89/919829db-9d44-4db4-a8a4-73523a1d66d3"
-          (reference "TP17") (unit 1)
+          (reference "TP14") (unit 1)
         )
       )
@@
   (symbol (lib_id "Connector:TestPoint") (at 125.73 160.02 0) (unit 1)
     (in_bom yes) (on_board yes) (dnp no) (fields_autoplaced)
-    (property "Reference" "TP18" (at 128.27 155.448 0)
+    (property "Reference" "TP15" (at 128.27 155.448 0)
       (effects (font (size 1.27 1.27)) (justify left))
     )
@@
       (project "nixieAccurateClock"
         (path "/55aab698-7558-4fe2-95ad-faa6da60ef89/919829db-9d44-4db4-a8a4-73523a1d66d3"
-          (reference "TP18") (unit 1)
+          (reference "TP15") (unit 1)
         )
       )
@@
   (symbol (lib_id "Connector:TestPoint") (at 107.95 176.53 90) (mirror x) (unit 1)
     (in_bom yes) (on_board yes) (dnp no)
-    (property "Reference" "TP19" (at 104.648 181.61 90)
+    (property "Reference" "TP16" (at 104.648 181.61 90)
       (effects (font (size 1.27 1.27)))
     )
@@
       (project "nixieAccurateClock"
         (path "/55aab698-7558-4fe2-95ad-faa6da60ef89/919829db-9d44-4db4-a8a4-73523a1d66d3"
-          (reference "TP19") (unit 1)
+          (reference "TP16") (unit 1)
         )
       )
@@
   (symbol (lib_id "Connector:TestPoint") (at 135.89 187.96 0) (unit 1)
     (in_bom yes) (on_board yes) (dnp no) (fields_autoplaced)
-    (property "Reference" "TP20" (at 138.43 183.388 0)
+    (property "Reference" "TP17" (at 138.43 183.388 0)
       (effects (font (size 1.27 1.27)) (justify left))
     )
@@
       (project "nixieAccurateClock"
         (path "/55aab698-7558-4fe2-95ad-faa6da60ef89/919829db-9d44-4db4-a8a4-73523a1d66d3"
-          (reference "TP20") (unit 1)
-        )
-      )
+          (reference "TP17") (unit 1)
+        )
+      )
