File: KiCad/nixieAccurateClock/20V_supply.kicad_sch (KiCad schematic)
At the start: 18 parts, among them Q4 BSP88

Commit message: simulate HV supply concept
LM5156 simulation is infeasible

LTSpice model demonstrating that a two stage buck from 5 to 210 is possible.  Both stages run away, but the LM5156 should provide feedback to keep it on target.
Parts:
- removed R?: 160k, Resistor_SMD:R_0201_0603Metric, symbol Device:R
- removed R?: 62k, Resistor_SMD:R_0201_0603Metric, symbol Device:R
- removed R?: 10k, Resistor_SMD:R_0201_0603Metric, symbol Device:R
- added R1: 100k, Resistor_SMD:R_0603_1608Metric, symbol Device:R
- added R2: 27k, Resistor_SMD:R_0603_1608Metric, symbol Device:R
- added R4: 62k, Resistor_SMD:R_0603_1608Metric, symbol Device:R
- gave numbers to parts that had none: 13
- renumbered Q4 to Q1
Connections:
- net +5V: now also U3.1 (BIAS), R4.2; no longer C3.2
- net GND: now also C3.2, R2.1
- net at TP1.1, U3.13 (PGOOD): now also R1.1
- net VCC_{LM5156_20V}: now reaches C3.1, U3.3 (VCC)
- net VCC_{LM5156_20V}: now also R1.2
- net at U3.14 (EN_UVLO_SYNC): now also R2.2, R4.1; no longer U3.1 (BIAS)
Other:
- moved on the sheet: C3, L1

Commit message: HV bleed circuit
Parts:
- renumbered C4 to C3, C3 to C4

Commit message: Add HV control
Stop tracking SPICE simulations
Connections:
- net VCC_{LM5156_20V}: no longer C4.1, U3.3 (VCC)
- net 20V_{RT}: now reaches R3.2, U3.12 (RT)
- net 20V_{PGOOD}: now reaches R1.1, TP1.1, U3.13 (PGOOD)
- net 20V_{COMP}: now reaches C3.1, R5.1, U3.8 (COMP)
- net 20V_{COMP-1}: now reaches C5.1, R5.2
- net 20V_{CS}: now reaches Q1.3 (S), R6.1, U3.7 (CS)
- net 20V_{GATE}: now reaches Q1.1 (G), U3.4 (GATE)
- net 20V_{BOOST}: now reaches D1.2 (A), L1.2, Q1.2 (D)
- net 20V_{FB}: now reaches R7.1, R8.2, U3.10 (FB)
- net 20V_{UVLO}: now reaches R2.2, R4.1, U3.14 (EN_UVLO_SYNC)
- net 20V_{SS}: now reaches C2.1, U3.11 (SS)
- new net 20V_{VCC}: C4.1, U3.3 (VCC)
Changed lines of the file:
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@@
-    (stroke (width 0) (type default))
-  )
-  (wire (pts (xy 125.73 44.45) (xy 107.95 44.45))
     (stroke (width 0) (type default))
   )
@@
     (stroke (width 0) (type default))
   )
-  (wire (pts (xy 52.07 52.07) (xy 62.23 52.07))
-    (stroke (width 0) (type default))
-  )
   (wire (pts (xy 144.78 44.45) (xy 147.32 44.45))
     (stroke (width 0) (type default))
@@
     (stroke (width 0) (type default))
   )
+  (wire (pts (xy 107.95 44.45) (xy 125.73 44.45))
+    (stroke (width 0) (type default))
+  )
   (wire (pts (xy 110.49 82.55) (xy 110.49 87.63))
     (stroke (width 0) (type default))
@@
   )
   (wire (pts (xy 58.42 74.93) (xy 64.77 74.93))
+    (stroke (width 0) (type default))
+  )
+  (wire (pts (xy 52.07 52.07) (xy 62.23 52.07))
     (stroke (width 0) (type default))
   )
@@
     (effects (font (size 1.27 1.27)) (justify left top))
   )
+  (label "20V_{UVLO}" (at 52.07 52.07 0) (fields_autoplaced)
+    (effects (font (size 1.27 1.27)) (justify left bottom))
+  )
+  (label "20V_{COMP}" (at 109.22 74.93 0) (fields_autoplaced)
+    (effects (font (size 1.27 1.27)) (justify left bottom))
+  )
+  (label "20V_{PGOOD}" (at 52.07 67.31 0) (fields_autoplaced)
+    (effects (font (size 1.27 1.27)) (justify left bottom))
+  )
   (label "VCC_{LM5156_20V}" (at 31.75 67.31 180) (fields_autoplaced)
     (effects (font (size 1.27 1.27)) (justify right bottom))
   )
-  (label "VCC_{LM5156_20V}" (at 107.95 44.45 0) (fields_autoplaced)
+  (label "20V_{BOOST}" (at 161.29 44.45 0) (fields_autoplaced)
     (effects (font (size 1.27 1.27)) (justify left bottom))
   )
+  (label "20V_{COMP-1}" (at 138.43 86.36 0) (fields_autoplaced)
+    (effects (font (size 1.27 1.27)) (justify left bottom))
+  )
+  (label "20V_{CS}" (at 109.22 59.69 0) (fields_autoplaced)
+    (effects (font (size 1.27 1.27)) (justify left bottom))
+  )
+  (label "20V_{SS}" (at 59.69 82.55 0) (fields_autoplaced)
+    (effects (font (size 1.27 1.27)) (justify left bottom))
+  )
+  (label "20V_{FB}" (at 109.22 67.31 0) (fields_autoplaced)
+    (effects (font (size 1.27 1.27)) (justify left bottom))
+  )
+  (label "20V_{GATE}" (at 109.22 52.07 0) (fields_autoplaced)
+    (effects (font (size 1.27 1.27)) (justify left bottom))
+  )
+  (label "20V_{VCC}" (at 109.22 44.45 0) (fields_autoplaced)
+    (effects (font (size 1.27 1.27)) (justify left bottom))
+  )
+  (label "20V_{RT}" (at 59.69 74.93 0) (fields_autoplaced)
+    (effects (font (size 1.27 1.27)) (justify left bottom))
+  )

Commit message: finish schematic features
Parts:
- added J8: Conn_01x02_Pin, Connector_PinHeader_2.54mm:PinHeader_1x02_P2.54mm_Vertical, symbol Connector:Conn_01x02_Pin
- added TP1, TP2, TP3, TP5, TP6, TP7: TestPoint, TestPoint:TestPoint_Loop_D2.54mm_Drill1.5mm_Beaded, symbol Connector:TestPoint
- renumbered C4 to C2, C6 to C3, C2 to C4, C3 to C5, C5 to C6, R4 to R1, R6 to R3, R1 to R4, R3 to R5, R7 to R6, R5 to R7, TP1 to TP4
Connections:
- net VCC_{LM5156_20V} is gone; now on net 20V_{VCC}: R4.2
- net +20V: now also J8.2 (Pin_2); no longer C3.1, D1.1 (K), R6.2
- net 20V_{BOOST}: now also TP1.1
- net 20V_{COMP}: now also TP6.1
- net 20V_{FB}: now also TP5.1
- net 20V_{GATE}: now also TP3.1
- net 20V_{UVLO}: now also TP2.1
- net GND: now also TP7.1
- new net 20V_{SENSE}: C3.1, D1.1 (K), J8.1 (Pin_1), R6.2
Other:
- company: (none) -> Paul Willis
- moved on the sheet: C2, R2

Commit message: ERC pass
Close look at pico iCE pinout
Add light sensor
Rough layout for non-HV
Parts:
- U5: renamed from U3; footprint 00_lib:PWP0014H-IPC_A -> 00_lib:PWP0014H-IPC_C
- renumbered C2 to C4, C3 to C5, C4 to C6, C5 to C7, C6 to C8, R8 to R10, R1 to R3, R2 to R4, R3 to R5, R4 to R6, R5 to R7, R6 to R8, R7 to R9

Commit message: DRC pass
it's messy
Parts:
- R5: footprint Resistor_SMD:R_0201_0603Metric -> Resistor_SMD:R_0603_1608Metric
Changed lines of the file:
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@@
       (effects (font (size 1.27 1.27)))
     )
-    (property "Footprint" "Resistor_SMD:R_0201_0603Metric" (at 161.798 66.04 90)
+    (property "Footprint" "Resistor_SMD:R_0603_1608Metric" (at 161.798 66.04 90)
       (effects (font (size 1.27 1.27)) hide)
     )

Commit message: Fill out BOM
Parts:
- C4, C7, C8: Price (none) -> 0.10
- C5: Price (none) -> 1.03
- C6: Model (none) -> CL10B104KB8NNWC; Price (none) -> 0.10
- D1: Model (none) -> SM4004; Price (none) -> 0.27
- J7: renamed from J8; Model (none) -> PH1-02-UA; Price (none) -> 0.10
- L1: Price (none) -> 0.41
- Q1: Model (none) -> BSP88; Price (none) -> 0.60
- R10: Model (none) -> RC0603JR-074K7L; Price (none) -> 0.10
- R3: Model (none) -> RMCF0603FT62K0; Price (none) -> 0.10
- R4: Model (none) -> RC0603FR-0727KL; Price (none) -> 0.10
- R5: Price (none) -> 0.74
- R6, R7, R8: Model (none) -> RC0603JR-07100KL; Price (none) -> 0.10
- R9: Model (none) -> RC0603JR-07470RL; Price (none) -> 0.10
- TP1, TP2, TP3, TP4, TP5, TP6, TP7: Price (none) -> 0.38
- U5: Model (none) -> LM51561HPWPR; Price (none) -> 2.18

Commit message: Add retailer links
Parts:
- C4, C6, C7, C8: Digikey link (none) -> https://www.digikey.com/en/products/detail/samsung-electro-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; Mouser link (none) -> https://www.mouser.com/ProductDetail/Samsung-Electro-Mechan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
- C5: Digikey link (none) -> https://www.digikey.com/en/products/detail/nichicon/UVC2G10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; Mouser link (none) -> https://www.mouser.com/ProductDetail/Nichicon/UVC2G100MPD1T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
- D1: Digikey link (none) -> https://www.digikey.com/en/products/detail/diotec-semicondu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; Mouser link (none) -> https://www.mouser.com/ProductDetail/Diotec-Semiconductor/S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
- J7: Digikey link (none) -> https://www.digikey.com/en/products/detail/adam-tech/PH1-02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; Mouser link (none) -> https://www.mouser.com/ProductDetail/Samtec/TSW-102-07-G-S?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
- L1: Digikey link (none) -> https://www.digikey.com/en/products/detail/tdk-corporation/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; Mouser link (none) -> https://www.mouser.com/ProductDetail/TDK/VLS6045EX-150M?qs=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
- Q1: Digikey link (none) -> https://www.digikey.com/en/products/detail/infineon-technol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; Mouser link (none) -> https://www.mouser.com/ProductDetail/Infineon-Technologies/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
- R10: Digikey link (none) -> https://www.digikey.com/en/products/detail/yageo/RC0603JR-0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; Mouser link (none) -> https://www.mouser.com/ProductDetail/YAGEO/RC0603JR-074K7L?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
- R3: Digikey link (none) -> https://www.digikey.com/en/products/detail/stackpole-electr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; Mouser link (none) -> https://www.mouser.com/ProductDetail/Panasonic/ERJ-3GEYJ623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
- R4: Digikey link (none) -> https://www.digikey.com/en/products/detail/yageo/RC0603FR-0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; Mouser link (none) -> https://www.mouser.com/ProductDetail/YAGEO/RC0603FR-0727KL?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
- R5: Digikey link (none) -> https://www.digikey.com/en/products/detail/vishay-dale/WSLP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; Mouser link (none) -> https://www.mouser.com/ProductDetail/Vishay-Dale/WSLP0603R0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
- R6, R7, R8: Digikey link (none) -> https://www.digikey.com/en/products/detail/yageo/RC0603JR-0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; Mouser link (none) -> https://www.mouser.com/ProductDetail/YAGEO/RC0603JR-07100KL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
- R9: Digikey link (none) -> https://www.digikey.com/en/products/detail/yageo/RC0603JR-0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; Mouser link (none) -> https://www.mouser.com/ProductDetail/YAGEO/RC0603JR-07470RL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
- TP1, TP2, TP3, TP4, TP5, TP6, TP7: Digikey link (none) -> https://www.digikey.com/en/products/detail/keystone-electro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; Mouser link (none) -> https://www.mouser.com/ProductDetail/Keystone-Electronics/5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
- U5: Digikey link (none) -> https://www.digikey.com/en/products/detail/texas-instrument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; Mouser link (none) -> https://www.mouser.com/ProductDetail/Texas-Instruments/LM51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
