File: KiCad/nixieAccurateClock/20V_supply.kicad_sch (KiCad schematic)
At the start: 25 parts, among them J7 Conn_01x02_Pin, Q1 BSP88, U5 LM51561HPWPR

Commit message: Switch to SMT test points
Parts:
- TP1, TP2, TP3, TP4, TP5, TP6, TP7: footprint TestPoint:TestPoint_Loop_D2.54mm_Drill1.5mm_Beaded -> 00_lib:TestPoint_Keystone_5019_Minature; Digikey link https://www.digikey.com/en/products/detail/keystone-electronics/5001/255327 -> https://www.digikey.com/en/products/detail/keystone-electronics/5019/3907343; Model 5001 -> 5019; Mouser link https://www.mouser.com/ProductDetail/Keystone-Electronics/5001?qs=q0tsjPZWdm%2FW0vdr%2FwowKg%3D%3D -> https://www.mouser.com/ProductDetail/Keystone-Electronics/5019?qs=wOxb8XianXjjCAsb90Ilzw%3D%3D; Price 0.38 -> 0.33

Commit message: switch to 27k R_anode
Add voltage rail jumpers for different 5V and 3.3V standby applications
Parts:
- added J8: Conn_01x02_Pin, Connector_PinHeader_2.54mm:PinHeader_1x02_P2.54mm_Vertical, symbol Connector:Conn_01x02_Pin
- renumbered J7 to J9
Connections:
- net +5V: now also J8.1 (Pin_1); no longer R3.2, U5.1 (BIAS)
- new net 5V_20V_{SENSE}: J8.2 (Pin_2), R3.2, U5.1 (BIAS)
Changed lines of the file:
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@@
   (junction (at 41.91 52.07) (diameter 0) (color 0 0 0 0)
   )
+  (junction (at 62.23 44.45) (diameter 0) (color 0 0 0 0)
+  )
   (junction (at 110.49 87.63) (diameter 0) (color 0 0 0 0)
   )
@@
   (junction (at 110.49 90.17) (diameter 0) (color 0 0 0 0)
   )
-  (junction (at 62.23 44.45) (diameter 0) (color 0 0 0 0)
-  )
   (junction (at 124.46 52.07) (diameter 0) (color 0 0 0 0)
   )
@@
     (stroke (width 0) (type default))
   )
+  (wire (pts (xy 44.45 44.45) (xy 62.23 44.45))
+    (stroke (width 0) (type default))
+  )
   (wire (pts (xy 107.95 87.63) (xy 110.49 87.63))
     (stroke (width 0) (type default))
@@
     (stroke (width 0) (type default))
   )
+  (wire (pts (xy 44.45 40.64) (xy 44.45 44.45))
+    (stroke (width 0) (type default))
+  )
   (wire (pts (xy 213.36 46.99) (xy 213.36 44.45))
     (stroke (width 0) (type default))
@@
     (stroke (width 0) (type default))
   )
+  (wire (pts (xy 41.91 44.45) (xy 41.91 40.64))
+    (stroke (width 0) (type default))
+  )
   (wire (pts (xy 160.02 59.69) (xy 160.02 57.15))
     (stroke (width 0) (type default))
@@
     (stroke (width 0) (type default))
   )
-  (wire (pts (xy 24.13 44.45) (xy 62.23 44.45))
-    (stroke (width 0) (type default))
-  )
   (wire (pts (xy 60.96 59.69) (xy 64.77 59.69))
     (stroke (width 0) (type default))
@@
   )
   (wire (pts (xy 107.95 44.45) (xy 113.03 44.45))
+    (stroke (width 0) (type default))
+  )
+  (wire (pts (xy 24.13 44.45) (xy 41.91 44.45))
     (stroke (width 0) (type default))
   )
@@
     (effects (font (size 1.27 1.27)) (justify left bottom))
   )
+  (label "5V_20V_{SENSE}" (at 46.99 44.45 0) (fields_autoplaced)
+    (effects (font (size 1.27 1.27)) (justify left bottom))
+  )
   (label "20V_{FB}" (at 109.22 67.31 0) (fields_autoplaced)
     (effects (font (size 1.27 1.27)) (justify left bottom))
@@
         (path "/55aab698-7558-4fe2-95ad-faa6da60ef89/33639105-1e30-4fa8-9335-500c2abdb54b"
           (reference "TP2") (unit 1)
+        )
+      )
+    )
+  )
+  (symbol (lib_id "Connector:Conn_01x02_Pin") (at 41.91 35.56 90) (mirror x) (unit 1)
+    (in_bom yes) (on_board yes) (dnp no)
+    (property "Reference" "J8" (at 45.72 37.465 90)
+      (effects (font (size 1.27 1.27)) (justify right))
+    )
+    (property "Value" "Conn_01x02_Pin" (at 45.72 34.925 90)
+      (effects (font (size 1.27 1.27)) (justify right))
+    )
+    (property "Footprint" "Connector_PinHeader_2.54mm:PinHeader_1x02_P2.54mm_Vertical" (at 41.91 35.56 0)
+      (effects (font (size 1.27 1.27)) hide)
+    )
+    (property "Datasheet" "https://app.adam-tech.com/products/download/data_sheet/201605/ph1-xx-ua-data-sheet.pdf" (at 41.91 35.56 0)
+      (effects (font (size 1.27 1.27)) hide)
+    )
+    (property "Sim.Enable" "0" (at 41.91 35.56 0)
+      (effects (font (size 1.27 1.27)) hide)
+    )
+    (property "Model" "PH1-02-UA" (at 41.91 35.56 0)
+      (effects (font (size 1.27 1.27)) hide)
+    )
+    (property "Price" "0.10" (at 41.91 35.56 0)
+      (effects (font (size 1.27 1.27)) hide)
+    )
+    (property "Digikey link" "https://www.digikey.com/en/products/detail/adam-tech/PH1-02-UA/9830266" (at 41.91 35.56 0)
+      (effects (font (size 1.27 1.27)) hide)
+    )
+    (property "Mouser link" "https://www.mouser.com/ProductDetail/Samtec/TSW-102-07-G-S?qs=iT52DjcXudsNPhlNCDp8vw%3D%3D" (at 41.91 35.56 0)
+      (effects (font (size 1.27 1.27)) hide)
+    )
+    (pin "1")
+    (pin "2")
+    (instances
+      (project "nixieAccurateClock"
+        (path "/55aab698-7558-4fe2-95ad-faa6da60ef89/f2852417-d6c8-4bbe-bd15-a29bc4083bd0"
+          (reference "J8") (unit 1)
+        )
+        (path "/55aab698-7558-4fe2-95ad-faa6da60ef89/33639105-1e30-4fa8-9335-500c2abdb54b"
+          (reference "J8") (unit 1)
         )
       )
@@
   (symbol (lib_id "Connector:Conn_01x02_Pin") (at 213.36 52.07 90) (unit 1)
     (in_bom yes) (on_board yes) (dnp no)
-    (property "Reference" "J7" (at 217.17 50.165 90)
+    (property "Reference" "J9" (at 217.17 50.165 90)
       (effects (font (size 1.27 1.27)) (justify right))
     )
@@
       (project "nixieAccurateClock"
         (path "/55aab698-7558-4fe2-95ad-faa6da60ef89/33639105-1e30-4fa8-9335-500c2abdb54b"
-          (reference "J7") (unit 1)
-        )
-      )
+          (reference "J9") (unit 1)
+        )
+      )

Commit message: clean up pico iCE traces
Parts:
- C5: footprint Capacitor_THT:CP_Radial_D10.0mm_P5.00mm -> Capacitor_SMD:CP_Elec_8x10; Digikey link https://www.digikey.com/en/products/detail/nichicon/UVC2G10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 -> https://www.digikey.com/en/products/detail/nichicon/ULR2E10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; Model UVC2G100MPD1TD -> ULR2E100MNL1GS; Mouser link https://www.mouser.com/ProductDetail/Nichicon/UVC2G100MPD1T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 -> https://www.mouser.com/ProductDetail/Nichicon/ULR2E100MNL1G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
Changed lines of the file:
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@@
       (effects (font (size 1.27 1.27)) (justify left))
     )
-    (property "Footprint" "Capacitor_THT:CP_Radial_D10.0mm_P5.00mm" (at 199.0852 55.88 0)
+    (property "Footprint" "Capacitor_SMD:CP_Elec_8x10" (at 199.0852 55.88 0)
       (effects (font (size 1.27 1.27)) hide)
     )
-    (property "Datasheet" "https://www.nichicon.co.jp/english/products/pdfs/e-uvc.pdf" (at 198.12 52.07 0)
+    (property "Datasheet" "https://www.nichicon.co.jp/english/series_items/catalog_pdf/e-ulr.pdf" (at 198.12 52.07 0)
       (effects (font (size 1.27 1.27)) hide)
     )
-    (property "Model" "UVC2G100MPD1TD" (at 198.12 52.07 0)
+    (property "Model" "ULR2E100MNL1GS" (at 198.12 52.07 0)
       (effects (font (size 1.27 1.27)) hide)
     )
@@
       (effects (font (size 1.27 1.27)) hide)
     )
-    (property "Digikey link" "https://www.digikey.com/en/products/detail/nichicon/UVC2G100MPD1TD/4312415" (at 198.12 52.07 0)
+    (property "Digikey link" "https://www.digikey.com/en/products/detail/nichicon/ULR2E100MNL1GS/3664123" (at 198.12 52.07 0)
       (effects (font (size 1.27 1.27)) hide)
     )
-    (property "Mouser link" "https://www.mouser.com/ProductDetail/Nichicon/UVC2G100MPD1TD?qs=dHDuPHwQO7%2FySlLjjH7nrA%3D%3D" (at 198.12 52.07 0)
+    (property "Mouser link" "https://www.mouser.com/ProductDetail/Nichicon/ULR2E100MNL1GS?qs=aoAypCcaRa8pBYU9738QBQ%3D%3D" (at 198.12 52.07 0)
       (effects (font (size 1.27 1.27)) hide)
     )

Commit message: clean up SMPS routing
Parts:
- removed TP4: TestPoint, 00_lib:TestPoint_Keystone_5019_Minature, symbol Connector:TestPoint
- renumbered TP5 to TP4, TP6 to TP5, TP7 to TP6
Changed lines of the file:
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@@
   (junction (at 124.46 52.07) (diameter 0) (color 0 0 0 0)
   )
-  (junction (at 41.91 67.31) (diameter 0) (color 0 0 0 0)
-  )
   (junction (at 124.46 74.93) (diameter 0) (color 0 0 0 0)
   )
@@
     (stroke (width 0) (type default))
   )
-  (wire (pts (xy 41.91 67.31) (xy 64.77 67.31))
-    (stroke (width 0) (type default))
-  )
   (wire (pts (xy 124.46 74.93) (xy 124.46 87.63))
     (stroke (width 0) (type default))
@@
     (stroke (width 0) (type default))
   )
-  (wire (pts (xy 40.64 67.31) (xy 41.91 67.31))
+  (wire (pts (xy 40.64 67.31) (xy 64.77 67.31))
     (stroke (width 0) (type default))
   )
@@
   )
   (wire (pts (xy 110.49 82.55) (xy 110.49 87.63))
-    (stroke (width 0) (type default))
-  )
-  (wire (pts (xy 41.91 64.77) (xy 41.91 67.31))
     (stroke (width 0) (type default))
   )
@@
         (path "/55aab698-7558-4fe2-95ad-faa6da60ef89/33639105-1e30-4fa8-9335-500c2abdb54b"
           (reference "#PWR035") (unit 1)
-        )
-      )
-    )
-  )
-  (symbol (lib_id "Connector:TestPoint") (at 41.91 64.77 0) (unit 1)
-    (in_bom yes) (on_board yes) (dnp no) (fields_autoplaced)
-    (property "Reference" "TP4" (at 44.45 60.198 0)
-      (effects (font (size 1.27 1.27)) (justify left))
-    )
-    (property "Value" "TestPoint" (at 44.45 62.738 0)
-      (effects (font (size 1.27 1.27)) (justify left))
-    )
-    (property "Footprint" "00_lib:TestPoint_Keystone_5019_Minature" (at 46.99 64.77 0)
-      (effects (font (size 1.27 1.27)) hide)
-    )
-    (property "Datasheet" "https://www.mouser.com/datasheet/2/215/019-743690.pdf" (at 46.99 64.77 0)
-      (effects (font (size 1.27 1.27)) hide)
-    )
-    (property "Model" "5019" (at 41.91 64.77 0)
-      (effects (font (size 1.27 1.27)) hide)
-    )
-    (property "Sim.Enable" "0" (at 41.91 64.77 0)
-      (effects (font (size 1.27 1.27)) hide)
-    )
-    (property "Price" "0.33" (at 41.91 64.77 0)
-      (effects (font (size 1.27 1.27)) hide)
-    )
-    (property "Digikey link" "https://www.digikey.com/en/products/detail/keystone-electronics/5019/3907343" (at 41.91 64.77 0)
-      (effects (font (size 1.27 1.27)) hide)
-    )
-    (property "Mouser link" "https://www.mouser.com/ProductDetail/Keystone-Electronics/5019?qs=wOxb8XianXjjCAsb90Ilzw%3D%3D" (at 41.91 64.77 0)
-      (effects (font (size 1.27 1.27)) hide)
-    )
-    (pin "1")
-    (instances
-      (project "nixieAccurateClock"
-        (path "/55aab698-7558-4fe2-95ad-faa6da60ef89/33639105-1e30-4fa8-9335-500c2abdb54b"
-          (reference "TP4") (unit 1)
         )
       )
@@
   (symbol (lib_id "Connector:TestPoint") (at 124.46 66.04 0) (unit 1)
     (in_bom yes) (on_board yes) (dnp no) (fields_autoplaced)
-    (property "Reference" "TP5" (at 127 61.468 0)
+    (property "Reference" "TP4" (at 127 61.468 0)
       (effects (font (size 1.27 1.27)) (justify left))
     )
@@
       (project "nixieAccurateClock"
         (path "/55aab698-7558-4fe2-95ad-faa6da60ef89/33639105-1e30-4fa8-9335-500c2abdb54b"
-          (reference "TP5") (unit 1)
+          (reference "TP4") (unit 1)
         )
       )
@@
   (symbol (lib_id "Connector:TestPoint") (at 223.52 101.6 0) (unit 1)
     (in_bom yes) (on_board yes) (dnp no) (fields_autoplaced)
-    (property "Reference" "TP7" (at 226.06 97.028 0)
+    (property "Reference" "TP6" (at 226.06 97.028 0)
       (effects (font (size 1.27 1.27)) (justify left))
     )
@@
       (project "nixieAccurateClock"
         (path "/55aab698-7558-4fe2-95ad-faa6da60ef89/33639105-1e30-4fa8-9335-500c2abdb54b"
-          (reference "TP7") (unit 1)
+          (reference "TP6") (unit 1)
         )
       )
@@
   (symbol (lib_id "Connector:TestPoint") (at 124.46 73.66 0) (unit 1)
     (in_bom yes) (on_board yes) (dnp no) (fields_autoplaced)
-    (property "Reference" "TP6" (at 127 69.088 0)
+    (property "Reference" "TP5" (at 127 69.088 0)
       (effects (font (size 1.27 1.27)) (justify left))
     )
@@
       (project "nixieAccurateClock"
         (path "/55aab698-7558-4fe2-95ad-faa6da60ef89/33639105-1e30-4fa8-9335-500c2abdb54b"
-          (reference "TP6") (unit 1)
-        )
-      )
+          (reference "TP5") (unit 1)
+        )
+      )

Commit message: inconsequential routing tweaks
Parts:
- renumbered J8 to J?
Changed lines of the file:
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@@
   (symbol (lib_id "Connector:Conn_01x02_Pin") (at 41.91 35.56 90) (mirror x) (unit 1)
     (in_bom yes) (on_board yes) (dnp no)
-    (property "Reference" "J8" (at 45.72 37.465 90)
+    (property "Reference" "J?" (at 45.72 37.465 90)
       (effects (font (size 1.27 1.27)) (justify right))
     )
@@
       (project "nixieAccurateClock"
         (path "/55aab698-7558-4fe2-95ad-faa6da60ef89/f2852417-d6c8-4bbe-bd15-a29bc4083bd0"
-          (reference "J8") (unit 1)
+          (reference "J?") (unit 1)
         )
         (path "/55aab698-7558-4fe2-95ad-faa6da60ef89/33639105-1e30-4fa8-9335-500c2abdb54b"
