File: KiCad/nixieAccurateClock/HV_bleed.kicad_sch (KiCad schematic)
At the start: 10 parts, among them Q3 BSP88, Q4 BSP88

Commit message: Add retailer links
Parts:
- C15: Digikey link (none) -> https://www.digikey.com/en/products/detail/samsung-electro-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; Mouser link (none) -> https://www.mouser.com/ProductDetail/Samsung-Electro-Mechan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
- D3: Digikey link (none) -> https://www.digikey.com/en/products/detail/diotec-semicondu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; Mouser link (none) -> https://www.mouser.com/ProductDetail/Diotec-Semiconductor/S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
- Q3, Q4: Digikey link (none) -> https://www.digikey.com/en/products/detail/infineon-technol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; Mouser link (none) -> https://www.mouser.com/ProductDetail/Infineon-Technologies/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
- R24: Digikey link (none) -> https://www.digikey.com/en/products/detail/stackpole-electr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; Mouser link (none) -> https://www.mouser.com/ProductDetail/SEI-Stackpole/RMCF0603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
- R25: Digikey link (none) -> https://www.digikey.com/en/products/detail/te-connectivity-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; Mouser link (none) -> https://www.mouser.com/ProductDetail/TE-Connectivity-Holswo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
- R26: Digikey link (none) -> https://www.digikey.com/en/products/detail/yageo/RC0603JR-0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; Mouser link (none) -> https://www.mouser.com/ProductDetail/YAGEO/RC0603JR-07100KL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
- TP14, TP15, TP16: Digikey link (none) -> https://www.digikey.com/en/products/detail/keystone-electro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; Mouser link (none) -> https://www.mouser.com/ProductDetail/Keystone-Electronics/5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
Changed lines of the file:
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@@
+      (effects (font (size 1.27 1.27)) hide)
+    )
+    (property "Digikey link" "https://www.digikey.com/en/products/detail/infineon-technologies/BSP88H6327XTSA1/5959955" (at 92.71 68.58 0)
+      (effects (font (size 1.27 1.27)) hide)
+    )
+    (property "Mouser link" "https://www.mouser.com/ProductDetail/Infineon-Technologies/BSP88H6327XTSA1?qs=LqwxS8kK3AsxJVC%2FVRfDmg%3D%3D" (at 92.71 68.58 0)
       (effects (font (size 1.27 1.27)) hide)
     )
@@
       (effects (font (size 1.27 1.27)) hide)
     )
+    (property "Digikey link" "https://www.digikey.com/en/products/detail/yageo/RC0603JR-07100KL/726698" (at 106.68 85.09 0)
+      (effects (font (size 1.27 1.27)) hide)
+    )
+    (property "Mouser link" "https://www.mouser.com/ProductDetail/YAGEO/RC0603JR-07100KL?qs=2cAdsCoAWRG9Rhqklpdeqg%3D%3D" (at 106.68 85.09 0)
+      (effects (font (size 1.27 1.27)) hide)
+    )
     (pin "1")
     (pin "2")
@@
       (effects (font (size 1.27 1.27)) hide)
     )
+    (property "Digikey link" "https://www.digikey.com/en/products/detail/keystone-electronics/5001/255327" (at 66.04 68.58 0)
+      (effects (font (size 1.27 1.27)) hide)
+    )
+    (property "Mouser link" "https://www.mouser.com/ProductDetail/Keystone-Electronics/5001?qs=q0tsjPZWdm%2FW0vdr%2FwowKg%3D%3D" (at 66.04 68.58 0)
+      (effects (font (size 1.27 1.27)) hide)
+    )
     (pin "1")
     (instances
@@
     )
     (property "Price" "0.60" (at 95.25 50.8 0)
+      (effects (font (size 1.27 1.27)) hide)
+    )
+    (property "Digikey link" "https://www.digikey.com/en/products/detail/te-connectivity-passive-product/ROX5SSJ10K/9926250" (at 95.25 50.8 0)
+      (effects (font (size 1.27 1.27)) hide)
+    )
+    (property "Mouser link" "https://www.mouser.com/ProductDetail/TE-Connectivity-Holsworthy/ROX5SSJ10K?qs=gZXFycFWdAPK2TCKEiyMYg%3D%3D" (at 95.25 50.8 0)
       (effects (font (size 1.27 1.27)) hide)
     )
@@
       (effects (font (size 1.27 1.27)) hide)
     )
+    (property "Digikey link" "https://www.digikey.com/en/products/detail/infineon-technologies/BSP88H6327XTSA1/5959955" (at 67.31 77.47 0)
+      (effects (font (size 1.27 1.27)) hide)
+    )
+    (property "Mouser link" "https://www.mouser.com/ProductDetail/Infineon-Technologies/BSP88H6327XTSA1?qs=LqwxS8kK3AsxJVC%2FVRfDmg%3D%3D" (at 67.31 77.47 0)
+      (effects (font (size 1.27 1.27)) hide)
+    )
     (pin "1")
     (pin "3")
@@
     )
     (property "Price" "0.10" (at 95.25 85.09 0)
+      (effects (font (size 1.27 1.27)) hide)
+    )
+    (property "Digikey link" "https://www.digikey.com/en/products/detail/samsung-electro-mechanics/CL10A105KA8NNNC/3886760" (at 95.25 85.09 0)
+      (effects (font (size 1.27 1.27)) hide)
+    )
+    (property "Mouser link" "https://www.mouser.com/ProductDetail/Samsung-Electro-Mechanics/CL10A105KA8NNNC?qs=hqM3L16%252BxldY%252BnK4KzDJVg%3D%3D" (at 95.25 85.09 0)
       (effects (font (size 1.27 1.27)) hide)
     )
@@
       (effects (font (size 1.27 1.27)) hide)
     )
+    (property "Digikey link" "https://www.digikey.com/en/products/detail/keystone-electronics/5001/255327" (at 90.17 77.47 0)
+      (effects (font (size 1.27 1.27)) hide)
+    )
+    (property "Mouser link" "https://www.mouser.com/ProductDetail/Keystone-Electronics/5001?qs=q0tsjPZWdm%2FW0vdr%2FwowKg%3D%3D" (at 90.17 77.47 0)
+      (effects (font (size 1.27 1.27)) hide)
+    )
     (pin "1")
     (instances
@@
       (effects (font (size 1.27 1.27)) hide)
     )
+    (property "Digikey link" "https://www.digikey.com/en/products/detail/stackpole-electronics-inc/RMCF0603FT1M00/1761036" (at 69.85 50.8 0)
+      (effects (font (size 1.27 1.27)) hide)
+    )
+    (property "Mouser link" "https://www.mouser.com/ProductDetail/SEI-Stackpole/RMCF0603FT1M00?qs=FESYatJ8odJNClY0wUC1cg%3D%3D" (at 69.85 50.8 0)
+      (effects (font (size 1.27 1.27)) hide)
+    )
     (pin "1")
     (pin "2")
@@
     )
     (property "Price" "0.27" (at 69.85 60.96 0)
+      (effects (font (size 1.27 1.27)) hide)
+    )
+    (property "Digikey link" "https://www.digikey.com/en/products/detail/diotec-semiconductor/SM4004/13155357" (at 69.85 60.96 0)
+      (effects (font (size 1.27 1.27)) hide)
+    )
+    (property "Mouser link" "https://www.mouser.com/ProductDetail/Diotec-Semiconductor/SM4004?qs=OlC7AqGiEDkXkiBPoivHAA%3D%3D" (at 69.85 60.96 0)
       (effects (font (size 1.27 1.27)) hide)
     )
@@
       (effects (font (size 1.27 1.27)) hide)
     )
+    (property "Digikey link" "https://www.digikey.com/en/products/detail/keystone-electronics/5001/255327" (at 90.17 58.42 0)
+      (effects (font (size 1.27 1.27)) hide)
+    )
+    (property "Mouser link" "https://www.mouser.com/ProductDetail/Keystone-Electronics/5001?qs=q0tsjPZWdm%2FW0vdr%2FwowKg%3D%3D" (at 90.17 58.42 0)
+      (effects (font (size 1.27 1.27)) hide)
+    )

Commit message: swap bleed resistor for SMD
Parts:
- R25: footprint Resistor_THT:R_Axial_DIN0617_L17.0mm_D6.0mm_P20.32mm_Horizontal -> Resistor_SMD:R_2512_6332Metric; Digikey link https://www.digikey.com/en/products/detail/te-connectivity-passive-product/ROX5SSJ10K/9926250 -> https://www.digikey.com/en/products/detail/te-connectivity-passive-product/352010KJT/2364839; Model ROX5SSJ10K -> 352010KJT; Mouser link https://www.mouser.com/ProductDetail/TE-Connectivity-Holsworthy/ROX5SSJ10K?qs=gZXFycFWdAPK2TCKEiyMYg%3D%3D -> https://www.mouser.com/ProductDetail/TE-Connectivity-Holsworthy/352010KJT?qs=DDevMFOh4ssnVH2d0oCe7g%3D%3D; Price 0.60 -> 0.43
Changed lines of the file:
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@@
       (effects (font (size 1.27 1.27)) (justify left))
     )
-    (property "Footprint" "Resistor_THT:R_Axial_DIN0617_L17.0mm_D6.0mm_P20.32mm_Horizontal" (at 93.472 50.8 90)
+    (property "Footprint" "Resistor_SMD:R_2512_6332Metric" (at 93.472 50.8 90)
       (effects (font (size 1.27 1.27)) hide)
     )
-    (property "Datasheet" "https://www.te.com/usa-en/product-8-2176412-0.datasheet.pdf" (at 95.25 50.8 0)
+    (property "Datasheet" "https://www.te.com/commerce/DocumentDelivery/DDEController?Action=srchrtrv&DocNm=1773139&DocType=DS&DocLang=English" (at 95.25 50.8 0)
       (effects (font (size 1.27 1.27)) hide)
     )
-    (property "Sim.Enable" "0" (at 95.25 50.8 0)
+    (property "Model" "352010KJT" (at 95.25 50.8 0)
       (effects (font (size 1.27 1.27)) hide)
     )
-    (property "Model" "ROX5SSJ10K" (at 95.25 50.8 0)
+    (property "Price" "0.43" (at 95.25 50.8 0)
       (effects (font (size 1.27 1.27)) hide)
     )
-    (property "Price" "0.60" (at 95.25 50.8 0)
+    (property "Digikey link" "https://www.digikey.com/en/products/detail/te-connectivity-passive-product/352010KJT/2364839" (at 95.25 50.8 0)
       (effects (font (size 1.27 1.27)) hide)
     )
-    (property "Digikey link" "https://www.digikey.com/en/products/detail/te-connectivity-passive-product/ROX5SSJ10K/9926250" (at 95.25 50.8 0)
+    (property "Mouser link" "https://www.mouser.com/ProductDetail/TE-Connectivity-Holsworthy/352010KJT?qs=DDevMFOh4ssnVH2d0oCe7g%3D%3D" (at 95.25 50.8 0)
       (effects (font (size 1.27 1.27)) hide)
     )
-    (property "Mouser link" "https://www.mouser.com/ProductDetail/TE-Connectivity-Holsworthy/ROX5SSJ10K?qs=gZXFycFWdAPK2TCKEiyMYg%3D%3D" (at 95.25 50.8 0)
-      (effects (font (size 1.27 1.27)) hide)
-    )

Commit message: Switch to SMT test points
Parts:
- TP14, TP15, TP16: footprint TestPoint:TestPoint_Loop_D2.54mm_Drill1.5mm_Beaded -> 00_lib:TestPoint_Keystone_5019_Minature; Digikey link https://www.digikey.com/en/products/detail/keystone-electronics/5001/255327 -> https://www.digikey.com/en/products/detail/keystone-electronics/5019/3907343; Model 5001 -> 5019; Mouser link https://www.mouser.com/ProductDetail/Keystone-Electronics/5001?qs=q0tsjPZWdm%2FW0vdr%2FwowKg%3D%3D -> https://www.mouser.com/ProductDetail/Keystone-Electronics/5019?qs=wOxb8XianXjjCAsb90Ilzw%3D%3D; Price 0.38 -> 0.33
Changed lines of the file:
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@@
       (effects (font (size 1.27 1.27)))
     )
-    (property "Footprint" "TestPoint:TestPoint_Loop_D2.54mm_Drill1.5mm_Beaded" (at 66.04 63.5 0)
-      (effects (font (size 1.27 1.27)) hide)
-    )
-    (property "Datasheet" "https://www.keyelco.com/userAssets/file/M65p56.pdf" (at 66.04 63.5 0)
-      (effects (font (size 1.27 1.27)) hide)
-    )
-    (property "Model" "5001" (at 66.04 68.58 0)
+    (property "Footprint" "00_lib:TestPoint_Keystone_5019_Minature" (at 66.04 63.5 0)
+      (effects (font (size 1.27 1.27)) hide)
+    )
+    (property "Datasheet" "https://www.mouser.com/datasheet/2/215/019-743690.pdf" (at 66.04 63.5 0)
+      (effects (font (size 1.27 1.27)) hide)
+    )
+    (property "Model" "5019" (at 66.04 68.58 0)
       (effects (font (size 1.27 1.27)) hide)
     )
@@
       (effects (font (size 1.27 1.27)) hide)
     )
-    (property "Price" "0.38" (at 66.04 68.58 0)
-      (effects (font (size 1.27 1.27)) hide)
-    )
-    (property "Digikey link" "https://www.digikey.com/en/products/detail/keystone-electronics/5001/255327" (at 66.04 68.58 0)
-      (effects (font (size 1.27 1.27)) hide)
-    )
-    (property "Mouser link" "https://www.mouser.com/ProductDetail/Keystone-Electronics/5001?qs=q0tsjPZWdm%2FW0vdr%2FwowKg%3D%3D" (at 66.04 68.58 0)
+    (property "Price" "0.33" (at 66.04 68.58 0)
+      (effects (font (size 1.27 1.27)) hide)
+    )
+    (property "Digikey link" "https://www.digikey.com/en/products/detail/keystone-electronics/5019/3907343" (at 66.04 68.58 0)
+      (effects (font (size 1.27 1.27)) hide)
+    )
+    (property "Mouser link" "https://www.mouser.com/ProductDetail/Keystone-Electronics/5019?qs=wOxb8XianXjjCAsb90Ilzw%3D%3D" (at 66.04 68.58 0)
       (effects (font (size 1.27 1.27)) hide)
     )
@@
       (effects (font (size 1.27 1.27)))
     )
-    (property "Footprint" "TestPoint:TestPoint_Loop_D2.54mm_Drill1.5mm_Beaded" (at 90.17 82.55 0)
-      (effects (font (size 1.27 1.27)) hide)
-    )
-    (property "Datasheet" "https://www.keyelco.com/userAssets/file/M65p56.pdf" (at 90.17 82.55 0)
-      (effects (font (size 1.27 1.27)) hide)
-    )
-    (property "Model" "5001" (at 90.17 77.47 0)
+    (property "Footprint" "00_lib:TestPoint_Keystone_5019_Minature" (at 90.17 82.55 0)
+      (effects (font (size 1.27 1.27)) hide)
+    )
+    (property "Datasheet" "https://www.mouser.com/datasheet/2/215/019-743690.pdf" (at 90.17 82.55 0)
+      (effects (font (size 1.27 1.27)) hide)
+    )
+    (property "Model" "5019" (at 90.17 77.47 0)
       (effects (font (size 1.27 1.27)) hide)
     )
@@
       (effects (font (size 1.27 1.27)) hide)
     )
-    (property "Price" "0.38" (at 90.17 77.47 0)
-      (effects (font (size 1.27 1.27)) hide)
-    )
-    (property "Digikey link" "https://www.digikey.com/en/products/detail/keystone-electronics/5001/255327" (at 90.17 77.47 0)
-      (effects (font (size 1.27 1.27)) hide)
-    )
-    (property "Mouser link" "https://www.mouser.com/ProductDetail/Keystone-Electronics/5001?qs=q0tsjPZWdm%2FW0vdr%2FwowKg%3D%3D" (at 90.17 77.47 0)
+    (property "Price" "0.33" (at 90.17 77.47 0)
+      (effects (font (size 1.27 1.27)) hide)
+    )
+    (property "Digikey link" "https://www.digikey.com/en/products/detail/keystone-electronics/5019/3907343" (at 90.17 77.47 0)
+      (effects (font (size 1.27 1.27)) hide)
+    )
+    (property "Mouser link" "https://www.mouser.com/ProductDetail/Keystone-Electronics/5019?qs=wOxb8XianXjjCAsb90Ilzw%3D%3D" (at 90.17 77.47 0)
       (effects (font (size 1.27 1.27)) hide)
     )
@@
       (effects (font (size 1.27 1.27)))
     )
-    (property "Footprint" "TestPoint:TestPoint_Loop_D2.54mm_Drill1.5mm_Beaded" (at 90.17 63.5 0)
-      (effects (font (size 1.27 1.27)) hide)
-    )
-    (property "Datasheet" "https://www.keyelco.com/userAssets/file/M65p56.pdf" (at 90.17 63.5 0)
-      (effects (font (size 1.27 1.27)) hide)
-    )
-    (property "Model" "5001" (at 90.17 58.42 0)
+    (property "Footprint" "00_lib:TestPoint_Keystone_5019_Minature" (at 90.17 63.5 0)
+      (effects (font (size 1.27 1.27)) hide)
+    )
+    (property "Datasheet" "https://www.mouser.com/datasheet/2/215/019-743690.pdf" (at 90.17 63.5 0)
+      (effects (font (size 1.27 1.27)) hide)
+    )
+    (property "Model" "5019" (at 90.17 58.42 0)
       (effects (font (size 1.27 1.27)) hide)
     )
@@
       (effects (font (size 1.27 1.27)) hide)
     )
-    (property "Price" "0.38" (at 90.17 58.42 0)
-      (effects (font (size 1.27 1.27)) hide)
-    )
-    (property "Digikey link" "https://www.digikey.com/en/products/detail/keystone-electronics/5001/255327" (at 90.17 58.42 0)
-      (effects (font (size 1.27 1.27)) hide)
-    )
-    (property "Mouser link" "https://www.mouser.com/ProductDetail/Keystone-Electronics/5001?qs=q0tsjPZWdm%2FW0vdr%2FwowKg%3D%3D" (at 90.17 58.42 0)
-      (effects (font (size 1.27 1.27)) hide)
-    )
+    (property "Price" "0.33" (at 90.17 58.42 0)
+      (effects (font (size 1.27 1.27)) hide)
+    )
+    (property "Digikey link" "https://www.digikey.com/en/products/detail/keystone-electronics/5019/3907343" (at 90.17 58.42 0)
+      (effects (font (size 1.27 1.27)) hide)
+    )
+    (property "Mouser link" "https://www.mouser.com/ProductDetail/Keystone-Electronics/5019?qs=wOxb8XianXjjCAsb90Ilzw%3D%3D" (at 90.17 58.42 0)
+      (effects (font (size 1.27 1.27)) hide)
+    )

Commit message: clean up SMPS routing
Parts:
- renumbered TP14 to TP11, TP15 to TP12, TP16 to TP13
Changed lines of the file:
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@@
   (symbol (lib_id "Connector:TestPoint") (at 66.04 68.58 90) (unit 1)
     (in_bom yes) (on_board yes) (dnp no) (fields_autoplaced)
-    (property "Reference" "TP15" (at 62.738 63.5 90)
+    (property "Reference" "TP12" (at 62.738 63.5 90)
       (effects (font (size 1.27 1.27)))
     )
@@
       (project "nixieAccurateClock"
         (path "/55aab698-7558-4fe2-95ad-faa6da60ef89/21095f53-01f6-40ea-bb6b-e8b09c532104"
-          (reference "TP15") (unit 1)
+          (reference "TP12") (unit 1)
         )
       )
@@
   (symbol (lib_id "Connector:TestPoint") (at 90.17 77.47 90) (mirror x) (unit 1)
     (in_bom yes) (on_board yes) (dnp no)
-    (property "Reference" "TP16" (at 86.868 82.4284 90)
+    (property "Reference" "TP13" (at 86.868 82.4284 90)
       (effects (font (size 1.27 1.27)))
     )
@@
       (project "nixieAccurateClock"
         (path "/55aab698-7558-4fe2-95ad-faa6da60ef89/21095f53-01f6-40ea-bb6b-e8b09c532104"
-          (reference "TP16") (unit 1)
+          (reference "TP13") (unit 1)
         )
       )
@@
   (symbol (lib_id "Connector:TestPoint") (at 90.17 58.42 90) (mirror x) (unit 1)
     (in_bom yes) (on_board yes) (dnp no)
-    (property "Reference" "TP14" (at 86.868 63.5 90)
+    (property "Reference" "TP11" (at 86.868 63.5 90)
       (effects (font (size 1.27 1.27)))
     )
@@
       (project "nixieAccurateClock"
         (path "/55aab698-7558-4fe2-95ad-faa6da60ef89/21095f53-01f6-40ea-bb6b-e8b09c532104"
-          (reference "TP14") (unit 1)
-        )
-      )
+          (reference "TP11") (unit 1)
+        )
+      )
