File: KiCad/nixieAccurateClock/nixieAccurateClock-rounded.kicad_pcb (KiCad board)
At the start: 4 copper layers, 152.4 x 101.6 mm, 114 parts, among them J1 Conn_01x02_Pin, J10 Conn_01x02_Pin, J11 Conn_02x05_Odd_Even, J2 Conn_01x02_Pin, J3 Conn_01x02_Pin, J4 Conn_01x02_Pin, J5 Conn_01x02_Pin, J6 Conn_Coaxial, J7 Conn_01x02_Pin, J8 Conn_01x02_Pin, J9 Conn_01x02_Pin, Q1 BSP88, Q2 BSP88, Q3 BSP88, Q4 BSP88, Q5 BSP88, SW1 SW_DIP_x08, U1 MCP23008-xSO, U13 ADC0820BCWMX, U14 TXB0108PWR, U15 TXB0108PWR, U2 pico iCE, U3 LTR-329ALS-01, U4 PX1125T, U5 LM51561HPWPR, U6 LM51561HPWPR

Commit message: some trace cleanup
Routing:
- net CLOCK_{HV}: track 243.2 -> 245.8 mm
- net PPS_{TRIMMED}: track 224.6 -> 225.9 mm
- net /DST_force: track 6.99 -> 6.13 mm
- net /24h_mode: track 5.28 -> 4.45 mm
- net /Nixies/DAISY_{HV-2}: track 32.3 -> 33.0 mm
- net /Nixies/DAISY_{HV-1}: track 27.9 -> 28.6 mm
- net /RESERVED_2: track 6.57 -> 7.22 mm

Commit message: change I2C pins
Avoid conflict with RP2040/iCE UART
Parts:
- moved R1 0.19 mm to (116.0, 65.7)
Connections:
- U2 pad 45: I2C_{CLOCK} -> unconnected-(U2-ICE_25/RP_1-Pad45)
- U2 pad 46: unconnected-(U2-ICE_23/RP_5-Pad46) -> I2C_{CLOCK}
- U2 pad 49: I2C_{DATA} -> unconnected-(U2-ICE_27/RP_0-Pad49)
- U2 pad 50: unconnected-(U2-ICE_26/RP_4-Pad50) -> I2C_{DATA}
Routing:
- net I2C_{CLOCK}: track 76.8 -> 73.2 mm
- net I2C_{DATA}: track 81.3 -> 78.8 mm
