File: KiCad/nixieAccurateClock/IN-14-daughter/IN-14-daughter.kicad_pcb (KiCad board)
At the start: 2 copper layers, 22.5 x 29.8 mm, 6 parts, among them J1 Conn_02x11_Top_Bottom, U1 HV509K6-G

Commit message: WIP final feature push
Routing:
- net /N_LHDP: track 48.3 -> 45.6 mm
- net /N_2: track 19.3 -> 20.7 mm
- net /N_3: track 14.7 -> 16.0 mm
- net /~{LATCH}: track 37.8 -> 38.6 mm, vias 0 -> 1
- net /~{POLARITY}: track 31.6 -> 31.9 mm, vias 0 -> 1
- added copper zone on In1.Cu, net GND
- added copper zone on In2.Cu, net GND
Other:
- copper layers 2 -> 4

Commit message: reroute daughter board
Swapped standoffs and pin header orientation on IN-14 daughter board so that standoffs face outward.  This allows using the daughter board mounting for the mother board mounting.
Parts:
- J1: value Conn_02x11_Top_Bottom -> Conn_02x11_Odd_Even
- moved H2 35.9 mm to (15.5, 3.50)
- moved N1 34.2 mm to (9.50, 14.0), turned to 0 degrees
- moved U1 34.2 mm to (9.50, 14.0), turned to -45 degrees
- moved J1 33.7 mm to (3.12, 26.0)
- moved H1 32.7 mm to (3.50, 3.50)
- moved R1 32.2 mm to (9.50, 23.0), turned to 0 degrees
Connections:
- J1 pad 1: VPP -> /N_7
- J1 pad 10: /N_1 -> +5V
- J1 pad 11: /N_6 -> /ANODE
- J1 pad 12: /~{LATCH} -> VPP
- J1 pad 13: /N_7 -> /N_LHDP
- J1 pad 14: /DOUT -> /HVGND
- J1 pad 15: /N_8 -> /N_1
- J1 pad 16: /ANODE -> /DIN
- J1 pad 17: /N_9 -> /N_2
- J1 pad 18: /N_LHDP -> /CLOCK
- J1 pad 19: /N_0 -> /N_3
- J1 pad 2: /DIN -> /N_6
- J1 pad 20: /N_RHDP -> +3.3V
- J1 pad 21: /HVGND -> /N_4
- J1 pad 22: +5V -> /N_5
- J1 pad 3: /N_2 -> /N_8
- J1 pad 4: /CLOCK -> /~{POLARITY}
- J1 pad 5: /N_3 -> /N_9
- J1 pad 6: +3.3V -> /~{LATCH}
- J1 pad 7: /N_4 -> /N_0
- J1 pad 8: /~{POLARITY} -> /DOUT
- J1 pad 9: /N_5 -> /N_RHDP
Routing:
- net /ANODE: track 49.3 -> 7.59 mm, vias 1 -> 0
- net /N_LHDP: track 45.6 -> 16.7 mm
- net /N_RHDP: track 35.7 -> 12.6 mm, vias 1 -> 0
- net /N_5: track 9.89 -> 32.6 mm
- net /N_6: track 10.2 -> 31.0 mm
- net /N_1: track 38.6 -> 18.1 mm
- net VPP: track 11.7 -> 29.4 mm, vias 1 -> 0
- net /DOUT: track 40.6 -> 26.1 mm, vias 1 -> 2
- net /N_4: track 11.9 -> 24.8 mm
- net /~{LATCH}: track 38.6 -> 26.1 mm
- net /N_7: track 11.6 -> 23.7 mm
- net /ANODE_DRIVE: track 18.2 -> 7.72 mm, vias 2 -> 0
- net +3.3V: track 27.3 -> 17.8 mm
- net /N_0: track 21.9 -> 13.2 mm
- net /DIN: track 16.9 -> 23.7 mm
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Other:
- board size 22.5 x 29.8 mm -> 19 x 29.5 mm

Commit message: fix daughter board HV compat
Increase copper weight on IN-14 daughter board to PCBWay's 4 layer 2 oz outer / 1.5 oz inner stackup.  This has a 0.22 mm prepreg rather than 0.11 mm prepreg, which helps maintain 200 V clearance (0.2 mm inner, 0.4 mm outer)
Routing:
- net /DOUT: track 26.1 -> 23.8 mm
- net /ANODE_DRIVE: track 7.72 -> 8.89 mm
- net +5V: track 27.6 -> 26.4 mm
- net /N_LHDP: track 16.7 -> 16.1 mm
- net /~{LATCH}: track 26.1 -> 26.4 mm, vias 1 -> 2
Other:
- board text added: "Rev A"

Commit message: simplify nixie daughter board
Remove cathode pins that would not be usable for current sensing anyway.
Pivot to using anode pin as shunt measurement with a R2R flash ADC (not yet implemented).
Parts:
- added REF**: Symbol_Highvoltage_Type1_CopperTop_Small, Symbol:Symbol_Highvoltage_Type1_CopperTop_Small, F.Cu at (16.5, 25.2)
- J1: value Conn_02x11_Odd_Even -> Conn_02x05_Odd_Even; footprint Connector_PinHeader_1.27mm:PinHeader_2x11_P1.27mm_Vertical -> Connector_PinHeader_2.54mm:PinHeader_2x05_P2.54mm_Vertical
- moved R1 3.46 mm to (13.0, 23.0), turned to 180 degrees
- moved J1 1.16 mm to (4.25, 26.2)
Connections:
- J1 pad 1: /N_7 -> /DOUT
- J1 pad 10: +5V -> GND
- J1 pad 2: /N_6 -> +5V
- J1 pad 3: /N_8 -> /~{LATCH}
- J1 pad 4: /~{POLARITY} -> /DIN
- J1 pad 5: /N_9 -> GND
- J1 pad 6: /~{LATCH} -> +3.3V
- J1 pad 7: /N_0 -> /ANODE
- J1 pad 8: /DOUT -> /CLOCK
- J1 pad 9: /N_RHDP -> VPP
- R1 pad 1: /ANODE_DRIVE -> VPP
- U1 pad 21: /~{POLARITY} -> GND
- U1 pad 27: /HVGND -> unconnected-(U1-HVGND-Pad27)
- U1 pad 28: /ANODE_DRIVE -> unconnected-(U1-BP-Pad28)
Routing:
- net /~{POLARITY}: track 28.3 -> 0.00 mm, vias 1 -> 0
- net /N_5: track 32.6 -> 6.15 mm
- net /N_6: track 31.0 -> 5.34 mm
- net /HVGND: track 23.3 -> 0.00 mm
- net /N_4: track 24.8 -> 5.28 mm
- net /N_7: track 23.7 -> 4.41 mm
- net /N_3: track 21.9 -> 6.04 mm
- net /N_8: track 19.2 -> 3.53 mm
- net /~{LATCH}: track 26.4 -> 12.9 mm, vias 2 -> 1
- net VPP: track 29.4 -> 16.3 mm
- net /N_2: track 20.0 -> 7.52 mm, vias 0 -> 1
- net /N_9: track 15.5 -> 3.29 mm
- net /DOUT: track 23.8 -> 12.7 mm, vias 2 -> 1
- net /N_1: track 18.1 -> 8.55 mm
- net /N_0: track 13.2 -> 3.71 mm
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Other:
- board size 19 x 29.5 mm -> 19 x 32 mm
- board text added: "IN-14 daughter board Rev A"
- board text removed: "Rev A"

Commit message: fix clearance rules on daughter board
0.4 mm clearance is not possible to obey with an HV driver IC package that has 0.25 mm pad spacing, but all HV lines can be kept at least 0.25 mm away from everything else and inner layers can be preferentially used.

WIP ADC interface, logic level convertor has been chosen.
Routing:
- net /N_4: track 5.28 -> 10.7 mm, vias 0 -> 1
- net /N_1: track 8.55 -> 13.1 mm, vias 0 -> 2
- net /DIN: track 29.6 -> 34.0 mm
- net /N_3: track 6.04 -> 10.1 mm, vias 0 -> 1
- net VPP: track 16.3 -> 17.4 mm, vias 0 -> 2
- net /N_2: track 7.52 -> 8.53 mm

Commit message: Add decoupling caps
Parts:
- added C1: 0.1u, Capacitor_SMD:C_0603_1608Metric, B.Cu at (17.8, 23.5)
- added C2: 0.1u, Capacitor_SMD:C_0603_1608Metric, B.Cu at (1.91, 20.3)
Connections:
- net /CLOCK renamed /CLK
- net /~{LATCH} renamed /~{LE}
- U1 pad 20: +3.3V -> /VDD
- U1 pad 26: +5V -> /VBIAS
Routing:
- net /VDD: track 0.00 -> 10.9 mm, vias 0 -> 2
- net +3.3V: track 25.1 -> 14.7 mm, vias 1 -> 0
- net +5V: track 18.6 -> 9.54 mm, vias 1 -> 0
- net /VBIAS: track 0.00 -> 9.05 mm, vias 0 -> 2

Commit message: clean up decoupling caps
Parts:
- moved C1 4.49 mm to (17.1, 19.1), turned to 0 degrees
- moved C2 0.85 mm to (2.25, 19.5), turned to 180 degrees
Routing:
- net +3.3V: track 14.7 -> 20.0 mm
- net /VDD: track 10.9 -> 6.97 mm, vias 2 -> 0
- net /VBIAS: track 9.05 -> 7.13 mm, vias 2 -> 0
- net +5V: track 9.54 -> 11.3 mm
- net /N_2: track 8.53 -> 7.94 mm
- net /N_RHDP: track 5.30 -> 5.06 mm, vias 0 -> 1
- net GND: vias 0 -> 2
