File: KiCad/nixieAccurateClock/IN-14-daughter/IN-14-daughter.kicad_pcb (KiCad board)
At the start: 4 copper layers, 19 x 32 mm, 12 parts, among them J1 Conn_02x05_Odd_Even, U1 HV509K6-G

Commit message: clean up IN-14 teardrops
Routing:
- net /DIN: track 33.7 -> 34.6 mm
- net +3.3V: track 19.9 -> 20.6 mm
- net /CLK: track 24.5 -> 25.2 mm

Commit message: round tracks plugin
Parts:
- moved C1 15.9 mm to (48.9, 34.9)
- moved C2 15.9 mm to (34.0, 35.4)
- moved FID1 15.9 mm to (33.0, 46.6)
- moved FID2 15.9 mm to (49.5, 46.6)
- moved FID3 15.9 mm to (41.2, 17.1)
- moved H1 15.9 mm to (35.2, 19.4)
- moved H2 15.9 mm to (47.2, 19.4)
- moved J1 15.9 mm to (36.0, 42.1)
- moved N1 15.9 mm to (41.2, 29.9)
- moved R1 15.9 mm to (44.7, 38.9)
- moved REF** 15.9 mm to (48.2, 41.8)
- moved U1 15.9 mm to (41.2, 29.9)
Routing:
- net /DIN: track 34.6 -> 35.3 mm
