File: KiCad/nixieAccurateClock/IN-14-daughter/IN-14-daughter.kicad_sch (KiCad schematic)
At the start: 6 parts, among them J1 Conn_02x11_Top_Bottom, U1 HV509K6-G

Commit message: reroute daughter board
Swapped standoffs and pin header orientation on IN-14 daughter board so that standoffs face outward.  This allows using the daughter board mounting for the mother board mounting.
Parts:
- removed J1: Conn_02x11_Top_Bottom, Connector_PinHeader_1.27mm:PinHeader_2x11_P1.27mm_Vertical, symbol Connector_Generic:Conn_02x11_Top_Bottom
- added J1: Conn_02x11_Odd_Even, Connector_PinHeader_1.27mm:PinHeader_2x11_P1.27mm_Vertical, symbol Connector_Generic:Conn_02x11_Odd_Even
Connections:
- net +3.3V: now also J1.20 (Pin_20)
- net +5V: now also J1.10 (Pin_10)
- net ANODE: now also J1.11 (Pin_11)
- net CLOCK: now also J1.18 (Pin_18)
- net DIN: now also J1.16 (Pin_16)
- net DOUT: now also J1.8 (Pin_8)
- net HVGND: now also J1.14 (Pin_14)
- net N_0: now also J1.7 (Pin_7)
- net N_1: now also J1.15 (Pin_15)
- net N_2: now also J1.17 (Pin_17)
- net N_3: now also J1.19 (Pin_19)
- net N_4: now also J1.21 (Pin_21)
- net N_5: now also J1.22 (Pin_22)
- net N_6: now also J1.2 (Pin_2)
- net N_7: now also J1.1 (Pin_1)
- net N_8: now also J1.3 (Pin_3)
- net N_9: now also J1.5 (Pin_5)
- net N_LHDP: now also J1.13 (Pin_13)
- net N_RHDP: now also J1.9 (Pin_9)
- net VPP: now also J1.12 (Pin_12)
- net ~{LATCH}: now also J1.6 (Pin_6)
- net ~{POLARITY}: now also J1.4 (Pin_4)

Commit message: simplify nixie daughter board
Remove cathode pins that would not be usable for current sensing anyway.
Pivot to using anode pin as shunt measurement with a R2R flash ADC (not yet implemented).
Parts:
- removed J1: Conn_02x11_Odd_Even, Connector_PinHeader_1.27mm:PinHeader_2x11_P1.27mm_Vertical, symbol Connector_Generic:Conn_02x11_Odd_Even
- added J1: Conn_02x05_Odd_Even, Connector_PinHeader_2.54mm:PinHeader_2x05_P2.54mm_Vertical, symbol Connector_Generic:Conn_02x05_Odd_Even
Connections:
- net ~{POLARITY} is gone; now on net GND: U1.21 (*POL)
- net +3.3V: now also J1.6 (Pin_6)
- net +5V: now also J1.2 (Pin_2)
- net ANODE: now also J1.7 (Pin_7)
- net CLOCK: now also J1.8 (Pin_8)
- net DIN: now also J1.4 (Pin_4)
- net DOUT: now also J1.1 (Pin_1)
- net GND: now also J1.10 (Pin_10), J1.5 (Pin_5)
- net VPP: now also R1.1, J1.9 (Pin_9)
- net ~{LATCH}: now also J1.3 (Pin_3)
- net ANODE_DRIVE: no longer names the net of U1.28 (BP)
- net ANODE_DRIVE: no longer R1.1
- net HVGND: no longer names the net of U1.27 (HVGND)
Other:
- moved on the sheet: N1, R1

Commit message: fix clearance rules on daughter board
0.4 mm clearance is not possible to obey with an HV driver IC package that has 0.25 mm pad spacing, but all HV lines can be kept at least 0.25 mm away from everything else and inner layers can be preferentially used.

WIP ADC interface, logic level convertor has been chosen.
Changed lines of the file:
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@@
   (title_block
     (title "IN-14 daughter board")
+    (rev "A")
   )
   (wire (pts (xy 57.15 88.9) (xy 57.15 93.98))
@@
     (effects (font (size 1.27 1.27)) (justify right bottom))
   )
-  (label "N_2" (at 63.5 59.69 90) (fields_autoplaced)
-    (effects (font (size 1.27 1.27)) (justify left bottom))
+  (label "N_2" (at 63.5 59.69 270) (fields_autoplaced)
+    (effects (font (size 1.27 1.27)) (justify right bottom))
   )
   (label "DOUT" (at 139.7 59.69 180) (fields_autoplaced)
     (effects (font (size 1.27 1.27)) (justify right bottom))
   )
-  (label "N_4" (at 68.58 59.69 90) (fields_autoplaced)
-    (effects (font (size 1.27 1.27)) (justify left bottom))
+  (label "N_4" (at 68.58 59.69 270) (fields_autoplaced)
+    (effects (font (size 1.27 1.27)) (justify right bottom))
   )
   (label "DIN" (at 52.07 156.21 90) (fields_autoplaced)
     (effects (font (size 1.27 1.27)) (justify left bottom))
   )
-  (label "N_1" (at 60.96 59.69 90) (fields_autoplaced)
-    (effects (font (size 1.27 1.27)) (justify left bottom))
+  (label "N_1" (at 60.96 59.69 270) (fields_autoplaced)
+    (effects (font (size 1.27 1.27)) (justify right bottom))
   )
   (label "ANODE" (at 139.7 67.31 180) (fields_autoplaced)
@@
     (effects (font (size 1.27 1.27)) (justify left bottom))
   )
-  (label "N_3" (at 66.04 59.69 90) (fields_autoplaced)
-    (effects (font (size 1.27 1.27)) (justify left bottom))
+  (label "N_3" (at 66.04 59.69 270) (fields_autoplaced)
+    (effects (font (size 1.27 1.27)) (justify right bottom))
   )
   (label "N_3" (at 72.39 88.9 90) (fields_autoplaced)
@@
     (effects (font (size 1.27 1.27)) (justify right bottom))
   )
-  (label "N_5" (at 71.12 59.69 90) (fields_autoplaced)
-    (effects (font (size 1.27 1.27)) (justify left bottom))
+  (label "N_5" (at 71.12 59.69 270) (fields_autoplaced)
+    (effects (font (size 1.27 1.27)) (justify right bottom))
   )
   (label "N_1" (at 64.77 88.9 90) (fields_autoplaced)
@@
     (effects (font (size 1.27 1.27)) (justify left bottom))
   )
-  (label "N_9" (at 81.28 59.69 90) (fields_autoplaced)
-    (effects (font (size 1.27 1.27)) (justify left bottom))
+  (label "N_9" (at 81.28 59.69 270) (fields_autoplaced)
+    (effects (font (size 1.27 1.27)) (justify right bottom))
   )
   (label "CLOCK" (at 57.15 156.21 90) (fields_autoplaced)
@@
     (effects (font (size 1.27 1.27)) (justify left bottom))
   )
-  (label "N_7" (at 76.2 59.69 90) (fields_autoplaced)
-    (effects (font (size 1.27 1.27)) (justify left bottom))
+  (label "N_7" (at 76.2 59.69 270) (fields_autoplaced)
+    (effects (font (size 1.27 1.27)) (justify right bottom))
   )
   (label "N_LHDP" (at 60.96 33.02 90) (fields_autoplaced)
     (effects (font (size 1.27 1.27)) (justify left bottom))
   )
-  (label "N_8" (at 78.74 59.69 90) (fields_autoplaced)
-    (effects (font (size 1.27 1.27)) (justify left bottom))
+  (label "N_8" (at 78.74 59.69 270) (fields_autoplaced)
+    (effects (font (size 1.27 1.27)) (justify right bottom))
   )
   (label "N_LHDP" (at 82.55 148.59 270) (fields_autoplaced)
@@
     (effects (font (size 1.27 1.27)) (justify left bottom))
   )
-  (label "N_6" (at 73.66 59.69 90) (fields_autoplaced)
-    (effects (font (size 1.27 1.27)) (justify left bottom))
+  (label "N_6" (at 73.66 59.69 270) (fields_autoplaced)
+    (effects (font (size 1.27 1.27)) (justify right bottom))
   )
   (label "N_RHDP" (at 83.82 33.02 90) (fields_autoplaced)
@@
     (effects (font (size 1.27 1.27)) (justify left bottom))
   )
-  (label "N_0" (at 83.82 59.69 90) (fields_autoplaced)
-    (effects (font (size 1.27 1.27)) (justify left bottom))
+  (label "N_0" (at 83.82 59.69 270) (fields_autoplaced)
+    (effects (font (size 1.27 1.27)) (justify right bottom))
   )
   (symbol (lib_id "power:GND") (at 137.16 29.21 0) (mirror y) (unit 1)

Commit message: Add decoupling caps
Parts:
- added C1, C2: 0.1u, Capacitor_SMD:C_0603_1608Metric, symbol Device:C_Small
Connections:
- net +3.3V: now also C1.2; no longer U1.20 (VDD)
- net +5V: now also C2.2; no longer U1.26 (VBIAS)
- net CLOCK renamed CLK
- net ~{LATCH} renamed ~{LE}
- new net VBIAS: C2.1, U1.26 (VBIAS)
- new net VDD: C1.1, U1.20 (VDD)

Commit message: Fill out BOM
Parts:
- C1, C2: Model (none) -> CL10B104KB8NNWC; Price (none) -> 0.10
- H1, H2: now left out of the parts list
- J1: Model (none) -> PPPC052LFBN-RC; Price (none) -> 0.72
- N1: Model (none) -> IN-14; Price (none) -> 17.50
- R1: Model (none) -> RC1206JR-0733KL; Price (none) -> 0.10
- U1: Price (none) -> 2.89
Changed lines of the file:
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@@
       (effects (font (size 1.27 1.27)) hide)
     )
-    (property "Datasheet" "~" (at 59.69 167.64 0)
+    (property "Datasheet" "https://mm.digikey.com/Volume0/opasdata/d220001/medias/docus/658/CL10B104KB8NNWC_Spec.pdf" (at 59.69 167.64 0)
+      (effects (font (size 1.27 1.27)) hide)
+    )
+    (property "Model" "CL10B104KB8NNWC" (at 59.69 167.64 0)
+      (effects (font (size 1.27 1.27)) hide)
+    )
+    (property "Price" "0.10" (at 59.69 167.64 0)
       (effects (font (size 1.27 1.27)) hide)
     )
@@
   )
   (symbol (lib_id "Mechanical:MountingHole_Pad") (at 137.16 24.13 0) (unit 1)
-    (in_bom yes) (on_board yes) (dnp no) (fields_autoplaced)
+    (in_bom no) (on_board yes) (dnp no) (fields_autoplaced)
     (property "Reference" "H1" (at 139.7 21.59 0)
       (effects (font (size 1.27 1.27)) (justify left))
@@
     )
   )
-  (symbol (lib_id "Device:C_Small") (at 74.93 167.64 0) (unit 1)
+  (symbol (lib_name "C_Small_1") (lib_id "Device:C_Small") (at 74.93 167.64 0) (unit 1)
     (in_bom yes) (on_board yes) (dnp no) (fields_autoplaced)
     (property "Reference" "C2" (at 77.47 166.3763 0)
@@
       (effects (font (size 1.27 1.27)) hide)
     )
-    (property "Datasheet" "~" (at 74.93 167.64 0)
+    (property "Datasheet" "https://mm.digikey.com/Volume0/opasdata/d220001/medias/docus/658/CL10B104KB8NNWC_Spec.pdf" (at 74.93 167.64 0)
+      (effects (font (size 1.27 1.27)) hide)
+    )
+    (property "Model" "CL10B104KB8NNWC" (at 74.93 167.64 0)
+      (effects (font (size 1.27 1.27)) hide)
+    )
+    (property "Price" "0.10" (at 74.93 167.64 0)
       (effects (font (size 1.27 1.27)) hide)
     )
@@
   )
   (symbol (lib_name "MountingHole_Pad_1") (lib_id "Mechanical:MountingHole_Pad") (at 166.37 24.13 0) (unit 1)
-    (in_bom yes) (on_board yes) (dnp no) (fields_autoplaced)
+    (in_bom no) (on_board yes) (dnp no) (fields_autoplaced)
     (property "Reference" "H2" (at 168.91 21.59 0)
       (effects (font (size 1.27 1.27)) (justify left))
@@
       (effects (font (size 0.508 0.508)) hide)
     )
-    (property "Datasheet" "" (at 71.12 46.99 0)
+    (property "Datasheet" "https://download.elektronicastynus.be/57/in-14_datasheet.pdf" (at 71.12 46.99 0)
+      (effects (font (size 1.27 1.27)) hide)
+    )
+    (property "Model" "IN-14" (at 71.12 46.99 90)
+      (effects (font (size 1.27 1.27)) hide)
+    )
+    (property "Price" "17.50" (at 71.12 46.99 90)
       (effects (font (size 1.27 1.27)) hide)
     )
@@
     (property "Datasheet" "https://ww1.microchip.com/downloads/en/DeviceDoc/hv509.pdf" (at 44.45 120.65 0)
       (effects (font (size 1.27 1.27) italic) hide)
+    )
+    (property "Price" "2.89" (at 92.71 93.98 90)
+      (effects (font (size 1.27 1.27)) hide)
     )
     (pin "27")
@@
       (effects (font (size 1.27 1.27)) hide)
     )
-    (property "Datasheet" "~" (at 73.66 29.21 0)
+    (property "Datasheet" "https://www.yageo.com/upload/media/product/app/datasheet/rchip/pyu-rc_group_51_rohs_l.pdf" (at 73.66 29.21 0)
+      (effects (font (size 1.27 1.27)) hide)
+    )
+    (property "Model" "RC1206JR-0733KL" (at 73.66 29.21 0)
+      (effects (font (size 1.27 1.27)) hide)
+    )
+    (property "Price" "0.10" (at 73.66 29.21 0)
       (effects (font (size 1.27 1.27)) hide)
     )
@@
       (effects (font (size 1.27 1.27)) hide)
     )
-    (property "Datasheet" "~" (at 148.59 64.77 0)
-      (effects (font (size 1.27 1.27)) hide)
-    )
+    (property "Datasheet" "https://mm.digikey.com/Volume0/opasdata/d220001/medias/docus/937/Female_Headers.100_DS.pdf" (at 148.59 64.77 0)
+      (effects (font (size 1.27 1.27)) hide)
+    )
+    (property "Model" "PPPC052LFBN-RC" (at 148.59 64.77 0)
+      (effects (font (size 1.27 1.27)) hide)
+    )
+    (property "Price" "0.72" (at 148.59 64.77 0)
+      (effects (font (size 1.27 1.27)) hide)
+    )

Commit message: Add retailer links
Parts:
- C1, C2: Digikey link (none) -> https://www.digikey.com/en/products/detail/samsung-electro-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; Mouser link (none) -> https://www.mouser.com/ProductDetail/Samsung-Electro-Mechan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
- J1: Digikey link (none) -> https://www.digikey.com/en/products/detail/sullins-connecto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; Mouser link (none) -> N/A
- N1: Digikey link (none) -> N/A; Mouser link (none) -> N/A
- R1: Digikey link (none) -> https://www.digikey.com/en/products/detail/yageo/RC1206JR-0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; Mouser link (none) -> https://www.mouser.com/ProductDetail/YAGEO/RC1206JR-0733KL?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
- U1: Digikey link (none) -> https://www.digikey.com/en/products/detail/microchip-techno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; Model (none) -> HV509K6-G; Mouser link (none) -> https://www.mouser.com/ProductDetail/Microchip-Technology/H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
Other:
- moved on the sheet: C1, C2, H1, H2, J1, N1, R1, U1

Commit message: Add fiducials
Parts:
- added FID1, FID2, FID3: Fiducial, Fiducial:Fiducial_0.5mm_Mask1.5mm, symbol Mechanical:Fiducial
Changed lines of the file:
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@@
     (stroke (width 0) (type default))
   )
-  (wire (pts (xy 59.69 48.26) (xy 48.26 48.26))
+  (wire (pts (xy 59.69 48.26) (xy 54.61 48.26))
     (stroke (width 0) (type default))
   )
@@
     (stroke (width 0) (type default))
   )
-  (wire (pts (xy 59.69 43.18) (xy 48.26 43.18))
+  (wire (pts (xy 59.69 43.18) (xy 54.61 43.18))
     (stroke (width 0) (type default))
   )
@@
     (stroke (width 0) (type default))
   )
-  (wire (pts (xy 59.69 55.88) (xy 48.26 55.88))
+  (wire (pts (xy 59.69 55.88) (xy 54.61 55.88))
     (stroke (width 0) (type default))
   )
@@
     (stroke (width 0) (type default))
   )
-  (wire (pts (xy 59.69 60.96) (xy 48.26 60.96))
+  (wire (pts (xy 59.69 60.96) (xy 54.61 60.96))
     (stroke (width 0) (type default))
   )
@@
     (effects (font (size 1.27 1.27)) (justify right bottom))
   )
-  (label "DIN" (at 48.26 43.18 0) (fields_autoplaced)
-    (effects (font (size 1.27 1.27)) (justify left bottom))
+  (label "DIN" (at 54.61 43.18 180) (fields_autoplaced)
+    (effects (font (size 1.27 1.27)) (justify right bottom))
   )
   (label "N_1" (at 135.89 59.69 180) (fields_autoplaced)
@@
     (effects (font (size 1.27 1.27)) (justify right bottom))
   )
-  (label "DOUT" (at 48.26 60.96 0) (fields_autoplaced)
-    (effects (font (size 1.27 1.27)) (justify left bottom))
+  (label "DOUT" (at 54.61 60.96 180) (fields_autoplaced)
+    (effects (font (size 1.27 1.27)) (justify right bottom))
   )
   (label "N_3" (at 135.89 64.77 180) (fields_autoplaced)
@@
     (effects (font (size 1.27 1.27)) (justify left bottom))
   )
-  (label "~{LE}" (at 48.26 55.88 0) (fields_autoplaced)
-    (effects (font (size 1.27 1.27)) (justify left bottom))
+  (label "~{LE}" (at 54.61 55.88 180) (fields_autoplaced)
+    (effects (font (size 1.27 1.27)) (justify right bottom))
   )
   (label "N_9" (at 135.89 80.01 180) (fields_autoplaced)
     (effects (font (size 1.27 1.27)) (justify right bottom))
   )
-  (label "CLK" (at 48.26 48.26 0) (fields_autoplaced)
-    (effects (font (size 1.27 1.27)) (justify left bottom))
+  (label "CLK" (at 54.61 48.26 180) (fields_autoplaced)
+    (effects (font (size 1.27 1.27)) (justify right bottom))
   )
   (label "N_9" (at 55.88 81.28 180) (fields_autoplaced)
@@
     (effects (font (size 1.27 1.27)) (justify left bottom))
   )
-  (label "VDD" (at 48.26 50.8 0) (fields_autoplaced)
-    (effects (font (size 1.27 1.27)) (justify left bottom))
+  (label "VDD" (at 54.61 50.8 180) (fields_autoplaced)
+    (effects (font (size 1.27 1.27)) (justify right bottom))
   )
   (label "N_8" (at 135.89 77.47 180) (fields_autoplaced)
@@
     (effects (font (size 1.27 1.27)) (justify right bottom))
   )
-  (label "VBIAS" (at 53.34 66.04 180) (fields_autoplaced)
+  (label "VBIAS" (at 54.61 66.04 180) (fields_autoplaced)
     (effects (font (size 1.27 1.27)) (justify right bottom))
   )
@@
     )
   )
+  (symbol (lib_id "Mechanical:Fiducial") (at 161.29 143.51 0) (unit 1)
+    (in_bom yes) (on_board yes) (dnp no) (fields_autoplaced)
+    (property "Reference" "FID2" (at 163.83 142.24 0)
+      (effects (font (size 1.27 1.27)) (justify left))
+    )
+    (property "Value" "Fiducial" (at 163.83 144.78 0)
+      (effects (font (size 1.27 1.27)) (justify left))
+    )
+    (property "Footprint" "Fiducial:Fiducial_0.5mm_Mask1.5mm" (at 161.29 143.51 0)
+      (effects (font (size 1.27 1.27)) hide)
+    )
+    (property "Datasheet" "~" (at 161.29 143.51 0)
+      (effects (font (size 1.27 1.27)) hide)
+    )
+    (instances
+      (project "IN-14-daughter"
+        (path "/0bdf933d-3de8-451a-be8d-fbdb2becffac"
+          (reference "FID2") (unit 1)
+        )
+      )
+    )
+  )
+  (symbol (lib_id "Mechanical:Fiducial") (at 161.29 138.43 0) (unit 1)
+    (in_bom yes) (on_board yes) (dnp no) (fields_autoplaced)
+    (property "Reference" "FID1" (at 163.83 137.16 0)
+      (effects (font (size 1.27 1.27)) (justify left))
+    )
+    (property "Value" "Fiducial" (at 163.83 139.7 0)
+      (effects (font (size 1.27 1.27)) (justify left))
+    )
+    (property "Footprint" "Fiducial:Fiducial_0.5mm_Mask1.5mm" (at 161.29 138.43 0)
+      (effects (font (size 1.27 1.27)) hide)
+    )
+    (property "Datasheet" "~" (at 161.29 138.43 0)
+      (effects (font (size 1.27 1.27)) hide)
+    )
+    (instances
+      (project "IN-14-daughter"
+        (path "/0bdf933d-3de8-451a-be8d-fbdb2becffac"
+          (reference "FID1") (unit 1)
+        )
+      )
+    )
+  )
   (symbol (lib_id "power:VPP") (at 179.07 72.39 270) (unit 1)
     (in_bom yes) (on_board yes) (dnp no)
@@
         (path "/0bdf933d-3de8-451a-be8d-fbdb2becffac"
           (reference "#PWR06") (unit 1)
+        )
+      )
+    )
+  )
+  (symbol (lib_id "Mechanical:Fiducial") (at 161.29 148.59 0) (unit 1)
+    (in_bom yes) (on_board yes) (dnp no) (fields_autoplaced)
+    (property "Reference" "FID3" (at 163.83 147.32 0)
+      (effects (font (size 1.27 1.27)) (justify left))
+    )
+    (property "Value" "Fiducial" (at 163.83 149.86 0)
+      (effects (font (size 1.27 1.27)) (justify left))
+    )
+    (property "Footprint" "Fiducial:Fiducial_0.5mm_Mask1.5mm" (at 161.29 148.59 0)
+      (effects (font (size 1.27 1.27)) hide)
+    )
+    (property "Datasheet" "~" (at 161.29 148.59 0)
+      (effects (font (size 1.27 1.27)) hide)
+    )
+    (instances
+      (project "IN-14-daughter"
+        (path "/0bdf933d-3de8-451a-be8d-fbdb2becffac"
+          (reference "FID3") (unit 1)
         )
       )
@@
   (symbol (lib_id "00_lib:HV509K6-G") (at 110.49 83.82 180) (unit 1)
     (in_bom yes) (on_board yes) (dnp no)
-    (property "Reference" "U1" (at 71.12 35.56 0)
+    (property "Reference" "U1" (at 71.12 40.64 0)
       (effects (font (size 1.524 1.524)) (justify left))
     )
-    (property "Value" "HV509K6-G" (at 90.17 91.44 0)
+    (property "Value" "HV509K6-G" (at 91.44 58.42 0)
       (effects (font (size 1.524 1.524)) (justify left))
     )
-    (property "Footprint" "Package_DFN_QFN:QFN-32-1EP_5x5mm_P0.5mm_EP3.1x3.1mm_ThermalVias" (at 85.09 44.45 0)
+    (property "Footprint" "Package_DFN_QFN:QFN-32-1EP_5x5mm_P0.5mm_EP3.1x3.1mm_ThermalVias" (at 85.09 38.1 0)
       (effects (font (size 1.27 1.27) italic) hide)
     )
@@
       (effects (font (size 1.27 1.27) italic) hide)
     )
-    (property "Price" "2.89" (at 110.49 83.82 90)
-      (effects (font (size 1.27 1.27)) hide)
-    )
-    (property "Digikey link" "https://www.digikey.com/en/products/detail/microchip-technology/HV509K6-G/4902492" (at 110.49 83.82 0)
-      (effects (font (size 1.27 1.27)) hide)
-    )
-    (property "Model" "HV509K6-G" (at 110.49 83.82 0)
-      (effects (font (size 1.27 1.27)) hide)
-    )
-    (property "Mouser link" "https://www.mouser.com/ProductDetail/Microchip-Technology/HV509K6-G?qs=073BFnXyqnuDeexnfjhPaQ%3D%3D" (at 110.49 83.82 0)
-      (effects (font (size 1.27 1.27)) hide)
-    )
+    (property "Price" "2.89" (at 85.09 44.45 0)
+      (effects (font (size 1.27 1.27)) hide)
+    )
+    (property "Digikey link" "https://www.digikey.com/en/products/detail/microchip-technology/HV509K6-G/4902492" (at 81.28 30.48 0)
+      (effects (font (size 1.27 1.27)) hide)
+    )
+    (property "Model" "HV509K6-G" (at 83.82 63.5 0)
+      (effects (font (size 1.27 1.27)) hide)
+    )
+    (property "Mouser link" "https://www.mouser.com/ProductDetail/Microchip-Technology/HV509K6-G?qs=073BFnXyqnuDeexnfjhPaQ%3D%3D" (at 85.09 33.02 0)
+      (effects (font (size 1.27 1.27)) hide)
+    )

Commit message: switch to 27k R_anode
Add voltage rail jumpers for different 5V and 3.3V standby applications
Parts:
- R1: value 33k -> 27k; Digikey link https://www.digikey.com/en/products/detail/yageo/RC1206JR-0733KL/729282 -> https://www.digikey.com/en/products/detail/yageo/RC1206JR-0727KL/729262; Model RC1206JR-0733KL -> RC1206JR-0727KL; Mouser link https://www.mouser.com/ProductDetail/YAGEO/RC1206JR-0733KL?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 -> https://www.mouser.com/ProductDetail/YAGEO/RC1206JR-0727KL?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
Changed lines of the file:
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@@
       (effects (font (size 1.27 1.27)) (justify left))
     )
-    (property "Value" "33k" (at 171.45 74.93 90)
+    (property "Value" "27k" (at 171.45 74.93 90)
       (effects (font (size 1.27 1.27)) (justify left))
     )
@@
       (effects (font (size 1.27 1.27)) hide)
     )
-    (property "Model" "RC1206JR-0733KL" (at 172.72 72.39 0)
+    (property "Model" "RC1206JR-0727KL" (at 172.72 72.39 0)
       (effects (font (size 1.27 1.27)) hide)
     )
@@
       (effects (font (size 1.27 1.27)) hide)
     )
-    (property "Digikey link" "https://www.digikey.com/en/products/detail/yageo/RC1206JR-0733KL/729282" (at 172.72 72.39 90)
+    (property "Digikey link" "https://www.digikey.com/en/products/detail/yageo/RC1206JR-0727KL/729262" (at 172.72 72.39 90)
       (effects (font (size 1.27 1.27)) hide)
     )
-    (property "Mouser link" "https://www.mouser.com/ProductDetail/YAGEO/RC1206JR-0733KL?qs=4sq2y2bXwtTBbhYRyjZ6aQ%3D%3D" (at 172.72 72.39 90)
+    (property "Mouser link" "https://www.mouser.com/ProductDetail/YAGEO/RC1206JR-0727KL?qs=CteSnpDdeuBg3%2FC0aG6GFQ%3D%3D" (at 172.72 72.39 90)
       (effects (font (size 1.27 1.27)) hide)
     )
