File: hardware/KiCad/nixieAccurateClock/20V_supply.kicad_sch (KiCad schematic)
At the start: 25 parts, among them J9 Conn_01x02_Pin, Q1 BSP88, U5 LM51561HPWPR

Commit message: switch all components to SMT
layout is a mess
Parts:
- J9, J?: footprint Connector_PinHeader_2.54mm:PinHeader_1x02_P2.54mm_Vertical -> Connector_PinHeader_2.54mm:PinHeader_1x02_P2.54mm_Vertical_SMD_Pin1Left; Digikey link https://www.digikey.com/en/products/detail/adam-tech/PH1-02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 -> https://www.digikey.com/en/products/detail/samtec-inc/TSM-1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; Model PH1-02-UA -> TSM-102-01-L-SV; Mouser link https://www.mouser.com/ProductDetail/Samtec/TSW-102-07-G-S?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 -> https://www.mouser.com/ProductDetail/Samtec/TSM-102-01-L-SV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; Price 0.10 -> 0.42
Changed lines of the file:
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@@
       (effects (font (size 1.27 1.27)) (justify right))
     )
-    (property "Footprint" "Connector_PinHeader_2.54mm:PinHeader_1x02_P2.54mm_Vertical" (at 41.91 35.56 0)
-      (effects (font (size 1.27 1.27)) hide)
-    )
-    (property "Datasheet" "https://app.adam-tech.com/products/download/data_sheet/201605/ph1-xx-ua-data-sheet.pdf" (at 41.91 35.56 0)
+    (property "Footprint" "Connector_PinHeader_2.54mm:PinHeader_1x02_P2.54mm_Vertical_SMD_Pin1Left" (at 41.91 35.56 0)
+      (effects (font (size 1.27 1.27)) hide)
+    )
+    (property "Datasheet" "https://suddendocs.samtec.com/catalog_english/tsm.pdf" (at 41.91 35.56 0)
       (effects (font (size 1.27 1.27)) hide)
     )
@@
       (effects (font (size 1.27 1.27)) hide)
     )
-    (property "Model" "PH1-02-UA" (at 41.91 35.56 0)
-      (effects (font (size 1.27 1.27)) hide)
-    )
-    (property "Price" "0.10" (at 41.91 35.56 0)
-      (effects (font (size 1.27 1.27)) hide)
-    )
-    (property "Digikey link" "https://www.digikey.com/en/products/detail/adam-tech/PH1-02-UA/9830266" (at 41.91 35.56 0)
-      (effects (font (size 1.27 1.27)) hide)
-    )
-    (property "Mouser link" "https://www.mouser.com/ProductDetail/Samtec/TSW-102-07-G-S?qs=iT52DjcXudsNPhlNCDp8vw%3D%3D" (at 41.91 35.56 0)
+    (property "Model" "TSM-102-01-L-SV" (at 41.91 35.56 0)
+      (effects (font (size 1.27 1.27)) hide)
+    )
+    (property "Price" "0.42" (at 41.91 35.56 0)
+      (effects (font (size 1.27 1.27)) hide)
+    )
+    (property "Digikey link" "https://www.digikey.com/en/products/detail/samtec-inc/TSM-102-01-L-SV/2685520" (at 41.91 35.56 0)
+      (effects (font (size 1.27 1.27)) hide)
+    )
+    (property "Mouser link" "https://www.mouser.com/ProductDetail/Samtec/TSM-102-01-L-SV?qs=FESYatJ8odJ%252BIhPvKBkuBA%3D%3D" (at 41.91 35.56 0)
       (effects (font (size 1.27 1.27)) hide)
     )
@@
       (effects (font (size 1.27 1.27)) (justify right))
     )
-    (property "Footprint" "Connector_PinHeader_2.54mm:PinHeader_1x02_P2.54mm_Vertical" (at 213.36 52.07 0)
-      (effects (font (size 1.27 1.27)) hide)
-    )
-    (property "Datasheet" "https://app.adam-tech.com/products/download/data_sheet/201605/ph1-xx-ua-data-sheet.pdf" (at 213.36 52.07 0)
+    (property "Footprint" "Connector_PinHeader_2.54mm:PinHeader_1x02_P2.54mm_Vertical_SMD_Pin1Left" (at 213.36 52.07 0)
+      (effects (font (size 1.27 1.27)) hide)
+    )
+    (property "Datasheet" "https://suddendocs.samtec.com/catalog_english/tsm.pdf" (at 213.36 52.07 0)
       (effects (font (size 1.27 1.27)) hide)
     )
@@
       (effects (font (size 1.27 1.27)) hide)
     )
-    (property "Model" "PH1-02-UA" (at 213.36 52.07 0)
-      (effects (font (size 1.27 1.27)) hide)
-    )
-    (property "Price" "0.10" (at 213.36 52.07 0)
-      (effects (font (size 1.27 1.27)) hide)
-    )
-    (property "Digikey link" "https://www.digikey.com/en/products/detail/adam-tech/PH1-02-UA/9830266" (at 213.36 52.07 0)
-      (effects (font (size 1.27 1.27)) hide)
-    )
-    (property "Mouser link" "https://www.mouser.com/ProductDetail/Samtec/TSW-102-07-G-S?qs=iT52DjcXudsNPhlNCDp8vw%3D%3D" (at 213.36 52.07 0)
-      (effects (font (size 1.27 1.27)) hide)
-    )
+    (property "Model" "TSM-102-01-L-SV" (at 213.36 52.07 0)
+      (effects (font (size 1.27 1.27)) hide)
+    )
+    (property "Price" "0.42" (at 213.36 52.07 0)
+      (effects (font (size 1.27 1.27)) hide)
+    )
+    (property "Digikey link" "https://www.digikey.com/en/products/detail/samtec-inc/TSM-102-01-L-SV/2685520" (at 213.36 52.07 0)
+      (effects (font (size 1.27 1.27)) hide)
+    )
+    (property "Mouser link" "https://www.mouser.com/ProductDetail/Samtec/TSM-102-01-L-SV?qs=FESYatJ8odJ%252BIhPvKBkuBA%3D%3D" (at 213.36 52.07 0)
+      (effects (font (size 1.27 1.27)) hide)
+    )

Commit message: switch to all SM components
Parts:
- renumbered J9 to J11, U5 to U4
Changed lines of the file:
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@@
   (symbol (lib_id "power:GND") (at 111.76 90.17 90) (unit 1)
     (in_bom yes) (on_board yes) (dnp no) (fields_autoplaced)
-    (property "Reference" "#PWR035" (at 118.11 90.17 0)
+    (property "Reference" "#PWR052" (at 118.11 90.17 0)
       (effects (font (size 1.27 1.27)) hide)
     )
@@
       (project "nixieAccurateClock"
         (path "/55aab698-7558-4fe2-95ad-faa6da60ef89/33639105-1e30-4fa8-9335-500c2abdb54b"
-          (reference "#PWR035") (unit 1)
+          (reference "#PWR052") (unit 1)
         )
       )
@@
         )
         (path "/55aab698-7558-4fe2-95ad-faa6da60ef89/33639105-1e30-4fa8-9335-500c2abdb54b"
-          (reference "J8") (unit 1)
+          (reference "J10") (unit 1)
         )
       )
@@
   (symbol (lib_id "power:GND") (at 160.02 73.66 0) (unit 1)
     (in_bom yes) (on_board yes) (dnp no) (fields_autoplaced)
-    (property "Reference" "#PWR032" (at 160.02 80.01 0)
+    (property "Reference" "#PWR049" (at 160.02 80.01 0)
       (effects (font (size 1.27 1.27)) hide)
     )
@@
       (project "nixieAccurateClock"
         (path "/55aab698-7558-4fe2-95ad-faa6da60ef89/33639105-1e30-4fa8-9335-500c2abdb54b"
-          (reference "#PWR032") (unit 1)
+          (reference "#PWR049") (unit 1)
         )
       )
@@
   (symbol (lib_id "power:GND") (at 138.43 100.33 0) (unit 1)
     (in_bom yes) (on_board yes) (dnp no) (fields_autoplaced)
-    (property "Reference" "#PWR036" (at 138.43 106.68 0)
+    (property "Reference" "#PWR053" (at 138.43 106.68 0)
       (effects (font (size 1.27 1.27)) hide)
     )
@@
       (project "nixieAccurateClock"
         (path "/55aab698-7558-4fe2-95ad-faa6da60ef89/33639105-1e30-4fa8-9335-500c2abdb54b"
-          (reference "#PWR036") (unit 1)
+          (reference "#PWR053") (unit 1)
         )
       )
@@
   (symbol (lib_id "power:GND") (at 198.12 60.96 0) (unit 1)
     (in_bom yes) (on_board yes) (dnp no) (fields_autoplaced)
-    (property "Reference" "#PWR031" (at 198.12 67.31 0)
+    (property "Reference" "#PWR048" (at 198.12 67.31 0)
       (effects (font (size 1.27 1.27)) hide)
     )
@@
       (project "nixieAccurateClock"
         (path "/55aab698-7558-4fe2-95ad-faa6da60ef89/33639105-1e30-4fa8-9335-500c2abdb54b"
-          (reference "#PWR031") (unit 1)
+          (reference "#PWR048") (unit 1)
         )
       )
@@
   (symbol (lib_id "power:GND") (at 24.13 52.07 270) (unit 1)
     (in_bom yes) (on_board yes) (dnp no) (fields_autoplaced)
-    (property "Reference" "#PWR029" (at 17.78 52.07 0)
+    (property "Reference" "#PWR046" (at 17.78 52.07 0)
       (effects (font (size 1.27 1.27)) hide)
     )
@@
       (project "nixieAccurateClock"
         (path "/55aab698-7558-4fe2-95ad-faa6da60ef89/33639105-1e30-4fa8-9335-500c2abdb54b"
-          (reference "#PWR029") (unit 1)
+          (reference "#PWR046") (unit 1)
         )
       )
@@
   (symbol (lib_id "00_lib:+20V") (at 218.44 44.45 270) (unit 1)
     (in_bom no) (on_board no) (dnp no) (fields_autoplaced)
-    (property "Reference" "#PWR028" (at 215.9 44.45 0)
+    (property "Reference" "#PWR045" (at 215.9 44.45 0)
       (effects (font (size 1.27 1.27)) hide)
     )
@@
       (project "nixieAccurateClock"
         (path "/55aab698-7558-4fe2-95ad-faa6da60ef89/33639105-1e30-4fa8-9335-500c2abdb54b"
-          (reference "#PWR028") (unit 1)
+          (reference "#PWR045") (unit 1)
         )
       )
@@
   (symbol (lib_id "power:+5V") (at 144.78 39.37 0) (unit 1)
     (in_bom yes) (on_board yes) (dnp no) (fields_autoplaced)
-    (property "Reference" "#PWR025" (at 144.78 43.18 0)
+    (property "Reference" "#PWR042" (at 144.78 43.18 0)
       (effects (font (size 1.27 1.27)) hide)
     )
@@
       (project "nixieAccurateClock"
         (path "/55aab698-7558-4fe2-95ad-faa6da60ef89/33639105-1e30-4fa8-9335-500c2abdb54b"
-          (reference "#PWR025") (unit 1)
+          (reference "#PWR042") (unit 1)
         )
       )
@@
   (symbol (lib_id "00_lib:LM51561HPWPR") (at 64.77 44.45 0) (unit 1)
     (in_bom yes) (on_board yes) (dnp no)
-    (property "Reference" "U5" (at 86.36 34.29 0)
+    (property "Reference" "U4" (at 86.36 34.29 0)
       (effects (font (size 1.524 1.524)))
     )
@@
       (project "nixieAccurateClock"
         (path "/55aab698-7558-4fe2-95ad-faa6da60ef89/33639105-1e30-4fa8-9335-500c2abdb54b"
-          (reference "U5") (unit 1)
+          (reference "U4") (unit 1)
         )
       )
@@
   (symbol (lib_id "power:GND") (at 121.92 44.45 90) (unit 1)
     (in_bom yes) (on_board yes) (dnp no)
-    (property "Reference" "#PWR027" (at 128.27 44.45 0)
+    (property "Reference" "#PWR044" (at 128.27 44.45 0)
       (effects (font (size 1.27 1.27)) hide)
     )
@@
       (project "nixieAccurateClock"
         (path "/55aab698-7558-4fe2-95ad-faa6da60ef89/33639105-1e30-4fa8-9335-500c2abdb54b"
-          (reference "#PWR027") (unit 1)
+          (reference "#PWR044") (unit 1)
         )
       )
@@
   (symbol (lib_id "power:GND") (at 48.26 74.93 270) (unit 1)
     (in_bom yes) (on_board yes) (dnp no) (fields_autoplaced)
-    (property "Reference" "#PWR033" (at 41.91 74.93 0)
+    (property "Reference" "#PWR050" (at 41.91 74.93 0)
       (effects (font (size 1.27 1.27)) hide)
     )
@@
       (project "nixieAccurateClock"
         (path "/55aab698-7558-4fe2-95ad-faa6da60ef89/33639105-1e30-4fa8-9335-500c2abdb54b"
-          (reference "#PWR033") (unit 1)
+          (reference "#PWR050") (unit 1)
         )
       )
@@
   (symbol (lib_id "power:GND") (at 48.26 82.55 270) (unit 1)
     (in_bom yes) (on_board yes) (dnp no) (fields_autoplaced)
-    (property "Reference" "#PWR034" (at 41.91 82.55 0)
+    (property "Reference" "#PWR051" (at 41.91 82.55 0)
       (effects (font (size 1.27 1.27)) hide)
     )
@@
       (project "nixieAccurateClock"
         (path "/55aab698-7558-4fe2-95ad-faa6da60ef89/33639105-1e30-4fa8-9335-500c2abdb54b"
-          (reference "#PWR034") (unit 1)
+          (reference "#PWR051") (unit 1)
         )
       )
@@
   (symbol (lib_id "power:GND") (at 223.52 104.14 0) (unit 1)
     (in_bom yes) (on_board yes) (dnp no) (fields_autoplaced)
-    (property "Reference" "#PWR038" (at 223.52 110.49 0)
+    (property "Reference" "#PWR055" (at 223.52 110.49 0)
       (effects (font (size 1.27 1.27)) hide)
     )
@@
       (project "nixieAccurateClock"
         (path "/55aab698-7558-4fe2-95ad-faa6da60ef89/33639105-1e30-4fa8-9335-500c2abdb54b"
-          (reference "#PWR038") (unit 1)
+          (reference "#PWR055") (unit 1)
         )
       )
@@
   (symbol (lib_id "Connector:Conn_01x02_Pin") (at 213.36 52.07 90) (unit 1)
     (in_bom yes) (on_board yes) (dnp no)
-    (property "Reference" "J9" (at 217.17 50.165 90)
+    (property "Reference" "J11" (at 217.17 50.165 90)
       (effects (font (size 1.27 1.27)) (justify right))
     )
@@
       (project "nixieAccurateClock"
         (path "/55aab698-7558-4fe2-95ad-faa6da60ef89/33639105-1e30-4fa8-9335-500c2abdb54b"
-          (reference "J9") (unit 1)
+          (reference "J11") (unit 1)
         )
       )
@@
   (symbol (lib_id "power:+5V") (at 24.13 44.45 90) (unit 1)
     (in_bom yes) (on_board yes) (dnp no) (fields_autoplaced)
-    (property "Reference" "#PWR026" (at 27.94 44.45 0)
+    (property "Reference" "#PWR043" (at 27.94 44.45 0)
       (effects (font (size 1.27 1.27)) hide)
     )
@@
       (project "nixieAccurateClock"
         (path "/55aab698-7558-4fe2-95ad-faa6da60ef89/33639105-1e30-4fa8-9335-500c2abdb54b"
-          (reference "#PWR026") (unit 1)
+          (reference "#PWR043") (unit 1)
         )
       )
@@
   (symbol (lib_id "power:GND") (at 184.15 104.14 0) (unit 1)
     (in_bom yes) (on_board yes) (dnp no) (fields_autoplaced)
-    (property "Reference" "#PWR037" (at 184.15 110.49 0)
+    (property "Reference" "#PWR054" (at 184.15 110.49 0)
       (effects (font (size 1.27 1.27)) hide)
     )
@@
       (project "nixieAccurateClock"
         (path "/55aab698-7558-4fe2-95ad-faa6da60ef89/33639105-1e30-4fa8-9335-500c2abdb54b"
-          (reference "#PWR037") (unit 1)
+          (reference "#PWR054") (unit 1)
         )
       )
@@
   (symbol (lib_id "power:GND") (at 60.96 59.69 270) (unit 1)
     (in_bom yes) (on_board yes) (dnp no) (fields_autoplaced)
-    (property "Reference" "#PWR030" (at 54.61 59.69 0)
+    (property "Reference" "#PWR047" (at 54.61 59.69 0)
       (effects (font (size 1.27 1.27)) hide)
     )
@@
       (project "nixieAccurateClock"
         (path "/55aab698-7558-4fe2-95ad-faa6da60ef89/33639105-1e30-4fa8-9335-500c2abdb54b"
-          (reference "#PWR030") (unit 1)
-        )
-      )
+          (reference "#PWR047") (unit 1)
+        )
+      )
