File: hardware/KiCad/nixieAccurateClock/Boost_quad.kicad_sch (KiCad schematic)
At the start: 14 parts

Commit message: single stage HV supply
Also switch to a MOSFET with a reasonable footprint
Parts:
- removed U?: SIB452DK-T1-GE3, 00_lib:SON_K-T1-GE3_VIS, symbol 00_lib:SIB452DK-T1-GE3
- added Q1: IRLH5030TRPBF, 00_lib:Infineon-PG-TDSON-8-0-0-MFG, symbol 00_lib:IRLH5030TRPBF
Connections:
- net GATE_{HV}: now also Q1.4 (G)
- net GND: now also Q1.1 (S), Q1.2 (S), Q1.3 (S)
- net HV_{HALF-BOOST}: now also Q1.5-6-7-8 (D)
