File: hardware/KiCad/nixieAccurateClock/nixieAccurateClock.kicad_pcb (KiCad board)
At the start: 4 copper layers, 152.4 x 101.6 mm, 114 parts, among them J1 Conn_01x02_Pin, J10 Conn_01x02_Pin, J11 Conn_02x05_Odd_Even, J2 Conn_01x02_Pin, J3 Conn_01x02_Pin, J4 Conn_01x02_Pin, J5 Conn_01x02_Pin, J6 Conn_Coaxial, J7 Conn_01x02_Pin, J8 Conn_01x02_Pin, J9 Conn_01x02_Pin, Q1 BSP88, Q2 BSP88, Q3 BSP88, Q4 BSP88, Q5 BSP88, SW1 SW_DIP_x08, U1 MCP23008-xSO, U13 ADC0820BCWMX, U14 TXB0108PWR, U15 TXB0108PWR, U2 pico iCE, U3 LTR-329ALS-01, U4 PX1125T, U5 LM51561HPWPR, U6 LM51561HPWPR

Commit message: WIP pinout config
Connections:
- U2 pad 63: GPS_{TXD} -> HV_{CONTROL}
- U2 pad 64: HV_{CONTROL} -> GPS_{TXD}
- U2 pad 67: GPS_{RXD} -> /INT_{IO-expander}
- U2 pad 68: /INT_{IO-expander} -> GPS_{RXD}
Routing:
- net HV_{CONTROL}: track 56.6 -> 53.0 mm
- net GPS_{TXD}: track 21.4 -> 17.9 mm
- net /INT_{IO-expander}: track 48.6 -> 51.2 mm
- net GPS_{RXD}: track 17.5 -> 15.0 mm
Changed lines of the file:
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@@
       (net 128 "unconnected-(U2-RP_12_LED_G-Pad62)") (pinfunction "RP_12_LED_G") (pintype "no_connect"))
     (pad "63" thru_hole oval (at 7.62 5.08) (size 1.7 1.7) (drill 1) (layers "*.Cu" "*.Mask")
-      (net 31 "GPS_{TXD}") (pinfunction "RP_17") (pintype "input"))
+      (net 110 "HV_{CONTROL}") (pinfunction "RP_17") (pintype "output"))
     (pad "64" thru_hole oval (at 10.16 5.08) (size 1.7 1.7) (drill 1) (layers "*.Cu" "*.Mask")
-      (net 110 "HV_{CONTROL}") (pinfunction "RP_21") (pintype "output"))
+      (net 31 "GPS_{TXD}") (pinfunction "RP_21") (pintype "input"))
     (pad "65" thru_hole oval (at 7.62 7.62) (size 1.7 1.7) (drill 1) (layers "*.Cu" "*.Mask")
       (net 32 "GPS_{RSTN}") (pinfunction "RP_19") (pintype "output"))
@@
       (net 127 "unconnected-(U2-RP_23-Pad66)") (pinfunction "RP_23") (pintype "no_connect"))
     (pad "67" thru_hole oval (at 7.62 10.16) (size 1.7 1.7) (drill 1) (layers "*.Cu" "*.Mask")
-      (net 30 "GPS_{RXD}") (pinfunction "RP_16") (pintype "output"))
+      (net 95 "/INT_{IO-expander}") (pinfunction "RP_16") (pintype "input"))
     (pad "68" thru_hole oval (at 10.16 10.16) (size 1.7 1.7) (drill 1) (layers "*.Cu" "*.Mask")
-      (net 95 "/INT_{IO-expander}") (pinfunction "RP_20") (pintype "input"))
+      (net 30 "GPS_{RXD}") (pinfunction "RP_20") (pintype "output"))
     (pad "69" thru_hole oval (at 7.62 12.7) (size 1.7 1.7) (drill 1) (layers "*.Cu" "*.Mask")
       (net 29 "GPS_{BOOT_SEL}") (pinfunction "RP_18") (pintype "output"))
@@
   (segment (start 121.591 96.331) (end 121.591 92.635) (width 0.25) (layer "F.Cu") (net 30))
   (via (at 121.591 92.635) (size 0.8) (drill 0.4) (layers "F.Cu" "B.Cu") (net 30))
-  (segment (start 113.314 92.635) (end 112.794 93.155) (width 0.25) (layer "B.Cu") (net 30))
-  (segment (start 112.794 93.155) (end 109.765 93.155) (width 0.25) (layer "B.Cu") (net 30))
-  (segment (start 121.591 92.635) (end 113.314 92.635) (width 0.25) (layer "B.Cu") (net 30))
-  (segment (start 109.765 93.155) (end 108.495 94.425) (width 0.25) (layer "B.Cu") (net 30))
-  (segment (start 122.691 90.687) (end 120.079 88.075) (width 0.25) (layer "F.Cu") (net 31))
-  (segment (start 120.079 88.075) (end 109.765 88.075) (width 0.25) (layer "F.Cu") (net 31))
+  (segment (start 112.825 92.635) (end 111.035 94.425) (width 0.25) (layer "B.Cu") (net 30))
+  (segment (start 121.591 92.635) (end 112.825 92.635) (width 0.25) (layer "B.Cu") (net 30))
   (segment (start 122.691 96.331) (end 122.691 90.687) (width 0.25) (layer "F.Cu") (net 31))
-  (segment (start 109.765 88.075) (end 108.495 89.345) (width 0.25) (layer "F.Cu") (net 31))
+  (segment (start 122.691 90.687) (end 121.349 89.345) (width 0.25) (layer "F.Cu") (net 31))
+  (segment (start 121.349 89.345) (end 111.035 89.345) (width 0.25) (layer "F.Cu") (net 31))
   (segment (start 118.999 102.235) (end 114.427 102.235) (width 0.25) (layer "F.Cu") (net 32))
   (segment (start 112.903 100.711) (end 112.903 94.152) (width 0.25) (layer "F.Cu") (net 32))
@@
   (segment (start 130.4825 67.945) (end 129.003 67.945) (width 0.25) (layer "F.Cu") (net 95))
   (via (at 128.27 92.583) (size 0.8) (drill 0.4) (layers "F.Cu" "B.Cu") (net 95))
-  (segment (start 128.27 92.583) (end 125.222 95.631) (width 0.25) (layer "B.Cu") (net 95))
-  (segment (start 112.241 95.631) (end 111.035 94.425) (width 0.25) (layer "B.Cu") (net 95))
-  (segment (start 125.222 95.631) (end 112.241 95.631) (width 0.25) (layer "B.Cu") (net 95))
+  (segment (start 125.158 95.695) (end 109.765 95.695) (width 0.25) (layer "B.Cu") (net 95))
+  (segment (start 128.27 92.583) (end 125.158 95.695) (width 0.25) (layer "B.Cu") (net 95))
+  (segment (start 109.765 95.695) (end 108.495 94.425) (width 0.25) (layer "B.Cu") (net 95))
   (segment (start 134.375 69.351) (end 130.429 65.405) (width 0.25) (layer "F.Cu") (net 97))
   (segment (start 130.667 92.583) (end 134.375 88.875) (width 0.25) (layer "F.Cu") (net 97))
@@
   (segment (start 59.963452 80.915384) (end 59.963452 83.163452) (width 0.25) (layer "F.Cu") (net 108))
   (segment (start 60.115 84.965) (end 61.865 84.965) (width 0.25) (layer "F.Cu") (net 109))
-  (segment (start 102.12 88.075) (end 102.12 88.12) (width 0.25) (layer "F.Cu") (net 110))
-  (segment (start 109.765 90.615) (end 111.035 89.345) (width 0.25) (layer "F.Cu") (net 110))
   (segment (start 68.045 66.14) (end 67.31 66.14) (width 0.25) (layer "F.Cu") (net 110))
-  (segment (start 104.615 90.615) (end 109.765 90.615) (width 0.25) (layer "F.Cu") (net 110))
-  (segment (start 102.12 88.12) (end 104.615 90.615) (width 0.25) (layer "F.Cu") (net 110))
+  (segment (start 102.12 88.12) (end 103.345 89.345) (width 0.25) (layer "F.Cu") (net 110))
+  (segment (start 103.345 89.345) (end 108.495 89.345) (width 0.25) (layer "F.Cu") (net 110))
   (segment (start 69.215 67.31) (end 68.045 66.14) (width 0.25) (layer "F.Cu") (net 110))
+  (segment (start 102.12 88.075) (end 102.12 88.12) (width 0.25) (layer "F.Cu") (net 110))
   (via (at 102.12 88.075) (size 0.8) (drill 0.4) (layers "F.Cu" "B.Cu") (net 110))
   (via (at 69.215 67.31) (size 0.8) (drill 0.4) (layers "F.Cu" "B.Cu") (net 110))

Commit message: add thermal reliefs
Parts:
- moved L1 0.83 mm to (34.0, 99.1)
- moved D1 0.50 mm to (41.1, 102.4)
Routing:
- net /High voltage supply/HV_{BOOST}: track 21.5 -> 19.3 mm
- net HV_{SENSE}: track 10.1 -> 9.44 mm

Commit message: daughter board no TH components
Parts:
- moved U12 6.56 mm to (25.8, 46.7)

Commit message: switch all components to SMT
layout is a mess
Parts:
- BT1: footprint Battery:BatteryHolder_Keystone_103_1x20mm -> Battery:BatteryHolder_Keystone_3002_1x2032
- J1, J10, J2, J3, J4, J5, J7, J8, J9: footprint Connector_PinHeader_2.54mm:PinHeader_1x02_P2.54mm_Vertical -> Connector_PinHeader_2.54mm:PinHeader_1x02_P2.54mm_Vertical_SMD_Pin1Left
- J11: footprint Connector_PinSocket_2.54mm:PinSocket_2x05_P2.54mm_Horizontal -> 00_lib:M207920542R
- RV1: footprint Potentiometer_THT:Potentiometer_Bourns_3266Z_Horizontal -> Potentiometer_SMD:Potentiometer_Bourns_3269X_Horizontal
- moved BT1 11.6 mm to (151.9, 87.0)
- moved J11 7.31 mm to (23.5, 31.8), turned to 90 degrees
- moved U8 6.56 mm to (133.4, 46.7)
- moved U10 6.56 mm to (79.6, 46.7)
- moved U11 6.56 mm to (50.6, 46.7)
- moved U9 6.56 mm to (104.4, 46.7)
- moved U7 6.56 mm to (158.2, 46.7)
- moved RV1 2.83 mm to (142.2, 112.4)
- moved J4 1.81 mm to (116.8, 53.3)
Routing:
- net CLOCK_{HV}: track 245.4 -> 57.6 mm, vias 2 -> 0
- net +5V: track 51.7 -> 216.1 mm
- net LSD_{SHUNT}: track 11.8 -> 26.4 mm
- net +3.3V: track 36.6 -> 45.5 mm, vias 7 -> 9
- net /~{USB_BOOT}: track 10.5 -> 8.52 mm

Commit message: switch to all SM components
Parts:
- added H10: MountingHole_Pad, MountingHole:MountingHole_2.7mm_M2.5_Pad_Via, F.Cu at (56.7, 19.9)
- added H11: MountingHole_Pad, MountingHole:MountingHole_2.7mm_M2.5_Pad_Via, F.Cu at (73.7, 19.9)
- added H12: MountingHole_Pad, MountingHole:MountingHole_2.7mm_M2.5_Pad_Via, F.Cu at (85.7, 19.9)
- added H13: MountingHole_Pad, MountingHole:MountingHole_2.7mm_M2.5_Pad_Via, F.Cu at (98.5, 19.9)
- added H14: MountingHole_Pad, MountingHole:MountingHole_2.7mm_M2.5_Pad_Via, F.Cu at (110.5, 19.9)
- added H15: MountingHole_Pad, MountingHole:MountingHole_2.7mm_M2.5_Pad_Via, F.Cu at (127.5, 19.9)
- added H16: MountingHole_Pad, MountingHole:MountingHole_2.7mm_M2.5_Pad_Via, F.Cu at (139.5, 19.9)
- added H17: MountingHole_Pad, MountingHole:MountingHole_2.7mm_M2.5_Pad_Via, F.Cu at (152.3, 19.9)
- added H18: MountingHole_Pad, MountingHole:MountingHole_2.7mm_M2.5_Pad_Via, F.Cu at (164.3, 19.9)
- added H3: MountingHole_Pad, MountingHole:MountingHole_2.7mm_M2.5_Pad_Via, F.Cu at (109.8, 113.5)
- added H4: MountingHole_Pad, MountingHole:MountingHole_2.7mm_M2.5_Pad_Via, F.Cu at (164.3, 113.5)
- added H5: MountingHole_Pad, MountingHole:MountingHole_2.7mm_M2.5_Pad_Via, F.Cu at (92.0, 57.6)
- added H6: MountingHole_Pad, MountingHole:MountingHole_2.7mm_M2.5_Pad_Via, F.Cu at (109.8, 57.6)
- added H7: MountingHole_Pad, MountingHole:MountingHole_2.7mm_M2.5_Pad_Via, F.Cu at (19.9, 19.9)
- added H8: MountingHole_Pad, MountingHole:MountingHole_2.7mm_M2.5_Pad_Via, F.Cu at (31.9, 19.9)
- added H9: MountingHole_Pad, MountingHole:MountingHole_2.7mm_M2.5_Pad_Via, F.Cu at (44.7, 19.9)
- added J5: pico iCE (B), 00_lib:pico iCE (B), F.Cu at (109.8, 84.3)
- J4: renamed from U2; value pico iCE -> pico iCE (A); footprint 00_lib:pico iCE -> 00_lib:pico iCE (A)
- moved H2 72.3 mm to (92.0, 113.5)
- moved J4 8.91 mm to (92.0, 84.3)
- renumbered J4 to J1, J8 to J10, J9 to J11, J10 to J12, U7 to J13, U8 to J14, U9 to J15, U10 to J16, U11 to J17, U12 to J18, J11 to J19, J1 to J3, J3 to J6, J5 to J7, J6 to J8, J7 to J9, U3 to U2, U4 to U3, U5 to U4, U6 to U5, U13 to U6, U14 to U7, U15 to U8
Routing:
- net SENSE_{PRECISE}: track 123.6 -> 0.00 mm, vias 1 -> 0
- net +5V: track 216.1 -> 339.7 mm, vias 10 -> 11
- net unconnected-(J5-ICE_14_SO/RP_8-Pad2): track 0.00 -> 107.8 mm, vias 0 -> 3
- net DATA_{PRECISE}: track 107.8 -> 0.00 mm, vias 3 -> 0
- net /3.3V_{SENSE}: track 26.2 -> 14.4 mm, vias 3 -> 2
- net GND: track 124.1 -> 135.9 mm, vias 25 -> 26

Commit message: switch to static level shifting
Parts:
- added C21: 0.1u, Capacitor_SMD:C_0603_1608Metric, F.Cu at (104.1, 23.5)
- added C22: 0.1u, Capacitor_SMD:C_0603_1608Metric, F.Cu at (113.7, 25.4)
- added C23: 0.1u, Capacitor_SMD:C_0603_1608Metric, F.Cu at (73.7, 34.3)
- added C24: 0.1u, Capacitor_SMD:C_0603_1608Metric, F.Cu at (81.3, 34.3)
- added U10: ~, Package_SO:TSSOP-14_4.4x5mm_P0.65mm, F.Cu at (77.5, 38.1)
- added U9: ~, Package_SO:TSSOP-14_4.4x5mm_P0.65mm, F.Cu at (108.0, 27.3)
- R27: value 100k -> 10M
- R29: value 10M -> 10k
- R30: value 100k -> 10k
- U6: value ADC0820BCWMX -> ~; footprint Package_SO:SOIC-20W_7.5x12.8mm_P1.27mm -> Package_SO:TSSOP-14_4.4x5mm_P0.65mm
- U7: value TXB0108PWR -> ~; footprint Package_SO:TSSOP-20_4.4x6.5mm_P0.65mm -> Package_SO:TSSOP-14_4.4x5mm_P0.65mm
- U8: value TXB0108PWR -> ADC0820BCWMX; footprint Package_SO:TSSOP-20_4.4x6.5mm_P0.65mm -> Package_SO:SOIC-20W_7.5x12.8mm_P1.27mm
- moved R27 59.1 mm to (55.2, 32.4)
- moved C18 37.6 mm to (73.7, 31.1), turned to 0 degrees
- moved C17 32.9 mm to (81.3, 31.1), turned to 180 degrees
- moved R28 28.3 mm to (60.3, 32.4), turned to 0 degrees
- moved U6 24.3 mm to (77.5, 27.3)
- moved C20 21.4 mm to (111.8, 34.3), turned to 180 degrees
- moved TP14 19.9 mm to (22.5, 60.3)
- moved TP15 18.2 mm to (30.1, 60.3)
- moved C19 16.7 mm to (104.1, 34.3), turned to 0 degrees
- moved TP6 14.8 mm to (38.0, 53.7)
- moved C16 13.3 mm to (96.5, 25.4)
- moved Q5 7.48 mm to (43.1, 30.4)
- moved R29 7.48 mm to (43.7, 35.6)
- moved R30 7.48 mm to (46.3, 35.6)
- moved U7 6.88 mm to (108.0, 38.1), turned to 0 degrees
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Connections:
- C17 pad 1: +3.3V -> +5V
- C18 pad 1: +5V -> +3.3V
- C19 pad 1: +3.3V -> +5V
- C20 pad 1: +5V -> +3.3V
- J5 pad 7: CLOCK_{PRECISE} -> DATA_{PRECISE}
- J5 pad 8: DATA_{PRECISE} -> CLOCK_{PRECISE}
- R27 pad 1: GND -> LSD_{SHUNT}
- R27 pad 2: /LSD ADC/OE_{lvl-shift-1} -> /LSD ADC/LSD_{SHUNT_div}
- R28 pad 1: GND -> /LSD ADC/LSD_{SHUNT_div}
- R28 pad 2: /LSD ADC/OE_{lvl-shift-2} -> VPP
- R29 pad 1: LSD_{SHUNT} -> HV_{MEASURE}
- R29 pad 2: /LSD ADC/LSD_{SHUNT_div} -> /LSD ADC/V_{SHUNT}
- R30 pad 1: /LSD ADC/LSD_{SHUNT_div} -> /LSD ADC/LSD_{SHUNT_SC_Emitter}
- R30 pad 2: VPP -> GND
- U6 pad 1: /LSD ADC/V_{SHUNT} -> /LSD ADC/VCC_{lvl-shift-A-1}
- U6 pad 10: GND -> LSD_{ADC_D0}
- U6 pad 11: GND -> LSD_{ADC_D1}
- U6 pad 12: HV_{MEASURE} -> LSD_{ADC_D2}
- U6 pad 13: /LSD ADC/LSD_{ADC_5V_~{CS}} -> LSD_{ADC_D3}
- U6 pad 14: /LSD ADC/LSD_{ADC_5V_D4} -> /LSD ADC/VCC_{lvl-shift-B-1}
- U6 pad 2: /LSD ADC/LSD_{ADC_5V_D0} -> /LSD ADC/LSD_{ADC_5V_D3}
- U6 pad 3: /LSD ADC/LSD_{ADC_5V_D1} -> /LSD ADC/LSD_{ADC_5V_D2}
- U6 pad 4: /LSD ADC/LSD_{ADC_5V_D2} -> /LSD ADC/LSD_{ADC_5V_D1}
- U6 pad 5: /LSD ADC/LSD_{ADC_5V_D3} -> /LSD ADC/LSD_{ADC_5V_D0}
- U6 pad 6: /LSD ADC/LSD_{ADC_5V_~{WR}/RDY} -> unconnected-(U6-NC-Pad6)
- U6 pad 7: /LSD ADC/LSD_{ADC_5V_MODE} -> GND
- U6 pad 8: /LSD ADC/LSD_{ADC_5V_~{RD}} -> +3.3V
- U6 pad 9: /LSD ADC/LSD_{ADC_5V_~{INT}} -> unconnected-(U6-NC-Pad9)
- U7 pad 1: LSD_{ADC_D3} -> /LSD ADC/VCC_{lvl-shift-A-2}
- U7 pad 10: /LSD ADC/OE_{lvl-shift-1} -> LSD_{ADC_D4}
- U7 pad 11: GND -> LSD_{ADC_D5}
- U7 pad 12: /LSD ADC/LSD_{ADC_5V_~{INT}} -> LSD_{ADC_D6}
- U7 pad 13: /LSD ADC/LSD_{ADC_5V_~{RD}} -> LSD_{ADC_D7}
- U7 pad 14: /LSD ADC/LSD_{ADC_5V_MODE} -> /LSD ADC/VCC_{lvl-shift-B-2}
- U7 pad 2: /LSD ADC/VCC_{lvl-shift-A-1} -> /LSD ADC/LSD_{ADC_5V_D7}
- U7 pad 3: LSD_{ADC_D2} -> /LSD ADC/LSD_{ADC_5V_D6}
- U7 pad 4: LSD_{ADC_D1} -> /LSD ADC/LSD_{ADC_5V_D5}
- U7 pad 5: LSD_{ADC_D0} -> /LSD ADC/LSD_{ADC_5V_D4}
- U7 pad 6: LSD_{ADC_~{WR}/RDY} -> unconnected-(U7-NC-Pad6)
- U7 pad 7: LSD_{ADC_MODE} -> GND
- U7 pad 8: LSD_{ADC_~{RD}} -> +3.3V
- U7 pad 9: LSD_{ADC_~{INT}} -> unconnected-(U7-NC-Pad9)
- U8 pad 1: unconnected-(U8-A1-Pad1) -> /LSD ADC/V_{SHUNT}
- U8 pad 10: /LSD ADC/OE_{lvl-shift-2} -> GND
- U8 pad 12: unconnected-(U8-B8-Pad12) -> HV_{MEASURE}
- U8 pad 13: /LSD ADC/LSD_{ADC_5V_~{OFL}} -> /LSD ADC/LSD_{ADC_5V_~{CS}}
- U8 pad 14: /LSD ADC/LSD_{ADC_5V_D7} -> /LSD ADC/LSD_{ADC_5V_D4}
- U8 pad 15: /LSD ADC/LSD_{ADC_5V_D6} -> /LSD ADC/LSD_{ADC_5V_D5}
- U8 pad 16: /LSD ADC/LSD_{ADC_5V_D5} -> /LSD ADC/LSD_{ADC_5V_D6}
- U8 pad 17: /LSD ADC/LSD_{ADC_5V_D4} -> /LSD ADC/LSD_{ADC_5V_D7}
- U8 pad 18: /LSD ADC/LSD_{ADC_5V_~{CS}} -> /LSD ADC/LSD_{ADC_5V_~{OFL}}
- U8 pad 19: /LSD ADC/VCC_{lvl-shift-B-2} -> unconnected-(U8-NC-Pad19)
- U8 pad 2: /LSD ADC/VCC_{lvl-shift-A-2} -> /LSD ADC/LSD_{ADC_5V_D0}
- U8 pad 20: unconnected-(U8-B1-Pad20) -> /LSD ADC/VCC_{ADC}
- U8 pad 3: LSD_{ADC_~{CS}} -> /LSD ADC/LSD_{ADC_5V_D1}
- U8 pad 4: LSD_{ADC_D4} -> /LSD ADC/LSD_{ADC_5V_D2}
- U8 pad 5: LSD_{ADC_D5} -> /LSD ADC/LSD_{ADC_5V_D3}
- U8 pad 6: LSD_{ADC_D6} -> /LSD ADC/LSD_{ADC_5V_~{WR}/RDY}
- U8 pad 7: LSD_{ADC_D7} -> /LSD ADC/LSD_{ADC_5V_MODE}
- U8 pad 8: LSD_{ADC_~{OFL}} -> /LSD ADC/LSD_{ADC_5V_~{RD}}
- U8 pad 9: unconnected-(U8-A8-Pad9) -> /LSD ADC/LSD_{ADC_5V_~{INT}}
Routing:
- net +5V: track 339.7 -> 11.2 mm, vias 11 -> 7
- net PPS_{TRIMMED}: track 224.2 -> 47.9 mm, vias 0 -> 1
- net VPP: track 195.1 -> 27.2 mm, vias 1 -> 0
- net /LSD ADC/V_{SHUNT}: track 112.2 -> 0.00 mm
- net unconnected-(J5-ICE_14_SO/RP_8-Pad2): track 107.8 -> 0.00 mm, vias 3 -> 0
- net DATA_{HV}: track 104.8 -> 0.00 mm
- net CLOCK_{PRECISE}: track 110.9 -> 8.67 mm, vias 3 -> 0
- net LSD_{ADC_~{WR}/RDY}: track 93.6 -> 0.00 mm, vias 1 -> 0
- net LSD_{ADC_D1}: track 87.6 -> 0.00 mm
- net LSD_{ADC_~{INT}}: track 86.6 -> 0.00 mm, vias 1 -> 0
- net LSD_{ADC_~{RD}}: track 85.8 -> 0.00 mm, vias 1 -> 0
- net LSD_{ADC_D0}: track 84.2 -> 0.00 mm
- net LSD_{ADC_MODE}: track 80.1 -> 0.00 mm, vias 1 -> 0
- net HV_{MEASURE}: track 134.5 -> 70.4 mm
- net LSD_{ADC_D4}: track 60.7 -> 0.00 mm
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- removed copper zone on F.Cu, net +3V3_STDBY

Commit message: HV overhaul
Parallel single stage boost convertor
Need to find replacement MOSFET because SiB452BK footprint is too small for reasonable manufacturing and HV clearance.
Parts:
- removed C22, C23, C24: 0.1u, Capacitor_SMD:C_0603_1608Metric
- removed J18: ~, 00_lib:IN-14 daughter board
- removed J19: Conn_02x05_Odd_Even, 00_lib:M207920542R
- removed Q1, Q2, Q3, Q4, Q5: BSP88, Package_TO_SOT_SMD:SOT-223-3_TabPin2
- removed R10, R13: 4.7k, Resistor_SMD:R_0603_1608Metric
- removed R11: 62k, Resistor_SMD:R_0603_1608Metric
- removed R12, R27: 10M, Resistor_SMD:R_0603_1608Metric
- removed R14, R15: 1k, Resistor_SMD:R_0603_1608Metric
- removed R16, R18, R22, R26, R28: 100k, Resistor_SMD:R_0603_1608Metric
- removed R17: 40m, Resistor_SMD:R_0603_1608Metric
- removed R19: 220k, Resistor_SMD:R_0603_1608Metric
- removed R20: 2.7M, Resistor_SMD:R_0603_1608Metric
- removed R21, R29, R30, R31, R32: 10k, Resistor_SMD:R_0603_1608Metric
- removed R23: 15k, Resistor_SMD:R_0603_1608Metric
- removed R24: 1M, Resistor_SMD:R_0603_1608Metric
- removed R25: 10k, Resistor_SMD:R_2512_6332Metric
- removed TP14, TP15, TP16, TP17: TestPoint, 00_lib:TestPoint_Keystone_5019_Minature
- added D4: SM4004, Diode_SMD:D_MELF, F.Cu at (81.9, 84.5)
- added D5: SM4004, Diode_SMD:D_MELF, F.Cu at (23.4, 78.7)
- added D6: SM4004, Diode_SMD:D_MELF, F.Cu at (35.5, 71.8)
- added D7: SM4004, Diode_SMD:D_MELF, F.Cu at (37.4, 78.1)
- added D8: SM4004, Diode_SMD:D_MELF, F.Cu at (46.3, 84.5)
- added D9: SM4004, Diode_SMD:D_MELF, F.Cu at (3.44, 23.7)
- added U11: ~, Package_SO:TSSOP-14_4.4x5mm_P0.65mm, F.Cu at (105.4, 29.8)
- added U12: ~, Package_SO:TSSOP-14_4.4x5mm_P0.65mm, F.Cu at (79.1, 37.5)
- C10, C5: value 10u -> 1u
- C11, C4, C7, C8, C9: footprint Capacitor_SMD:C_0603_1608Metric -> Capacitor_SMD:CP_Elec_8x10
- C12: value 1n -> 1u
- C13, C15: value 1u -> 0.1u
- C6: value 0.1u -> 1u; footprint Capacitor_SMD:C_0603_1608Metric -> Capacitor_SMD:CP_Elec_8x10
- J11, J12: value Conn_01x02_Pin -> ~; footprint Connector_PinHeader_2.54mm:PinHeader_1x02_P2.54mm_Vertical_SMD_Pin1Left -> 00_lib:IN-14 daughter board
- J17: value ~ -> Conn_02x05_Odd_Even; footprint 00_lib:IN-14 daughter board -> 00_lib:M207920542R
- L1: value 15u -> 10u; footprint 00_lib:IND_VLS6045EX-150M -> 00_lib:IND_BOURNS_SRR1280
- L2: value 820u -> 10u; footprint 00_lib:IND_MSS1583_COC -> 00_lib:IND_BOURNS_SRR1280
- R3: value 62k -> 10M
- R4: value 27k -> 100k
- R5: value 40m -> 1M
- R6: value 100k -> 10k; footprint Resistor_SMD:R_0603_1608Metric -> Resistor_SMD:R_2512_6332Metric
- R8: value 100k -> 1M
- R9: value 470 -> 47k
- U10: value ~ -> ADC0820BCWMX; footprint Package_SO:TSSOP-14_4.4x5mm_P0.65mm -> Package_SO:SOIC-20W_7.5x12.8mm_P1.27mm
- U4, U5: value LM51561HPWPR -> SIB452DK-T1-GE3; footprint 00_lib:PWP0014H-IPC_C -> 00_lib:SON_K-T1-GE3_VIS
- U6, U7: value ~ -> SIB452DK-T1-GE3; footprint Package_SO:TSSOP-14_4.4x5mm_P0.65mm -> 00_lib:SON_K-T1-GE3_VIS
- U8: value ADC0820BCWMX -> ~; footprint Package_SO:SOIC-20W_7.5x12.8mm_P1.27mm -> Package_SO:TSSOP-14_4.4x5mm_P0.65mm
- moved J11 121.5 mm to (158.2, 46.7)
- moved U7 103.0 mm to (5.16, 30.9)
- moved R8 101.7 mm to (-16.0, 25.4), turned to 0 degrees
- moved TP10 81.3 mm to (-3.41, 22.5), turned to 0 degrees
- moved TP12 79.3 mm to (-11.2, 18.6)
- moved TP9 78.2 mm to (-3.41, 18.6), turned to 0 degrees
- moved C12 78.0 mm to (1.47, 27.1), turned to 0 degrees
- moved R9 78.0 mm to (-16.0, 27.9)
- moved U6 72.3 mm to (5.16, 27.5), turned to 0 degrees
- moved TP13 65.6 mm to (-11.2, 22.5)
- moved TP11 64.9 mm to (-3.41, 26.5)
- moved R5 63.7 mm to (1.47, 29.6), turned to 0 degrees
- moved R6 62.7 mm to (3.81, 19.1), turned to 0 degrees
- moved J12 62.4 mm to (133.4, 46.7)
- moved R7 54.9 mm to (1.47, 32.1), turned to 0 degrees
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Connections:
- C11 pad 1: GND -> /High voltage supply/Boost Quadrupler 2/HV_{HALF-SUPPLY}
- C11 pad 2: /High voltage supply/HV_{SS} -> GND
- C12 pad 1: /High voltage supply/HV_{COMP} -> /HV bleed/HV_bleed_{source}
- C13 pad 1: /High voltage supply/HV_{COMP-1} -> +5V
- C13 pad 2: GND -> /LSD ADC/VCC_{ADC}
- C14 pad 1: /High voltage supply/HV_{FB} -> +5V
- C14 pad 2: GND -> /LSD ADC/VCC_{lvl-shift-A-1}
- C15 pad 1: /HV bleed/HV_bleed_{source} -> +3.3V
- C15 pad 2: GND -> /LSD ADC/VCC_{lvl-shift-B-1}
- C16 pad 2: /LSD ADC/VCC_{ADC} -> /LSD ADC/VCC_{lvl-shift-A-2}
- C17 pad 1: +5V -> +3.3V
- C17 pad 2: /LSD ADC/VCC_{lvl-shift-A-1} -> /LSD ADC/VCC_{lvl-shift-B-2}
- C18 pad 1: +3.3V -> +5V
- C18 pad 2: /LSD ADC/VCC_{lvl-shift-B-1} -> /LSD ADC/VCC_{lvl-shift-A-3}
- C19 pad 1: +5V -> +3.3V
- C19 pad 2: /LSD ADC/VCC_{lvl-shift-A-2} -> /LSD ADC/VCC_{lvl-shift-B-3}
- C20 pad 2: /LSD ADC/VCC_{lvl-shift-B-2} -> /LSD ADC/VCC_{lvl-shift-A-4}
- C21 pad 2: /LSD ADC/VCC_{lvl-shift-A-3} -> /LSD ADC/VCC_{lvl-shift-B-4}
- C4 pad 1: /20V supply/20V_{VCC} -> /High voltage supply/Boost Quadrupler 1/HV_{FULL-BOOST}
- C4 pad 2: GND -> /High voltage supply/Boost Quadrupler 1/HV_{HALF-BOOST}
- C5 pad 1: /20V supply/20V_{SENSE} -> /High voltage supply/Boost Quadrupler 1/HV_{QUARTER-BOOST}
- C5 pad 2: GND -> /High voltage supply/Boost Quadrupler 1/HV_{HALF-BOOST}
- C6 pad 1: /20V supply/20V_{SS} -> HV_{SENSE}
- C7 pad 1: /20V supply/20V_{COMP} -> /High voltage supply/Boost Quadrupler 1/HV_{HALF-SUPPLY}
- C8 pad 1: /20V supply/20V_{COMP-1} -> /High voltage supply/Boost Quadrupler 2/HV_{FULL-BOOST}
- C8 pad 2: GND -> /High voltage supply/Boost Quadrupler 2/HV_{HALF-BOOST}
- C9 pad 1: /High voltage supply/HV_{VCC} -> /High voltage supply/Boost Quadrupler 2/HV_{QUARTER-BOOST}
- C9 pad 2: GND -> /High voltage supply/Boost Quadrupler 2/HV_{HALF-BOOST}
- D1 pad 1: /20V supply/20V_{SENSE} -> HV_{SENSE}
- D1 pad 2: /20V supply/20V_{BOOST} -> /High voltage supply/Boost Quadrupler 1/HV_{FULL-BOOST}
- D2 pad 1: HV_{SENSE} -> /High voltage supply/Boost Quadrupler 1/HV_{FULL-BOOST}
- D2 pad 2: /High voltage supply/HV_{BOOST} -> /High voltage supply/Boost Quadrupler 1/HV_{HALF-SUPPLY}
- D3 pad 1: /HV bleed/HV_bleed_{gate} -> /High voltage supply/Boost Quadrupler 1/HV_{HALF-SUPPLY}
- D3 pad 2: /HV bleed/HV_bleed_{pulldown} -> /High voltage supply/Boost Quadrupler 1/HV_{QUARTER-BOOST}
- J10 pad 1: +5V -> HV_{SENSE}
- J10 pad 2: /20V supply/5V_20V_{SENSE} -> VPP
- J11 pad 1: /20V supply/20V_{SENSE} -> /Nixies/DAISY_{HV-1}
- J11 pad 2: +20V -> +5V
- J12 pad 1: HV_{SENSE} -> /Nixies/DAISY_{HV-2}
- J12 pad 2: VPP -> +5V
- J13 pad 1: /Nixies/DAISY_{HV-1} -> /Nixies/DAISY_{HV-3}
- J13 pad 4: DATA_{HV} -> /Nixies/DAISY_{HV-2}
- J14 pad 1: /Nixies/DAISY_{HV-2} -> /Nixies/DAISY_{HV-4}
- J14 pad 4: /Nixies/DAISY_{HV-1} -> /Nixies/DAISY_{HV-3}
- J15 pad 1: /Nixies/DAISY_{HV-3} -> /Nixies/DAISY_{HV-5}
- J15 pad 4: /Nixies/DAISY_{HV-2} -> /Nixies/DAISY_{HV-4}
- J16 pad 1: /Nixies/DAISY_{HV-4} -> /Nixies/D_{IN-PRECISE}
- J16 pad 4: /Nixies/DAISY_{HV-3} -> /Nixies/DAISY_{HV-5}
- J16 pad 7: unconnected-(J16-ANODE-Pad7) -> LSD_{SHUNT}
- J17 pad 1: /Nixies/DAISY_{HV-5} -> DATA_{PRECISE}
- J17 pad 10: GND -> SENSE_{PRECISE}
- J17 pad 4: /Nixies/DAISY_{HV-4} -> /Nixies/D_{IN-PRECISE}
- J17 pad 7: unconnected-(J17-ANODE-Pad7) -> CLOCK_{PRECISE}
- J5 pad 19: HV_{MEASURE} -> MEASURE_{HV}
- J5 pad 23: HV_{CONTROL} -> GATE_{HV}
- L1 pad 2: /20V supply/20V_{BOOST} -> /High voltage supply/Boost Quadrupler 1/HV_{HALF-BOOST}
- L2 pad 1: +20V -> +5V
- L2 pad 2: /High voltage supply/HV_{BOOST} -> /High voltage supply/Boost Quadrupler 2/HV_{HALF-BOOST}
- R3 pad 1: /20V supply/20V_{UVLO} -> VPP
- R3 pad 2: /20V supply/5V_20V_{SENSE} -> MEASURE_{HV}
- R4 pad 1: GND -> MEASURE_{HV}
- R4 pad 2: /20V supply/20V_{UVLO} -> GND
- R5 pad 1: /20V supply/20V_{CS} -> /HV bleed/HV_bleed_{pulldown}
- R5 pad 2: GND -> HV_{SENSE}
- R6 pad 1: /20V supply/20V_{PGOOD} -> HV_{SENSE}
- R6 pad 2: /20V supply/20V_{VCC} -> /HV bleed/HV_bleed_{drain}
- R7 pad 1: GND -> /HV bleed/HV_bleed_{source}
- R7 pad 2: /20V supply/20V_{RT} -> GND
- R8 pad 1: /20V supply/20V_{FB} -> /LSD ADC/V_{SHUNT}
- R8 pad 2: /20V supply/20V_{SENSE} -> LSD_{SHUNT}
- R9 pad 1: /20V supply/20V_{COMP} -> GND
- R9 pad 2: /20V supply/20V_{COMP-1} -> /LSD ADC/V_{SHUNT}
- TP1 pad 1: /20V supply/20V_{BOOST} -> /High voltage supply/Boost Quadrupler 1/HV_{HALF-BOOST}
- TP10 pad 1: /High voltage supply/HV_{COMP} -> /HV bleed/HV_bleed_{gate}
- TP11 pad 1: /HV bleed/HV_bleed_{drain} -> /HV bleed/HV_bleed_{source}
- TP12 pad 1: /HV bleed/HV_bleed_{gate} -> /LSD ADC/V_{SHUNT}
- TP13 pad 1: /HV bleed/HV_bleed_{source} -> GND
- TP2 pad 1: /20V supply/20V_{UVLO} -> /High voltage supply/Boost Quadrupler 1/HV_{FULL-BOOST}
- TP3 pad 1: /20V supply/20V_{GATE} -> /High voltage supply/Boost Quadrupler 1/HV_{QUARTER-BOOST}
- TP4 pad 1: /20V supply/20V_{FB} -> /High voltage supply/Boost Quadrupler 1/HV_{HALF-SUPPLY}
- TP5 pad 1: /20V supply/20V_{COMP} -> /High voltage supply/Boost Quadrupler 2/HV_{HALF-BOOST}
- TP6 pad 1: GND -> /High voltage supply/Boost Quadrupler 2/HV_{FULL-BOOST}
- TP7 pad 1: /High voltage supply/HV_{BOOST} -> /High voltage supply/Boost Quadrupler 2/HV_{QUARTER-BOOST}
- TP8 pad 1: /High voltage supply/HV_{GATE} -> /High voltage supply/Boost Quadrupler 2/HV_{HALF-SUPPLY}
- TP9 pad 1: /High voltage supply/HV_{FB} -> /HV bleed/HV_bleed_{drain}
- U10 pad 1: /LSD ADC/VCC_{lvl-shift-A-4} -> /LSD ADC/V_{SHUNT}
- U10 pad 10: /LSD ADC/LSD_{ADC_5V_~{CS}} -> GND
- U10 pad 11: /LSD ADC/LSD_{ADC_5V_~{RD}} -> GND
- U10 pad 12: /LSD ADC/LSD_{ADC_5V_MODE} -> MEASURE_{HV}
- U10 pad 13: /LSD ADC/LSD_{ADC_5V_~{WR}/RDY} -> /LSD ADC/LSD_{ADC_5V_~{CS}}
- U10 pad 14: /LSD ADC/VCC_{lvl-shift-B-4} -> /LSD ADC/LSD_{ADC_5V_D4}
- U10 pad 2: LSD_{ADC_~{WR}/RDY} -> /LSD ADC/LSD_{ADC_5V_D0}
- U10 pad 3: LSD_{ADC_MODE} -> /LSD ADC/LSD_{ADC_5V_D1}
- U10 pad 4: LSD_{ADC_~{RD}} -> /LSD ADC/LSD_{ADC_5V_D2}
- U10 pad 5: LSD_{ADC_~{CS}} -> /LSD ADC/LSD_{ADC_5V_D3}
- U10 pad 6: unconnected-(U10-NC-Pad6) -> /LSD ADC/LSD_{ADC_5V_~{WR}/RDY}
- U10 pad 7: GND -> /LSD ADC/LSD_{ADC_5V_MODE}
- U10 pad 8: +3.3V -> /LSD ADC/LSD_{ADC_5V_~{RD}}
- U10 pad 9: unconnected-(U10-NC-Pad9) -> /LSD ADC/LSD_{ADC_5V_~{INT}}
- U4 pad 1: /20V supply/5V_20V_{SENSE} -> /High voltage supply/Boost Quadrupler 1/HV_{HALF-BOOST}
- U4 pad 2: unconnected-(U4-NC-Pad2) -> /High voltage supply/Boost Quadrupler 1/HV_{HALF-BOOST}
- U4 pad 3: /20V supply/20V_{VCC} -> GATE_{HV}
- U4 pad 4: /20V supply/20V_{GATE} -> GND
- U4 pad 5: GND -> /High voltage supply/Boost Quadrupler 1/HV_{HALF-BOOST}
- U4 pad 6: GND -> /High voltage supply/Boost Quadrupler 1/HV_{HALF-BOOST}
- U4 pad 7: /20V supply/20V_{CS} -> GND
- U5 pad 1: +20V -> /High voltage supply/Boost Quadrupler 2/HV_{HALF-BOOST}
- U5 pad 2: unconnected-(U5-NC-Pad2) -> /High voltage supply/Boost Quadrupler 2/HV_{HALF-BOOST}
- U5 pad 3: /High voltage supply/HV_{VCC} -> GATE_{HV}
- U5 pad 4: /High voltage supply/HV_{GATE} -> GND
- U5 pad 5: GND -> /High voltage supply/Boost Quadrupler 2/HV_{HALF-BOOST}
- U5 pad 6: GND -> /High voltage supply/Boost Quadrupler 2/HV_{HALF-BOOST}
- U5 pad 7: /High voltage supply/HV_{CS} -> GND
- U6 pad 1: /LSD ADC/VCC_{lvl-shift-A-1} -> /HV bleed/HV_bleed_{drain}
- U6 pad 2: /LSD ADC/LSD_{ADC_5V_D3} -> /HV bleed/HV_bleed_{drain}
- U6 pad 3: /LSD ADC/LSD_{ADC_5V_D2} -> /HV bleed/HV_bleed_{gate}
- U6 pad 4: /LSD ADC/LSD_{ADC_5V_D1} -> /HV bleed/HV_bleed_{source}
- U6 pad 5: /LSD ADC/LSD_{ADC_5V_D0} -> /HV bleed/HV_bleed_{drain}
- U6 pad 6: unconnected-(U6-NC-Pad6) -> /HV bleed/HV_bleed_{drain}
- U6 pad 7: GND -> /HV bleed/HV_bleed_{source}
- U7 pad 1: /LSD ADC/VCC_{lvl-shift-A-2} -> /HV bleed/HV_bleed_{gate}
- U7 pad 2: /LSD ADC/LSD_{ADC_5V_D7} -> /HV bleed/HV_bleed_{gate}
- U7 pad 3: /LSD ADC/LSD_{ADC_5V_D6} -> +5V
- U7 pad 4: /LSD ADC/LSD_{ADC_5V_D5} -> GND
- U7 pad 5: /LSD ADC/LSD_{ADC_5V_D4} -> /HV bleed/HV_bleed_{gate}
- U7 pad 6: unconnected-(U7-NC-Pad6) -> /HV bleed/HV_bleed_{gate}
- U8 pad 1: /LSD ADC/V_{SHUNT} -> /LSD ADC/VCC_{lvl-shift-A-1}
- U8 pad 10: GND -> LSD_{ADC_D0}
- U8 pad 11: GND -> LSD_{ADC_D1}
- U8 pad 12: HV_{MEASURE} -> LSD_{ADC_D2}
- U8 pad 13: /LSD ADC/LSD_{ADC_5V_~{CS}} -> LSD_{ADC_D3}
- U8 pad 14: /LSD ADC/LSD_{ADC_5V_D4} -> /LSD ADC/VCC_{lvl-shift-B-1}
- U8 pad 2: /LSD ADC/LSD_{ADC_5V_D0} -> /LSD ADC/LSD_{ADC_5V_D3}
- U8 pad 3: /LSD ADC/LSD_{ADC_5V_D1} -> /LSD ADC/LSD_{ADC_5V_D2}
- U8 pad 4: /LSD ADC/LSD_{ADC_5V_D2} -> /LSD ADC/LSD_{ADC_5V_D1}
- U8 pad 5: /LSD ADC/LSD_{ADC_5V_D3} -> /LSD ADC/LSD_{ADC_5V_D0}
- U8 pad 6: /LSD ADC/LSD_{ADC_5V_~{WR}/RDY} -> unconnected-(U8-NC-Pad6)
- U8 pad 7: /LSD ADC/LSD_{ADC_5V_MODE} -> GND
- U8 pad 8: /LSD ADC/LSD_{ADC_5V_~{RD}} -> +3.3V
- U8 pad 9: /LSD ADC/LSD_{ADC_5V_~{INT}} -> unconnected-(U8-NC-Pad9)
- U9 pad 1: /LSD ADC/VCC_{lvl-shift-A-3} -> /LSD ADC/VCC_{lvl-shift-A-2}
- U9 pad 10: LSD_{ADC_~{INT}} -> LSD_{ADC_D4}
- U9 pad 11: LSD_{ADC_~{OFL}} -> LSD_{ADC_D5}
- U9 pad 12: unconnected-(U9-B2Y-Pad12) -> LSD_{ADC_D6}
- U9 pad 13: unconnected-(U9-B1Y-Pad13) -> LSD_{ADC_D7}
- U9 pad 14: /LSD ADC/VCC_{lvl-shift-B-3} -> /LSD ADC/VCC_{lvl-shift-B-2}
- U9 pad 2: /LSD ADC/VCC_{lvl-shift-A-3} -> /LSD ADC/LSD_{ADC_5V_D7}
- U9 pad 3: /LSD ADC/VCC_{lvl-shift-A-3} -> /LSD ADC/LSD_{ADC_5V_D6}
- U9 pad 4: /LSD ADC/LSD_{ADC_5V_~{OFL}} -> /LSD ADC/LSD_{ADC_5V_D5}
- U9 pad 5: /LSD ADC/LSD_{ADC_5V_~{INT}} -> /LSD ADC/LSD_{ADC_5V_D4}
Routing:
- net HV_{MEASURE}: track 70.4 -> 0.00 mm, vias 1 -> 0
- net GND: track 126.6 -> 64.7 mm, vias 22 -> 9
- net +20V: track 36.5 -> 0.00 mm
- net /HV bleed/HV_bleed_{drain}: track 34.8 -> 0.00 mm, vias 2 -> 0
- net /20V supply/20V_{FB}: track 33.7 -> 0.00 mm
- net /High voltage supply/HV_{UVLO}: track 32.3 -> 0.00 mm, vias 2 -> 0
- net HV_{CONTROL}: track 30.2 -> 0.00 mm, vias 1 -> 0
- net /High voltage supply/HV_{GATE}: track 27.8 -> 0.00 mm, vias 2 -> 0
- net VPP: track 27.2 -> 0.00 mm
- net /High voltage supply/HV_{FB}: track 24.1 -> 0.00 mm
- net /HV bleed/HV_bleed_{gate}: track 21.7 -> 0.00 mm
- net /LSD ADC/LSD_{ADC_5V_~{CS}}: track 19.4 -> 0.00 mm
- net /High voltage supply/HV_{BOOST}: track 19.3 -> 0.00 mm
- net /20V supply/20V_{VCC}: track 16.5 -> 0.00 mm, vias 2 -> 0
- net /20V supply/20V_{UVLO}: track 13.9 -> 0.00 mm
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- removed copper zone on F.Cu, net +20V
- removed copper zone on F.Cu, net +5V
- removed copper zone on F.Cu, net /20V supply/20V_{BOOST}
- removed copper zone on F.Cu, net /20V supply/20V_{SENSE}
- removed copper zone on F.Cu, net /20V supply/5V_20V_{SENSE}
- removed copper zone on F.Cu, net /High voltage supply/HV_{BOOST}
- removed copper zone on F.Cu, net HV_{SENSE}
Other:
- board text added: "+200V"
- board text added: "Nixie Accurate Clock, Rev B https://github.com/willis936/nixie-clock-ice"
- board text removed: "+20V"
- board text removed: "+210V"
- board text removed: "Nixie Accurate Clock, Rev A https://github.com/willis936/nixie-clock-ice"
