File: hardware/KiCad/nixieAccurateClock/nixieAccurateClock.kicad_pcb (KiCad board)
At the start: 4 copper layers, 152.4 x 101.6 mm, 108 parts, among them J1 Conn_01x02_Pin, J10 Conn_01x02_Pin, J17 Conn_02x05_Odd_Even, J2 Conn_01x02_Pin, J3 Conn_01x02_Pin, J4 pico iCE (A), J5 pico iCE (B), J6 Conn_01x02_Pin, J7 Conn_01x02_Pin, J8 Conn_Coaxial, J9 Conn_01x02_Pin, SW1 SW_DIP_x08, U1 MCP23008-xSO, U10 ADC0820BCWMX, U2 LTR-329ALS-01, U3 PX1125T, U4 SIB452DK-T1-GE3, U5 SIB452DK-T1-GE3, U6 SIB452DK-T1-GE3, U7 SIB452DK-T1-GE3

Commit message: single stage HV supply
Also switch to a MOSFET with a reasonable footprint
Parts:
- removed C18, C19, C20, C21: 0.1u, Capacitor_SMD:C_0603_1608Metric
- removed D6, D7, D8, D9: SM4004, Diode_SMD:D_MELF
- removed L2: 10u, 00_lib:IND_BOURNS_SRR1280
- removed TP10, TP11, TP12, TP13: TestPoint, 00_lib:TestPoint_Keystone_5019_Minature
- removed U10: ADC0820BCWMX, Package_SO:SOIC-20W_7.5x12.8mm_P1.27mm
- removed U11, U12, U9: ~, Package_SO:TSSOP-14_4.4x5mm_P0.65mm
- added Q1: IRLH5030TRPBF, 00_lib:Infineon-PG-TDSON-8-0-0-MFG, F.Cu at (59.4, 89.7)
- added Q2: BSP88, Package_TO_SOT_SMD:SOT-223-3_TabPin2, F.Cu at (-10.6, 22.0)
- added Q3: BSP88, Package_TO_SOT_SMD:SOT-223-3_TabPin2, F.Cu at (-10.6, 30.2)
- C10, C11, C9: value 1u -> 0.1u; footprint Capacitor_SMD:CP_Elec_8x10 -> Capacitor_SMD:C_0603_1608Metric
- C12: value 1u -> 0.1u
- C8: footprint Capacitor_SMD:CP_Elec_8x10 -> Capacitor_SMD:C_0603_1608Metric
- U4, U5, U7: value SIB452DK-T1-GE3 -> ~; footprint 00_lib:SON_K-T1-GE3_VIS -> Package_SO:TSSOP-14_4.4x5mm_P0.65mm
- U6: value SIB452DK-T1-GE3 -> ADC0820BCWMX; footprint 00_lib:SON_K-T1-GE3_VIS -> Package_SO:SOIC-20W_7.5x12.8mm_P1.27mm
- moved U4 123.3 mm to (-35.7, 21.1), turned to 0 degrees
- moved U8 115.2 mm to (-35.7, 40.8), turned to 0 degrees
- moved C9 95.6 mm to (-29.3, 19.1), turned to 0 degrees
- moved C13 94.7 mm to (-29.3, 29.1)
- moved C14 94.7 mm to (-29.3, 31.6)
- moved U5 92.6 mm to (-35.7, 27.7), turned to 0 degrees
- moved C15 91.8 mm to (-25.3, 19.1)
- moved C16 91.8 mm to (-25.3, 21.6)
- moved C17 91.8 mm to (-25.3, 24.1)
- moved C11 90.4 mm to (-29.3, 24.1)
- moved TP5 86.0 mm to (-2.81, 19.8)
- moved TP8 75.5 mm to (-20.4, 19.8)
- moved C8 72.3 mm to (2.07, 19.1), turned to 0 degrees
- moved C10 70.6 mm to (-29.3, 21.6), turned to 0 degrees
- moved TP7 62.7 mm to (-2.81, 27.7)
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Connections:
- C10 pad 1: HV_{SENSE} -> +5V
- C10 pad 2: GND -> /LSD ADC/VCC_{lvl-shift-A-1}
- C11 pad 1: /High voltage supply/Boost Quadrupler 2/HV_{HALF-SUPPLY} -> +3.3V
- C11 pad 2: GND -> /LSD ADC/VCC_{lvl-shift-B-1}
- C12 pad 1: /HV bleed/HV_bleed_{source} -> +5V
- C12 pad 2: GND -> /LSD ADC/VCC_{lvl-shift-A-2}
- C13 pad 1: +5V -> +3.3V
- C13 pad 2: /LSD ADC/VCC_{ADC} -> /LSD ADC/VCC_{lvl-shift-B-2}
- C14 pad 2: /LSD ADC/VCC_{lvl-shift-A-1} -> /LSD ADC/VCC_{lvl-shift-A-3}
- C15 pad 2: /LSD ADC/VCC_{lvl-shift-B-1} -> /LSD ADC/VCC_{lvl-shift-B-3}
- C16 pad 1: +5V -> +3.3V
- C16 pad 2: /LSD ADC/VCC_{lvl-shift-A-2} -> /LSD ADC/VCC_{lvl-shift-A-4}
- C17 pad 1: +3.3V -> +5V
- C17 pad 2: /LSD ADC/VCC_{lvl-shift-B-2} -> /LSD ADC/VCC_{lvl-shift-B-4}
- C8 pad 1: /High voltage supply/Boost Quadrupler 2/HV_{FULL-BOOST} -> /HV bleed/HV_bleed_{source}
- C8 pad 2: /High voltage supply/Boost Quadrupler 2/HV_{HALF-BOOST} -> GND
- C9 pad 1: /High voltage supply/Boost Quadrupler 2/HV_{QUARTER-BOOST} -> +5V
- C9 pad 2: /High voltage supply/Boost Quadrupler 2/HV_{HALF-BOOST} -> /LSD ADC/VCC_{ADC}
- D5 pad 1: HV_{SENSE} -> /HV bleed/HV_bleed_{gate}
- D5 pad 2: /High voltage supply/Boost Quadrupler 2/HV_{FULL-BOOST} -> /HV bleed/HV_bleed_{pulldown}
- TP5 pad 1: /High voltage supply/Boost Quadrupler 2/HV_{HALF-BOOST} -> /HV bleed/HV_bleed_{drain}
- TP6 pad 1: /High voltage supply/Boost Quadrupler 2/HV_{FULL-BOOST} -> /HV bleed/HV_bleed_{gate}
- TP7 pad 1: /High voltage supply/Boost Quadrupler 2/HV_{QUARTER-BOOST} -> /HV bleed/HV_bleed_{source}
- TP8 pad 1: /High voltage supply/Boost Quadrupler 2/HV_{HALF-SUPPLY} -> /LSD ADC/V_{SHUNT}
- TP9 pad 1: /HV bleed/HV_bleed_{drain} -> GND
- U4 pad 1: /High voltage supply/Boost Quadrupler 1/HV_{HALF-BOOST} -> /LSD ADC/VCC_{lvl-shift-A-1}
- U4 pad 2: /High voltage supply/Boost Quadrupler 1/HV_{HALF-BOOST} -> /LSD ADC/LSD_{ADC_5V_D3}
- U4 pad 3: GATE_{HV} -> /LSD ADC/LSD_{ADC_5V_D2}
- U4 pad 4: GND -> /LSD ADC/LSD_{ADC_5V_D1}
- U4 pad 5: /High voltage supply/Boost Quadrupler 1/HV_{HALF-BOOST} -> /LSD ADC/LSD_{ADC_5V_D0}
- U4 pad 6: /High voltage supply/Boost Quadrupler 1/HV_{HALF-BOOST} -> unconnected-(U4-NC-Pad6)
- U5 pad 1: /High voltage supply/Boost Quadrupler 2/HV_{HALF-BOOST} -> /LSD ADC/VCC_{lvl-shift-A-2}
- U5 pad 2: /High voltage supply/Boost Quadrupler 2/HV_{HALF-BOOST} -> /LSD ADC/LSD_{ADC_5V_D7}
- U5 pad 3: GATE_{HV} -> /LSD ADC/LSD_{ADC_5V_D6}
- U5 pad 4: GND -> /LSD ADC/LSD_{ADC_5V_D5}
- U5 pad 5: /High voltage supply/Boost Quadrupler 2/HV_{HALF-BOOST} -> /LSD ADC/LSD_{ADC_5V_D4}
- U5 pad 6: /High voltage supply/Boost Quadrupler 2/HV_{HALF-BOOST} -> unconnected-(U5-NC-Pad6)
- U6 pad 1: /HV bleed/HV_bleed_{drain} -> /LSD ADC/V_{SHUNT}
- U6 pad 2: /HV bleed/HV_bleed_{drain} -> /LSD ADC/LSD_{ADC_5V_D0}
- U6 pad 3: /HV bleed/HV_bleed_{gate} -> /LSD ADC/LSD_{ADC_5V_D1}
- U6 pad 4: /HV bleed/HV_bleed_{source} -> /LSD ADC/LSD_{ADC_5V_D2}
- U6 pad 5: /HV bleed/HV_bleed_{drain} -> /LSD ADC/LSD_{ADC_5V_D3}
- U6 pad 6: /HV bleed/HV_bleed_{drain} -> /LSD ADC/LSD_{ADC_5V_~{WR}/RDY}
- U6 pad 7: /HV bleed/HV_bleed_{source} -> /LSD ADC/LSD_{ADC_5V_MODE}
- U7 pad 1: /HV bleed/HV_bleed_{gate} -> /LSD ADC/VCC_{lvl-shift-A-3}
- U7 pad 2: /HV bleed/HV_bleed_{gate} -> /LSD ADC/VCC_{lvl-shift-A-3}
- U7 pad 3: +5V -> /LSD ADC/VCC_{lvl-shift-A-3}
- U7 pad 4: GND -> /LSD ADC/LSD_{ADC_5V_~{OFL}}
- U7 pad 5: /HV bleed/HV_bleed_{gate} -> /LSD ADC/LSD_{ADC_5V_~{INT}}
- U7 pad 6: /HV bleed/HV_bleed_{gate} -> unconnected-(U7-NC-Pad6)
- U8 pad 1: /LSD ADC/VCC_{lvl-shift-A-1} -> /LSD ADC/VCC_{lvl-shift-A-4}
- U8 pad 10: LSD_{ADC_D0} -> /LSD ADC/LSD_{ADC_5V_~{CS}}
- U8 pad 11: LSD_{ADC_D1} -> /LSD ADC/LSD_{ADC_5V_~{RD}}
- U8 pad 12: LSD_{ADC_D2} -> /LSD ADC/LSD_{ADC_5V_MODE}
- U8 pad 13: LSD_{ADC_D3} -> /LSD ADC/LSD_{ADC_5V_~{WR}/RDY}
- U8 pad 14: /LSD ADC/VCC_{lvl-shift-B-1} -> /LSD ADC/VCC_{lvl-shift-B-4}
- U8 pad 2: /LSD ADC/LSD_{ADC_5V_D3} -> LSD_{ADC_~{WR}/RDY}
- U8 pad 3: /LSD ADC/LSD_{ADC_5V_D2} -> LSD_{ADC_MODE}
- U8 pad 4: /LSD ADC/LSD_{ADC_5V_D1} -> LSD_{ADC_~{RD}}
- U8 pad 5: /LSD ADC/LSD_{ADC_5V_D0} -> LSD_{ADC_~{CS}}
