File: hardware/KiCad/nixieAccurateClock/nixieAccurateClock.kicad_pcb (KiCad board)
At the start: 4 copper layers, 152.4 x 101.6 mm, 94 parts, among them J1 Conn_01x02_Pin, J10 Conn_01x02_Pin, J17 Conn_02x05_Odd_Even, J2 Conn_01x02_Pin, J3 Conn_01x02_Pin, J4 pico iCE (A), J5 pico iCE (B), J6 Conn_01x02_Pin, J7 Conn_01x02_Pin, J8 Conn_Coaxial, J9 Conn_01x02_Pin, Q1 IRLH5030TRPBF, Q2 BSP88, Q3 BSP88, SW1 SW_DIP_x08, U1 MCP23008-xSO, U2 LTR-329ALS-01, U3 PX1125T, U6 ADC0820BCWMX

Commit message: proper HVPS
Parts:
- added D6: SM4004, Diode_SMD:D_MELF, F.Cu at (21.0, 61.0)
- added Q4: PZTA42, Package_TO_SOT_SMD:SOT-223-3_TabPin2, F.Cu at (34.9, 97.2)
- added Q5: PZTA42, Package_TO_SOT_SMD:SOT-223-3_TabPin2, F.Cu at (24.1, 75.6)
- added Q6: PZTA42, Package_TO_SOT_SMD:SOT-223-3_TabPin2, F.Cu at (23.5, 85.1)
- added R10: 10k, Resistor_SMD:R_2512_6332Metric, F.Cu at (27.3, 61.0)
- added R11: 100k, Resistor_SMD:R_0603_1608Metric, F.Cu at (31.8, 78.7)
- added R12: 1M, Resistor_SMD:R_0603_1608Metric, F.Cu at (61.0, 29.8)
- added R13: 47k, Resistor_SMD:R_0603_1608Metric, F.Cu at (61.0, 24.8)
- C9: value 0.1u -> locked
- D4: value SM4004 -> 1SMB5956B-13; footprint Diode_SMD:D_MELF -> Diode_SMD:D_SMB
- Q1: value IRLH5030TRPBF -> PZTA42; footprint 00_lib:Infineon-PG-TDSON-8-0-0-MFG -> Package_TO_SOT_SMD:SOT-223-3_TabPin2
- Q2, Q3: value BSP88 -> PZTA42
- R5, R8: value 1M -> 0.5; footprint Resistor_SMD:R_0603_1608Metric -> Resistor_SMD:R_2010_5025Metric
- R6: value 10k -> 0.5; footprint Resistor_SMD:R_2512_6332Metric -> Resistor_SMD:R_2010_5025Metric
- R7: value 100k -> 0.5; footprint Resistor_SMD:R_0603_1608Metric -> Resistor_SMD:R_2010_5025Metric
- R9: value 47k -> 1M
- moved U5 141.0 mm to (105.1, 36.2)
- moved U7 140.9 mm to (105.1, 28.5)
- moved C13 137.9 mm to (108.6, 32.4), turned to 180 degrees
- moved C15 132.7 mm to (107.3, 24.8)
- moved C12 132.3 mm to (102.9, 32.4), turned to 180 degrees
- moved C14 131.1 mm to (101.6, 24.8)
- moved C9 126.6 mm to (97.2, 24.8), turned to 180 degrees
- moved U6 116.5 mm to (91.4, 32.4)
- moved U4 113.4 mm to (77.5, 28.6), turned to 180 degrees
- moved U8 113.2 mm to (77.5, 36.2)
- moved C10 112.3 mm to (82.5, 31.8), turned to 90 degrees
- moved R4 106.9 mm to (93.3, 41.9)
- moved C17 105.0 mm to (79.4, 32.4), turned to 180 degrees
- moved R3 103.1 mm to (89.5, 41.9)
- moved R5 102.7 mm to (62.2, 104.8), turned to -90 degrees
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Connections:
- net /High voltage supply/Boost Quadrupler 1/HV_{FULL-BOOST} renamed /High voltage supply/HV_{FULL-BOOST}
- net /High voltage supply/Boost Quadrupler 1/HV_{HALF-SUPPLY} renamed /High voltage supply/HV_{HALF-SUPPLY}
- C4 pad 2: /High voltage supply/Boost Quadrupler 1/HV_{HALF-BOOST} -> /High voltage supply/HV_{HALF-BOOST}
- C5 pad 1: /High voltage supply/Boost Quadrupler 1/HV_{QUARTER-BOOST} -> /High voltage supply/HV_{QUARTER-BOOST}
- C5 pad 2: /High voltage supply/Boost Quadrupler 1/HV_{HALF-BOOST} -> /High voltage supply/HV_{HALF-BOOST}
- C6 pad 1: HV_{SENSE} -> /High voltage supply/HV_{SENSE}
- D1 pad 1: HV_{SENSE} -> /High voltage supply/HV_{SENSE}
- D3 pad 2: /High voltage supply/Boost Quadrupler 1/HV_{QUARTER-BOOST} -> /High voltage supply/HV_{QUARTER-BOOST}
- D4 pad 1: /High voltage supply/Boost Quadrupler 1/HV_{QUARTER-BOOST} -> /High voltage supply/HV_{SENSE}
- D5 pad 1: /HV bleed/HV_bleed_{gate} -> /High voltage supply/HV_{QUARTER-BOOST}
- D5 pad 2: /HV bleed/HV_bleed_{pulldown} -> GND
- J10 pad 1: HV_{SENSE} -> /High voltage supply/HV_{SENSE}
- L1 pad 2: /High voltage supply/Boost Quadrupler 1/HV_{HALF-BOOST} -> /High voltage supply/HV_{HALF-BOOST}
- Q1 pad 1: GND -> GATE_{HV}
- Q1 pad 2: GND -> /High voltage supply/HV_{HALF-BOOST}
- Q1 pad 3: GND -> /High voltage supply/RE_{HV-1}
- Q2 pad 1: /HV bleed/HV_bleed_{gate} -> GATE_{HV}
- Q2 pad 2: /HV bleed/HV_bleed_{drain} -> /High voltage supply/HV_{HALF-BOOST}
- Q2 pad 3: /HV bleed/HV_bleed_{source} -> /High voltage supply/RE_{HV-2}
- Q3 pad 1: +5V -> GATE_{HV}
- Q3 pad 2: /HV bleed/HV_bleed_{gate} -> /High voltage supply/HV_{HALF-BOOST}
- Q3 pad 3: GND -> /High voltage supply/RE_{HV-3}
- R3 pad 1: VPP -> /High voltage supply/HV_{SENSE}
- R5 pad 1: /HV bleed/HV_bleed_{pulldown} -> /High voltage supply/RE_{HV-1}
- R5 pad 2: HV_{SENSE} -> GND
- R6 pad 1: HV_{SENSE} -> /High voltage supply/RE_{HV-2}
- R6 pad 2: /HV bleed/HV_bleed_{drain} -> GND
- R7 pad 1: /HV bleed/HV_bleed_{source} -> /High voltage supply/RE_{HV-3}
- R8 pad 1: /LSD ADC/V_{SHUNT} -> /High voltage supply/RE_{HV-4}
- R8 pad 2: LSD_{SHUNT} -> GND
- R9 pad 1: GND -> /HV bleed/HV_bleed_{pulldown}
- R9 pad 2: /LSD ADC/V_{SHUNT} -> HV_{SENSE}
- TP1 pad 1: /High voltage supply/Boost Quadrupler 1/HV_{HALF-BOOST} -> /High voltage supply/HV_{HALF-BOOST}
- TP3 pad 1: /High voltage supply/Boost Quadrupler 1/HV_{QUARTER-BOOST} -> /High voltage supply/HV_{QUARTER-BOOST}
Routing:
- net GATE_{HV}: track 0.00 -> 78.8 mm
- net /LSD ADC/LSD_{ADC_5V_~{INT}}: track 0.00 -> 18.6 mm, vias 0 -> 2
- net /LSD ADC/LSD_{ADC_5V_~{CS}}: track 0.00 -> 16.8 mm, vias 0 -> 2
- net MEASURE_{HV}: track 0.00 -> 9.58 mm
- net /LSD ADC/LSD_{ADC_5V_D7}: track 0.00 -> 8.72 mm
- net /LSD ADC/LSD_{ADC_5V_D6}: track 0.00 -> 8.46 mm
- net /LSD ADC/LSD_{ADC_5V_D5}: track 0.00 -> 8.20 mm
- net /LSD ADC/LSD_{ADC_5V_D4}: track 0.00 -> 7.95 mm
- net /LSD ADC/LSD_{ADC_5V_~{WR}/RDY}: track 0.00 -> 7.23 mm
- net /LSD ADC/LSD_{ADC_5V_D3}: track 0.00 -> 7.23 mm
- net +5V: track 2.54 -> 9.75 mm, vias 1 -> 4
- net /LSD ADC/LSD_{ADC_5V_MODE}: track 0.00 -> 6.98 mm
- net /LSD ADC/LSD_{ADC_5V_D2}: track 0.00 -> 6.98 mm
- net /LSD ADC/LSD_{ADC_5V_D1}: track 0.00 -> 6.72 mm
- net /LSD ADC/LSD_{ADC_5V_~{RD}}: track 0.00 -> 6.72 mm
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
Commit message: lay out HVPS
Parts:
- moved TP1 1.91 mm to (26.7, 97.2)
- moved TP7 1.91 mm to (35.6, 81.3)
- moved D4 1.27 mm to (37.5, 72.4)
- moved R9 1.04 mm to (21.8, 56.5), turned to 0 degrees
- moved D2 0.90 mm to (48.9, 74.3)
- moved D1 0.64 mm to (46.4, 67.9)
- moved TP4 0.63 mm to (52.7, 68.6)
- moved R5 0.23 mm to (62.0, 104.8)
- moved C5 0.08 mm to (55.2, 85.8)
Connections:
- C6 pad 1: /High voltage supply/HV_{SENSE} -> HV_{SENSE}
- D1 pad 1: /High voltage supply/HV_{SENSE} -> HV_{SENSE}
- D4 pad 1: /High voltage supply/HV_{SENSE} -> HV_{SENSE}
- J10 pad 1: /High voltage supply/HV_{SENSE} -> HV_{SENSE}
- R3 pad 1: /High voltage supply/HV_{SENSE} -> HV_{SENSE}
Routing:
- net /High voltage supply/HV_{HALF-BOOST}: track 0.00 -> 79.1 mm
- net /HV bleed/HV_bleed_{gate}: track 0.00 -> 32.1 mm
- net I2C_{CLOCK}: track 42.7 -> 70.0 mm
- net I2C_{DATA}: track 47.7 -> 75.0 mm
- net GND: track 70.8 -> 97.2 mm, vias 13 -> 23
- net /HV bleed/HV_bleed_{drain}: track 0.00 -> 17.9 mm
- net /HV bleed/HV_bleed_{source}: track 0.00 -> 17.5 mm
- net /High voltage supply/HV_{QUARTER-BOOST}: track 0.00 -> 15.7 mm
- net /High voltage supply/RE_{HV-4}: track 0.00 -> 3.01 mm
- net /High voltage supply/RE_{HV-3}: track 0.00 -> 3.01 mm
- net /High voltage supply/RE_{HV-2}: track 0.00 -> 3.01 mm
- net /High voltage supply/RE_{HV-1}: track 0.00 -> 3.00 mm
- net /HV bleed/HV_bleed_{pulldown}: track 0.00 -> 2.06 mm
- net +5V: track 9.75 -> 11.7 mm, vias 4 -> 8
- net GATE_{HV}: track 78.8 -> 79.7 mm
- added copper zone on F.Cu, net +5V
- added copper zone on F.Cu, net /High voltage supply/HV_{FULL-BOOST}
- added copper zone on F.Cu, net /High voltage supply/HV_{HALF-SUPPLY}
- added copper zone on F.Cu, net HV_{SENSE}

Commit message: route nixie daughter boards
Parts:
- moved R2 1.36 mm to (116.1, 70.4), turned to -90 degrees
Connections:
- net +3V3_STDBY renamed +3.3V_STDBY
- net /3.3V_STDBY_SRAM_{SENSE} renamed /+3.3V_STDBY_SRAM_{SENSE}
- net /3.3V_{SENSE} renamed /+3.3V_{SENSE}
- net /5V_{SENSE} renamed /+5V_{SENSE}
- net /GPS/3.3V_STDBY_GPS_{SENSE} renamed /GPS/+3.3V_STDBY_GPS_{SENSE}
- J4 pad 27: GPS_{1PPS2} -> GPS_{1PPS}
- J4 pad 28: GPS_{1PPS} -> GPS_{1PPS2}
Routing:
- net VPP: track 0.00 -> 184.3 mm, vias 0 -> 8
- net CLOCK_{HV}: track 0.00 -> 182.8 mm, vias 0 -> 8
- net PPS_{TRIMMED}: track 47.9 -> 220.7 mm, vias 1 -> 7
- net GND: track 97.2 -> 180.7 mm, vias 23 -> 40
- net LSD_{SHUNT}: track 0.00 -> 39.2 mm
- net /LSD ADC/V_{SHUNT}: track 0.00 -> 33.5 mm
- net /Nixies/DAISY_{HV-4}: track 0.00 -> 31.5 mm, vias 0 -> 2
- net /Nixies/DAISY_{HV-2}: track 0.00 -> 31.5 mm, vias 0 -> 2
- net /Nixies/DAISY_{HV-1}: track 0.00 -> 27.3 mm, vias 0 -> 2
- net /Nixies/DAISY_{HV-5}: track 0.00 -> 27.3 mm, vias 0 -> 2
- net /Nixies/DAISY_{HV-3}: track 0.00 -> 27.3 mm, vias 0 -> 2
- net GPS_{1PPS}: track 18.2 -> 42.2 mm
- net +5V: track 11.7 -> 30.8 mm, vias 8 -> 15
- net +3.3V: track 0.00 -> 18.4 mm, vias 0 -> 6
- net /+3.3V_{SENSE}: track 0.00 -> 15.6 mm, vias 0 -> 5
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
Commit message: WIP ADC routing
Parts:
- moved REF** 1.42 mm to (56.5, 58.4)
Connections:
- J4 pad 15: LSD_{ADC_D3} -> LSD_{ADC_D2}
- J4 pad 16: LSD_{ADC_D2} -> LSD_{ADC_D3}
Routing:
- net DATA_{HV}: track 0.00 -> 118.5 mm, vias 0 -> 2
- net LSD_{ADC_D1}: track 0.00 -> 97.2 mm, vias 0 -> 2
- net LSD_{ADC_D0}: track 0.00 -> 89.1 mm
- net CLOCK_{HV}: track 182.8 -> 255.3 mm
- net LSD_{ADC_D3}: track 0.00 -> 69.2 mm
- net LSD_{ADC_D2}: track 0.00 -> 67.6 mm
- net PPS_{TRIMMED}: track 220.7 -> 216.6 mm, vias 7 -> 8
- net +3.3V: track 18.4 -> 15.4 mm, vias 6 -> 4
- net GATE_{HV}: track 79.7 -> 81.4 mm, vias 0 -> 2
- net GND: track 180.7 -> 181.2 mm
- net GPS_{BOOT_SEL}: track 27.7 -> 28.2 mm

Commit message: update ADC pinout for improved routing
Connections:
- J4 pad 10: LSD_{ADC_D7} -> LSD_{ADC_D4}
- J4 pad 11: LSD_{ADC_D6} -> LSD_{ADC_~{RD}}
- J4 pad 13: LSD_{ADC_D4} -> LSD_{ADC_MODE}
- J4 pad 14: LSD_{ADC_~{CS}} -> LSD_{ADC_D6}
- J4 pad 15: LSD_{ADC_D2} -> LSD_{ADC_~{WR}/RDY}
- J4 pad 16: LSD_{ADC_D3} -> LSD_{ADC_D7}
- J4 pad 19: LSD_{ADC_~{RD}} -> LSD_{ADC_D3}
- J4 pad 20: LSD_{ADC_MODE} -> LSD_{ADC_~{INT}}
- J4 pad 22: LSD_{ADC_~{INT}} -> LSD_{ADC_~{OFL}}
- J4 pad 29: LSD_{ADC_D0} -> LSD_{ADC_D1}
- J4 pad 30: LSD_{ADC_D1} -> LSD_{ADC_D2}
- J4 pad 31: LSD_{ADC_~{WR}/RDY} -> LSD_{ADC_D0}
- J4 pad 9: LSD_{ADC_~{OFL}} -> LSD_{ADC_~{CS}}
Routing:
- net LSD_{ADC_~{WR}/RDY}: track 0.00 -> 62.7 mm
- net LSD_{ADC_MODE}: track 0.00 -> 58.1 mm
- net LSD_{ADC_~{RD}}: track 0.00 -> 52.8 mm
- net LSD_{ADC_~{CS}}: track 0.00 -> 46.7 mm
- net LSD_{ADC_D2}: track 67.6 -> 96.9 mm, vias 0 -> 2
- net LSD_{ADC_D1}: track 97.2 -> 85.9 mm, vias 2 -> 0
- net +3.3V: track 15.4 -> 22.4 mm, vias 4 -> 6
- net GND: track 181.2 -> 184.4 mm
- net LSD_{ADC_D3}: track 69.2 -> 72.2 mm
- net LSD_{ADC_D0}: track 89.1 -> 90.5 mm

Commit message: DRC pass
Parts:
- moved J1 2.54 mm to (116.8, 55.9)
- moved Q1 1.91 mm to (63.2, 97.2)
- moved L1 1.91 mm to (75.6, 97.2)
- moved Q3 1.91 mm to (43.2, 97.2)
- moved R5 1.91 mm to (60.1, 104.8)
- moved R6 1.91 mm to (50.2, 104.8)
- moved R7 1.91 mm to (40.0, 104.8)
- moved TP1 1.91 mm to (24.8, 97.2)
- moved R8 1.90 mm to (29.9, 104.8)
- moved Q2 1.90 mm to (53.3, 97.2)
- moved Q4 1.90 mm to (33.0, 97.2)
- moved C7 0.64 mm to (62.2, 69.8)
- moved REF** 0.63 mm to (56.5, 59.1)
Routing:
- net LSD_{ADC_~{OFL}}: track 0.00 -> 144.6 mm, vias 0 -> 4
- net SENSE_{PRECISE}: track 0.00 -> 143.7 mm, vias 0 -> 2
- net DATA_{PRECISE}: track 0.00 -> 142.1 mm, vias 0 -> 2
- net LSD_{ADC_~{INT}}: track 0.00 -> 139.5 mm, vias 0 -> 4
- net CLOCK_{PRECISE}: track 0.00 -> 139.4 mm, vias 0 -> 2
- net LSD_{ADC_D7}: track 0.00 -> 79.5 mm
- net LSD_{ADC_D6}: track 0.00 -> 75.2 mm
- net LSD_{ADC_D5}: track 0.00 -> 71.0 mm
- net LSD_{ADC_D4}: track 0.00 -> 66.8 mm
- net HV_{SENSE}: track 0.00 -> 58.2 mm, vias 0 -> 2
- net MEASURE_{HV}: track 9.58 -> 62.1 mm, vias 0 -> 2
- net GND: track 184.4 -> 200.2 mm, vias 40 -> 43
- net +3.3V: track 22.4 -> 33.3 mm
- net +3.3V_STDBY: track 44.0 -> 51.3 mm
- net /+3.3V_{SENSE}: track 15.6 -> 20.7 mm, vias 5 -> 7
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
Commit message: Rev B prep
Parts:
- moved TP9 13.8 mm to (19.9, 102.9)
- moved H7 0.25 mm to (19.9, 19.9)
- moved H8 0.25 mm to (31.9, 19.9)
Routing:
- net GND: track 200.2 -> 210.8 mm
- net LSD_{SHUNT}: track 39.2 -> 39.7 mm

Commit message: update to KiCAD 8
Parts:
- C9: value locked -> 0.1u
- turned C3 to -90 degrees
Connections:
- C3 pad 1: /GPS/VCC_{GPS} -> +3.3V
- C3 pad 2: +3.3V -> /GPS/VCC_{GPS}
