File: hardware/KiCad/nixieAccurateClock/nixieAccurateClock.kicad_pcb (KiCad board)
At the start: 4 copper layers, 152.4 x 101.6 mm, 103 parts, among them J1 Conn_01x02_Pin, J10 Conn_01x02_Pin, J17 Conn_02x05_Odd_Even, J2 Conn_01x02_Pin, J3 Conn_01x02_Pin, J4 pico iCE (A), J5 pico iCE (B), J6 Conn_01x02_Pin, J7 Conn_01x02_Pin, J8 Conn_Coaxial, J9 Conn_01x02_Pin, Q1 PZTA42, Q2 PZTA42, Q3 PZTA42, Q4 PZTA42, Q5 PZTA42, Q6 PZTA42, SW1 SW_DIP_x08, U1 MCP23008-xSO, U2 LTR-329ALS-01, U3 PX1125T, U6 ADC0820BCWMX

Commit message: add alignment holes to 2x20 SM headers
Routing:
- net GND: track 210.8 -> 196.3 mm, vias 43 -> 45
- net /Pico Ice/~{USB_BOOT}: track 13.3 -> 26.0 mm
- net /GPS/GPS_{BOOT_SEL}: track 28.2 -> 26.7 mm
Changed lines of the file:
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@@
 			)
 		)
+		(pad "" np_thru_hole circle
+			(at 0 -21.59 270)
+			(size 1.09 1.09)
+			(drill 1.09)
+			(layers "F&B.Cu" "*.Mask")
+		)
+		(pad "" np_thru_hole circle
+			(at 0 24.13 270)
+			(size 1.09 1.09)
+			(drill 1.09)
+			(layers "F&B.Cu" "*.Mask")
+		)
 		(pad "1" smd rect
 			(at -2.54 -22.86)
@@
 			)
 		)
+		(pad "" np_thru_hole circle
+			(at 0 -21.59 90)
+			(size 1.09 1.09)
+			(drill 1.09)
+			(layers "F&B.Cu" "*.Mask")
+		)
+		(pad "" np_thru_hole circle
+			(at 0 24.13 90)
+			(size 1.09 1.09)
+			(drill 1.09)
+			(layers "F&B.Cu" "*.Mask")
+		)
 		(pad "1" smd rect
 			(at -2.5 -22.86)
@@
 	)
 	(segment
-		(start 94.025 113.475)
-		(end 91.985 113.475)
-		(width 0.5)
-		(layer "F.Cu")
-		(net 2)
-	)
-	(segment
 		(start 25.795 44.125)
 		(end 25.795 41.625)
@@
 	)
 	(segment
-		(start 131.191 105.791)
-		(end 130.091 106.891)
+		(start 94.505 107.125)
+		(end 97.663 107.125)
 		(width 0.5)
 		(layer "F.Cu")
@@
 	)
 	(segment
-		(start 97.375 110.125)
-		(end 94.025 113.475)
+		(start 131.191 105.791)
+		(end 130.091 106.891)
 		(width 0.5)
 		(layer "F.Cu")
@@
 	)
 	(segment
-		(start 96.625 107.125)
-		(end 97.375 107.875)
-		(width 0.5)
-		(layer "F.Cu")
-		(net 2)
-	)
-	(segment
-		(start 97.375 107.875)
-		(end 97.375 110.125)
-		(width 0.5)
-		(layer "F.Cu")
-		(net 2)
-	)
-	(segment
 		(start 74.6075 38.145)
 		(end 74.6075 39.0475)
@@
 	)
 	(segment
-		(start 92.52 63.945)
-		(end 91.985 63.41)
-		(width 0.5)
-		(layer "F.Cu")
-		(net 2)
-	)
-	(segment
 		(start 90.525 59.055)
 		(end 91.985 57.595)
@@
 	)
 	(segment
-		(start 94.505 107.125)
-		(end 96.625 107.125)
-		(width 0.5)
-		(layer "F.Cu")
-		(net 2)
-	)
-	(segment
 		(start 74.6075 39.0475)
 		(end 74.93 39.37)
@@
 	)
 	(segment
-		(start 91.985 63.41)
-		(end 91.985 57.595)
-		(width 0.5)
-		(layer "F.Cu")
-		(net 2)
-	)
-	(segment
 		(start 163.275 52.07)
 		(end 163.275 49.165)
@@
 	)
 	(segment
-		(start 94.505 63.945)
-		(end 92.52 63.945)
-		(width 0.5)
-		(layer "F.Cu")
-		(net 2)
-	)
-	(segment
 		(start 40.03 108.585)
 		(end 40.03 107.0875)
@@
 	)
 	(segment
+		(start 94.505 63.945)
+		(end 97.663 63.945)
+		(width 0.5)
+		(layer "F.Cu")
+		(net 2)
+	)
+	(segment
 		(start 30.875 52.07)
 		(end 30.875 49.165)
@@
 	)
 	(via
+		(at 97.663 107.125)
+		(size 0.8)
+		(drill 0.4)
+		(layers "F.Cu" "B.Cu")
+		(free yes)
+		(net 2)
+	)
+	(via
 		(at 80.01 25.4)
 		(size 0.8)
@@
 	)
 	(via
+		(at 97.663 63.945)
+		(size 0.8)
+		(drill 0.4)
+		(layers "F.Cu" "B.Cu")
+		(free yes)
+		(net 2)
+	)
+	(via
 		(at 158.195 40.005)
 		(size 0.8)
@@
 	)
 	(segment
-		(start 83.82 108.93)
-		(end 84.375 108.375)
+		(start 98.235 105.855)
+		(end 86.2975 105.855)
 		(width 0.25)
 		(layer "F.Cu")
@@
 	)
 	(segment
-		(start 92.415 109.665)
-		(end 94.505 109.665)
+		(start 98.17 109.665)
+		(end 99.06 108.775)
 		(width 0.25)
 		(layer "F.Cu")
@@
 	)
 	(segment
-		(start 84.375 108.375)
-		(end 91.125 108.375)
+		(start 94.505 109.665)
+		(end 98.17 109.665)
 		(width 0.25)
 		(layer "F.Cu")
@@
 	)
 	(segment
-		(start 83.82 110.74)
-		(end 83.82 108.93)
+		(start 83.82 108.3325)
+		(end 83.82 110.74)
 		(width 0.25)
 		(layer "F.Cu")
@@
 	)
 	(segment
-		(start 91.125 108.375)
-		(end 92.415 109.665)
+		(start 99.06 108.775)
+		(end 99.06 106.68)
+		(width 0.25)
+		(layer "F.Cu")
+		(net 12)
+	)
+	(segment
+		(start 99.06 106.68)
+		(end 98.235 105.855)
+		(width 0.25)
+		(layer "F.Cu")
+		(net 12)
+	)
+	(segment
+		(start 86.2975 105.855)
+		(end 83.82 108.3325)
 		(width 0.25)
 		(layer "F.Cu")
@@
 	)
 	(segment
-		(start 98.815 103.315)
-		(end 101.355 105.855)
+		(start 92.815 103.315)
+		(end 117.285 103.315)
 		(width 0.25)
 		(layer "F.Cu")
@@
 	)
 	(segment
-		(start 119.825 105.855)
-		(end 120.491 106.521)
-		(width 0.25)
-		(layer "F.Cu")
-		(net 19)
-	)
-	(segment
-		(start 91.425 94.425)
-		(end 91.985 94.985)
-		(width 0.25)
-		(layer "F.Cu")
-		(net 19)
-	)
-	(segment
 		(start 120.491 106.521)
 		(end 120.491 108.331)
@@
 	)
 	(segment
-		(start 92.815 103.315)
-		(end 98.815 103.315)
+		(start 89.465 94.425)
+		(end 91.425 94.425)
 		(width 0.25)
 		(layer "F.Cu")
@@
 	)
 	(segment
-		(start 89.465 94.425)
-		(end 91.425 94.425)
+		(start 91.425 94.425)
+		(end 91.985 94.985)
 		(width 0.25)
 		(layer "F.Cu")
@@
 	)
 	(segment
-		(start 101.355 105.855)
-		(end 119.825 105.855)
+		(start 91.985 94.985)
+		(end 91.985 102.485)
 		(width 0.25)
 		(layer "F.Cu")
@@
 	)
 	(segment
-		(start 91.985 94.985)
-		(end 91.985 102.485)
+		(start 117.285 103.315)
+		(end 120.491 106.521)
 		(width 0.25)
 		(layer "F.Cu")
@@
 	)
 	(segment
-		(start 118.555 103.315)
-		(end 121.591 106.351)
+		(start 103.025 100.775)
+		(end 114.3 100.775)
 		(width 0.25)
 		(layer "F.Cu")
@@
 	)
 	(segment
-		(start 105.565 103.315)
-		(end 118.555 103.315)
+		(start 114.3 100.775)
+		(end 115.57 102.045)
+		(width 0.25)
+		(layer "F.Cu")
+		(net 46)
+	)
+	(segment
+		(start 96.675 94.425)
+		(end 103.025 100.775)
 		(width 0.25)
 		(layer "F.Cu")
@@
 	)
 	(segment
-		(start 96.675 94.425)
-		(end 105.565 103.315)
+		(start 117.285 102.045)
+		(end 121.591 106.351)
+		(width 0.25)
+		(layer "F.Cu")
+		(net 46)
+	)
+	(segment
+		(start 115.57 102.045)
+		(end 117.285 102.045)
 		(width 0.25)
 		(layer "F.Cu")
@@
 	)
 	(segment
-		(start 111.701 109.061)
+		(start 109.765 107.125)
+		(end 113.475 107.125)
+		(width 0.5)
+		(layer "B.Cu")
+		(net 57)
+	)
+	(segment
+		(start 115.411 109.061)
 		(end 136.525 109.061)
 		(width 0.5)
@@
 	)
 	(segment
-		(start 109.765 107.125)
-		(end 111.701 109.061)
+		(start 113.475 107.125)
+		(end 115.411 109.061)
 		(width 0.5)
 		(layer "B.Cu")
@@
 	)
 	(segment
-		(start 118.291 108.331)
-		(end 118.227 108.395)
+		(start 104.375 96.965)
+		(end 107.245 96.965)
+		(width 0.25)
+		(layer "F.Cu")
+		(net 61)
+	)
+	(segment
+		(start 116.8035 108.331)
+		(end 118.291 108.331)
 		(width 0.25)
 		(layer "F.Cu")
@@
 	)
 	(segment
-		(start 104.375 96.965)
-		(end 107.245 96.965)
+		(start 114.3275 105.855)
+		(end 116.8035 108.331)
 		(width 0.25)
 		(layer "F.Cu")
@@
 	)
 	(segment
-		(start 118.227 108.395)
-		(end 104.375 108.395)
+		(start 104.375 105.855)
+		(end 114.3275 105.855)
 		(width 0.25)
 		(layer "F.Cu")
@@
 	)
 	(via
-		(at 104.375 108.395)
+		(at 104.375 105.855)
 		(size 0.8)
 		(drill 0.4)
@@
 	)
 	(segment
-		(start 104.375 108.395)
+		(start 104.375 105.855)
 		(end 104.375 96.965)
 		(width 0.25)

Commit message: fix 2x1 SM header chirality
Parts:
- J1, J10, J2, J3, J6, J7, J9: footprint Connector_PinHeader_2.54mm:PinHeader_1x02_P2.54mm_Vertical_SMD_Pin1Left -> Connector_PinHeader_2.54mm:PinHeader_1x02_P2.54mm_Vertical_SMD_Pin1Right
- moved J10 3.87 mm to (45.7, 55.9), turned to 180 degrees
Routing:
- net GND: track 196.3 -> 181.1 mm, vias 45 -> 47
- net +3.3V_STDBY: track 51.3 -> 56.0 mm
- net /Pico Ice/~{USB_BOOT}: track 26.0 -> 29.3 mm
- net /Pico Ice/+3.3V_{SENSE}: track 20.7 -> 23.8 mm, vias 7 -> 9
- net +3.3V: track 33.3 -> 36.0 mm, vias 6 -> 8
- net /Pico Ice/~{ICE_RST}: track 23.2 -> 25.8 mm
- net /GPS/+3.3V_STDBY_GPS_{SENSE}: track 18.1 -> 20.6 mm
- net /Pico Ice/+5V_{SENSE}: track 14.7 -> 15.5 mm
- net /Pico Ice/+3.3V_STDBY_SRAM_{SENSE}: track 32.6 -> 33.2 mm

Commit message: more detailed build notes, drop HV divider by 10x
Parts:
- R3: value 10M -> 1M
- R4: value 100k -> 10k
Changed lines of the file:
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@@
 			)
 		)
-		(property "Value" "10M"
+		(property "Value" "1M"
 			(at 0 1.43 0)
 			(layer "F.Fab")
@@
 			)
 		)
-		(property "Digikey link" "https://www.digikey.com/en/products/detail/stackpole-electronics-inc/RMCF0603FT10M0/1761206"
+		(property "Digikey link" "https://www.digikey.com/en/products/detail/stackpole-electronics-inc/RMCF0603FT1M00/1761036"
 			(at 0 0 0)
 			(layer "F.Fab")
@@
 			)
 		)
-		(property "Model" "RMCF0603FT10M0"
+		(property "Model" "RMCF0603FT1M00"
 			(at 0 0 0)
 			(layer "F.Fab")
@@
 			)
 		)
-		(property "Mouser link" "https://www.mouser.com/ProductDetail/SEI-Stackpole/RMCF0603FT10M0?qs=FESYatJ8odIf0bWpBT4vKw%3D%3D"
+		(property "Mouser link" "https://www.mouser.com/ProductDetail/SEI-Stackpole/RMCF0603FT1M00?qs=FESYatJ8odJNClY0wUC1cg%3D%3D"
 			(at 0 0 0)
 			(layer "F.Fab")
@@
 			)
 		)
-		(property "Footprint" ""
+		(property "Footprint" "Symbol:Symbol_HighVoltage_Type2_CopperTop_VerySmall"
 			(at 0 0 0)
 			(unlocked yes)
@@
 			)
 		)
-		(property "Value" "100k"
+		(property "Value" "10k"
 			(at 0 1.43 0)
 			(layer "F.Fab")
@@
 			)
 		)
-		(property "Digikey link" "https://www.digikey.com/en/products/detail/yageo/RC0603JR-07100KL/726698"
+		(property "Digikey link" "https://www.digikey.com/en/products/detail/yageo/RC0603FR-0710KL/726880"
 			(at 0 0 0)
 			(layer "F.Fab")
@@
 			)
 		)
-		(property "Model" "RC0603JR-07100KL"
+		(property "Model" "RC0603FR-0710KL"
 			(at 0 0 0)
 			(layer "F.Fab")
@@
 			)
 		)
-		(property "Mouser link" "https://www.mouser.com/ProductDetail/YAGEO/RC0603JR-07100KL?qs=2cAdsCoAWRG9Rhqklpdeqg%3D%3D"
+		(property "Mouser link" "https://www.mouser.com/ProductDetail/YAGEO/RC0603FR-0710KL?qs=grNVn54RoB%252B3GtjbJj3wJQ%3D%3D"
 			(at 0 0 0)
 			(layer "F.Fab")
@@
 		)
 	)
-	(gr_text_box "Fabrication notes:\n1. Use ENIG coating.\n2. Use black solder mask.\n3. All vias are tented.\n4. All vias are 0.4 mm.\n5. 1.6 mm thick board.\n6. Use FR4 core.\n7. Use 1 oz copper on outer layers.\n8. Use 1 oz copper on inner layers.\n9. Use 0.2 mm thick prepreg.\n\nAssembly notes:\n1. Single side assembly (top).\n2. Use lead free solder.\n3. Do not procure or install pico ICE in J4/J5.\n   Install only 2x 2x20 0.1{dblquote} pin sockets.\n4. Do not procure or install nixie daughter boards in J11-J17.\n   Install only 6x 2x5 0.1{dblquote} pin sockets.\n5. No special component handling."
+	(gr_text_box "Fabrication notes:\n 1. Fabricate in accordance with IPC-4012 Class 2.\n 2. Inspect PCB in accordance with IPC-A-600 Class 2.\n 3. Test Requirements: 100% netlist electrical verification using supplied IPC-356 netlist for opens and shorts.\n 4. Flame class to be UL94 HB or greater.\n 5. 1.6 mm nominal board thickness.\n 6. Use FR4 core.\n 7. Use 1 oz copper on outer layers.\n 8. Use 1 oz copper on inner layers.\n 9. Use 0.2 mm thick prepreg.\n10. Use ENIG coating per IPC-4552.\n11. Use black solder mask.\n12. All vias are tented.\n13. All vias are 0.4 mm.\n\nAssembly notes:\n 1. Assemble in accordance with IPC-J-STD-001 Class 2.\n 2. Inspect PCBA in accordance with IPC-A-610 Class 2.\n 3. Clean flux residue after soldering per IPC-J-STD-001 Section 8, Cleaning Designator C-22.\n 4. Single side assembly (top).\n 5. Use lead-free solder.\n 6. Do not procure or install pico ICE in J4/J5.\n    Install only 2x 2x20 0.1{dblquote} pin sockets.\n 7. Do not procure or install nixie daughter boards in J11-J17.\n    Install only 6x 2x5 0.1{dblquote} pin sockets.\n 8. No special component handling."
 		(start 175.26 55.375)
-		(end 279.76 103.125)
+		(end 279.76 125.35)
 		(layer "Cmts.User")
 		(effects
