File: hardware/KiCad/nixieAccurateClock/nixieAccurateClock.kicad_sch (KiCad schematic)
At the start: 36 parts, among them J1 Conn_01x02_Pin, J2 Conn_01x02_Pin, J3 Conn_01x02_Pin, J4 pico iCE (A), J5 pico iCE (B), J6 Conn_01x02_Pin, SW1 SW_DIP_x08, U1 MCP23008-xSO, U2 LTR-329ALS-01

Commit message: route nixie daughter boards
Connections:
- net GPS_{1PPS2}: now also J4.28 (ICE_45); no longer J4.27 (ICE_44_G6)
- net GPS_{1PPS}: now also J4.27 (ICE_44_G6); no longer J4.28 (ICE_45)
- net +3V3_STDBY renamed +3.3V_STDBY
- net 3.3V_STDBY_SRAM_{SENSE} renamed +3.3V_STDBY_SRAM_{SENSE}
- net 3.3V_{SENSE} renamed +3.3V_{SENSE}
- net 5V_{SENSE} renamed +5V_{SENSE}

Commit message: WIP ADC routing
Connections:
- net LSD_{ADC_D2}: now also J4.15 (ICE_42); no longer J4.16 (ICE_43)
- net LSD_{ADC_D3}: now also J4.16 (ICE_43); no longer J4.15 (ICE_42)
Changed lines of the file:
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@@
+    (stroke (width 0) (type default))
+  )
+  (wire (pts (xy 116.84 55.88) (xy 120.65 55.88))
     (stroke (width 0) (type default))
   )
@@
     (stroke (width 0) (type default))
   )
-  (wire (pts (xy 120.65 53.34) (xy 116.84 53.34))
-    (stroke (width 0) (type default))
-  )
   (wire (pts (xy 240.03 144.78) (xy 243.84 144.78))
     (stroke (width 0) (type default))
@@
     (stroke (width 0) (type default))
   )
+  (wire (pts (xy 116.84 53.34) (xy 120.65 53.34))
+    (stroke (width 0) (type default))
+  )
   (wire (pts (xy 133.35 118.11) (xy 133.35 120.65))
     (stroke (width 0) (type default))
@@
   )
   (wire (pts (xy 215.9 148.59) (xy 215.9 144.78))
-    (stroke (width 0) (type default))
-  )
-  (wire (pts (xy 120.65 55.88) (xy 116.84 55.88))
     (stroke (width 0) (type default))
   )
@@
     )
   )
-  (global_label "LSD_{ADC_D3}" (shape input) (at 120.65 53.34 0) (fields_autoplaced)
-    (effects (font (size 1.27 1.27)) (justify left))
-    (property "Intersheetrefs" "${INTERSHEET_REFS}" (at 132.8542 53.34 0)
+  (global_label "LSD_{ADC_D3}" (shape input) (at 120.65 55.88 0) (fields_autoplaced)
+    (effects (font (size 1.27 1.27)) (justify left))
+    (property "Intersheetrefs" "${INTERSHEET_REFS}" (at 132.8542 55.88 0)
       (effects (font (size 1.27 1.27)) (justify left) hide)
     )
@@
     )
   )
-  (global_label "LSD_{ADC_D2}" (shape input) (at 120.65 55.88 0) (fields_autoplaced)
-    (effects (font (size 1.27 1.27)) (justify left))
-    (property "Intersheetrefs" "${INTERSHEET_REFS}" (at 132.8542 55.88 0)
-      (effects (font (size 1.27 1.27)) (justify left) hide)
-    )
+  (global_label "LSD_{ADC_D2}" (shape input) (at 120.65 53.34 0) (fields_autoplaced)
+    (effects (font (size 1.27 1.27)) (justify left))
+    (property "Intersheetrefs" "${INTERSHEET_REFS}" (at 132.8542 53.34 0)
+      (effects (font (size 1.27 1.27)) (justify left) hide)
+    )

Commit message: update ADC pinout for improved routing
Connections:
- net LSD_{ADC_D0}: now also J4.31 (ICE_48); no longer J4.29 (ICE_46)
- net LSD_{ADC_D1}: now also J4.29 (ICE_46); no longer J4.30 (ICE_47)
- net LSD_{ADC_D2}: now also J4.30 (ICE_47); no longer J4.15 (ICE_42)
- net LSD_{ADC_D3}: now also J4.19 (ICE_11); no longer J4.16 (ICE_43)
- net LSD_{ADC_D4}: now also J4.10 (ICE_31); no longer J4.13 (ICE_36)
- net LSD_{ADC_D6}: now also J4.14 (ICE_38); no longer J4.11 (ICE_32)
- net LSD_{ADC_D7}: now also J4.16 (ICE_43); no longer J4.10 (ICE_31)
- net LSD_{ADC_MODE}: now also J4.13 (ICE_36); no longer J4.20 (ICE_6)
- net LSD_{ADC_~{CS}}: now also J4.9 (ICE_28); no longer J4.14 (ICE_38)
- net LSD_{ADC_~{INT}}: now also J4.20 (ICE_6); no longer J4.22 (ICE_9)
- net LSD_{ADC_~{OFL}}: now also J4.22 (ICE_9); no longer J4.9 (ICE_28)
- net LSD_{ADC_~{RD}}: now also J4.11 (ICE_32); no longer J4.19 (ICE_11)
- net LSD_{ADC_~{WR}/RDY}: now also J4.15 (ICE_42); no longer J4.31 (ICE_48)

Commit message: update to KiCAD 8
Parts:
- removed J?: Conn_01x02_Pin, Connector_PinHeader_2.54mm:PinHeader_1x02_P2.54mm_Vertical_SMD_Pin1Left, symbol Connector:Conn_01x02_Pin
- added J7: Conn_01x02_Pin, Connector_PinHeader_2.54mm:PinHeader_1x02_P2.54mm_Vertical_SMD_Pin1Left, symbol Connector:Conn_01x02_Pin
- FID1, FID2, FID3: now left out of the parts list
Connections:
- net +3.3V_STDBY: now also J7.1 (Pin_1)
- net +3.3V_STDBY_SRAM_{SENSE}: now also J7.2 (Pin_2)

Commit message: add polyfuse to HVPS
WIP hierarchy overhaul
Parts:
- removed J1, J2, J3, J6, J7: Conn_01x02_Pin, Connector_PinHeader_2.54mm:PinHeader_1x02_P2.54mm_Vertical_SMD_Pin1Left, symbol Connector:Conn_01x02_Pin
- removed J4: pico iCE (A), 00_lib:pico iCE (A), symbol 00_lib:pico_iCE (A)
- removed J5: pico iCE (B), 00_lib:pico iCE (B), symbol 00_lib:pico_iCE (B)
- removed R1, R2: 1k, Resistor_SMD:R_0603_1608Metric, symbol Device:R
- removed RV1: 100k, Potentiometer_SMD:Potentiometer_Bourns_3269X_Horizontal, symbol Device:R_Potentiometer
Other:
- added sheet Pico Ice (pico_ce.kicad_sch)

Commit message: fuse HV, refactor schematic hierarchy
Parts:
- removed C1, C2: 0.1u, Capacitor_SMD:C_0603_1608Metric, symbol Device:C_Small
- removed SW1: SW_DIP_x08, Button_Switch_SMD:SW_DIP_SPSTx08_Slide_6.7x21.88mm_W8.61mm_P2.54mm_LowProfile, symbol Switch:SW_DIP_x08
- removed U1: MCP23008-xSO, Package_SO:SOIC-18W_7.5x11.6mm_P1.27mm, symbol Interface_Expansion:MCP23008-xSO
- removed U2: LTR-329ALS-01, 00_lib:LTR-329ALS-01_LTO, symbol 00_lib:LTR-329ALS-01
Other:
- added sheet Peripherals (peripherals.kicad_sch)
- sheet GPS ports: added GPS_{1PPS2}, GPS_{1PPS}, GPS_{BOOT_SEL}, GPS_{RSTN}, GPS_{RXD}, GPS_{TXD}; removed none
- sheet HV bleed ports: added HV_{SENSE}; removed none
- sheet High voltage supply ports: added GATE_{HV}, HV_{SENSE}, MEASURE_{HV}; removed none
- sheet LSD ADC ports: added LSD_{ADC_D0}, LSD_{ADC_D1}, LSD_{ADC_D2}, LSD_{ADC_D3}, LSD_{ADC_D4}, LSD_{ADC_D5}, LSD_{ADC_D6}, LSD_{ADC_D7}, LSD_{ADC_MODE}, LSD_{ADC_~{CS}}, LSD_{ADC_~{INT}}, LSD_{ADC_~{OFL}}, LSD_{ADC_~{RD}}, LSD_{ADC_~{WR}/RDY}, LSD_{SHUNT}, MEASURE_{HV}; removed none
- sheet Nixies ports: added CLOCK_{HV}, CLOCK_{PRECISE}, DATA_{HV}, DATA_{PRECISE}, LSD_{SHUNT}, PPS_{TRIMMED}, SENSE_{PRECISE}; removed none
- sheet Pico Ice ports: added CLOCK_{HV}, CLOCK_{PRECISE}, DATA_{HV}, DATA_{PRECISE}, GATE_{HV}, GPS_{1PPS2}, GPS_{1PPS}, GPS_{BOOT_SEL}, GPS_{RSTN}, GPS_{RXD}, GPS_{TXD}, I2C_{CLOCK}, I2C_{DATA}, INT_{IO-expander}, LSD_{ADC_D0}, LSD_{ADC_D1}, LSD_{ADC_D2}, LSD_{ADC_D3}, LSD_{ADC_D4}, LSD_{ADC_D5}, LSD_{ADC_D6}, LSD_{ADC_D7}, LSD_{ADC_MODE}, LSD_{ADC_~{CS}}, LSD_{ADC_~{INT}}, LSD_{ADC_~{OFL}}, LSD_{ADC_~{RD}}, LSD_{ADC_~{WR}/RDY}, MEASURE_{HV}, PPS_{TRIMMED}, SENSE_{PRECISE}, brightness_control, ~{RESET}_{IO-expander}; removed none
