File: hardware/KiCad/nixieAccurateClock/LSD_ADC.kicad_sch (KiCad schematic)
At the start: 19 parts, among them Q5 BSP88, U13 ADC0820BCWMX, U14 TXB0108PWR, U15 TXB0108PWR

Commit message: switch to all SM components
Parts:
- renumbered U13 to U6, U14 to U7, U15 to U8
Changed lines of the file:
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@@
   (symbol (lib_id "power:GND") (at 87.63 30.48 180) (unit 1)
     (in_bom yes) (on_board yes) (dnp no)
-    (property "Reference" "#PWR084" (at 87.63 24.13 0)
+    (property "Reference" "#PWR0101" (at 87.63 24.13 0)
       (effects (font (size 1.27 1.27)) hide)
     )
@@
       (project "nixieAccurateClock"
         (path "/55aab698-7558-4fe2-95ad-faa6da60ef89/919829db-9d44-4db4-a8a4-73523a1d66d3"
-          (reference "#PWR084") (unit 1)
+          (reference "#PWR0101") (unit 1)
         )
       )
@@
   (symbol (lib_id "power:+3.3V") (at 241.3 50.8 0) (unit 1)
     (in_bom yes) (on_board yes) (dnp no)
-    (property "Reference" "#PWR088" (at 241.3 54.61 0)
+    (property "Reference" "#PWR0105" (at 241.3 54.61 0)
       (effects (font (size 1.27 1.27)) hide)
     )
@@
       (project "nixieAccurateClock"
         (path "/55aab698-7558-4fe2-95ad-faa6da60ef89/919829db-9d44-4db4-a8a4-73523a1d66d3"
-          (reference "#PWR088") (unit 1)
+          (reference "#PWR0105") (unit 1)
         )
       )
@@
   (symbol (lib_id "00_lib:TXB0108PWR") (at 168.91 80.01 0) (unit 1)
     (in_bom yes) (on_board yes) (dnp no) (fields_autoplaced)
-    (property "Reference" "U14" (at 171.1041 97.79 0)
+    (property "Reference" "U7" (at 171.1041 97.79 0)
       (effects (font (size 1.27 1.27)) (justify left))
     )
@@
       (project "nixieAccurateClock"
         (path "/55aab698-7558-4fe2-95ad-faa6da60ef89/919829db-9d44-4db4-a8a4-73523a1d66d3"
-          (reference "U14") (unit 1)
+          (reference "U7") (unit 1)
         )
       )
@@
   (symbol (lib_id "power:GND") (at 133.35 69.85 270) (unit 1)
     (in_bom yes) (on_board yes) (dnp no)
-    (property "Reference" "#PWR090" (at 127 69.85 0)
+    (property "Reference" "#PWR0107" (at 127 69.85 0)
       (effects (font (size 1.27 1.27)) hide)
     )
@@
       (project "nixieAccurateClock"
         (path "/55aab698-7558-4fe2-95ad-faa6da60ef89/919829db-9d44-4db4-a8a4-73523a1d66d3"
-          (reference "#PWR090") (unit 1)
+          (reference "#PWR0107") (unit 1)
         )
       )
@@
   (symbol (lib_id "power:+5V") (at 246.38 50.8 0) (unit 1)
     (in_bom yes) (on_board yes) (dnp no)
-    (property "Reference" "#PWR089" (at 246.38 54.61 0)
+    (property "Reference" "#PWR0106" (at 246.38 54.61 0)
       (effects (font (size 1.27 1.27)) hide)
     )
@@
       (project "nixieAccurateClock"
         (path "/55aab698-7558-4fe2-95ad-faa6da60ef89/919829db-9d44-4db4-a8a4-73523a1d66d3"
-          (reference "#PWR089") (unit 1)
+          (reference "#PWR0106") (unit 1)
         )
       )
@@
   (symbol (lib_id "power:GND") (at 135.89 190.5 0) (unit 1)
     (in_bom yes) (on_board yes) (dnp no) (fields_autoplaced)
-    (property "Reference" "#PWR096" (at 135.89 196.85 0)
+    (property "Reference" "#PWR0113" (at 135.89 196.85 0)
       (effects (font (size 1.27 1.27)) hide)
     )
@@
       (project "nixieAccurateClock"
         (path "/55aab698-7558-4fe2-95ad-faa6da60ef89/919829db-9d44-4db4-a8a4-73523a1d66d3"
-          (reference "#PWR096") (unit 1)
+          (reference "#PWR0113") (unit 1)
         )
       )
@@
   (symbol (lib_id "power:+3.3V") (at 166.37 50.8 0) (unit 1)
     (in_bom yes) (on_board yes) (dnp no)
-    (property "Reference" "#PWR086" (at 166.37 54.61 0)
+    (property "Reference" "#PWR0103" (at 166.37 54.61 0)
       (effects (font (size 1.27 1.27)) hide)
     )
@@
       (project "nixieAccurateClock"
         (path "/55aab698-7558-4fe2-95ad-faa6da60ef89/919829db-9d44-4db4-a8a4-73523a1d66d3"
-          (reference "#PWR086") (unit 1)
+          (reference "#PWR0103") (unit 1)
         )
       )
@@
   (symbol (lib_id "power:GND") (at 114.3 190.5 0) (unit 1)
     (in_bom yes) (on_board yes) (dnp no) (fields_autoplaced)
-    (property "Reference" "#PWR095" (at 114.3 196.85 0)
+    (property "Reference" "#PWR0112" (at 114.3 196.85 0)
       (effects (font (size 1.27 1.27)) hide)
     )
@@
       (project "nixieAccurateClock"
         (path "/55aab698-7558-4fe2-95ad-faa6da60ef89/919829db-9d44-4db4-a8a4-73523a1d66d3"
-          (reference "#PWR095") (unit 1)
+          (reference "#PWR0112") (unit 1)
         )
       )
@@
   (symbol (lib_id "power:GND") (at 168.91 101.6 0) (unit 1)
     (in_bom yes) (on_board yes) (dnp no) (fields_autoplaced)
-    (property "Reference" "#PWR092" (at 168.91 107.95 0)
+    (property "Reference" "#PWR0109" (at 168.91 107.95 0)
       (effects (font (size 1.27 1.27)) hide)
     )
@@
       (project "nixieAccurateClock"
         (path "/55aab698-7558-4fe2-95ad-faa6da60ef89/919829db-9d44-4db4-a8a4-73523a1d66d3"
-          (reference "#PWR092") (unit 1)
+          (reference "#PWR0109") (unit 1)
         )
       )
@@
   (symbol (lib_id "power:VPP") (at 93.98 144.78 180) (unit 1)
     (in_bom yes) (on_board yes) (dnp no) (fields_autoplaced)
-    (property "Reference" "#PWR094" (at 93.98 140.97 0)
+    (property "Reference" "#PWR0111" (at 93.98 140.97 0)
       (effects (font (size 1.27 1.27)) hide)
     )
@@
       (project "nixieAccurateClock"
         (path "/55aab698-7558-4fe2-95ad-faa6da60ef89/919829db-9d44-4db4-a8a4-73523a1d66d3"
-          (reference "#PWR094") (unit 1)
+          (reference "#PWR0111") (unit 1)
         )
       )
@@
   (symbol (lib_id "power:+5V") (at 171.45 50.8 0) (unit 1)
     (in_bom yes) (on_board yes) (dnp no)
-    (property "Reference" "#PWR087" (at 171.45 54.61 0)
+    (property "Reference" "#PWR0104" (at 171.45 54.61 0)
       (effects (font (size 1.27 1.27)) hide)
     )
@@
       (project "nixieAccurateClock"
         (path "/55aab698-7558-4fe2-95ad-faa6da60ef89/919829db-9d44-4db4-a8a4-73523a1d66d3"
-          (reference "#PWR087") (unit 1)
+          (reference "#PWR0104") (unit 1)
         )
       )
@@
   (symbol (lib_id "power:GND") (at 243.84 101.6 0) (unit 1)
     (in_bom yes) (on_board yes) (dnp no) (fields_autoplaced)
-    (property "Reference" "#PWR093" (at 243.84 107.95 0)
+    (property "Reference" "#PWR0110" (at 243.84 107.95 0)
       (effects (font (size 1.27 1.27)) hide)
     )
@@
       (project "nixieAccurateClock"
         (path "/55aab698-7558-4fe2-95ad-faa6da60ef89/919829db-9d44-4db4-a8a4-73523a1d66d3"
-          (reference "#PWR093") (unit 1)
+          (reference "#PWR0110") (unit 1)
         )
       )
@@
   (symbol (lib_id "power:GND") (at 68.58 43.18 270) (unit 1)
     (in_bom yes) (on_board yes) (dnp no)
-    (property "Reference" "#PWR085" (at 62.23 43.18 0)
+    (property "Reference" "#PWR0102" (at 62.23 43.18 0)
       (effects (font (size 1.27 1.27)) hide)
     )
@@
       (project "nixieAccurateClock"
         (path "/55aab698-7558-4fe2-95ad-faa6da60ef89/919829db-9d44-4db4-a8a4-73523a1d66d3"
-          (reference "#PWR085") (unit 1)
+          (reference "#PWR0102") (unit 1)
         )
       )
@@
   (symbol (lib_id "power:+5V") (at 83.82 24.13 0) (unit 1)
     (in_bom yes) (on_board yes) (dnp no)
-    (property "Reference" "#PWR083" (at 83.82 27.94 0)
+    (property "Reference" "#PWR0100" (at 83.82 27.94 0)
       (effects (font (size 1.27 1.27)) hide)
     )
@@
       (project "nixieAccurateClock"
         (path "/55aab698-7558-4fe2-95ad-faa6da60ef89/919829db-9d44-4db4-a8a4-73523a1d66d3"
-          (reference "#PWR083") (unit 1)
+          (reference "#PWR0100") (unit 1)
         )
       )
@@
   (symbol (lib_name "TXB0108PWR_1") (lib_id "00_lib:TXB0108PWR") (at 243.84 80.01 0) (unit 1)
     (in_bom yes) (on_board yes) (dnp no) (fields_autoplaced)
-    (property "Reference" "U15" (at 246.0341 97.79 0)
+    (property "Reference" "U8" (at 246.0341 97.79 0)
       (effects (font (size 1.27 1.27)) (justify left))
     )
@@
       (project "nixieAccurateClock"
         (path "/55aab698-7558-4fe2-95ad-faa6da60ef89/919829db-9d44-4db4-a8a4-73523a1d66d3"
-          (reference "U15") (unit 1)
+          (reference "U8") (unit 1)
         )
       )
@@
   (symbol (lib_id "00_lib:ADC0820-N") (at 73.66 62.23 0) (unit 1)
     (in_bom yes) (on_board yes) (dnp no)
-    (property "Reference" "U13" (at 73.66 35.56 0)
+    (property "Reference" "U6" (at 73.66 35.56 0)
       (effects (font (size 1.27 1.27)) (justify left))
     )
@@
       (project "nixieAccurateClock"
         (path "/55aab698-7558-4fe2-95ad-faa6da60ef89/919829db-9d44-4db4-a8a4-73523a1d66d3"
-          (reference "U13") (unit 1)
+          (reference "U6") (unit 1)
         )
       )
@@
   (symbol (lib_id "power:GND") (at 208.28 69.85 270) (unit 1)
     (in_bom yes) (on_board yes) (dnp no)
-    (property "Reference" "#PWR091" (at 201.93 69.85 0)
+    (property "Reference" "#PWR0108" (at 201.93 69.85 0)
       (effects (font (size 1.27 1.27)) hide)
     )
@@
       (project "nixieAccurateClock"
         (path "/55aab698-7558-4fe2-95ad-faa6da60ef89/919829db-9d44-4db4-a8a4-73523a1d66d3"
-          (reference "#PWR091") (unit 1)
-        )
-      )
+          (reference "#PWR0108") (unit 1)
+        )
+      )

Commit message: switch to static level shifting
Parts:
- removed R27, R28: 100k, Resistor_SMD:R_0603_1608Metric, symbol Device:R
- removed U7, U8: TXB0108PWR, Package_SO:TSSOP-20_4.4x6.5mm_P0.65mm, symbol 00_lib:TXB0108PWR
- added C21, C22, C23, C24: 0.1u, Capacitor_SMD:C_0603_1608Metric, symbol Device:C_Small
- added U10, U6, U7, U9: ~, Package_SO:TSSOP-14_4.4x5mm_P0.65mm, symbol 00_lib:TXU0104PWR
- renumbered R29 to R27, R30 to R28, R31 to R29, R32 to R30, U6 to U8
Connections:
- net +3.3V: now also C18.1, C20.1, C22.1, C23.1, U10.8 (OE), U6.8 (OE), U7.8 (OE), U9.8 (OE); no longer C17.1, C19.1
- net +5V: now also C17.1, C19.1, C21.1, C24.1; no longer C18.1, C20.1
- net GND: now also U10.7 (GND), U6.7 (GND), U7.7 (GND), U9.7 (GND)
- net LSD_{ADC_5V_D0}: now also U6.5 (A4)
- net LSD_{ADC_5V_D1}: now also U6.4 (A3)
- net LSD_{ADC_5V_D2}: now also U6.3 (A2)
- net LSD_{ADC_5V_D3}: now also U6.2 (A1)
- net LSD_{ADC_5V_D4}: now also U7.5 (A4)
- net LSD_{ADC_5V_D5}: now also U7.4 (A3)
- net LSD_{ADC_5V_D6}: now also U7.3 (A2)
- net LSD_{ADC_5V_D7}: now also U7.2 (A1)
- net LSD_{ADC_5V_MODE}: now also U10.12 (B2Y)
- net LSD_{ADC_5V_~{CS}}: now also U10.10 (B4Y)
- net LSD_{ADC_5V_~{INT}}: now also U9.5 (A4)
- net LSD_{ADC_5V_~{OFL}}: now also U9.4 (A3)
- net LSD_{ADC_5V_~{RD}}: now also U10.11 (B3Y)
- net LSD_{ADC_5V_~{WR}/RDY}: now also U10.13 (B1Y)
- net LSD_{ADC_D0}: now also U6.10 (B4Y)
- net LSD_{ADC_D1}: now also U6.11 (B3Y)
- net LSD_{ADC_D2}: now also U6.12 (B2Y)
- net LSD_{ADC_D3}: now also U6.13 (B1Y)
- net LSD_{ADC_D4}: now also U7.10 (B4Y)
- net LSD_{ADC_D5}: now also U7.11 (B3Y)
- net LSD_{ADC_D6}: now also U7.12 (B2Y)
- net LSD_{ADC_D7}: now also U7.13 (B1Y)
- net LSD_{ADC_MODE}: now also U10.3 (A2)
- net LSD_{ADC_~{CS}}: now also U10.5 (A4)
- net LSD_{ADC_~{INT}}: now also U9.10 (B4Y)
- net LSD_{ADC_~{OFL}}: now also U9.11 (B3Y)
- net LSD_{ADC_~{RD}}: now also U10.4 (A3)
- net LSD_{ADC_~{WR}/RDY}: now also U10.2 (A1)
- net VCC_{lvl-shift-A-1}: now also U6.1 (V_{CCA})
- net VCC_{lvl-shift-A-2}: now also U7.1 (V_{CCA})
- net VCC_{lvl-shift-B-1}: now also U6.14 (V_{CCB})
- net VCC_{lvl-shift-B-2}: now also U7.14 (V_{CCB})
- new net VCC_{lvl-shift-A-3}: C21.2, U9.1 (V_{CCA}), U9.2 (A1), U9.3 (A2)
- new net VCC_{lvl-shift-A-4}: C23.2, U10.1 (V_{CCA})
- new net VCC_{lvl-shift-B-3}: C22.2, U9.14 (V_{CCB})
- new net VCC_{lvl-shift-B-4}: C24.2, U10.14 (V_{CCB})
Other:
- moved on the sheet: Q5, R27, R28, R29, R30, TP14, TP15, TP16, TP17

Commit message: WIP HV overhaul
Parts:
- removed R30: 10k, Resistor_SMD:R_0603_1608Metric, symbol Device:R
- added R?: 100k, Resistor_SMD:R_0603_1608Metric, symbol Device:R
- renumbered R28 to R27, R27 to R28
Connections:
- net GND: now also R29.2
- net HV_{MEASURE}: now also R?.1; no longer R29.1
- net LSD_{SHUNT_SC_Emitter}: now also R29.1
- net LSD_{SHUNT_div}: now also R27.2, R28.1; no longer R27.1, R28.2
- net LSD_{SHUNT}: now also R27.1; no longer R28.1
- net VPP: now also R28.2; no longer R27.2
- net V_{SHUNT}: now also R?.2; no longer R29.2
Other:
- moved on the sheet: R27, R28, R29

Commit message: HV overhaul
Parallel single stage boost convertor
Need to find replacement MOSFET because SiB452BK footprint is too small for reasonable manufacturing and HV clearance.
Parts:
- removed Q5: BSP88, Package_TO_SOT_SMD:SOT-223-3_TabPin2, symbol 00_lib:BSP88
- removed R27, R?: 100k, Resistor_SMD:R_0603_1608Metric, symbol Device:R
- removed R28: 10M, Resistor_SMD:R_0603_1608Metric, symbol Device:R
- removed R29: 10k, Resistor_SMD:R_0603_1608Metric, symbol Device:R
- removed TP15, TP16: TestPoint, 00_lib:TestPoint_Keystone_5019_Minature, symbol Connector:TestPoint
- added R?: 1M, Resistor_SMD:R_0603_1608Metric, symbol Device:R
- added R?: 47k, Resistor_SMD:R_0603_1608Metric, symbol Device:R
- renumbered C16 to C13, C17 to C14, C18 to C15, C19 to C16, C20 to C17, C21 to C18, C22 to C19, C23 to C20, C24 to C21, TP14 to TP12, TP17 to TP13, U8 to U10, U9 to U11, U10 to U12, U6 to U8, U7 to U9
Connections:
- net LSD_{SHUNT_div} is gone; now on net V_{SHUNT}: TP12.1
- net GND: now also R?.1
- net LSD_{SHUNT}: now also R?.2
- net V_{SHUNT}: now also R?.1, R?.2
- net HV_{MEASURE} renamed MEASURE_{HV}
Other:
- moved on the sheet: TP13

Commit message: single stage HV supply
Also switch to a MOSFET with a reasonable footprint
Parts:
- renumbered C14 to C10, C15 to C11, C16 to C12, C17 to C13, C18 to C14, C19 to C15, C20 to C16, C21 to C17, C13 to C9, TP12 to TP8, TP13 to TP9, U8 to U4, U9 to U5, U10 to U6, U11 to U7, U12 to U8
