File: hardware/KiCad/nixieAccurateClock/LSD_ADC.kicad_sch (KiCad schematic)
At the start: 18 parts, among them U6 ADC0820BCWMX

Commit message: update to KiCAD 8
Parts:
- gave numbers to parts that had none: 2
