File: hardware/KiCad/nixieAccurateClock/hv_supply.kicad_sch (KiCad schematic)
At the start: 3 parts, among them J10 Conn_01x02_Pin

Commit message: proper HVPS
Parts:
- added C4, C5, C6, C7: 1u, Capacitor_SMD:CP_Elec_8x10, symbol Device:C_Polarized
- added D4: 1SMB5956B-13, Diode_SMD:D_SMB, symbol Device:D_Zener
- added D? (x4): SM4004, Diode_SMD:D_MELF, symbol Diode:SM4004
- added L1: 10u, 00_lib:IND_BOURNS_SRR1280, symbol Device:L
- added Q1, Q2, Q3, Q4: PZTA42, Package_TO_SOT_SMD:SOT-223-3_TabPin2, symbol Transistor_BJT:PZTA42
- added R5, R6, R7, R8: 0.5, Resistor_SMD:R_2010_5025Metric, symbol Device:R
- added TP1, TP2, TP3, TP4: TestPoint, 00_lib:TestPoint_Keystone_5019_Minature, symbol Connector:TestPoint
Connections:
- net GND: now also C6.2, C7.2, D4.2 (A), D?.2 (A), R5.2, R6.2, R7.2, R8.2
- net HV_{SENSE}: now also R3.1, C6.1, D4.1 (K), D?.1 (K)
- net VPP: no longer R3.1
- new net +5V: L1.1
- new net GATE_{HV}: Q1.1 (B), Q2.1 (B), Q3.1 (B), Q4.1 (B)
- new net HV_{FULL-BOOST}: C4.1, D?.1 (K), D?.2 (A), TP2.1
- new net HV_{HALF-BOOST}: C4.2, C5.2, L1.2, Q1.2 (C), Q2.2 (C), Q3.2 (C), Q4.2 (C), TP1.1
- new net HV_{HALF-SUPPLY}: C7.1, D?.1 (K), D?.2 (A), TP4.1
- new net HV_{QUARTER-BOOST}: C5.1, D?.1 (K), D?.2 (A), TP3.1
- new net RE_{HV-1}: Q1.3 (E), R5.1
- new net RE_{HV-2}: Q2.3 (E), R6.1
- new net RE_{HV-3}: Q3.3 (E), R7.1
- new net RE_{HV-4}: Q4.3 (E), R8.1
Other:
- removed sheet Boost Quadrupler 1
- moved on the sheet: J10, R3, R4

Commit message: lay out HVPS
Changed lines of the file:
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@@
   (title_block
     (title "Nixie Accurate Clock")
-    (rev "A")
+    (rev "B")
     (company "Paul Willis")
   )
@@
   (junction (at 96.52 46.99) (diameter 0) (color 0 0 0 0)
   )
+  (junction (at 177.8 46.99) (diameter 0) (color 0 0 0 0)
+  )
   (junction (at 96.52 63.5) (diameter 0) (color 0 0 0 0)
   )
@@
     (stroke (width 0) (type default))
   )
-  (wire (pts (xy 153.67 46.99) (xy 210.82 46.99))
+  (wire (pts (xy 153.67 46.99) (xy 177.8 46.99))
     (stroke (width 0) (type default))
   )
@@
     (stroke (width 0) (type default))
   )
+  (wire (pts (xy 177.8 46.99) (xy 210.82 46.99))
+    (stroke (width 0) (type default))
+  )
   (wire (pts (xy 210.82 69.85) (xy 210.82 77.47))
     (stroke (width 0) (type default))
@@
     (stroke (width 0) (type default))
   )
+  (wire (pts (xy 180.34 50.8) (xy 177.8 50.8))
+    (stroke (width 0) (type default))
+  )
   (wire (pts (xy 124.46 46.99) (xy 124.46 52.07))
     (stroke (width 0) (type default))
@@
   )
   (wire (pts (xy 124.46 63.5) (xy 124.46 67.31))
+    (stroke (width 0) (type default))
+  )
+  (wire (pts (xy 177.8 50.8) (xy 177.8 46.99))
     (stroke (width 0) (type default))
   )
@@
     (effects (font (size 1.27 1.27)) (justify left top))
   )
-  (text_box "Some nixie power supplies online are based on single stage flyback with 1:10 transformers.  Transformers are expensive and not well stocked compared to inductors.  This boost convertor with voltage quadrupler resembles LT AN47 Appendix D with a voltage quadrupler (Art of Electronics 3E 1.6.5 Regulators, Figure 1.67).\n\nOpt to just use the RP2040 PIO PWM and ADC rather than a discrete SMPS IC.\n\nAn exotic MOSFET or parallel boost convertor stages could be used.  Instead I am using a cheap, robust BJT in parallel with biasing resistors to current share for worst case loads."
-    (at 29.21 128.27 0) (size 60.96 30.48)
+  (text_box "Some nixie power supplies online are based on single stage flyback with 1:10 transformers.  Transformers are expensive and not well stocked compared to inductors.  This boost convertor with voltage quadrupler resembles LT AN47 Appendix D with a voltage quadrupler (Art of Electronics 3E 1.6.5 Regulators, Figure 1.67).\n\nOpt to just use the RP2040 PIO PWM and ADC rather than a discrete SMPS IC.\n\nAn exotic MOSFET or parallel boost convertor stages could be used.  Instead I am using a cheap, robust BJT in parallel with biasing resistors to current share for worst case loads (AoE 3E 2.4.4 Current sharing in paralleled BJTs)."
+    (at 29.21 128.27 0) (size 60.96 33.02)
     (stroke (width 0) (type default))
     (fill (type none))
@@
   (label "HV_{QUARTER-BOOST}" (at 95.25 63.5 180) (fields_autoplaced)
     (effects (font (size 1.27 1.27)) (justify right bottom))
-  )
-  (label "HV_{SENSE}" (at 163.83 46.99 0) (fields_autoplaced)
-    (effects (font (size 1.27 1.27)) (justify left bottom))
   )
   (label "HV_{HALF-SUPPLY}" (at 125.73 63.5 0) (fields_autoplaced)
@@
     )
   )
+  (global_label "HV_{SENSE}" (shape output) (at 180.34 50.8 0) (fields_autoplaced)
+    (effects (font (size 1.27 1.27)) (justify left))
+    (property "Intersheetrefs" "${INTERSHEET_REFS}" (at 190.6331 50.8 0)
+      (effects (font (size 1.27 1.27)) (justify left) hide)
+    )
+  )

Commit message: route nixie daughter boards
Parts:
- Q1, Q2, Q3, Q4: Digikey link (none) -> https://www.digikey.com/en/products/detail/micro-commercial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; Mouser link (none) -> https://www.mouser.com/ProductDetail/Diotec-Semiconductor/P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; Price (none) -> 0.41
- R5, R6, R7, R8: Model (none) -> CSRN2010FKR500
Changed lines of the file:
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@@
+      (effects (font (size 1.27 1.27)) hide)
+    )
+    (property "Model" "CSRN2010FKR500" (at 152.4 139.7 0)
       (effects (font (size 1.27 1.27)) hide)
     )
@@
       (effects (font (size 1.27 1.27)) (justify left) hide)
     )
+    (property "Digikey link" "https://www.digikey.com/en/products/detail/micro-commercial-co/PZTA42-TP/10054674" (at 184.15 128.27 0)
+      (effects (font (size 1.27 1.27)) hide)
+    )
+    (property "Mouser link" "https://www.mouser.com/ProductDetail/Diotec-Semiconductor/PZTA42?qs=OlC7AqGiEDlNqlN7791aVQ%3D%3D" (at 184.15 128.27 0)
+      (effects (font (size 1.27 1.27)) hide)
+    )
+    (property "Price" "0.41" (at 184.15 128.27 0)
+      (effects (font (size 1.27 1.27)) hide)
+    )
     (pin "3")
     (pin "2")
@@
       (effects (font (size 1.27 1.27)) (justify left) hide)
     )
+    (property "Digikey link" "https://www.digikey.com/en/products/detail/micro-commercial-co/PZTA42-TP/10054674" (at 115.57 128.27 0)
+      (effects (font (size 1.27 1.27)) hide)
+    )
+    (property "Mouser link" "https://www.mouser.com/ProductDetail/Diotec-Semiconductor/PZTA42?qs=OlC7AqGiEDlNqlN7791aVQ%3D%3D" (at 115.57 128.27 0)
+      (effects (font (size 1.27 1.27)) hide)
+    )
+    (property "Price" "0.41" (at 115.57 128.27 0)
+      (effects (font (size 1.27 1.27)) hide)
+    )
     (pin "3")
     (pin "2")
@@
     (property "Datasheet" "https://www.onsemi.com/pub/Collateral/PZTA42T1-D.PDF" (at 218.44 128.27 0)
       (effects (font (size 1.27 1.27)) (justify left) hide)
+    )
+    (property "Digikey link" "https://www.digikey.com/en/products/detail/micro-commercial-co/PZTA42-TP/10054674" (at 218.44 128.27 0)
+      (effects (font (size 1.27 1.27)) hide)
+    )
+    (property "Mouser link" "https://www.mouser.com/ProductDetail/Diotec-Semiconductor/PZTA42?qs=OlC7AqGiEDlNqlN7791aVQ%3D%3D" (at 218.44 128.27 0)
+      (effects (font (size 1.27 1.27)) hide)
+    )
+    (property "Price" "0.41" (at 218.44 128.27 0)
+      (effects (font (size 1.27 1.27)) hide)
     )
     (pin "3")
@@
       (effects (font (size 1.27 1.27)) hide)
     )
+    (property "Model" "CSRN2010FKR500" (at 220.98 139.7 0)
+      (effects (font (size 1.27 1.27)) hide)
+    )
     (pin "1")
     (pin "2")
@@
     (property "Datasheet" "https://www.onsemi.com/pub/Collateral/PZTA42T1-D.PDF" (at 149.86 128.27 0)
       (effects (font (size 1.27 1.27)) (justify left) hide)
+    )
+    (property "Digikey link" "https://www.digikey.com/en/products/detail/micro-commercial-co/PZTA42-TP/10054674" (at 149.86 128.27 0)
+      (effects (font (size 1.27 1.27)) hide)
+    )
+    (property "Mouser link" "https://www.mouser.com/ProductDetail/Diotec-Semiconductor/PZTA42?qs=OlC7AqGiEDlNqlN7791aVQ%3D%3D" (at 149.86 128.27 0)
+      (effects (font (size 1.27 1.27)) hide)
+    )
+    (property "Price" "0.41" (at 149.86 128.27 0)
+      (effects (font (size 1.27 1.27)) hide)
     )
     (pin "3")
@@
       (effects (font (size 1.27 1.27)) hide)
     )
+    (property "Model" "CSRN2010FKR500" (at 118.11 139.7 0)
+      (effects (font (size 1.27 1.27)) hide)
+    )
     (pin "1")
     (pin "2")
@@
       (effects (font (size 1.27 1.27)) hide)
     )
+    (property "Model" "CSRN2010FKR500" (at 186.69 139.7 0)
+      (effects (font (size 1.27 1.27)) hide)
+    )
