File: hardware/KiCad/nixieAccurateClock/hv_supply.kicad_sch (KiCad schematic)
At the start: 25 parts, among them J10 Conn_01x02_Pin, Q1 PZTA42, Q2 PZTA42, Q3 PZTA42, Q4 PZTA42

Commit message: update to KiCAD 8
Parts:
- gave numbers to parts that had none: 4

Commit message: add polyfuse to HVPS
WIP hierarchy overhaul
Parts:
- added F1: 1A, Fuse:Fuse_1206_3216Metric, symbol Device:Polyfuse
Connections:
- net +5V: now also F1.1; no longer L1.1
- new net 5V_{BOOST-FUSE}: F1.2, L1.1
Other:
- moved on the sheet: L1
Changed lines of the file:
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@@
 	(wire
 		(pts
-			(xy 177.8 46.99) (xy 210.82 46.99)
+			(xy 35.56 46.99) (xy 53.34 46.99)
 		)
 		(stroke
@@
 	(wire
 		(pts
-			(xy 210.82 69.85) (xy 210.82 77.47)
+			(xy 177.8 46.99) (xy 210.82 46.99)
 		)
 		(stroke
@@
 	(wire
 		(pts
-			(xy 33.02 46.99) (xy 41.91 46.99)
+			(xy 210.82 69.85) (xy 210.82 77.47)
 		)
 		(stroke
@@
 	(wire
 		(pts
+			(xy 24.13 46.99) (xy 27.94 46.99)
+		)
+		(stroke
+			(width 0)
+			(type default)
+		)
+	)
+	(wire
+		(pts
 			(xy 152.4 143.51) (xy 152.4 146.05)
 		)
@@
 	(wire
 		(pts
-			(xy 49.53 46.99) (xy 96.52 46.99)
+			(xy 60.96 46.99) (xy 96.52 46.99)
 		)
 		(stroke
@@
 		)
 	)
+	(text_box "Polyfuse input with 1A hold current and 1.8A trip current.\n\nSimulation shows this will hold up to 110 mA load and trip on 170 mA load.\n\n12 Nixie tubes @ 2.8 mA each would be 33.6 mA worst case load.\n\nThe goal is to allow max load driving while tripping on faults.\nThis is limits the energy delivered to humans / environment during shocks to be ~12 J / 2.9 cal (300 ms trip time * 200 V^2 / 1 kOhm)."
+		(exclude_from_sim no)
+		(at 19.05 17.78 0)
+		(size 78.74 20.32)
+		(stroke
+			(width 0)
+			(type default)
+		)
+		(fill
+			(type none)
+		)
+		(effects
+			(font
+				(size 1.27 1.27)
+			)
+			(justify left top)
+		)
+	)
 	(text_box "100:1 divider to bring (0-333.3 V) down to (0-3.3V) for feedback ADC"
 		(exclude_from_sim no)
@@
 		)
 	)
+	(label "5V_{BOOST-FUSE}"
+		(at 36.83 46.99 0)
+		(fields_autoplaced yes)
+		(effects
+			(font
+				(size 1.27 1.27)
+			)
+			(justify left bottom)
+		)
+	)
 	(label "HV_{QUARTER-BOOST}"
 		(at 95.25 63.5 180)
@@
 	)
 	(label "HV_{HALF-BOOST}"
-		(at 58.42 46.99 0)
+		(at 67.31 46.99 0)
 		(fields_autoplaced yes)
 		(effects
@@
 	(symbol
 		(lib_id "power:+5V")
-		(at 33.02 46.99 90)
+		(at 24.13 46.99 90)
 		(unit 1)
 		(exclude_from_sim yes)
@@
 		(fields_autoplaced yes)
 		(property "Reference" "#PWR043"
-			(at 36.83 46.99 0)
+			(at 27.94 46.99 0)
 			(effects
 				(font
@@
 		)
 		(property "Value" "+5V"
-			(at 29.21 46.99 90)
+			(at 20.32 46.99 90)
 			(effects
 				(font
@@
 		)
 		(property "Footprint" ""
-			(at 33.02 46.99 0)
+			(at 24.13 46.99 0)
 			(effects
 				(font
@@
 		)
 		(property "Datasheet" ""
-			(at 33.02 46.99 0)
+			(at 24.13 46.99 0)
 			(effects
 				(font
@@
 		)
 		(property "Description" "Power symbol creates a global label with name \"+5V\""
-			(at 33.02 46.99 0)
+			(at 24.13 46.99 0)
 			(effects
 				(font
@@
 	)
 	(symbol
+		(lib_id "Device:Polyfuse")
+		(at 31.75 46.99 90)
+		(unit 1)
+		(exclude_from_sim no)
+		(in_bom yes)
+		(on_board yes)
+		(dnp no)
+		(fields_autoplaced yes)
+		(property "Reference" "F1"
+			(at 31.75 40.64 90)
+			(effects
+				(font
+					(size 1.27 1.27)
+				)
+			)
+		)
+		(property "Value" "1A"
+			(at 31.75 43.18 90)
+			(effects
+				(font
+					(size 1.27 1.27)
+				)
+			)
+		)
+		(property "Footprint" "Fuse:Fuse_1206_3216Metric"
+			(at 36.83 45.72 0)
+			(effects
+				(font
+					(size 1.27 1.27)
+				)
+				(justify left)
+				(hide yes)
+			)
+		)
+		(property "Datasheet" "https://www.belfuse.com/resources/datasheets/circuitprotection/ds-cp-0zcj-series.pdf"
+			(at 31.75 46.99 0)
+			(effects
+				(font
+					(size 1.27 1.27)
+				)
+				(hide yes)
+			)
+		)
+		(property "Description" "Resettable fuse, polymeric positive temperature coefficient"
+			(at 31.75 46.99 0)
+			(effects
+				(font
+					(size 1.27 1.27)
+				)
+				(hide yes)
+			)
+		)
+		(property "Model" "0ZCJ0100FF2E"
+			(at 31.75 46.99 90)
+			(effects
+				(font
+					(size 1.27 1.27)
+				)
+				(hide yes)
+			)
+		)
+		(property "Digikey link" "https://www.digikey.com/en/products/detail/bel-fuse-inc/0ZCJ0100FF2E/4156136"
+			(at 31.75 46.99 90)
+			(effects
+				(font
+					(size 1.27 1.27)
+				)
+				(hide yes)
+			)
+		)
+		(property "Mouser link" "https://www.mouser.com/ProductDetail/Bel-Fuse/0ZCJ0100FF2E?qs=SRYZG9HaIQ16trCtSE8WyA%3D%3D"
+			(at 31.75 46.99 90)
+			(effects
+				(font
+					(size 1.27 1.27)
+				)
+				(hide yes)
+			)
+		)
+		(property "Price" "0.23"
+			(at 31.75 46.99 90)
+			(effects
+				(font
+					(size 1.27 1.27)
+				)
+				(hide yes)
+			)
+		)
+		(pin "1"
+		)
+		(pin "2"
+		)
+		(instances
+			(project "nixieAccurateClock"
+				(path "/55aab698-7558-4fe2-95ad-faa6da60ef89/f2852417-d6c8-4bbe-bd15-a29bc4083bd0"
+					(reference "F1")
+					(unit 1)
+				)
+			)
+		)
+	)
+	(symbol
 		(lib_id "Device:R")
 		(at 231.14 59.69 0)
@@
 	(symbol
 		(lib_id "Device:L")
-		(at 45.72 46.99 90)
+		(at 57.15 46.99 90)
 		(unit 1)
 		(exclude_from_sim no)
@@
 		(fields_autoplaced yes)
 		(property "Reference" "L1"
-			(at 45.72 41.91 90)
+			(at 57.15 41.91 90)
 			(effects
 				(font
@@
 		)
 		(property "Value" "10u"
-			(at 45.72 44.45 90)
+			(at 57.15 44.45 90)
 			(effects
 				(font
@@
 		)
 		(property "Footprint" "00_lib:IND_BOURNS_SRR1280"
-			(at 45.72 46.99 0)
+			(at 57.15 46.99 0)
 			(effects
 				(font
@@
 		)
 		(property "Datasheet" "https://www.bourns.com/docs/Product-Datasheets/SRR1280.pdf"
-			(at 45.72 46.99 0)
+			(at 57.15 46.99 0)
 			(effects
 				(font
@@
 		)
 		(property "Description" "Inductor"
-			(at 45.72 46.99 0)
+			(at 57.15 46.99 0)
 			(effects
 				(font
@@
 		)
 		(property "Model" "SRR1280-100M"
-			(at 45.72 46.99 90)
+			(at 57.15 46.99 90)
 			(effects
 				(font
@@
 		)
 		(property "Price" "1.02"
-			(at 45.72 46.99 0)
+			(at 57.15 46.99 0)
 			(effects
 				(font
@@
 		)
 		(property "Digikey link" "https://www.digikey.com/en/products/detail/bourns-inc/SRR1280-100M/1969992"
-			(at 45.72 46.99 0)
+			(at 57.15 46.99 0)
 			(effects
 				(font
@@
 		)
 		(property "Mouser link" "https://www.mouser.com/ProductDetail/Bourns/SRR1280-100M?qs=brMhP%2FMjUfe%2FtbNTKcGHiQ%3D%3D"
-			(at 45.72 46.99 0)
+			(at 57.15 46.99 0)
 			(effects
 				(font

Commit message: fuse HV, refactor schematic hierarchy
Changed lines of the file:
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@@
 	(title_block
 		(title "Nixie Accurate Clock")
-		(date "2024-02-25")
+		(date "2024-03-07")
 		(rev "B")
 		(company "Paul Willis")
@@
 		)
 	)
-	(global_label "GATE_{HV}"
+	(hierarchical_label "GATE_{HV}"
 		(shape input)
 		(at 107.95 128.27 180)
@@
 			(justify right)
 		)
-		(property "Intersheetrefs" "${INTERSHEET_REFS}"
-			(at 98.5035 128.27 0)
-			(effects
-				(font
-					(size 1.27 1.27)
-				)
-				(justify right)
-				(hide yes)
-			)
-		)
-	)
-	(global_label "MEASURE_{HV}"
+	)
+	(hierarchical_label "GATE_{HV}"
+		(shape input)
+		(at 176.53 128.27 180)
+		(fields_autoplaced yes)
+		(effects
+			(font
+				(size 1.27 1.27)
+			)
+			(justify right)
+		)
+	)
+	(hierarchical_label "MEASURE_{HV}"
 		(shape output)
 		(at 233.68 66.04 0)
@@
 			(justify left)
 		)
-		(property "Intersheetrefs" "${INTERSHEET_REFS}"
-			(at 247.2993 66.04 0)
-			(effects
-				(font
-					(size 1.27 1.27)
-				)
-				(justify left)
-				(hide yes)
-			)
-		)
-	)
-	(global_label "GATE_{HV}"
+	)
+	(hierarchical_label "HV_{SENSE}"
+		(shape output)
+		(at 180.34 50.8 0)
+		(fields_autoplaced yes)
+		(effects
+			(font
+				(size 1.27 1.27)
+			)
+			(justify left)
+		)
+	)
+	(hierarchical_label "GATE_{HV}"
 		(shape input)
 		(at 210.82 128.27 180)
@@
 			(justify right)
 		)
-		(property "Intersheetrefs" "${INTERSHEET_REFS}"
-			(at 201.3735 128.27 0)
-			(effects
-				(font
-					(size 1.27 1.27)
-				)
-				(justify right)
-				(hide yes)
-			)
-		)
-	)
-	(global_label "GATE_{HV}"
+	)
+	(hierarchical_label "GATE_{HV}"
 		(shape input)
 		(at 142.24 128.27 180)
@@
 			(justify right)
 		)
-		(property "Intersheetrefs" "${INTERSHEET_REFS}"
-			(at 132.7935 128.27 0)
-			(effects
-				(font
-					(size 1.27 1.27)
-				)
-				(justify right)
-				(hide yes)
-			)
-		)
-	)
-	(global_label "GATE_{HV}"
-		(shape input)
-		(at 176.53 128.27 180)
-		(fields_autoplaced yes)
-		(effects
-			(font
-				(size 1.27 1.27)
-			)
-			(justify right)
-		)
-		(property "Intersheetrefs" "${INTERSHEET_REFS}"
-			(at 167.0835 128.27 0)
-			(effects
-				(font
-					(size 1.27 1.27)
-				)
-				(justify right)
-				(hide yes)
-			)
-		)
-	)
-	(global_label "HV_{SENSE}"
-		(shape output)
-		(at 180.34 50.8 0)
-		(fields_autoplaced yes)
-		(effects
-			(font
-				(size 1.27 1.27)
-			)
-			(justify left)
-		)
-		(property "Intersheetrefs" "${INTERSHEET_REFS}"
-			(at 190.6331 50.8 0)
-			(effects
-				(font
-					(size 1.27 1.27)
-				)
-				(justify left)
-				(hide yes)
-			)
-		)
-	)
+	)
