File: hardware/KiCad/nixieAccurateClock/hv_supply.kicad_sch (KiCad schematic)
At the start: 26 parts, among them J10 Conn_01x02_Pin, Q1 PZTA42, Q2 PZTA42, Q3 PZTA42, Q4 PZTA42

Commit message: fix 2x1 SM header chirality
Parts:
- J10: footprint Connector_PinHeader_2.54mm:PinHeader_1x02_P2.54mm_Vertical_SMD_Pin1Left -> Connector_PinHeader_2.54mm:PinHeader_1x02_P2.54mm_Vertical_SMD_Pin1Right
Changed lines of the file:
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@@
 			)
 		)
-		(property "Footprint" "Connector_PinHeader_2.54mm:PinHeader_1x02_P2.54mm_Vertical_SMD_Pin1Left"
+		(property "Footprint" "Connector_PinHeader_2.54mm:PinHeader_1x02_P2.54mm_Vertical_SMD_Pin1Right"
 			(at 246.38 54.61 0)
 			(effects

Commit message: more detailed build notes, drop HV divider by 10x
Parts:
- R3: value 10M -> 1M; Digikey link https://www.digikey.com/en/products/detail/stackpole-electronics-inc/RMCF0603FT10M0/1761206 -> https://www.digikey.com/en/products/detail/stackpole-electronics-inc/RMCF0603FT1M00/1761036; Model RMCF0603FT10M0 -> RMCF0603FT1M00; Mouser link https://www.mouser.com/ProductDetail/SEI-Stackpole/RMCF0603FT10M0?qs=FESYatJ8odIf0bWpBT4vKw%3D%3D -> https://www.mouser.com/ProductDetail/SEI-Stackpole/RMCF0603FT1M00?qs=FESYatJ8odJNClY0wUC1cg%3D%3D
- R4: value 100k -> 10k; Digikey link https://www.digikey.com/en/products/detail/yageo/RC0603JR-0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 -> https://www.digikey.com/en/products/detail/yageo/RC0603FR-0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; Model RC0603JR-07100KL -> RC0603FR-0710KL; Mouser link https://www.mouser.com/ProductDetail/YAGEO/RC0603JR-07100KL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 -> https://www.mouser.com/ProductDetail/YAGEO/RC0603FR-0710KL?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
Changed lines of the file:
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@@
 			)
 		)
-		(property "Value" "10M"
+		(property "Value" "1M"
 			(at 233.68 60.96 0)
 			(effects
@@
 			)
 		)
-		(property "Model" "RMCF0603FT10M0"
+		(property "Model" "RMCF0603FT1M00"
 			(at 231.14 59.69 0)
 			(effects
@@
 			)
 		)
-		(property "Digikey link" "https://www.digikey.com/en/products/detail/stackpole-electronics-inc/RMCF0603FT10M0/1761206"
+		(property "Digikey link" "https://www.digikey.com/en/products/detail/stackpole-electronics-inc/RMCF0603FT1M00/1761036"
 			(at 231.14 59.69 0)
 			(effects
@@
 			)
 		)
-		(property "Mouser link" "https://www.mouser.com/ProductDetail/SEI-Stackpole/RMCF0603FT10M0?qs=FESYatJ8odIf0bWpBT4vKw%3D%3D"
+		(property "Mouser link" "https://www.mouser.com/ProductDetail/SEI-Stackpole/RMCF0603FT1M00?qs=FESYatJ8odJNClY0wUC1cg%3D%3D"
 			(at 231.14 59.69 0)
 			(effects
@@
 			)
 		)
-		(property "Value" "100k"
+		(property "Value" "10k"
 			(at 233.68 73.66 0)
 			(effects
@@
 			)
 		)
-		(property "Model" "RC0603JR-07100KL"
+		(property "Model" "RC0603FR-0710KL"
 			(at 231.14 72.39 0)
 			(effects
@@
 			)
 		)
-		(property "Digikey link" "https://www.digikey.com/en/products/detail/yageo/RC0603JR-07100KL/726698"
+		(property "Digikey link" "https://www.digikey.com/en/products/detail/yageo/RC0603FR-0710KL/726880"
 			(at 231.14 72.39 0)
 			(effects
@@
 			)
 		)
-		(property "Mouser link" "https://www.mouser.com/ProductDetail/YAGEO/RC0603JR-07100KL?qs=2cAdsCoAWRG9Rhqklpdeqg%3D%3D"
+		(property "Mouser link" "https://www.mouser.com/ProductDetail/YAGEO/RC0603FR-0710KL?qs=grNVn54RoB%252B3GtjbJj3wJQ%3D%3D"
 			(at 231.14 72.39 0)
 			(effects

Commit message: Modify HV supply to attempt to solve weak IC
Parts:
- removed Q1, Q2, Q3, Q4: PZTA42, Package_TO_SOT_SMD:SOT-223-3_TabPin2, symbol Transistor_BJT:PZTA42
- removed R5, R6, R7, R8: 0.5, Resistor_SMD:R_2010_5025Metric, symbol Device:R
- added Q1, Q2, Q3, Q4: BSP296N, Package_TO_SOT_SMD:SOT-223-3_TabPin2, symbol Transistor_FET:BSP89
- D1, D2, D3, D5: value SM4004 -> EGL41G; Digikey link https://www.digikey.com/en/products/detail/diotec-semicondu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 -> https://www.digikey.com/en/products/detail/vishay-general-s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; Model SM4004 -> EGL41G; Mouser link https://www.mouser.com/ProductDetail/Diotec-Semiconductor/S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 -> https://www.mouser.com/ProductDetail/Vishay-General-Semicon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; Price 0.27 -> 0.47
- F1: value 1A -> 2A; Digikey link https://www.digikey.com/en/products/detail/bel-fuse-inc/0ZCJ0100FF2E/4156136 -> https://www.digikey.com/en/products/detail/bel-fuse-inc/0ZCJ0200FF2C/4156138; Model 0ZCJ0100FF2E -> 0ZCJ0200FF2C; Mouser link https://www.mouser.com/ProductDetail/Bel-Fuse/0ZCJ0100FF2E?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 -> https://www.mouser.com/ProductDetail/Bel-Fuse/0ZCJ0200FF2C?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; Price 0.23 -> 0.46
Connections:
- net GATE_{HV}: now also Q1.1 (G), Q2.1 (G), Q3.1 (G), Q4.1 (G)
- net GND: now also Q1.3 (S), Q2.3 (S), Q3.3 (S), Q4.3 (S)
- net HV_{HALF-BOOST}: now also Q1.2 (D), Q2.2 (D), Q3.2 (D), Q4.2 (D)
Other:
- moved on the sheet: C5, C7, TP1, TP2, TP3
