File: hardware/KiCad/nixieAccurateClock/nixies.kicad_sch (KiCad schematic)
At the start: 7 parts, among them J11 Conn_02x05_Odd_Even

Commit message: switch all components to SMT
layout is a mess
Parts:
- J11: footprint Connector_PinSocket_2.54mm:PinSocket_2x05_P2.54mm_Horizontal -> 00_lib:M207920542R; Digikey link https://www.digikey.com/en/products/detail/sullins-connecto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 -> https://www.digikey.com/en/products/detail/harwin-inc/M20-7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; Model SFH11-PBPC-D05-RA-BK -> M20-7920542R; Mouser link N/A -> https://www.mouser.com/ProductDetail/Harwin/M20-7920542R?qs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; Price 0.81 -> 1.71
Changed lines of the file:
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@@
       (effects (font (size 1.27 1.27)))
     )
-    (property "Footprint" "Connector_PinSocket_2.54mm:PinSocket_2x05_P2.54mm_Horizontal" (at 45.72 135.89 0)
+    (property "Footprint" "00_lib:M207920542R" (at 45.72 135.89 0)
       (effects (font (size 1.27 1.27)) hide)
     )
-    (property "Datasheet" "https://s3.amazonaws.com/catalogspreads-pdf/PAGE123%20.100%20SFH11%20SERIES%20FEMALE%20HDR%20ST%20RA.pdf" (at 45.72 135.89 0)
+    (property "Datasheet" "https://cdn.harwin.com/pdfs/Harwin_Datasheet-INDESS.pdf" (at 45.72 135.89 0)
       (effects (font (size 1.27 1.27)) hide)
     )
-    (property "Model" "SFH11-PBPC-D05-RA-BK" (at 45.72 135.89 0)
+    (property "Model" "M20-7920542R" (at 45.72 135.89 0)
       (effects (font (size 1.27 1.27)) hide)
     )
-    (property "Price" "0.81" (at 45.72 135.89 0)
+    (property "Price" "1.71" (at 45.72 135.89 0)
       (effects (font (size 1.27 1.27)) hide)
     )
-    (property "Digikey link" "https://www.digikey.com/en/products/detail/sullins-connector-solutions/SFH11-PBPC-D05-RA-BK/1990095" (at 45.72 135.89 0)
+    (property "Digikey link" "https://www.digikey.com/en/products/detail/harwin-inc/M20-7920542R/6559290" (at 45.72 135.89 0)
       (effects (font (size 1.27 1.27)) hide)
     )
-    (property "Mouser link" "N/A" (at 45.72 135.89 0)
+    (property "Mouser link" "https://www.mouser.com/ProductDetail/Harwin/M20-7920542R?qs=k41KVqW3ymqj80AqJ%2FxUlA%3D%3D" (at 45.72 135.89 0)
       (effects (font (size 1.27 1.27)) hide)
     )

Commit message: switch to all SM components
Parts:
- J13: renamed from U7; Digikey link N/A -> https://www.digikey.com/en/products/detail/samtec-inc/SSM-1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; Model (none) -> SSM-105-L-DV; Mouser link N/A -> https://www.mouser.com/ProductDetail/Samtec/SSM-105-L-DV?qs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; Price 21.41 -> 21.30
- J14: renamed from U8; Digikey link N/A -> https://www.digikey.com/en/products/detail/samtec-inc/SSM-1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; Model (none) -> SSM-105-L-DV; Mouser link N/A -> https://www.mouser.com/ProductDetail/Samtec/SSM-105-L-DV?qs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; Price 21.41 -> 21.30
- J15: renamed from U9; Digikey link N/A -> https://www.digikey.com/en/products/detail/samtec-inc/SSM-1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; Model (none) -> SSM-105-L-DV; Mouser link N/A -> https://www.mouser.com/ProductDetail/Samtec/SSM-105-L-DV?qs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; Price 21.41 -> 21.30
- J16: renamed from U10; Digikey link N/A -> https://www.digikey.com/en/products/detail/samtec-inc/SSM-1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; Model (none) -> SSM-105-L-DV; Mouser link N/A -> https://www.mouser.com/ProductDetail/Samtec/SSM-105-L-DV?qs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; Price 21.41 -> 21.30
- J17: renamed from U11; Digikey link N/A -> https://www.digikey.com/en/products/detail/samtec-inc/SSM-1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; Model (none) -> SSM-105-L-DV; Mouser link N/A -> https://www.mouser.com/ProductDetail/Samtec/SSM-105-L-DV?qs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; Price 21.41 -> 21.30
- J18: renamed from U12; Digikey link N/A -> https://www.digikey.com/en/products/detail/samtec-inc/SSM-1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; Model (none) -> SSM-105-L-DV; Mouser link N/A -> https://www.mouser.com/ProductDetail/Samtec/SSM-105-L-DV?qs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; Price 21.41 -> 21.30
- renumbered J11 to J19

Commit message: HV overhaul
Parallel single stage boost convertor
Need to find replacement MOSFET because SiB452BK footprint is too small for reasonable manufacturing and HV clearance.
Parts:
- J11: renamed from J13; Price 21.30 -> 2.59
- J12: renamed from J14; Price 21.30 -> 2.59
- J13: renamed from J15; Price 21.30 -> 2.59
- J14: renamed from J16; Price 21.30 -> 2.59
- J15: renamed from J17; Price 21.30 -> 2.59
- J16: renamed from J18; Price 21.30 -> 2.59
- renumbered J19 to J17
