File: hardware/KiCad/nixieAccurateClock/HV_bleed.kicad_sch (KiCad schematic)
At the start: 10 parts, among them Q3 BSP88, Q4 BSP88

Commit message: HV overhaul
Parallel single stage boost convertor
Need to find replacement MOSFET because SiB452BK footprint is too small for reasonable manufacturing and HV clearance.
Parts:
- removed Q3, Q4: BSP88, Package_TO_SOT_SMD:SOT-223-3_TabPin2, symbol 00_lib:BSP88
- added U6, U7: SIB452DK-T1-GE3, 00_lib:SON_K-T1-GE3_VIS, symbol 00_lib:SIB452DK-T1-GE3
- renumbered C15 to C12, D3 to D9, R24 to R5, R25 to R6, R26 to R7, TP12 to TP10, TP13 to TP11, TP11 to TP9
Connections:
- net +5V: now also U7.3 (G)
- net GND: now also U7.4 (S), U7.7 (S)
- net HV_bleed_{drain}: now also U6.1 (D), U6.2 (D), U6.5 (D), U6.6 (D)
- net HV_bleed_{gate}: now also U6.3 (G), U7.1 (D), U7.2 (D), U7.5 (D), U7.6 (D)
- net HV_bleed_{source}: now also U6.4 (S), U6.7 (S)
Other:
- moved on the sheet: C12, R6, R7, TP10, TP9

Commit message: single stage HV supply
Also switch to a MOSFET with a reasonable footprint
Parts:
- removed U6, U7: SIB452DK-T1-GE3, 00_lib:SON_K-T1-GE3_VIS, symbol 00_lib:SIB452DK-T1-GE3
- added Q2, Q3: BSP88, Package_TO_SOT_SMD:SOT-223-3_TabPin2, symbol 00_lib:BSP88
- renumbered C12 to C8, D9 to D5, TP9 to TP5, TP10 to TP6, TP11 to TP7
Connections:
- net +5V: now also Q3.1 (G)
- net GND: now also Q3.3 (S)
- net HV_bleed_{drain}: now also Q2.2 (D)
- net HV_bleed_{gate}: now also Q2.1 (G), Q3.2 (D)
- net HV_bleed_{source}: now also Q2.3 (S)
Other:
- moved on the sheet: C8

Commit message: proper HVPS
Parts:
- removed Q2, Q3: BSP88, Package_TO_SOT_SMD:SOT-223-3_TabPin2, symbol 00_lib:BSP88
- added Q5, Q6: PZTA42, Package_TO_SOT_SMD:SOT-223-3_TabPin2, symbol Transistor_BJT:PZTA42
- renumbered D5 to D6, R6 to R10, R7 to R11, R5 to R9
Connections:
- net +5V: now also Q6.1 (B)
- net GND: now also Q6.3 (E)
- net HV_bleed_{drain}: now also Q5.2 (C)
- net HV_bleed_{gate}: now also Q5.1 (B), Q6.2 (C)
- net HV_bleed_{source}: now also Q5.3 (E)

Commit message: fuse HV, refactor schematic hierarchy
Changed lines of the file:
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@@
 	(title_block
 		(title "Nixie Accurate Clock")
-		(date "2024-02-25")
+		(date "2024-03-07")
 		(rev "B")
 		(company "Paul Willis")
@@
 		)
 	)
-	(global_label "HV_{SENSE}"
+	(hierarchical_label "HV_{SENSE}"
 		(shape input)
 		(at 66.04 43.18 180)
@@
 			(justify right)
 		)
-		(property "Intersheetrefs" "${INTERSHEET_REFS}"
-			(at 55.7469 43.18 0)
-			(effects
-				(font
-					(size 1.27 1.27)
-				)
-				(justify right)
-				(hide yes)
-			)
-		)
-	)
+	)
