File: hardware/KiCad/nixieAccurateClock/gps.kicad_sch (KiCad schematic)
At the start: 5 parts, among them J6 Conn_Coaxial, J7 Conn_01x02_Pin, U4 PX1125T

Commit message: switch all components to SMT
layout is a mess
Parts:
- BT1: footprint Battery:BatteryHolder_Keystone_103_1x20mm -> Battery:BatteryHolder_Keystone_3002_1x2032; Digikey link https://www.digikey.com/en/products/detail/103/36-103-ND/33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 -> https://www.digikey.com/en/products/detail/keystone-electro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; Model 103 -> 3002; Mouser link https://www.mouser.com/ProductDetail/Keystone-Electronics/1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 -> https://www.mouser.com/ProductDetail/Keystone-Electronics/3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; Price 1.50 -> 0.46
- J7: footprint Connector_PinHeader_2.54mm:PinHeader_1x02_P2.54mm_Vertical -> Connector_PinHeader_2.54mm:PinHeader_1x02_P2.54mm_Vertical_SMD_Pin1Left; Digikey link https://www.digikey.com/en/products/detail/adam-tech/PH1-02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 -> https://www.digikey.com/en/products/detail/samtec-inc/TSM-1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; Model PH1-02-UA -> TSM-102-01-L-SV; Mouser link https://www.mouser.com/ProductDetail/Samtec/TSW-102-07-G-S?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 -> https://www.mouser.com/ProductDetail/Samtec/TSM-102-01-L-SV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; Price 0.10 -> 0.42
Changed lines of the file:
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@@
       (effects (font (size 1.27 1.27)) (justify right))
     )
-    (property "Footprint" "Connector_PinHeader_2.54mm:PinHeader_1x02_P2.54mm_Vertical" (at 62.23 113.03 0)
+    (property "Footprint" "Connector_PinHeader_2.54mm:PinHeader_1x02_P2.54mm_Vertical_SMD_Pin1Left" (at 62.23 113.03 0)
       (effects (font (size 1.27 1.27)) hide)
     )
-    (property "Datasheet" "https://app.adam-tech.com/products/download/data_sheet/201605/ph1-xx-ua-data-sheet.pdf" (at 62.23 113.03 0)
+    (property "Datasheet" "https://suddendocs.samtec.com/catalog_english/tsm.pdf" (at 62.23 113.03 0)
       (effects (font (size 1.27 1.27)) hide)
     )
@@
       (effects (font (size 1.27 1.27)) hide)
     )
-    (property "Model" "PH1-02-UA" (at 62.23 113.03 0)
+    (property "Model" "TSM-102-01-L-SV" (at 62.23 113.03 0)
       (effects (font (size 1.27 1.27)) hide)
     )
-    (property "Price" "0.10" (at 62.23 113.03 0)
+    (property "Price" "0.42" (at 62.23 113.03 0)
       (effects (font (size 1.27 1.27)) hide)
     )
-    (property "Digikey link" "https://www.digikey.com/en/products/detail/adam-tech/PH1-02-UA/9830266" (at 62.23 113.03 0)
+    (property "Digikey link" "https://www.digikey.com/en/products/detail/samtec-inc/TSM-102-01-L-SV/2685520" (at 62.23 113.03 0)
       (effects (font (size 1.27 1.27)) hide)
     )
-    (property "Mouser link" "https://www.mouser.com/ProductDetail/Samtec/TSW-102-07-G-S?qs=iT52DjcXudsNPhlNCDp8vw%3D%3D" (at 62.23 113.03 0)
+    (property "Mouser link" "https://www.mouser.com/ProductDetail/Samtec/TSM-102-01-L-SV?qs=FESYatJ8odJ%252BIhPvKBkuBA%3D%3D" (at 62.23 113.03 0)
       (effects (font (size 1.27 1.27)) hide)
     )
@@
       (effects (font (size 1.27 1.27)) (justify left))
     )
-    (property "Footprint" "Battery:BatteryHolder_Keystone_103_1x20mm" (at 72.39 126.746 90)
+    (property "Footprint" "Battery:BatteryHolder_Keystone_3002_1x2032" (at 72.39 126.746 90)
       (effects (font (size 1.27 1.27)) hide)
     )
-    (property "Datasheet" "https://www.keyelco.com/userAssets/file/M65p3.pdf" (at 72.39 126.746 90)
+    (property "Datasheet" "https://www.keyelco.com/userAssets/file/M65p9.pdf" (at 72.39 126.746 90)
       (effects (font (size 1.27 1.27)) hide)
     )
@@
       (effects (font (size 1.27 1.27)) hide)
     )
-    (property "Model" "103" (at 72.39 128.27 0)
+    (property "Model" "3002" (at 72.39 128.27 0)
       (effects (font (size 1.27 1.27)) hide)
     )
-    (property "Price" "1.50" (at 72.39 128.27 0)
+    (property "Price" "0.46" (at 72.39 128.27 0)
       (effects (font (size 1.27 1.27)) hide)
     )
-    (property "Digikey link" "https://www.digikey.com/en/products/detail/103/36-103-ND/331620" (at 72.39 128.27 0)
+    (property "Digikey link" "https://www.digikey.com/en/products/detail/keystone-electronics/3002/227444" (at 72.39 128.27 0)
       (effects (font (size 1.27 1.27)) hide)
     )
-    (property "Mouser link" "https://www.mouser.com/ProductDetail/Keystone-Electronics/103?qs=Q3RoVmURDolsdXuDGYj49g%3D%3D" (at 72.39 128.27 0)
+    (property "Mouser link" "https://www.mouser.com/ProductDetail/Keystone-Electronics/3002?qs=Mn60vILZNNZWJpgHXc3g8Q%3D%3D" (at 72.39 128.27 0)
       (effects (font (size 1.27 1.27)) hide)
     )

Commit message: switch to all SM components
Parts:
- renumbered J6 to J8, J7 to J9, U4 to U3
Changed lines of the file:
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@@
   (symbol (lib_id "power:GND") (at 160.02 92.71 90) (mirror x) (unit 1)
     (in_bom yes) (on_board yes) (dnp no)
-    (property "Reference" "#PWR020" (at 166.37 92.71 0)
+    (property "Reference" "#PWR037" (at 166.37 92.71 0)
       (effects (font (size 1.27 1.27)) hide)
     )
@@
       (project "nixieAccurateClock"
         (path "/55aab698-7558-4fe2-95ad-faa6da60ef89/9610945c-9df3-4d66-a574-d19433fdc707"
-          (reference "#PWR020") (unit 1)
+          (reference "#PWR037") (unit 1)
         )
       )
@@
   (symbol (lib_id "Connector:Conn_01x02_Pin") (at 62.23 113.03 0) (mirror x) (unit 1)
     (in_bom yes) (on_board yes) (dnp no)
-    (property "Reference" "J7" (at 64.77 114.3 0)
+    (property "Reference" "J9" (at 64.77 114.3 0)
       (effects (font (size 1.27 1.27)) (justify right))
     )
@@
       (project "nixieAccurateClock"
         (path "/55aab698-7558-4fe2-95ad-faa6da60ef89/9610945c-9df3-4d66-a574-d19433fdc707"
-          (reference "J7") (unit 1)
+          (reference "J9") (unit 1)
         )
       )
@@
   (symbol (lib_id "power:GND") (at 72.39 135.89 0) (mirror y) (unit 1)
     (in_bom yes) (on_board yes) (dnp no)
-    (property "Reference" "#PWR024" (at 72.39 142.24 0)
+    (property "Reference" "#PWR041" (at 72.39 142.24 0)
       (effects (font (size 1.27 1.27)) hide)
     )
@@
       (project "nixieAccurateClock"
         (path "/55aab698-7558-4fe2-95ad-faa6da60ef89/9610945c-9df3-4d66-a574-d19433fdc707"
-          (reference "#PWR024") (unit 1)
+          (reference "#PWR041") (unit 1)
         )
       )
@@
   (symbol (lib_id "power:GND") (at 184.15 99.06 0) (mirror y) (unit 1)
     (in_bom yes) (on_board yes) (dnp no)
-    (property "Reference" "#PWR021" (at 184.15 105.41 0)
+    (property "Reference" "#PWR038" (at 184.15 105.41 0)
       (effects (font (size 1.27 1.27)) hide)
     )
@@
       (project "nixieAccurateClock"
         (path "/55aab698-7558-4fe2-95ad-faa6da60ef89/9610945c-9df3-4d66-a574-d19433fdc707"
-          (reference "#PWR021") (unit 1)
+          (reference "#PWR038") (unit 1)
         )
       )
@@
   (symbol (lib_id "power:GND") (at 106.68 82.55 180) (unit 1)
     (in_bom yes) (on_board yes) (dnp no)
-    (property "Reference" "#PWR018" (at 106.68 76.2 0)
+    (property "Reference" "#PWR035" (at 106.68 76.2 0)
       (effects (font (size 1.27 1.27)) hide)
     )
@@
       (project "nixieAccurateClock"
         (path "/55aab698-7558-4fe2-95ad-faa6da60ef89/9610945c-9df3-4d66-a574-d19433fdc707"
-          (reference "#PWR018") (unit 1)
+          (reference "#PWR035") (unit 1)
         )
       )
@@
   (symbol (lib_id "power:+3.3V") (at 96.52 128.27 180) (unit 1)
     (in_bom yes) (on_board yes) (dnp no) (fields_autoplaced)
-    (property "Reference" "#PWR023" (at 96.52 124.46 0)
+    (property "Reference" "#PWR040" (at 96.52 124.46 0)
       (effects (font (size 1.27 1.27)) hide)
     )
@@
       (project "nixieAccurateClock"
         (path "/55aab698-7558-4fe2-95ad-faa6da60ef89/9610945c-9df3-4d66-a574-d19433fdc707"
-          (reference "#PWR023") (unit 1)
+          (reference "#PWR040") (unit 1)
         )
       )
@@
   (symbol (lib_id "power:GND") (at 156.21 82.55 0) (mirror x) (unit 1)
     (in_bom yes) (on_board yes) (dnp no)
-    (property "Reference" "#PWR019" (at 156.21 76.2 0)
+    (property "Reference" "#PWR036" (at 156.21 76.2 0)
       (effects (font (size 1.27 1.27)) hide)
     )
@@
       (project "nixieAccurateClock"
         (path "/55aab698-7558-4fe2-95ad-faa6da60ef89/9610945c-9df3-4d66-a574-d19433fdc707"
-          (reference "#PWR019") (unit 1)
+          (reference "#PWR036") (unit 1)
         )
       )
@@
   (symbol (lib_id "00_lib:PX1125T") (at 109.22 87.63 0) (unit 1)
     (in_bom yes) (on_board yes) (dnp no) (fields_autoplaced)
-    (property "Reference" "U4" (at 132.08 80.01 0)
+    (property "Reference" "U3" (at 132.08 80.01 0)
       (effects (font (size 1.27 1.27)))
     )
@@
       (project "nixieAccurateClock"
         (path "/55aab698-7558-4fe2-95ad-faa6da60ef89/9610945c-9df3-4d66-a574-d19433fdc707"
-          (reference "U4") (unit 1)
+          (reference "U3") (unit 1)
         )
       )
@@
   (symbol (lib_id "power:GND") (at 106.68 120.65 0) (mirror y) (unit 1)
     (in_bom yes) (on_board yes) (dnp no)
-    (property "Reference" "#PWR022" (at 106.68 127 0)
+    (property "Reference" "#PWR039" (at 106.68 127 0)
       (effects (font (size 1.27 1.27)) hide)
     )
@@
       (project "nixieAccurateClock"
         (path "/55aab698-7558-4fe2-95ad-faa6da60ef89/9610945c-9df3-4d66-a574-d19433fdc707"
-          (reference "#PWR022") (unit 1)
+          (reference "#PWR039") (unit 1)
         )
       )
@@
   (symbol (lib_id "Connector:Conn_Coaxial") (at 184.15 90.17 0) (unit 1)
     (in_bom yes) (on_board yes) (dnp no) (fields_autoplaced)
-    (property "Reference" "J6" (at 187.96 89.1932 0)
+    (property "Reference" "J8" (at 187.96 89.1932 0)
       (effects (font (size 1.27 1.27)) (justify left))
     )
@@
       (project "nixieAccurateClock"
         (path "/55aab698-7558-4fe2-95ad-faa6da60ef89/9610945c-9df3-4d66-a574-d19433fdc707"
-          (reference "J6") (unit 1)
-        )
-      )
+          (reference "J8") (unit 1)
+        )
+      )

Commit message: route nixie daughter boards
Connections:
- net +3V3_STDBY renamed +3.3V_STDBY
- net 3.3V_STDBY_GPS_{SENSE} renamed +3.3V_STDBY_GPS_{SENSE}
Changed lines of the file:
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@@
     (effects (font (size 1.27 1.27)) (justify right bottom))
   )
-  (label "3.3V_STDBY_GPS_{SENSE}" (at 73.66 110.49 0) (fields_autoplaced)
+  (label "+3.3V_STDBY_GPS_{SENSE}" (at 73.66 110.49 0) (fields_autoplaced)
     (effects (font (size 1.27 1.27)) (justify left bottom))
   )
@@
     )
   )
-  (global_label "+3V3_STDBY" (shape output) (at 67.31 120.65 180) (fields_autoplaced)
+  (global_label "+3.3V_STDBY" (shape output) (at 67.31 120.65 180) (fields_autoplaced)
     (effects (font (size 1.27 1.27)) (justify right))
-    (property "Intersheetrefs" "${INTERSHEET_REFS}" (at 52.4715 120.65 0)
+    (property "Intersheetrefs" "${INTERSHEET_REFS}" (at 51.8667 120.65 0)
       (effects (font (size 1.27 1.27)) (justify right) hide)
     )

Commit message: update to KiCAD 8
Connections:
- net +3.3V: now also C3.1; no longer C3.2
- net VCC_{GPS}: now also C3.2; no longer C3.1

Commit message: fuse HV, refactor schematic hierarchy
Changed lines of the file:
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@@
 	(title_block
 		(title "Nixie Accurate Clock")
-		(date "2024-02-25")
+		(date "2024-03-07")
 		(rev "B")
 		(company "Paul Willis")
@@
 			)
 			(justify left bottom)
-		)
-	)
-	(global_label "GPS_{RSTN}"
-		(shape input)
-		(at 157.48 97.79 0)
-		(fields_autoplaced yes)
-		(effects
-			(font
-				(size 1.27 1.27)
-			)
-			(justify left)
-		)
-		(property "Intersheetrefs" "${INTERSHEET_REFS}"
-			(at 168.0876 97.79 0)
-			(effects
-				(font
-					(size 1.27 1.27)
-				)
-				(justify left)
-				(hide yes)
-			)
-		)
-	)
-	(global_label "GPS_{TXD}"
-		(shape output)
-		(at 106.68 105.41 180)
-		(fields_autoplaced yes)
-		(effects
-			(font
-				(size 1.27 1.27)
-			)
-			(justify right)
-		)
-		(property "Intersheetrefs" "${INTERSHEET_REFS}"
-			(at 97.1368 105.41 0)
-			(effects
-				(font
-					(size 1.27 1.27)
-				)
-				(justify right)
-				(hide yes)
-			)
 		)
 	)
@@
 		)
 	)
-	(global_label "GPS_{BOOT_SEL}"
+	(hierarchical_label "GPS_{1PPS2}"
+		(shape output)
+		(at 157.48 107.95 0)
+		(fields_autoplaced yes)
+		(effects
+			(font
+				(size 1.27 1.27)
+			)
+			(justify left)
+		)
+	)
+	(hierarchical_label "GPS_{1PPS}"
+		(shape output)
+		(at 157.48 110.49 0)
+		(fields_autoplaced yes)
+		(effects
+			(font
+				(size 1.27 1.27)
+			)
+			(justify left)
+		)
+	)
+	(hierarchical_label "GPS_{BOOT_SEL}"
 		(shape input)
 		(at 157.48 115.57 0)
@@
 			(justify left)
 		)
-		(property "Intersheetrefs" "${INTERSHEET_REFS}"
-			(at 171.6678 115.57 0)
-			(effects
-				(font
-					(size 1.27 1.27)
-				)
-				(justify left)
-				(hide yes)
-			)
-		)
-	)
-	(global_label "GPS_{1PPS2}"
+	)
+	(hierarchical_label "GPS_{TXD}"
 		(shape output)
-		(at 157.48 107.95 0)
+		(at 106.68 105.41 180)
+		(fields_autoplaced yes)
+		(effects
+			(font
+				(size 1.27 1.27)
+			)
+			(justify right)
+		)
+	)
+	(hierarchical_label "GPS_{RSTN}"
+		(shape input)
+		(at 157.48 97.79 0)
 		(fields_autoplaced yes)
 		(effects
@@
 			(justify left)
 		)
-		(property "Intersheetrefs" "${INTERSHEET_REFS}"
-			(at 169.2003 107.95 0)
-			(effects
-				(font
-					(size 1.27 1.27)
-				)
-				(justify left)
-				(hide yes)
-			)
-		)
-	)
-	(global_label "GPS_{1PPS}"
-		(shape output)
-		(at 157.48 110.49 0)
-		(fields_autoplaced yes)
-		(effects
-			(font
-				(size 1.27 1.27)
-			)
-			(justify left)
-		)
-		(property "Intersheetrefs" "${INTERSHEET_REFS}"
-			(at 168.2327 110.49 0)
-			(effects
-				(font
-					(size 1.27 1.27)
-				)
-				(justify left)
-				(hide yes)
-			)
-		)
-	)
-	(global_label "GPS_{RXD}"
+	)
+	(hierarchical_label "GPS_{RXD}"
 		(shape input)
 		(at 106.68 107.95 180)
@@
 			(justify right)
 		)
-		(property "Intersheetrefs" "${INTERSHEET_REFS}"
-			(at 96.8949 107.95 0)
-			(effects
-				(font
-					(size 1.27 1.27)
-				)
-				(justify right)
-				(hide yes)
-			)
-		)
-	)
+	)
