File: hardware/KiCad/nixieAccurateClock/gps.kicad_sch (KiCad schematic)
At the start: 5 parts, among them J8 Conn_Coaxial, J9 Conn_01x02_Pin, U3 PX1125T

Commit message: fix 2x1 SM header chirality
Parts:
- J9: footprint Connector_PinHeader_2.54mm:PinHeader_1x02_P2.54mm_Vertical_SMD_Pin1Left -> Connector_PinHeader_2.54mm:PinHeader_1x02_P2.54mm_Vertical_SMD_Pin1Right
Changed lines of the file:
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@@
 			)
 		)
-		(property "Footprint" "Connector_PinHeader_2.54mm:PinHeader_1x02_P2.54mm_Vertical_SMD_Pin1Left"
+		(property "Footprint" "Connector_PinHeader_2.54mm:PinHeader_1x02_P2.54mm_Vertical_SMD_Pin1Right"
 			(at 62.23 113.03 0)
 			(effects

Commit message: Modify HV supply to attempt to solve weak IC
Changed lines of the file:
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@@
 (kicad_sch
-	(version 20231120)
+	(version 20250114)
 	(generator "eeschema")
-	(generator_version "8.0")
+	(generator_version "9.0")
 	(paper "A4")
 	(title_block
@@
 	(label "VCC_{GPS}"
 		(at 105.41 113.03 180)
-		(fields_autoplaced yes)
 		(effects
 			(font
@@
 	(label "+3.3V_STDBY_GPS_{SENSE}"
 		(at 73.66 110.49 0)
-		(fields_autoplaced yes)
 		(effects
 			(font
@@
 	(label "RF_IN"
 		(at 157.48 90.17 0)
-		(fields_autoplaced yes)
 		(effects
 			(font
@@
 		(shape output)
 		(at 157.48 107.95 0)
-		(fields_autoplaced yes)
 		(effects
 			(font
@@
 		(shape output)
 		(at 157.48 110.49 0)
-		(fields_autoplaced yes)
 		(effects
 			(font
@@
 		(shape input)
 		(at 157.48 115.57 0)
-		(fields_autoplaced yes)
 		(effects
 			(font
@@
 		(shape output)
 		(at 106.68 105.41 180)
-		(fields_autoplaced yes)
 		(effects
 			(font
@@
 		(shape input)
 		(at 157.48 97.79 0)
-		(fields_autoplaced yes)
 		(effects
 			(font
@@
 		(shape input)
 		(at 106.68 107.95 180)
-		(fields_autoplaced yes)
-		(effects
-			(font
+		(effects
+			(font
