File: hardware/KiCad/nixieAccurateClock/nixieAccurateClock-rounded.kicad_pcb (KiCad board)
At the start: 4 copper layers, 152.4 x 101.6 mm, 102 parts, among them J1 Conn_01x02_Pin, J10 Conn_01x02_Pin, J17 Conn_02x05_Odd_Even, J2 Conn_01x02_Pin, J3 Conn_01x02_Pin, J4 pico iCE (A), J5 pico iCE (B), J6 Conn_01x02_Pin, J7 Conn_01x02_Pin, J8 Conn_Coaxial, J9 Conn_01x02_Pin, Q1 PZTA42, Q2 PZTA42, Q3 PZTA42, Q4 PZTA42, Q5 PZTA42, Q6 PZTA42, SW1 SW_DIP_x08, U1 MCP23008-xSO, U2 LTR-329ALS-01, U3 PX1125T, U6 ADC0820BCWMX

Commit message: update to KiCAD 8
Parts:
- C9: value locked -> 0.1u
- turned C3 to -90 degrees
Connections:
- C3 pad 1: /GPS/VCC_{GPS} -> +3.3V
- C3 pad 2: +3.3V -> /GPS/VCC_{GPS}

Commit message: Update date
Parts:
- moved R2 0.66 mm to (115.6, 70.7), turned to 90 degrees
- moved R1 0.38 mm to (115.6, 65.7)
Routing:
- net I2C_{CLOCK}: track 70.3 -> 69.0 mm
- net I2C_{DATA}: track 74.8 -> 75.7 mm

Commit message: fuse HV, refactor schematic hierarchy
Parts:
- added F1: 1A, Fuse:Fuse_1206_3216Metric, F.Cu at (80.4, 87.8)
Connections:
- net /+3.3V_STDBY_SRAM_{SENSE} renamed /Pico Ice/+3.3V_STDBY_SRAM_{SENSE}
- net /+3.3V_{SENSE} renamed /Pico Ice/+3.3V_{SENSE}
- net /+5V_{SENSE} renamed /Pico Ice/+5V_{SENSE}
- net /24h_mode renamed /Peripherals/24h_mode
- net /DST_check renamed /Peripherals/DST_check
- net /DST_force renamed /Peripherals/DST_force
- net /INT_{IO-expander} renamed /Peripherals/INT_{IO-expander}
- net /RESERVED_1 renamed /Peripherals/RESERVED_1
- net /RESERVED_2 renamed /Peripherals/RESERVED_2
- net /VCC_{ALS} renamed /Peripherals/VCC_{ALS}
- net /VCC_{IO-expander} renamed /Peripherals/VCC_{IO-expander}
- net /anti-poison_force renamed /Peripherals/anti-poison_force
- net /anti-poison_routine renamed /Peripherals/anti-poison_routine
- net /brightness_control renamed /Peripherals/brightness_control
- net /manual_brightness renamed /Peripherals/manual_brightness
- net /~{ICE_RST} renamed /Pico Ice/~{ICE_RST}
- net /~{RESET}_{IO-expander} renamed /Peripherals/~{RESET}_{IO-expander}
- net /~{USB_BOOT} renamed /Pico Ice/~{USB_BOOT}
- net CLOCK_{HV} renamed /Nixies/CLOCK_{HV}
- net CLOCK_{PRECISE} renamed /Nixies/CLOCK_{PRECISE}
- net DATA_{HV} renamed /Nixies/DATA_{HV}
- net DATA_{PRECISE} renamed /Nixies/DATA_{PRECISE}
- net GATE_{HV} renamed /High voltage supply/GATE_{HV}
- net GPS_{1PPS2} renamed /GPS/GPS_{1PPS2}
- net GPS_{1PPS} renamed /GPS/GPS_{1PPS}
- net GPS_{BOOT_SEL} renamed /GPS/GPS_{BOOT_SEL}
- net GPS_{RSTN} renamed /GPS/GPS_{RSTN}
- net GPS_{RXD} renamed /GPS/GPS_{RXD}
- net GPS_{TXD} renamed /GPS/GPS_{TXD}
- net HV_{SENSE} renamed /HV bleed/HV_{SENSE}
- net I2C_{CLOCK} renamed /Peripherals/I2C_{CLOCK}
- net I2C_{DATA} renamed /Peripherals/I2C_{DATA}
- net LSD_{ADC_D0} renamed /LSD ADC/LSD_{ADC_D0}
- net LSD_{ADC_D1} renamed /LSD ADC/LSD_{ADC_D1}
- net LSD_{ADC_D2} renamed /LSD ADC/LSD_{ADC_D2}
- net LSD_{ADC_D3} renamed /LSD ADC/LSD_{ADC_D3}
- net LSD_{ADC_D4} renamed /LSD ADC/LSD_{ADC_D4}
- net LSD_{ADC_D5} renamed /LSD ADC/LSD_{ADC_D5}
- net LSD_{ADC_D6} renamed /LSD ADC/LSD_{ADC_D6}
- net LSD_{ADC_D7} renamed /LSD ADC/LSD_{ADC_D7}
- net LSD_{ADC_MODE} renamed /LSD ADC/LSD_{ADC_MODE}
- net LSD_{ADC_~{CS}} renamed /LSD ADC/LSD_{ADC_~{CS}}
- net LSD_{ADC_~{INT}} renamed /LSD ADC/LSD_{ADC_~{INT}}
- net LSD_{ADC_~{OFL}} renamed /LSD ADC/LSD_{ADC_~{OFL}}
- net LSD_{ADC_~{RD}} renamed /LSD ADC/LSD_{ADC_~{RD}}
- net LSD_{ADC_~{WR}/RDY} renamed /LSD ADC/LSD_{ADC_~{WR}/RDY}
- net LSD_{SHUNT} renamed /LSD ADC/LSD_{SHUNT}
- net MEASURE_{HV} renamed /High voltage supply/MEASURE_{HV}
- net PPS_{TRIMMED} renamed /Nixies/PPS_{TRIMMED}
- net SENSE_{PRECISE} renamed /Nixies/SENSE_{PRECISE}
- L1 pad 1: +5V -> /High voltage supply/5V_{BOOST-FUSE}
Routing:
- added copper zone on F.Cu, net /High voltage supply/5V_{BOOST-FUSE}
