File: hardware/KiCad/nixieAccurateClock/nixieAccurateClock-rounded.kicad_pcb (KiCad board)
At the start: 4 copper layers, 152.4 x 101.6 mm, 103 parts, among them J1 Conn_01x02_Pin, J10 Conn_01x02_Pin, J17 Conn_02x05_Odd_Even, J2 Conn_01x02_Pin, J3 Conn_01x02_Pin, J4 pico iCE (A), J5 pico iCE (B), J6 Conn_01x02_Pin, J7 Conn_01x02_Pin, J8 Conn_Coaxial, J9 Conn_01x02_Pin, Q1 PZTA42, Q2 PZTA42, Q3 PZTA42, Q4 PZTA42, Q5 PZTA42, Q6 PZTA42, SW1 SW_DIP_x08, U1 MCP23008-xSO, U2 LTR-329ALS-01, U3 PX1125T, U6 ADC0820BCWMX

Commit message: add alignment holes to 2x20 SM headers
Routing:
- net GND: track 209.9 -> 195.9 mm, vias 43 -> 45
- net /Pico Ice/~{USB_BOOT}: track 13.1 -> 25.8 mm
- net /GPS/GPS_{BOOT_SEL}: track 28.2 -> 26.6 mm

Commit message: fix 2x1 SM header chirality
Parts:
- J1, J10, J2, J3, J6, J7, J9: footprint Connector_PinHeader_2.54mm:PinHeader_1x02_P2.54mm_Vertical_SMD_Pin1Left -> Connector_PinHeader_2.54mm:PinHeader_1x02_P2.54mm_Vertical_SMD_Pin1Right
- moved J10 3.87 mm to (45.7, 55.9), turned to 180 degrees
Routing:
- net GND: track 195.9 -> 180.7 mm, vias 45 -> 47
- net +3.3V_STDBY: track 51.2 -> 55.9 mm
- net /Pico Ice/~{USB_BOOT}: track 25.8 -> 29.1 mm
- net /Pico Ice/+3.3V_{SENSE}: track 20.6 -> 23.8 mm, vias 7 -> 9
- net +3.3V: track 33.3 -> 36.0 mm, vias 6 -> 8
- net /Pico Ice/~{ICE_RST}: track 23.0 -> 25.6 mm
- net /GPS/+3.3V_STDBY_GPS_{SENSE}: track 18.1 -> 20.4 mm
- net /Pico Ice/+5V_{SENSE}: track 14.6 -> 15.5 mm
- net /Pico Ice/+3.3V_STDBY_SRAM_{SENSE}: track 32.5 -> 33.2 mm

Commit message: more detailed build notes, drop HV divider by 10x
Parts:
- R3: value 10M -> 1M
- R4: value 100k -> 10k
