File: hardware/KiCad/nixieAccurateClock/pico_ce.kicad_sch (KiCad schematic)
At the start: 10 parts, among them J1 Conn_01x02_Pin, J2 Conn_01x02_Pin, J3 Conn_01x02_Pin, J4 pico iCE (A), J5 pico iCE (B), J6 Conn_01x02_Pin, J7 Conn_01x02_Pin

Commit message: fuse HV, refactor schematic hierarchy
Parts:
- removed RV1: 100k, Potentiometer_SMD:Potentiometer_Bourns_3269X_Horizontal, symbol Device:R_Potentiometer
