File: hardware/KiCad/nixieAccurateClock/IN-14-daughter/IN-14-daughter-rounded.kicad_pcb (KiCad board)
At the start: 4 copper layers, 19 x 32 mm, 12 parts, among them J1 Conn_02x05_Odd_Even, U1 HV509K6-G

Commit message: daughter board no TH components
Parts:
- J1: footprint Connector_PinHeader_2.54mm:PinHeader_2x05_P2.54mm_Vertical -> Connector_PinHeader_2.54mm:PinHeader_2x05_P2.54mm_Vertical_SMD
- moved REF** 6.57 mm to (44.1, 46.9)
- moved J1 6.55 mm to (41.2, 46.1)
- moved FID1 3.00 mm to (33.0, 49.6)
- moved FID2 3.00 mm to (49.5, 49.6)
- moved R1 0.08 mm to (44.8, 38.9)
Routing:
- net /CLK: track 24.6 -> 29.2 mm
- net +5V: track 11.4 -> 15.0 mm
- net /~{LE}: track 12.7 -> 14.7 mm, vias 1 -> 2
- net VPP: track 17.0 -> 18.5 mm
- net /ANODE: track 7.58 -> 8.48 mm
- net /DOUT: track 12.5 -> 12.7 mm, vias 1 -> 0
- net GND: vias 2 -> 3
Other:
- board size 19 x 32 mm -> 19 x 36.4 mm

Commit message: Rev B prep
Other:
- board text added: "IN-14 daughter board Rev B"
- board text removed: "IN-14 daughter board Rev A"

Commit message: update to KiCAD 8
Parts:
- U1: footprint Package_DFN_QFN:QFN-32-1EP_5x5mm_P0.5mm_EP3.1x3.1mm_ThermalVias -> Package_DFN_QFN:QFN-32-1EP_5x5mm_P0.5mm_EP3.3x3.3mm_ThermalVias

Commit message: Clean up clearances
Set board clearances, add dimension annotations, clean up pour dimensions
Parts:
- moved FID1 0.25 mm to (33.2, 49.6)
- moved FID2 0.25 mm to (49.2, 49.6)
- moved FID3 0.25 mm to (41.2, 17.4)
Other:
- board text added: "0.2000 mm / 0.2000 mm"
- board text added: "19.0000 mm x 36.4450 mm"
- board text removed: "0.0000 mm / 0.0000 mm"
- board text removed: "19.0000 mm x 32.0000 mm"

Commit message: Switch to 2.4 mm stackup
PCBWAY001 is cheaper than PCBWAY209 (2 oz copper) for 0.2 mm prepreg (200 V clearance)
Other:
- board text added: "0.035 mm"
- board text added: "0.196 mm"
- board text added: "0.2200 mm / 0.2200 mm"
- board text added: "1.9 mm"
- board text added: "2.4520 mm"
- board text added: "Dielectric"
- board text removed: "0.0525 mm"
- board text removed: "0.07 mm"
- board text removed: "0.2000 mm / 0.2000 mm"
- board text removed: "0.22 mm"
- board text removed: "0.895 mm"
- board text removed: "1.6000 mm"
- board text removed: "Dielectric 1"
- board text removed: "Dielectric 2"
- board text removed: "Dielectric 3"
