File: hardware/KiCad/nixieAccurateClock/IN-14-daughter/IN-14-daughter-rounded.kicad_pcb (KiCad board)
At the start: 4 copper layers, 19 x 36.4 mm, 12 parts, among them J1 Conn_02x05_Odd_Even, U1 HV509K6-G

Commit message: Switch to stackup PCBWAY206
2.4 mm board is incompatible with SMA connector
Clean up outdated board notes
Other:
- board text added: "1.1 mm"
- board text added: "1.6520 mm"
- board text added: "Dielectric 1"
- board text added: "Dielectric 2"
- board text added: "Dielectric 3"
- board text added: "Epoxy"
- board text removed: "1.9 mm"
- board text removed: "2.4520 mm"
- board text removed: "Dielectric"
