File: hardware/KiCad/nixieAccurateClock/IN-14-daughter/IN-14-daughter.kicad_pcb (KiCad board)
At the start: 4 copper layers, 19 x 32 mm, 12 parts, among them J1 Conn_02x05_Odd_Even, U1 HV509K6-G

Commit message: add thermal reliefs
Changed lines of the file:
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@@
   (segment (start 43.503903 31.068243) (end 44.56066 32.125) (width 0.25) (layer "B.Cu") (net 33))
   (segment (start 45 32.125) (end 44.56066 32.125) (width 0.25) (layer "B.Cu") (net 33))
-  (segment (start 40.896446 39.978554) (end 42.915725 37.959275) (width 0.25) (layer "F.Cu") (net 34))
-  (segment (start 39.103553 39.978554) (end 38.54 40.542107) (width 0.25) (layer "F.Cu") (net 34))
+  (segment (start 39.457107 39.625) (end 38.54 40.542107) (width 0.25) (layer "F.Cu") (net 34))
+  (segment (start 42.915725 33.411533) (end 42.915725 37.959275) (width 0.25) (layer "F.Cu") (net 34))
+  (segment (start 42.915725 37.959275) (end 41.25 39.625) (width 0.25) (layer "F.Cu") (net 34))
+  (segment (start 41.25 39.625) (end 39.457107 39.625) (width 0.25) (layer "F.Cu") (net 34))
   (segment (start 38.54 40.542107) (end 38.54 42.125) (width 0.25) (layer "F.Cu") (net 34))
-  (segment (start 40.896446 39.978554) (end 39.103553 39.978554) (width 0.25) (layer "F.Cu") (net 34))
-  (segment (start 42.915725 33.411533) (end 42.915725 37.959275) (width 0.25) (layer "F.Cu") (net 34))
   (via (at 42.915725 33.411533) (size 0.6) (drill 0.3) (layers "F.Cu" "B.Cu") (net 34))
   (segment (start 42.769278 32.454938) (end 42.443243 32.128903) (width 0.25) (layer "B.Cu") (net 34))
   (segment (start 42.915725 33.411533) (end 42.915725 32.601385) (width 0.25) (layer "B.Cu") (net 34))
   (segment (start 42.915725 32.601385) (end 42.769278 32.454938) (width 0.25) (layer "B.Cu") (net 34))
+  (zone (net 3) (net_name "GND") (layers "F.Cu" "In1.Cu" "In2.Cu" "B.Cu") (hatch edge 0.5)
+    (priority 1)
+    (connect_pads (clearance 0.5))
+    (min_thickness 0.25) (filled_areas_thickness no)
+    (fill (thermal_gap 0.5) (thermal_bridge_width 0.5))
+    (polygon
+      (pts
+        (xy 31.75 47.875)
+        (xy 31.75 39.375)
+        (xy 50.75 39.375)
+        (xy 50.75 47.875)
+      )
+    )
+  )
   (zone (net 3) (net_name "GND") (layers "F.Cu" "In1.Cu" "In2.Cu" "B.Cu") (hatch edge 0.5)
     (connect_pads yes (clearance 0.5))
@@
         (xy 31.75 15.875)
         (xy 50.75 15.875)
-        (xy 50.75 47.875)
-        (xy 31.75 47.875)
+        (xy 50.75 39.375)
+        (xy 31.75 39.375)
       )
     )

Commit message: daughter board no TH components
Parts:
- J1: footprint Connector_PinHeader_2.54mm:PinHeader_2x05_P2.54mm_Vertical -> Connector_PinHeader_2.54mm:PinHeader_2x05_P2.54mm_Vertical_SMD
- moved REF** 6.57 mm to (44.1, 46.9)
- moved J1 6.55 mm to (41.2, 46.1)
- moved FID1 3.00 mm to (33.0, 49.6)
- moved FID2 3.00 mm to (49.5, 49.6)
- moved R1 0.08 mm to (44.8, 38.9)
Routing:
- net /CLK: track 25.3 -> 29.5 mm
- net +5V: track 11.5 -> 15.2 mm
- net /~{LE}: track 13.1 -> 15.0 mm, vias 1 -> 2
- net VPP: track 17.5 -> 18.9 mm
- net /ANODE: track 7.74 -> 8.58 mm
- net /DOUT: track 12.9 -> 13.1 mm, vias 1 -> 0
- net GND: vias 2 -> 3
Other:
- board size 19 x 32 mm -> 19 x 36.4 mm

Commit message: Rev B prep
Other:
- board text added: "IN-14 daughter board Rev B"
- board text removed: "IN-14 daughter board Rev A"
Changed lines of the file:
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@@
   (title_block
     (title "IN-14 daughter board")
-    (rev "A")
+    (date "2024-02-24")
+    (rev "B")
     (company "Paul Willis")
   )
@@
   (gr_rect (start 31.75 15.875) (end 50.75 52.32)
     (stroke (width 0.1) (type default)) (fill none) (layer "Edge.Cuts"))
-  (gr_text "IN-14\ndaughter board\nRev A" (at 37.75 47.875) (layer "F.SilkS")
+  (gr_text "IN-14\ndaughter board\nRev B" (at 37.75 47.875) (layer "F.SilkS")
     (effects (font (size 0.8 0.8) (thickness 0.125)) (justify bottom))
   )

Commit message: update to KiCAD 8
Parts:
- U1: footprint Package_DFN_QFN:QFN-32-1EP_5x5mm_P0.5mm_EP3.1x3.1mm_ThermalVias -> Package_DFN_QFN:QFN-32-1EP_5x5mm_P0.5mm_EP3.3x3.3mm_ThermalVias

Commit message: Clean up clearances
Set board clearances, add dimension annotations, clean up pour dimensions
Parts:
- moved FID1 0.25 mm to (33.2, 49.6)
- moved FID2 0.25 mm to (49.2, 49.6)
- moved FID3 0.25 mm to (41.2, 17.4)
Other:
- board text added: "0.2000 mm / 0.2000 mm"
- board text added: "19.0000 mm x 36.4450 mm"
- board text removed: "0.0000 mm / 0.0000 mm"
- board text removed: "19.0000 mm x 32.0000 mm"

Commit message: Switch to 2.4 mm stackup
PCBWAY001 is cheaper than PCBWAY209 (2 oz copper) for 0.2 mm prepreg (200 V clearance)
Other:
- board text added: "0.035 mm"
- board text added: "0.196 mm"
- board text added: "0.2200 mm / 0.2200 mm"
- board text added: "1.9 mm"
- board text added: "2.4520 mm"
- board text added: "Dielectric"
- board text removed: "0.0525 mm"
- board text removed: "0.07 mm"
- board text removed: "0.2000 mm / 0.2000 mm"
- board text removed: "0.22 mm"
- board text removed: "0.895 mm"
- board text removed: "1.6000 mm"
- board text removed: "Dielectric 1"
- board text removed: "Dielectric 2"
- board text removed: "Dielectric 3"
