File: hardware/KiCad/nixieAccurateClock/IN-14-daughter/IN-14-daughter.kicad_sch (KiCad schematic)
At the start: 11 parts, among them J1 Conn_02x05_Odd_Even, U1 HV509K6-G

Commit message: daughter board no TH components
Parts:
- J1: footprint Connector_PinHeader_2.54mm:PinHeader_2x05_P2.54mm_Vertical -> Connector_PinHeader_2.54mm:PinHeader_2x05_P2.54mm_Vertical_SMD; Digikey link https://www.digikey.com/en/products/detail/sullins-connecto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 -> https://www.digikey.com/en/products/detail/molex/0015916100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; Model PPPC052LFBN-RC -> 15-91-6100; Mouser link N/A -> https://www.mouser.com/ProductDetail/Molex/15-91-6100?qs=5A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; Price 0.72 -> 3.14
Changed lines of the file:
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@@
       (effects (font (size 1.27 1.27)))
     )
-    (property "Footprint" "Connector_PinHeader_2.54mm:PinHeader_2x05_P2.54mm_Vertical" (at 80.01 125.73 0)
+    (property "Footprint" "Connector_PinHeader_2.54mm:PinHeader_2x05_P2.54mm_Vertical_SMD" (at 80.01 125.73 0)
       (effects (font (size 1.27 1.27)) hide)
     )
-    (property "Datasheet" "https://mm.digikey.com/Volume0/opasdata/d220001/medias/docus/937/Female_Headers.100_DS.pdf" (at 80.01 125.73 0)
+    (property "Datasheet" "https://www.molex.com/content/dam/molex/molex-dot-com/products/automated/en-us/productspecificationpdf/713/71308/PS-71308-001.pdf?inline" (at 80.01 125.73 0)
       (effects (font (size 1.27 1.27)) hide)
     )
-    (property "Model" "PPPC052LFBN-RC" (at 80.01 125.73 0)
+    (property "Model" "15-91-6100" (at 80.01 125.73 0)
       (effects (font (size 1.27 1.27)) hide)
     )
-    (property "Price" "0.72" (at 80.01 125.73 0)
+    (property "Price" "3.14" (at 80.01 125.73 0)
       (effects (font (size 1.27 1.27)) hide)
     )
-    (property "Digikey link" "https://www.digikey.com/en/products/detail/sullins-connector-solutions/PPPC052LFBN-RC/810245" (at 80.01 125.73 0)
+    (property "Digikey link" "https://www.digikey.com/en/products/detail/molex/0015916100/3124523" (at 80.01 125.73 0)
       (effects (font (size 1.27 1.27)) hide)
     )
-    (property "Mouser link" "N/A" (at 80.01 125.73 0)
+    (property "Mouser link" "https://www.mouser.com/ProductDetail/Molex/15-91-6100?qs=5ADmCPbgZvxX3zRPE3%2FoVw%3D%3D" (at 80.01 125.73 0)
       (effects (font (size 1.27 1.27)) hide)
     )

Commit message: DRC pass
Other:
- company: (none) -> Paul Willis
Changed lines of the file:
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@@
     (title "IN-14 daughter board")
     (rev "A")
+    (company "Paul Willis")
   )
   (wire (pts (xy 115.57 48.26) (xy 110.49 48.26))

Commit message: update to KiCAD 8
Parts:
- FID1, FID2, FID3: now left out of the parts list
- N1: now not fitted
- U1: footprint Package_DFN_QFN:QFN-32-1EP_5x5mm_P0.5mm_EP3.1x3.1mm_ThermalVias -> Package_DFN_QFN:QFN-32-1EP_5x5mm_P0.5mm_EP3.3x3.3mm_ThermalVias
